File: kicad/cft/mem/mem.sch (KiCad schematic (older format))
At the start: 9 parts

Commit message: Planning and design for the MEM board.
Parts:
- added U104: 74HC138, alexios:SOIC-16, symbol alexios:74HC138
- added U111, U112: 29W040, Sockets:PLCC32, symbol Memory_Flash:29W040
- U101, U102, U105, U106, U107, U108, U109, U110: renamed from U?; footprint Package_SO:SOJ-36_10.16x23.49mm_P1.27mm -> Package_DIP:DIP-40_W15.24mm
- U103: renamed from U?; footprint (none) -> alexios:SOIC-16
Connections:
- net labels added: AB19, AB20, AB21, AB22, AB23, DB10, DB11, DB12, DB13, DB14, DB15, DB8, DB9, ~RBCE4, ~RBCE5, ~RBCE6, ~RBCE7, ~ROMCE
- net labels removed: PB10, PB11, PB12, PB13, PB14, PB15, PB8, PB9
- wire segments 300 -> 373
Other:
- note added: "Notes"
- note added: "Use DIP40 sockets for first 1024×16 bank of SRAM (four 512K chips), then\nleave land patterns for another 7M in smaller packages, SOJ or Flash TSSOP.\n\nThis implies only one MEM board need be used. RAM can be mapped to\n00:0000–0F:FFFF for the first (DIP) Megaword, then extending up to 7F:FFFF\nwith all 8 Megawords installed.\n\nFlash devices are in PLCC32 sockets and form a single 512K×16 ROM B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"

Commit message: Play around with new MEM board
Parts:
- added U?: 74HC138, alexios:SOIC-16, symbol alexios:74HC138
Connections:
- wire segments 373 -> 386
Changed lines of the file:
@@
 EESchema Schematic File Version 4
 LIBS:mem-cache
-EELAYER 26 0
+EELAYER 30 0
 EELAYER END
 $Descr A3 16535 11693
@@
 Text Label 5250 7650 2    50   ~ 0
 ~ROMCE
-Wire Bus Line
-	15050 3050 15050 3350
-Wire Bus Line
-	15050 3450 15050 3750
 Text Notes 6700 8050 0    100  ~ 20
 Notes
 Text Notes 6700 8900 0    50   ~ 0
 Use DIP40 sockets for first 1024×16 bank of SRAM (four 512K chips), then\nleave land patterns for another 7M in smaller packages, SOJ or Flash TSSOP.\n\nThis implies only one MEM board need be used. RAM can be mapped to\n00:0000–0F:FFFF for the first (DIP) Megaword, then extending up to 7F:FFFF\nwith all 8 Megawords installed.\n\nFlash devices are in PLCC32 sockets and form a single 512K×16 ROM Bank\nmapped to 80:0000–87:FFFF. This is hardwired.
+Wire Wire Line
+	1750 8950 1350 8950
+Wire Wire Line
+	1750 9050 1350 9050
+Wire Wire Line
+	1750 9150 1350 9150
+Wire Wire Line
+	1750 9650 1350 9650
+Wire Wire Line
+	1750 9550 1350 9550
+Text Label 1350 9550 0    50   ~ 0
+AB23
+Wire Wire Line
+	3150 8950 2750 8950
+Wire Wire Line
+	3150 9050 2750 9050
+Wire Wire Line
+	3150 9150 2750 9150
+Wire Wire Line
+	3150 9550 2750 9550
+Wire Wire Line
+	3150 9650 2750 9650
+Wire Wire Line
+	2750 9250 3150 9250
+Wire Wire Line
+	2750 9350 3150 9350
+Wire Wire Line
+	2750 9450 3150 9450
+$Comp
+L alexios:74HC138 U?
+U 1 1 5D65AD6B
+P 2250 9350
+F 0 "U?" H 2250 10017 50  0000 C CNN
+F 1 "74HC138" H 2250 9926 50  0000 C CNN
+F 2 "alexios:SOIC-16" H 2250 9350 50  0001 C CNN
+F 3 "http://www.ti.com/lit/gpn/sn74LS138" H 2250 9350 50  0001 C CNN
+	1    2250 9350
+	1    0    0    -1
+$EndComp
+Text Label 1350 9650 0    50   ~ 0
+AB22
+Text Label 1350 9150 0    50   ~ 0
+AB21
+Text Label 1350 9050 0    50   ~ 0
+AB20
+Text Label 1350 8950 0    50   ~ 0
+AB19
+$Comp
+L power:GND #PWR?
+U 1 1 5D6FAE34
+P 1750 9750
+F 0 "#PWR?" H 1750 9500 50  0001 C CNN
+F 1 "GND" H 1755 9577 50  0000 C CNN
+F 2 "" H 1750 9750 50  0001 C CNN
+F 3 "" H 1750 9750 50  0001 C CNN
+	1    1750 9750
+	1    0    0    -1
+$EndComp
+Wire Bus Line
+	15050 3450 15050 3750
+Wire Bus Line
+	15050 3050 15050 3350
 $EndSCHEMATC

Commit message: Experimenting with MEM board configurations and layouts.
Parts:
- removed U101, U102, U105, U106, U107, U108, U109, U110: IS64C5128AL-12KLA3, Package_DIP:DIP-40_W15.24mm, symbol Memory_RAM:IS64C5128AL-12KLA3
- removed U?: 74HC138, alexios:SOIC-16, symbol alexios:74HC138
- renumbered U111 to U1, U112 to U2, U103 to U3, U104 to U4
Connections:
- net labels added: AB[0..18]
- wire segments 386 -> 169
Other:
- moved on the sheet: U1, U2, U3A, U4A

Commit message: Working on MEM board.
Parts:
- added JP101: Jumper_3_Bridged12, Connector_PinHeader_2.54mm:PinHeader_1x03_P2.54mm_Vertical, symbol Jumper:Jumper_3_Bridged12
- added U29: 74HC138, alexios:SOIC-16, symbol alexios:74HC138
Connections:
- net labels added: ~CS0, ~CS1, ~CS10, ~CS11, ~CS2, ~CS3, ~CS4, ~CS5, ~CS6, ~CS7, ~CS8, ~CS9, ~ROMCS, ~ROMWE
- net labels removed: ~RBCE0, ~RBCE1, ~RBCE2, ~RBCE3, ~RBCE4, ~RBCE5, ~RBCE6, ~RBCE7, ~ROMCE
- wire segments 169 -> 186
- no-connect marks 10 -> 14
Other:
- note added: "AB=00AAAxxx:xxxxxxxx:xxxxxxxx\n(0–4096K, chunks of 512K)"
- note added: "AB=01AAAxxx:xxxxxxxx:xxxxxxxx\n(4096–8192K, chunks of 512K)"
- moved on the sheet: U1, U2

Commit message: Working on MEM schematics and board.
Parts:
- added C51, C52, C53, C54: 100nF, alexios:LED_0805_2012Metric_Pad1.15x1.40mm_HandSolder, symbol Device:C_Small
- added unit 2 of U29
- added unit 2 of U3
- added U30: 74AC32, alexios:SOIC-14, symbol alexios:74AC32
- added unit 2 of U4
Connections:
- net +5V: now also JP101.3 (B), C51.1, C52.1, C53.1, C54.1, U29.16 (VCC), U3.16 (VCC), U30.14 (VCC), U4.16 (VCC); no longer JP101.1 (A)
- net GND: now also C51.2, C52.2, C53.2, C54.2, U29.8 (GND), U3.8 (GND), U30.1, U30.2, U30.4, U30.5, U30.7 (GND), U4.8 (GND)
- net ~MEM: now also U30.10, U30.13
- net ~R: now also U30.12; no longer U1.32 (OE), U2.32 (OE)
- net ~W: now also U30.9; no longer JP101.3 (B)
- net ~ROMWE renamed ~ROMW
- new net ~MEMR: JP101.1 (A), U1.32 (OE), U2.32 (OE), U30.11
- new net ~MEMW: U30.8
- no-connect marks 14 -> 43
Other:
- note removed: "Power switch from front pane"
- moved on the sheet: JP101

Commit message: Routing MEM board.
Parts:
- removed U1, U2: 29W040, Sockets:PLCC32, symbol Memory_Flash:29W040
- added C55, C56: 100nF, alexios:SMD_0805_2012Metric_Pad1.15x1.40mm_HandSolder, symbol Device:C_Small
- added U1, U2: 29W040, alexios:PLCC32, symbol alexios:29W040
- C51, C52, C53, C54: footprint alexios:LED_0805_2012Metric_Pad1.15x1.40mm_HandSolder -> alexios:SMD_0805_2012Metric_Pad1.15x1.40mm_HandSolder
Connections:
- net +5V: now also C55.1, C56.1, U1.32 (VCC), U2.32 (VCC)
- net AB0: now also U1.12 (A0), U2.12 (A0)
- net AB1: now also U1.11 (A1), U2.11 (A1)
- net AB10: now also U1.23 (A10), U2.23 (A10)
- net AB11: now also U1.25 (A11), U2.25 (A11)
- net AB12: now also U1.4 (A12), U2.4 (A12)
- net AB13: now also U1.28 (A13), U2.28 (A13)
- net AB14: now also U1.29 (A14), U2.29 (A14)
- net AB15: now also U1.3 (A15), U2.3 (A15)
- net AB16: now also U1.2 (A16), U2.2 (A16)
- net AB17: now also U1.30 (A17), U2.30 (A17)
- net AB18: now also U1.1 (A18), U2.1 (A18)
- net AB2: now also U1.10 (A2), U2.10 (A2)
- net AB3: now also U1.9 (A3), U2.9 (A3)
- net AB4: now also U1.8 (A4), U2.8 (A4)
- net AB5: now also U1.7 (A5), U2.7 (A5)
- net AB6: now also U1.6 (A6), U2.6 (A6)
- net AB7: now also U1.5 (A7), U2.5 (A7)
- net AB8: now also U1.27 (A8), U2.27 (A8)
- net AB9: now also U1.26 (A9), U2.26 (A9)
- net DB0: now also U1.13 (D0)
- net DB1: now also U1.14 (D1)
- net DB10: now also U2.15 (D2)
- net DB11: now also U2.17 (D3)
- net DB12: now also U2.18 (D4)
- net DB13: now also U2.19 (D5)
- net DB14: now also U2.20 (D6)
- net DB15: now also U2.21 (D7)
- net DB2: now also U1.15 (D2)
- net DB3: now also U1.17 (D3)
- net DB4: now also U1.18 (D4)
- net DB5: now also U1.19 (D5)
- net DB6: now also U1.20 (D6)
- net DB7: now also U1.21 (D7)
- net DB8: now also U2.13 (D0)
- net DB9: now also U2.14 (D1)
- net GND: now also U30.10, U30.12, U30.13, U30.9, C55.2, C56.2, U1.16 (GND), U2.16 (GND); no longer U30.1, U30.2, U30.4, U30.5
- net ~MEM: now also U30.2, U30.5; no longer U30.10, U30.13
- net ~MEMR: now also U30.3, U1.24 (~OE), U2.24 (~OE); no longer U30.11
- net ~MEMW: now also U30.6; no longer U30.8
- net ~R: now also U30.1; no longer U30.12
- net ~ROMCS: now also U1.22 (~CE), U2.22 (~CE)
- net ~ROMW: now also U1.31 (~WE), U2.31 (~WE)
- net ~W: now also U30.4; no longer U30.9
Other:
- moved on the sheet: U30A, U30B, U30C, U30D

Commit message: Routing MEM board
Connections:
- no-connect marks 43 -> 44
Other:
- moved on the sheet: C51, C52, C53, U29A, U29B, U3A, U3B, U4A, U4B

Commit message: Fully routed MEM board.
Connections:
- net ~MEMR: no longer JP101.1 (A)
- net ~MEMW: now also JP101.1 (A)
Other:
- moved on the sheet: JP101
Changed lines of the file:
@@
 L Jumper:Jumper_3_Bridged12 JP101
 U 1 1 5D8A2F99
-P 25750 1950
-F 0 "JP101" V 25750 2016 50  0000 L CNN
-F 1 "Jumper_3_Bridged12" V 25795 2016 50  0001 L CNN
-F 2 "Connector_PinHeader_2.54mm:PinHeader_1x03_P2.54mm_Vertical" H 25750 1950 50  0001 C CNN
-F 3 "~" H 25750 1950 50  0001 C CNN
-	1    25750 1950
+P 25800 2150
+F 0 "JP101" V 25800 2216 50  0000 L CNN
+F 1 "Jumper_3_Bridged12" V 25845 2216 50  0001 L CNN
+F 2 "Connector_PinHeader_2.54mm:PinHeader_1x03_P2.54mm_Vertical" H 25800 2150 50  0001 C CNN
+F 3 "~" H 25800 2150 50  0001 C CNN
+	1    25800 2150
 	0    -1   -1   0
 $EndComp
@@
 L power:+5V #PWR0110
 U 1 1 5D8DB890
-P 25750 1700
-F 0 "#PWR0110" H 25750 1550 50  0001 C CNN
-F 1 "+5V" H 25765 1873 50  0000 C CNN
-F 2 "" H 25750 1700 50  0001 C CNN
-F 3 "" H 25750 1700 50  0001 C CNN
-	1    25750 1700
-	1    0    0    -1
-$EndComp
-Wire Wire Line
-	25900 1950 26200 1950
-Text Label 26200 1950 2    50   ~ 0
+P 25800 1900
+F 0 "#PWR0110" H 25800 1750 50  0001 C CNN
+F 1 "+5V" H 25815 2073 50  0000 C CNN
+F 2 "" H 25800 1900 50  0001 C CNN
+F 3 "" H 25800 1900 50  0001 C CNN
+	1    25800 1900
+	1    0    0    -1
+$EndComp
+Wire Wire Line
+	25950 2150 26250 2150
+Text Label 26250 2150 2    50   ~ 0
 ~ROMW
 Text Label -5150 1550 2    50   ~ 0
@@
 	1    0    0    -1
 $EndComp
-Wire Wire Line
-	25750 2600 26200 2600
-Text Label 26200 2600 2    50   ~ 0
-~MEMR
-Wire Wire Line
-	25750 3050 26200 3050
-Text Label 26200 3050 2    50   ~ 0
+Text Label 26250 2600 2    50   ~ 0
+~MEMR
+Wire Wire Line
+	25750 3050 25800 3050
+Text Label 26250 3050 2    50   ~ 0
 ~MEMW
 Wire Wire Line
@@
 $EndComp
 Connection ~ 26950 3000
-Wire Wire Line
-	25750 2200 25750 2600
-Connection ~ 25750 2600
 Text Label 1450 1450 0    50   ~ 0
 ~MEMR
@@
 	22500 5350 22650 5350
 NoConn ~ 22650 5350
+Wire Wire Line
+	25750 2600 26250 2600
+Wire Wire Line
+	25800 2400 25800 3050
+Connection ~ 25800 3050
+Wire Wire Line
+	25800 3050 26250 3050
 $EndSCHEMATC
