File: kicad/cft/mem/mem.kicad_pcb (KiCad board)
At the start: 2 copper layers, 131.9 x 164.6 mm, 93 parts, among them P1 CFT-2019-Bus, U1 29W040, U10 IS61C5128AL, U11 IS61C5128AL, U12 IS61C5128AL, U13 IS61C5128AL, U14 IS61C5128AL, U15 IS61C5128AL, U16 IS61C5128AL, U17 IS61C5128AL, U18 IS61C5128AL, U19 IS61C5128AL, U2 29W040, U20 IS61C5128AL, U21 IS61C5128AL, U22 IS61C5128AL, U23 IS61C5128AL, U24 IS61C5128AL, U25 IS61C5128AL, U26 IS61C5128AL, U27 IS61C5128AL, U28 IS61C5128AL, U29 74HC138, U3 74HC138, U30 74AC32, U4 74HC138, U5 IS61C5128AL, U6 IS61C5128AL, U7 IS61C5128AL, U8 IS61C5128AL, U9 IS61C5128AL

Commit message: Worked on MEM board.
Parts:
- moved JP101 5.08 mm to (146.1, 214.0), turned to 0 degrees
Connections:
- JP101 pad 1: /~MEMW -> +5V
- JP101 pad 3: +5V -> /~MEMW

Commit message: Worked on MEM board.
Routing:
- net /AB22: track 61.5 -> 49.0 mm
- net /AB23: track 65.6 -> 53.4 mm, vias 5 -> 4
- net /AB21: track 66.2 -> 56.7 mm
- net /AB20: track 56.5 -> 47.5 mm
- net /~CS2: track 130.6 -> 122.3 mm
- net /~CS1: track 172.4 -> 169.2 mm
- net /AB11: track 558.1 -> 560.3 mm
- net /AB12: track 525.2 -> 527.1 mm
- net /AB13: track 554.1 -> 555.6 mm
- net /AB5: track 564.6 -> 566.0 mm
- net GND: track 269.0 -> 270.2 mm
- net /AB14: track 552.4 -> 553.0 mm

Commit message: Fine-tuning MEM board.
Parts:
- added G***: LOGO, alexios:CFT, F.Cu at (106.7, 92.7)
- added REF**: OSHW-Logo2_14.6x12mm_SilkScreen, Symbol:OSHW-Logo2_14.6x12mm_SilkScreen, B.Cu at (196.8, 101.6)
- added REF**: ESD-Logo_6.6x6mm_SilkScreen, Symbol:ESD-Logo_6.6x6mm_SilkScreen, F.Cu at (200.7, 212.1)
- added REF**: QRCODE-CFT, alexios:QRCODE-CFT, B.Cu at (171.4, 218.4)
Routing:
- net /AB21: track 56.7 -> 45.4 mm
- net /AB15: track 542.1 -> 552.7 mm
- net /AB18: track 548.2 -> 556.5 mm
- net /~CS4: track 98.1 -> 106.1 mm
- net /~CS2: track 122.3 -> 115.6 mm
- net /AB10: track 628.2 -> 622.1 mm
- net /~MEMR: track 576.7 -> 570.8 mm
- net /AB20: track 47.5 -> 42.0 mm
- net /~CS1: track 169.2 -> 164.3 mm
- net /~ROMCS: track 241.4 -> 236.9 mm
- net /AB0: track 604.9 -> 600.8 mm
- net /DB14: track 372.8 -> 368.7 mm
- net /AB1: track 581.7 -> 577.6 mm
- net /DB13: track 367.9 -> 364.2 mm
- net /DB15: track 361.5 -> 358.4 mm
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Other:
- board text removed: "0 1 0 1"
- board text removed: "2 3 2 3"
- board text removed: "4 5 4 5"
- board text removed: "6 7 6 7"
- board text removed: "8 9 8 9"
- board text removed: "A B A B"
- board text removed: "LSB MSB"

Commit message: Fine-tuning MEM board.
Routing:
- net (no net): track 6.29 -> 0.00 mm
- net /AB23: track 53.4 -> 51.4 mm
- net GND: vias 609 -> 644
- net /AB9: vias 13 -> 12
- net /AB6: vias 11 -> 10

Commit message: Added card handles, fine tuned board.
Parts:
- added C57: 47µF, Capacitor_THT:CP_Radial_D6.3mm_P2.50mm, F.Cu at (200.7, 152.4)
- added C58: 47µF, Capacitor_THT:CP_Radial_D6.3mm_P2.50mm, F.Cu at (201.4, 205.8)
Routing:
- net /AB14: track 552.2 -> 545.5 mm
- net /DB0: track 369.8 -> 363.4 mm
- net /DB1: track 405.5 -> 400.0 mm
- net /DB2: track 404.7 -> 400.1 mm
- net /DB3: track 406.7 -> 402.9 mm
- net /~MEMR: track 570.8 -> 567.6 mm
- net /AB10: track 622.1 -> 619.4 mm
- net /~ROMCS: track 236.9 -> 234.3 mm
- net /AB1: track 577.6 -> 575.2 mm
- net /AB0: track 600.8 -> 598.7 mm
- net /AB3: track 569.9 -> 567.9 mm
- net /DB14: track 368.7 -> 366.7 mm
- net /AB2: track 594.7 -> 592.8 mm
- net /AB6: track 564.5 -> 562.7 mm
- net /AB9: track 628.3 -> 626.5 mm
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Other:
- board text added: "1"
- board text added: "1-2: Flash Write Protect"
- board text added: "2"
- board text added: "2-3: Flash Write Enable"
- board text added: "3"
- board text added: "6 MW RAM, 512 kW ROM Board"
- board text added: "This is NOT PCI Express! Do not plug into any slot meant for PCI Express."

Commit message: Switched to new PLCC socket. Fine tuned board. Added datecode.
Parts:
- added REF**: SIGNATURESILK, alexios:SIGNATURE, F.Cu at (200.7, 222.2)
- moved REF** 109.2 mm to (91.4, 212.1)
Other:
- board text added: "1939"
