File: kicad/cft/mem/rambank.sch (KiCad schematic (older format))
At the start: 6 parts, among them U5 IS61C5128AL, U6 IS61C5128AL

Commit message: Working on MEM board.
Changed lines of the file:
@@
 EESchema Schematic File Version 4
 LIBS:mem-cache
-EELAYER 30 0
+EELAYER 26 0
 EELAYER END
 $Descr A4 11693 8268
 encoding utf-8
-Sheet 4 14
+Sheet 3 14
 Title ""
 Date ""
@@
 AR Path="/5ECDEC6E/5EACCD3C" Ref="U26"  Part="1"
 AR Path="/5ECDEC7E/5EACCD3C" Ref="U28"  Part="1"
-F 0 "U8" H 6500 4517 50  0000 C CNN
+F 0 "U28" H 6500 4517 50  0000 C CNN
 F 1 "IS61C5128AL" H 6500 4426 50  0000 C CNN
 F 2 "Package_SO:SOJ-36_10.16x23.49mm_P1.27mm" V 6400 3375 50  0001 C CNN
@@
 AR Path="/5ECDEC6E/5EACCD43" Ref="U25"  Part="1"
 AR Path="/5ECDEC7E/5EACCD43" Ref="U27"  Part="1"
-F 0 "U7" H 4600 4517 50  0000 C CNN
+F 0 "U27" H 4600 4517 50  0000 C CNN
 F 1 "IS61C5128AL" H 4600 4426 50  0000 C CNN
 F 2 "Package_SO:SOJ-36_10.16x23.49mm_P1.27mm" V 4500 3375 50  0001 C CNN
@@
 AR Path="/5ECDEC6E/5EAD7016" Ref="U25"  Part="2"
 AR Path="/5ECDEC7E/5EAD7016" Ref="U27"  Part="2"
-F 0 "U7" H 4575 5917 50  0000 C CNN
+F 0 "U27" H 4575 5917 50  0000 C CNN
 F 1 "IS61C5128AL" H 4575 5826 50  0000 C CNN
 F 2 "Package_SO:SOJ-36_10.16x23.49mm_P1.27mm" V 4500 5675 50  0001 C CNN
@@
 AR Path="/5ECDEC6E/5EAD85F7" Ref="U26"  Part="2"
 AR Path="/5ECDEC7E/5EAD85F7" Ref="U28"  Part="2"
-F 0 "U8" H 6475 5917 50  0000 C CNN
+F 0 "U28" H 6475 5917 50  0000 C CNN
 F 1 "IS61C5128AL" H 6475 5826 50  0000 C CNN
 F 2 "Package_SO:SOJ-36_10.16x23.49mm_P1.27mm" V 6400 5675 50  0001 C CNN
@@
 AR Path="/5ECDEC6E/5EADE4AF" Ref="#PWR090"  Part="1"
 AR Path="/5ECDEC7E/5EADE4AF" Ref="#PWR098"  Part="1"
-F 0 "#PWR018" H 4150 5200 50  0001 C CNN
+F 0 "#PWR098" H 4150 5200 50  0001 C CNN
 F 1 "+5V" H 4165 5523 50  0000 C CNN
 F 2 "" H 4150 5350 50  0001 C CNN
@@
 AR Path="/5ECDEC6E/5EADE72D" Ref="#PWR092"  Part="1"
 AR Path="/5ECDEC7E/5EADE72D" Ref="#PWR0100"  Part="1"
-F 0 "#PWR020" H 5000 5200 50  0001 C CNN
+F 0 "#PWR0100" H 5000 5200 50  0001 C CNN
 F 1 "+5V" H 5015 5523 50  0000 C CNN
 F 2 "" H 5000 5350 50  0001 C CNN
@@
 AR Path="/5ECDEC6E/5EADE7CB" Ref="#PWR094"  Part="1"
 AR Path="/5ECDEC7E/5EADE7CB" Ref="#PWR0102"  Part="1"
-F 0 "#PWR022" H 6050 5200 50  0001 C CNN
+F 0 "#PWR0102" H 6050 5200 50  0001 C CNN
 F 1 "+5V" H 6065 5523 50  0000 C CNN
 F 2 "" H 6050 5350 50  0001 C CNN
@@
 AR Path="/5ECDEC6E/5EADE963" Ref="#PWR096"  Part="1"
 AR Path="/5ECDEC7E/5EADE963" Ref="#PWR0104"  Part="1"
-F 0 "#PWR024" H 6900 5200 50  0001 C CNN
+F 0 "#PWR0104" H 6900 5200 50  0001 C CNN
 F 1 "+5V" H 6915 5523 50  0000 C CNN
 F 2 "" H 6900 5350 50  0001 C CNN
@@
 AR Path="/5ECDEC6E/5EADEDDC" Ref="#PWR097"  Part="1"
 AR Path="/5ECDEC7E/5EADEDDC" Ref="#PWR0105"  Part="1"
-F 0 "#PWR025" H 6900 5300 50  0001 C CNN
+F 0 "#PWR0105" H 6900 5300 50  0001 C CNN
 F 1 "GND" H 6905 5377 50  0000 C CNN
 F 2 "" H 6900 5550 50  0001 C CNN
@@
 AR Path="/5ECDEC6E/5EADF1C4" Ref="#PWR095"  Part="1"
 AR Path="/5ECDEC7E/5EADF1C4" Ref="#PWR0103"  Part="1"
-F 0 "#PWR023" H 6050 5300 50  0001 C CNN
+F 0 "#PWR0103" H 6050 5300 50  0001 C CNN
 F 1 "GND" H 6055 5377 50  0000 C CNN
 F 2 "" H 6050 5550 50  0001 C CNN
@@
 AR Path="/5ECDEC6E/5EADF5B8" Ref="#PWR091"  Part="1"
 AR Path="/5ECDEC7E/5EADF5B8" Ref="#PWR099"  Part="1"
-F 0 "#PWR019" H 4150 5300 50  0001 C CNN
+F 0 "#PWR099" H 4150 5300 50  0001 C CNN
 F 1 "GND" H 4155 5377 50  0000 C CNN
 F 2 "" H 4150 5550 50  0001 C CNN
@@
 AR Path="/5ECDEC6E/5EADFE90" Ref="#PWR093"  Part="1"
 AR Path="/5ECDEC7E/5EADFE90" Ref="#PWR0101"  Part="1"
-F 0 "#PWR021" H 5000 5300 50  0001 C CNN
+F 0 "#PWR0101" H 5000 5300 50  0001 C CNN
 F 1 "GND" H 5005 5377 50  0000 C CNN
 F 2 "" H 5000 5550 50  0001 C CNN
@@
 AR Path="/5ECDEC6E/5EAE1505" Ref="C43"  Part="1"
 AR Path="/5ECDEC7E/5EAE1505" Ref="C47"  Part="1"
-F 0 "C7" H 4059 5496 50  0000 R CNN
+F 0 "C47" H 4059 5496 50  0000 R CNN
 F 1 "100nF" H 4059 5405 50  0000 R CNN
 F 2 "alexios:LED_0805_2012Metric_Pad1.15x1.40mm_HandSolder" H 4150 5450 50  0001 C CNN
@@
 AR Path="/5ECDEC6E/5EAE33D6" Ref="C44"  Part="1"
 AR Path="/5ECDEC7E/5EAE33D6" Ref="C48"  Part="1"
-F 0 "C8" H 5092 5496 50  0000 L CNN
+F 0 "C48" H 5092 5496 50  0000 L CNN
 F 1 "100nF" H 5092 5405 50  0000 L CNN
 F 2 "alexios:LED_0805_2012Metric_Pad1.15x1.40mm_HandSolder" H 5000 5450 50  0001 C CNN
@@
 AR Path="/5ECDEC6E/5EAE37CE" Ref="C45"  Part="1"
 AR Path="/5ECDEC7E/5EAE37CE" Ref="C49"  Part="1"
-F 0 "C9" H 5959 5496 50  0000 R CNN
+F 0 "C49" H 5959 5496 50  0000 R CNN
 F 1 "100nF" H 5959 5405 50  0000 R CNN
 F 2 "alexios:LED_0805_2012Metric_Pad1.15x1.40mm_HandSolder" H 6050 5450 50  0001 C CNN
@@
 AR Path="/5ECDEC6E/5EAE3E26" Ref="C46"  Part="1"
 AR Path="/5ECDEC7E/5EAE3E26" Ref="C50"  Part="1"
-F 0 "C10" H 6992 5496 50  0000 L CNN
+F 0 "C50" H 6992 5496 50  0000 L CNN
 F 1 "100nF" H 6992 5405 50  0000 L CNN
 F 2 "alexios:LED_0805_2012Metric_Pad1.15x1.40mm_HandSolder" H 6900 5450 50  0001 C CNN
@@
 Text HLabel 3100 4600 0    50   3State ~ 0
 ~DB[0..15]
+Text Label 3150 4600 0    50   ~ 0
+DB[0..15]
 Wire Bus Line
 	5350 2150 5350 4500
@@
 Wire Bus Line
 	5700 1700 5700 3750
-Text Label 3150 4600 0    50   ~ 0
-DB[0..15]
 $EndSCHEMATC

Commit message: Working on MEM schematics and board.
Changed lines of the file:
@@
 $Descr A4 11693 8268
 encoding utf-8
-Sheet 3 14
+Sheet 14 14
 Title ""
 Date ""
@@
 AR Path="/5ECDEC6E/5EACCD3C" Ref="U26"  Part="1"
 AR Path="/5ECDEC7E/5EACCD3C" Ref="U28"  Part="1"
-F 0 "U28" H 6500 4517 50  0000 C CNN
+F 0 "U6" H 6500 4517 50  0000 C CNN
 F 1 "IS61C5128AL" H 6500 4426 50  0000 C CNN
 F 2 "Package_SO:SOJ-36_10.16x23.49mm_P1.27mm" V 6400 3375 50  0001 C CNN
@@
 AR Path="/5ECDEC6E/5EACCD43" Ref="U25"  Part="1"
 AR Path="/5ECDEC7E/5EACCD43" Ref="U27"  Part="1"
-F 0 "U27" H 4600 4517 50  0000 C CNN
+F 0 "U5" H 4600 4517 50  0000 C CNN
 F 1 "IS61C5128AL" H 4600 4426 50  0000 C CNN
 F 2 "Package_SO:SOJ-36_10.16x23.49mm_P1.27mm" V 4500 3375 50  0001 C CNN
@@
 AR Path="/5ECDEC6E/5EAD7016" Ref="U25"  Part="2"
 AR Path="/5ECDEC7E/5EAD7016" Ref="U27"  Part="2"
-F 0 "U27" H 4575 5917 50  0000 C CNN
+F 0 "U5" H 4575 5917 50  0000 C CNN
 F 1 "IS61C5128AL" H 4575 5826 50  0000 C CNN
 F 2 "Package_SO:SOJ-36_10.16x23.49mm_P1.27mm" V 4500 5675 50  0001 C CNN
@@
 AR Path="/5ECDEC6E/5EAD85F7" Ref="U26"  Part="2"
 AR Path="/5ECDEC7E/5EAD85F7" Ref="U28"  Part="2"
-F 0 "U28" H 6475 5917 50  0000 C CNN
+F 0 "U6" H 6475 5917 50  0000 C CNN
 F 1 "IS61C5128AL" H 6475 5826 50  0000 C CNN
 F 2 "Package_SO:SOJ-36_10.16x23.49mm_P1.27mm" V 6400 5675 50  0001 C CNN
@@
 AR Path="/5ECDEC6E/5EAE1505" Ref="C43"  Part="1"
 AR Path="/5ECDEC7E/5EAE1505" Ref="C47"  Part="1"
-F 0 "C47" H 4059 5496 50  0000 R CNN
+F 0 "C3" H 4059 5496 50  0000 R CNN
 F 1 "100nF" H 4059 5405 50  0000 R CNN
 F 2 "alexios:LED_0805_2012Metric_Pad1.15x1.40mm_HandSolder" H 4150 5450 50  0001 C CNN
@@
 AR Path="/5ECDEC6E/5EAE33D6" Ref="C44"  Part="1"
 AR Path="/5ECDEC7E/5EAE33D6" Ref="C48"  Part="1"
-F 0 "C48" H 5092 5496 50  0000 L CNN
+F 0 "C4" H 5092 5496 50  0000 L CNN
 F 1 "100nF" H 5092 5405 50  0000 L CNN
 F 2 "alexios:LED_0805_2012Metric_Pad1.15x1.40mm_HandSolder" H 5000 5450 50  0001 C CNN
@@
 Connection ~ 5000 5350
 Connection ~ 5000 5550
-$Comp
-L Device:C_Small C5
-U 1 1 5EAE37CE
-P 6050 5450
-AR Path="/5E94D03A/5EAE37CE" Ref="C5"  Part="1"
-AR Path="/5EC68F14/5EAE37CE" Ref="C9"  Part="1"
-AR Path="/5EC75B87/5EAE37CE" Ref="C13"  Part="1"
-AR Path="/5EC75B97/5EAE37CE" Ref="C17"  Part="1"
-AR Path="/5EC8475C/5EAE37CE" Ref="C?"  Part="1"
-AR Path="/5EC8476C/5EAE37CE" Ref="C?"  Part="1"
-AR Path="/5EC8477C/5EAE37CE" Ref="C?"  Part="1"
-AR Path="/5EC8478C/5EAE37CE" Ref="C?"  Part="1"
-AR Path="/5ECB980E/5EAE37CE" Ref="C?"  Part="1"
-AR Path="/5ECB981E/5EAE37CE" Ref="C?"  Part="1"
-AR Path="/5ECCD509/5EAE37CE" Ref="C21"  Part="1"
-AR Path="/5ECCD519/5EAE37CE" Ref="C25"  Part="1"
-AR Path="/5ECCD529/5EAE37CE" Ref="C29"  Part="1"
-AR Path="/5ECCD539/5EAE37CE" Ref="C33"  Part="1"
-AR Path="/5ECDEC4E/5EAE37CE" Ref="C37"  Part="1"
-AR Path="/5ECDEC5E/5EAE37CE" Ref="C41"  Part="1"
-AR Path="/5ECDEC6E/5EAE37CE" Ref="C45"  Part="1"
-AR Path="/5ECDEC7E/5EAE37CE" Ref="C49"  Part="1"
-F 0 "C49" H 5959 5496 50  0000 R CNN
-F 1 "100nF" H 5959 5405 50  0000 R CNN
-F 2 "alexios:LED_0805_2012Metric_Pad1.15x1.40mm_HandSolder" H 6050 5450 50  0001 C CNN
-F 3 "~" H 6050 5450 50  0001 C CNN
-	1    6050 5450
-	1    0    0    -1
-$EndComp
-Connection ~ 6050 5350
-Connection ~ 6050 5550
 $Comp
 L Device:C_Small C6
@@
 AR Path="/5ECDEC6E/5EAE3E26" Ref="C46"  Part="1"
 AR Path="/5ECDEC7E/5EAE3E26" Ref="C50"  Part="1"
-F 0 "C50" H 6992 5496 50  0000 L CNN
+F 0 "C6" H 6992 5496 50  0000 L CNN
 F 1 "100nF" H 6992 5405 50  0000 L CNN
 F 2 "alexios:LED_0805_2012Metric_Pad1.15x1.40mm_HandSolder" H 6900 5450 50  0001 C CNN
@@
 DB[0..15]
 Wire Bus Line
-	5350 2150 5350 4500
+	5700 1700 5700 3750
+Wire Bus Line
+	3800 1700 3800 3750
 Wire Bus Line
 	7300 2150 7300 4500
 Wire Bus Line
-	3800 1700 3800 3750
-Wire Bus Line
-	5700 1700 5700 3750
+	5350 2150 5350 4500
+Connection ~ 6050 5550
+Connection ~ 6050 5350
+$Comp
+L Device:C_Small C5
+U 1 1 5EAE37CE
+P 6050 5450
+AR Path="/5E94D03A/5EAE37CE" Ref="C5"  Part="1"
+AR Path="/5EC68F14/5EAE37CE" Ref="C9"  Part="1"
+AR Path="/5EC75B87/5EAE37CE" Ref="C13"  Part="1"
+AR Path="/5EC75B97/5EAE37CE" Ref="C17"  Part="1"
+AR Path="/5EC8475C/5EAE37CE" Ref="C?"  Part="1"
+AR Path="/5EC8476C/5EAE37CE" Ref="C?"  Part="1"
+AR Path="/5EC8477C/5EAE37CE" Ref="C?"  Part="1"
+AR Path="/5EC8478C/5EAE37CE" Ref="C?"  Part="1"
+AR Path="/5ECB980E/5EAE37CE" Ref="C?"  Part="1"
+AR Path="/5ECB981E/5EAE37CE" Ref="C?"  Part="1"
+AR Path="/5ECCD509/5EAE37CE" Ref="C21"  Part="1"
+AR Path="/5ECCD519/5EAE37CE" Ref="C25"  Part="1"
+AR Path="/5ECCD529/5EAE37CE" Ref="C29"  Part="1"
+AR Path="/5ECCD539/5EAE37CE" Ref="C33"  Part="1"
+AR Path="/5ECDEC4E/5EAE37CE" Ref="C37"  Part="1"
+AR Path="/5ECDEC5E/5EAE37CE" Ref="C41"  Part="1"
+AR Path="/5ECDEC6E/5EAE37CE" Ref="C45"  Part="1"
+AR Path="/5ECDEC7E/5EAE37CE" Ref="C49"  Part="1"
+F 0 "C5" H 5959 5496 50  0000 R CNN
+F 1 "100nF" H 5959 5405 50  0000 R CNN
+F 2 "alexios:LED_0805_2012Metric_Pad1.15x1.40mm_HandSolder" H 6050 5450 50  0001 C CNN
+F 3 "~" H 6050 5450 50  0001 C CNN
+	1    6050 5450
+	1    0    0    -1
+$EndComp
 $EndSCHEMATC

Commit message: Routing MEM board.
Parts:
- C3, C4, C5, C6: footprint alexios:LED_0805_2012Metric_Pad1.15x1.40mm_HandSolder -> alexios:SMD_0805_2012Metric_Pad1.15x1.40mm_HandSolder
- U5, U6: footprint Package_SO:SOJ-36_10.16x23.49mm_P1.27mm -> alexios:SOJ-36_10.16x23.49mm_P1.27mm
Changed lines of the file:
@@
 EESchema Schematic File Version 4
 LIBS:mem-cache
-EELAYER 26 0
+EELAYER 30 0
 EELAYER END
 $Descr A4 11693 8268
 encoding utf-8
-Sheet 14 14
+Sheet 11 14
 Title ""
 Date ""
@@
 AR Path="/5ECDEC6E/5EACCD3C" Ref="U26"  Part="1"
 AR Path="/5ECDEC7E/5EACCD3C" Ref="U28"  Part="1"
-F 0 "U6" H 6500 4517 50  0000 C CNN
+F 0 "U22" H 6500 4517 50  0000 C CNN
 F 1 "IS61C5128AL" H 6500 4426 50  0000 C CNN
-F 2 "Package_SO:SOJ-36_10.16x23.49mm_P1.27mm" V 6400 3375 50  0001 C CNN
+F 2 "alexios:SOJ-36_10.16x23.49mm_P1.27mm" V 6400 3375 50  0001 C CNN
 F 3 "https://uk.mouser.com/datasheet/2/12/AS6C8008-1288432.pdf" H 6400 3450 50  0001 C CNN
 F 4 "870-61C5128AL-10KLI; €3.11" H 5700 1500 50  0001 L CNN "AC:BOM-Mouser"
@@
 AR Path="/5ECDEC6E/5EACCD43" Ref="U25"  Part="1"
 AR Path="/5ECDEC7E/5EACCD43" Ref="U27"  Part="1"
-F 0 "U5" H 4600 4517 50  0000 C CNN
+F 0 "U21" H 4600 4517 50  0000 C CNN
 F 1 "IS61C5128AL" H 4600 4426 50  0000 C CNN
-F 2 "Package_SO:SOJ-36_10.16x23.49mm_P1.27mm" V 4500 3375 50  0001 C CNN
+F 2 "alexios:SOJ-36_10.16x23.49mm_P1.27mm" V 4500 3375 50  0001 C CNN
 F 3 "https://uk.mouser.com/datasheet/2/12/AS6C8008-1288432.pdf" H 4500 3450 50  0001 C CNN
 F 4 "870-61C5128AL-10KLI; €3.11" H 3800 1500 50  0001 L CNN "AC:BOM-Mouser"
@@
 AR Path="/5ECDEC6E/5EAD7016" Ref="U25"  Part="2"
 AR Path="/5ECDEC7E/5EAD7016" Ref="U27"  Part="2"
-F 0 "U5" H 4575 5917 50  0000 C CNN
+F 0 "U21" H 4575 5917 50  0000 C CNN
 F 1 "IS61C5128AL" H 4575 5826 50  0000 C CNN
-F 2 "Package_SO:SOJ-36_10.16x23.49mm_P1.27mm" V 4500 5675 50  0001 C CNN
+F 2 "alexios:SOJ-36_10.16x23.49mm_P1.27mm" V 4500 5675 50  0001 C CNN
 F 3 "https://uk.mouser.com/datasheet/2/12/AS6C8008-1288432.pdf" H 4500 5750 50  0001 C CNN
 F 4 "870-61C5128AL-10KLI; €3.11" H 3800 3800 50  0001 L CNN "AC:BOM-Mouser"
@@
 AR Path="/5ECDEC6E/5EAD85F7" Ref="U26"  Part="2"
 AR Path="/5ECDEC7E/5EAD85F7" Ref="U28"  Part="2"
-F 0 "U6" H 6475 5917 50  0000 C CNN
+F 0 "U22" H 6475 5917 50  0000 C CNN
 F 1 "IS61C5128AL" H 6475 5826 50  0000 C CNN
-F 2 "Package_SO:SOJ-36_10.16x23.49mm_P1.27mm" V 6400 5675 50  0001 C CNN
+F 2 "alexios:SOJ-36_10.16x23.49mm_P1.27mm" V 6400 5675 50  0001 C CNN
 F 3 "https://uk.mouser.com/datasheet/2/12/AS6C8008-1288432.pdf" H 6400 5750 50  0001 C CNN
 F 4 "870-61C5128AL-10KLI; €3.11" H 5700 3800 50  0001 L CNN "AC:BOM-Mouser"
@@
 AR Path="/5ECDEC6E/5EADE4AF" Ref="#PWR090"  Part="1"
 AR Path="/5ECDEC7E/5EADE4AF" Ref="#PWR098"  Part="1"
-F 0 "#PWR098" H 4150 5200 50  0001 C CNN
+F 0 "#PWR074" H 4150 5200 50  0001 C CNN
 F 1 "+5V" H 4165 5523 50  0000 C CNN
 F 2 "" H 4150 5350 50  0001 C CNN
@@
 AR Path="/5ECDEC6E/5EADE72D" Ref="#PWR092"  Part="1"
 AR Path="/5ECDEC7E/5EADE72D" Ref="#PWR0100"  Part="1"
-F 0 "#PWR0100" H 5000 5200 50  0001 C CNN
+F 0 "#PWR076" H 5000 5200 50  0001 C CNN
 F 1 "+5V" H 5015 5523 50  0000 C CNN
 F 2 "" H 5000 5350 50  0001 C CNN
@@
 AR Path="/5ECDEC6E/5EADE7CB" Ref="#PWR094"  Part="1"
 AR Path="/5ECDEC7E/5EADE7CB" Ref="#PWR0102"  Part="1"
-F 0 "#PWR0102" H 6050 5200 50  0001 C CNN
+F 0 "#PWR078" H 6050 5200 50  0001 C CNN
 F 1 "+5V" H 6065 5523 50  0000 C CNN
 F 2 "" H 6050 5350 50  0001 C CNN
@@
 AR Path="/5ECDEC6E/5EADE963" Ref="#PWR096"  Part="1"
 AR Path="/5ECDEC7E/5EADE963" Ref="#PWR0104"  Part="1"
-F 0 "#PWR0104" H 6900 5200 50  0001 C CNN
+F 0 "#PWR080" H 6900 5200 50  0001 C CNN
 F 1 "+5V" H 6915 5523 50  0000 C CNN
 F 2 "" H 6900 5350 50  0001 C CNN
@@
 AR Path="/5ECDEC6E/5EADEDDC" Ref="#PWR097"  Part="1"
 AR Path="/5ECDEC7E/5EADEDDC" Ref="#PWR0105"  Part="1"
-F 0 "#PWR0105" H 6900 5300 50  0001 C CNN
+F 0 "#PWR081" H 6900 5300 50  0001 C CNN
 F 1 "GND" H 6905 5377 50  0000 C CNN
 F 2 "" H 6900 5550 50  0001 C CNN
@@
 AR Path="/5ECDEC6E/5EADF1C4" Ref="#PWR095"  Part="1"
 AR Path="/5ECDEC7E/5EADF1C4" Ref="#PWR0103"  Part="1"
-F 0 "#PWR0103" H 6050 5300 50  0001 C CNN
+F 0 "#PWR079" H 6050 5300 50  0001 C CNN
 F 1 "GND" H 6055 5377 50  0000 C CNN
 F 2 "" H 6050 5550 50  0001 C CNN
@@
 AR Path="/5ECDEC6E/5EADF5B8" Ref="#PWR091"  Part="1"
 AR Path="/5ECDEC7E/5EADF5B8" Ref="#PWR099"  Part="1"
-F 0 "#PWR099" H 4150 5300 50  0001 C CNN
+F 0 "#PWR075" H 4150 5300 50  0001 C CNN
 F 1 "GND" H 4155 5377 50  0000 C CNN
 F 2 "" H 4150 5550 50  0001 C CNN
@@
 AR Path="/5ECDEC6E/5EADFE90" Ref="#PWR093"  Part="1"
 AR Path="/5ECDEC7E/5EADFE90" Ref="#PWR0101"  Part="1"
-F 0 "#PWR0101" H 5000 5300 50  0001 C CNN
+F 0 "#PWR077" H 5000 5300 50  0001 C CNN
 F 1 "GND" H 5005 5377 50  0000 C CNN
 F 2 "" H 5000 5550 50  0001 C CNN
@@
 AR Path="/5ECDEC6E/5EAE1505" Ref="C43"  Part="1"
 AR Path="/5ECDEC7E/5EAE1505" Ref="C47"  Part="1"
-F 0 "C3" H 4059 5496 50  0000 R CNN
+F 0 "C35" H 4059 5496 50  0000 R CNN
 F 1 "100nF" H 4059 5405 50  0000 R CNN
-F 2 "alexios:LED_0805_2012Metric_Pad1.15x1.40mm_HandSolder" H 4150 5450 50  0001 C CNN
+F 2 "alexios:SMD_0805_2012Metric_Pad1.15x1.40mm_HandSolder" H 4150 5450 50  0001 C CNN
 F 3 "~" H 4150 5450 50  0001 C CNN
 	1    4150 5450
@@
 AR Path="/5ECDEC6E/5EAE33D6" Ref="C44"  Part="1"
 AR Path="/5ECDEC7E/5EAE33D6" Ref="C48"  Part="1"
-F 0 "C4" H 5092 5496 50  0000 L CNN
+F 0 "C36" H 5092 5496 50  0000 L CNN
 F 1 "100nF" H 5092 5405 50  0000 L CNN
-F 2 "alexios:LED_0805_2012Metric_Pad1.15x1.40mm_HandSolder" H 5000 5450 50  0001 C CNN
+F 2 "alexios:SMD_0805_2012Metric_Pad1.15x1.40mm_HandSolder" H 5000 5450 50  0001 C CNN
 F 3 "~" H 5000 5450 50  0001 C CNN
 	1    5000 5450
@@
 AR Path="/5ECDEC6E/5EAE3E26" Ref="C46"  Part="1"
 AR Path="/5ECDEC7E/5EAE3E26" Ref="C50"  Part="1"
-F 0 "C6" H 6992 5496 50  0000 L CNN
+F 0 "C38" H 6992 5496 50  0000 L CNN
 F 1 "100nF" H 6992 5405 50  0000 L CNN
-F 2 "alexios:LED_0805_2012Metric_Pad1.15x1.40mm_HandSolder" H 6900 5450 50  0001 C CNN
+F 2 "alexios:SMD_0805_2012Metric_Pad1.15x1.40mm_HandSolder" H 6900 5450 50  0001 C CNN
 F 3 "~" H 6900 5450 50  0001 C CNN
 	1    6900 5450
@@
 Text Label 3150 4600 0    50   ~ 0
 DB[0..15]
-Wire Bus Line
-	5700 1700 5700 3750
-Wire Bus Line
-	3800 1700 3800 3750
-Wire Bus Line
-	7300 2150 7300 4500
-Wire Bus Line
-	5350 2150 5350 4500
 Connection ~ 6050 5550
 Connection ~ 6050 5350
@@
 AR Path="/5ECDEC6E/5EAE37CE" Ref="C45"  Part="1"
 AR Path="/5ECDEC7E/5EAE37CE" Ref="C49"  Part="1"
-F 0 "C5" H 5959 5496 50  0000 R CNN
+F 0 "C37" H 5959 5496 50  0000 R CNN
 F 1 "100nF" H 5959 5405 50  0000 R CNN
-F 2 "alexios:LED_0805_2012Metric_Pad1.15x1.40mm_HandSolder" H 6050 5450 50  0001 C CNN
+F 2 "alexios:SMD_0805_2012Metric_Pad1.15x1.40mm_HandSolder" H 6050 5450 50  0001 C CNN
 F 3 "~" H 6050 5450 50  0001 C CNN
 	1    6050 5450
 	1    0    0    -1
 $EndComp
+Wire Bus Line
+	7300 2150 7300 4500
+Wire Bus Line
+	5350 2150 5350 4500
+Wire Bus Line
+	5700 1700 5700 3750
+Wire Bus Line
+	3800 1700 3800 3750
 $EndSCHEMATC

Commit message: Routing MEM board
Changed lines of the file:
@@
 $Descr A4 11693 8268
 encoding utf-8
-Sheet 11 14
+Sheet 3 14
 Title ""
 Date ""
@@
 AR Path="/5ECDEC6E/5EACCD3C" Ref="U26"  Part="1"
 AR Path="/5ECDEC7E/5EACCD3C" Ref="U28"  Part="1"
-F 0 "U22" H 6500 4517 50  0000 C CNN
+F 0 "U6" H 6500 4517 50  0000 C CNN
 F 1 "IS61C5128AL" H 6500 4426 50  0000 C CNN
 F 2 "alexios:SOJ-36_10.16x23.49mm_P1.27mm" V 6400 3375 50  0001 C CNN
@@
 AR Path="/5ECDEC6E/5EACCD43" Ref="U25"  Part="1"
 AR Path="/5ECDEC7E/5EACCD43" Ref="U27"  Part="1"
-F 0 "U21" H 4600 4517 50  0000 C CNN
+F 0 "U5" H 4600 4517 50  0000 C CNN
 F 1 "IS61C5128AL" H 4600 4426 50  0000 C CNN
 F 2 "alexios:SOJ-36_10.16x23.49mm_P1.27mm" V 4500 3375 50  0001 C CNN
@@
 AR Path="/5ECDEC6E/5EAD7016" Ref="U25"  Part="2"
 AR Path="/5ECDEC7E/5EAD7016" Ref="U27"  Part="2"
-F 0 "U21" H 4575 5917 50  0000 C CNN
+F 0 "U5" H 4575 5917 50  0000 C CNN
 F 1 "IS61C5128AL" H 4575 5826 50  0000 C CNN
 F 2 "alexios:SOJ-36_10.16x23.49mm_P1.27mm" V 4500 5675 50  0001 C CNN
@@
 AR Path="/5ECDEC6E/5EAD85F7" Ref="U26"  Part="2"
 AR Path="/5ECDEC7E/5EAD85F7" Ref="U28"  Part="2"
-F 0 "U22" H 6475 5917 50  0000 C CNN
+F 0 "U6" H 6475 5917 50  0000 C CNN
 F 1 "IS61C5128AL" H 6475 5826 50  0000 C CNN
 F 2 "alexios:SOJ-36_10.16x23.49mm_P1.27mm" V 6400 5675 50  0001 C CNN
@@
 AR Path="/5ECDEC6E/5EADE4AF" Ref="#PWR090"  Part="1"
 AR Path="/5ECDEC7E/5EADE4AF" Ref="#PWR098"  Part="1"
-F 0 "#PWR074" H 4150 5200 50  0001 C CNN
+F 0 "#PWR010" H 4150 5200 50  0001 C CNN
 F 1 "+5V" H 4165 5523 50  0000 C CNN
 F 2 "" H 4150 5350 50  0001 C CNN
@@
 AR Path="/5ECDEC6E/5EADE72D" Ref="#PWR092"  Part="1"
 AR Path="/5ECDEC7E/5EADE72D" Ref="#PWR0100"  Part="1"
-F 0 "#PWR076" H 5000 5200 50  0001 C CNN
+F 0 "#PWR012" H 5000 5200 50  0001 C CNN
 F 1 "+5V" H 5015 5523 50  0000 C CNN
 F 2 "" H 5000 5350 50  0001 C CNN
@@
 AR Path="/5ECDEC6E/5EADE7CB" Ref="#PWR094"  Part="1"
 AR Path="/5ECDEC7E/5EADE7CB" Ref="#PWR0102"  Part="1"
-F 0 "#PWR078" H 6050 5200 50  0001 C CNN
+F 0 "#PWR014" H 6050 5200 50  0001 C CNN
 F 1 "+5V" H 6065 5523 50  0000 C CNN
 F 2 "" H 6050 5350 50  0001 C CNN
@@
 AR Path="/5ECDEC6E/5EADE963" Ref="#PWR096"  Part="1"
 AR Path="/5ECDEC7E/5EADE963" Ref="#PWR0104"  Part="1"
-F 0 "#PWR080" H 6900 5200 50  0001 C CNN
+F 0 "#PWR016" H 6900 5200 50  0001 C CNN
 F 1 "+5V" H 6915 5523 50  0000 C CNN
 F 2 "" H 6900 5350 50  0001 C CNN
@@
 AR Path="/5ECDEC6E/5EADEDDC" Ref="#PWR097"  Part="1"
 AR Path="/5ECDEC7E/5EADEDDC" Ref="#PWR0105"  Part="1"
-F 0 "#PWR081" H 6900 5300 50  0001 C CNN
+F 0 "#PWR017" H 6900 5300 50  0001 C CNN
 F 1 "GND" H 6905 5377 50  0000 C CNN
 F 2 "" H 6900 5550 50  0001 C CNN
@@
 AR Path="/5ECDEC6E/5EADF1C4" Ref="#PWR095"  Part="1"
 AR Path="/5ECDEC7E/5EADF1C4" Ref="#PWR0103"  Part="1"
-F 0 "#PWR079" H 6050 5300 50  0001 C CNN
+F 0 "#PWR015" H 6050 5300 50  0001 C CNN
 F 1 "GND" H 6055 5377 50  0000 C CNN
 F 2 "" H 6050 5550 50  0001 C CNN
@@
 AR Path="/5ECDEC6E/5EADF5B8" Ref="#PWR091"  Part="1"
 AR Path="/5ECDEC7E/5EADF5B8" Ref="#PWR099"  Part="1"
-F 0 "#PWR075" H 4150 5300 50  0001 C CNN
+F 0 "#PWR011" H 4150 5300 50  0001 C CNN
 F 1 "GND" H 4155 5377 50  0000 C CNN
 F 2 "" H 4150 5550 50  0001 C CNN
@@
 AR Path="/5ECDEC6E/5EADFE90" Ref="#PWR093"  Part="1"
 AR Path="/5ECDEC7E/5EADFE90" Ref="#PWR0101"  Part="1"
-F 0 "#PWR077" H 5000 5300 50  0001 C CNN
+F 0 "#PWR013" H 5000 5300 50  0001 C CNN
 F 1 "GND" H 5005 5377 50  0000 C CNN
 F 2 "" H 5000 5550 50  0001 C CNN
@@
 AR Path="/5ECDEC6E/5EAE1505" Ref="C43"  Part="1"
 AR Path="/5ECDEC7E/5EAE1505" Ref="C47"  Part="1"
-F 0 "C35" H 4059 5496 50  0000 R CNN
+F 0 "C3" H 4059 5496 50  0000 R CNN
 F 1 "100nF" H 4059 5405 50  0000 R CNN
 F 2 "alexios:SMD_0805_2012Metric_Pad1.15x1.40mm_HandSolder" H 4150 5450 50  0001 C CNN
@@
 AR Path="/5ECDEC6E/5EAE33D6" Ref="C44"  Part="1"
 AR Path="/5ECDEC7E/5EAE33D6" Ref="C48"  Part="1"
-F 0 "C36" H 5092 5496 50  0000 L CNN
+F 0 "C4" H 5092 5496 50  0000 L CNN
 F 1 "100nF" H 5092 5405 50  0000 L CNN
 F 2 "alexios:SMD_0805_2012Metric_Pad1.15x1.40mm_HandSolder" H 5000 5450 50  0001 C CNN
@@
 AR Path="/5ECDEC6E/5EAE3E26" Ref="C46"  Part="1"
 AR Path="/5ECDEC7E/5EAE3E26" Ref="C50"  Part="1"
-F 0 "C38" H 6992 5496 50  0000 L CNN
+F 0 "C6" H 6992 5496 50  0000 L CNN
 F 1 "100nF" H 6992 5405 50  0000 L CNN
 F 2 "alexios:SMD_0805_2012Metric_Pad1.15x1.40mm_HandSolder" H 6900 5450 50  0001 C CNN
@@
 AR Path="/5ECDEC6E/5EAE37CE" Ref="C45"  Part="1"
 AR Path="/5ECDEC7E/5EAE37CE" Ref="C49"  Part="1"
-F 0 "C37" H 5959 5496 50  0000 R CNN
+F 0 "C5" H 5959 5496 50  0000 R CNN
 F 1 "100nF" H 5959 5405 50  0000 R CNN
 F 2 "alexios:SMD_0805_2012Metric_Pad1.15x1.40mm_HandSolder" H 6050 5450 50  0001 C CNN
