File: kicad/cft/mem/rambank.sch (KiCad schematic (older format))
At the start: 6 parts, among them U5 IS61C5128AL, U6 IS61C5128AL

Commit message: Fully routed MEM board.
Changed lines of the file:
@@
 $Descr A4 11693 8268
 encoding utf-8
-Sheet 3 14
+Sheet 14 14
 Title ""
 Date ""
@@
 AR Path="/5ECDEC6E/5EACCD3C" Ref="U26"  Part="1"
 AR Path="/5ECDEC7E/5EACCD3C" Ref="U28"  Part="1"
-F 0 "U6" H 6500 4517 50  0000 C CNN
+F 0 "U28" H 6500 4517 50  0000 C CNN
 F 1 "IS61C5128AL" H 6500 4426 50  0000 C CNN
 F 2 "alexios:SOJ-36_10.16x23.49mm_P1.27mm" V 6400 3375 50  0001 C CNN
@@
 AR Path="/5ECDEC6E/5EACCD43" Ref="U25"  Part="1"
 AR Path="/5ECDEC7E/5EACCD43" Ref="U27"  Part="1"
-F 0 "U5" H 4600 4517 50  0000 C CNN
+F 0 "U27" H 4600 4517 50  0000 C CNN
 F 1 "IS61C5128AL" H 4600 4426 50  0000 C CNN
 F 2 "alexios:SOJ-36_10.16x23.49mm_P1.27mm" V 4500 3375 50  0001 C CNN
@@
 AR Path="/5ECDEC6E/5EAD7016" Ref="U25"  Part="2"
 AR Path="/5ECDEC7E/5EAD7016" Ref="U27"  Part="2"
-F 0 "U5" H 4575 5917 50  0000 C CNN
+F 0 "U27" H 4575 5917 50  0000 C CNN
 F 1 "IS61C5128AL" H 4575 5826 50  0000 C CNN
 F 2 "alexios:SOJ-36_10.16x23.49mm_P1.27mm" V 4500 5675 50  0001 C CNN
@@
 AR Path="/5ECDEC6E/5EAD85F7" Ref="U26"  Part="2"
 AR Path="/5ECDEC7E/5EAD85F7" Ref="U28"  Part="2"
-F 0 "U6" H 6475 5917 50  0000 C CNN
+F 0 "U28" H 6475 5917 50  0000 C CNN
 F 1 "IS61C5128AL" H 6475 5826 50  0000 C CNN
 F 2 "alexios:SOJ-36_10.16x23.49mm_P1.27mm" V 6400 5675 50  0001 C CNN
@@
 AR Path="/5ECDEC6E/5EADE4AF" Ref="#PWR090"  Part="1"
 AR Path="/5ECDEC7E/5EADE4AF" Ref="#PWR098"  Part="1"
-F 0 "#PWR010" H 4150 5200 50  0001 C CNN
+F 0 "#PWR098" H 4150 5200 50  0001 C CNN
 F 1 "+5V" H 4165 5523 50  0000 C CNN
 F 2 "" H 4150 5350 50  0001 C CNN
@@
 AR Path="/5ECDEC6E/5EADE72D" Ref="#PWR092"  Part="1"
 AR Path="/5ECDEC7E/5EADE72D" Ref="#PWR0100"  Part="1"
-F 0 "#PWR012" H 5000 5200 50  0001 C CNN
+F 0 "#PWR0100" H 5000 5200 50  0001 C CNN
 F 1 "+5V" H 5015 5523 50  0000 C CNN
 F 2 "" H 5000 5350 50  0001 C CNN
@@
 AR Path="/5ECDEC6E/5EADE7CB" Ref="#PWR094"  Part="1"
 AR Path="/5ECDEC7E/5EADE7CB" Ref="#PWR0102"  Part="1"
-F 0 "#PWR014" H 6050 5200 50  0001 C CNN
+F 0 "#PWR0102" H 6050 5200 50  0001 C CNN
 F 1 "+5V" H 6065 5523 50  0000 C CNN
 F 2 "" H 6050 5350 50  0001 C CNN
@@
 AR Path="/5ECDEC6E/5EADE963" Ref="#PWR096"  Part="1"
 AR Path="/5ECDEC7E/5EADE963" Ref="#PWR0104"  Part="1"
-F 0 "#PWR016" H 6900 5200 50  0001 C CNN
+F 0 "#PWR0104" H 6900 5200 50  0001 C CNN
 F 1 "+5V" H 6915 5523 50  0000 C CNN
 F 2 "" H 6900 5350 50  0001 C CNN
@@
 AR Path="/5ECDEC6E/5EADEDDC" Ref="#PWR097"  Part="1"
 AR Path="/5ECDEC7E/5EADEDDC" Ref="#PWR0105"  Part="1"
-F 0 "#PWR017" H 6900 5300 50  0001 C CNN
+F 0 "#PWR0105" H 6900 5300 50  0001 C CNN
 F 1 "GND" H 6905 5377 50  0000 C CNN
 F 2 "" H 6900 5550 50  0001 C CNN
@@
 AR Path="/5ECDEC6E/5EADF1C4" Ref="#PWR095"  Part="1"
 AR Path="/5ECDEC7E/5EADF1C4" Ref="#PWR0103"  Part="1"
-F 0 "#PWR015" H 6050 5300 50  0001 C CNN
+F 0 "#PWR0103" H 6050 5300 50  0001 C CNN
 F 1 "GND" H 6055 5377 50  0000 C CNN
 F 2 "" H 6050 5550 50  0001 C CNN
@@
 AR Path="/5ECDEC6E/5EADF5B8" Ref="#PWR091"  Part="1"
 AR Path="/5ECDEC7E/5EADF5B8" Ref="#PWR099"  Part="1"
-F 0 "#PWR011" H 4150 5300 50  0001 C CNN
+F 0 "#PWR099" H 4150 5300 50  0001 C CNN
 F 1 "GND" H 4155 5377 50  0000 C CNN
 F 2 "" H 4150 5550 50  0001 C CNN
@@
 AR Path="/5ECDEC6E/5EADFE90" Ref="#PWR093"  Part="1"
 AR Path="/5ECDEC7E/5EADFE90" Ref="#PWR0101"  Part="1"
-F 0 "#PWR013" H 5000 5300 50  0001 C CNN
+F 0 "#PWR0101" H 5000 5300 50  0001 C CNN
 F 1 "GND" H 5005 5377 50  0000 C CNN
 F 2 "" H 5000 5550 50  0001 C CNN
@@
 AR Path="/5ECDEC6E/5EAE1505" Ref="C43"  Part="1"
 AR Path="/5ECDEC7E/5EAE1505" Ref="C47"  Part="1"
-F 0 "C3" H 4059 5496 50  0000 R CNN
+F 0 "C47" H 4059 5496 50  0000 R CNN
 F 1 "100nF" H 4059 5405 50  0000 R CNN
 F 2 "alexios:SMD_0805_2012Metric_Pad1.15x1.40mm_HandSolder" H 4150 5450 50  0001 C CNN
@@
 AR Path="/5ECDEC6E/5EAE33D6" Ref="C44"  Part="1"
 AR Path="/5ECDEC7E/5EAE33D6" Ref="C48"  Part="1"
-F 0 "C4" H 5092 5496 50  0000 L CNN
+F 0 "C48" H 5092 5496 50  0000 L CNN
 F 1 "100nF" H 5092 5405 50  0000 L CNN
 F 2 "alexios:SMD_0805_2012Metric_Pad1.15x1.40mm_HandSolder" H 5000 5450 50  0001 C CNN
@@
 AR Path="/5ECDEC6E/5EAE3E26" Ref="C46"  Part="1"
 AR Path="/5ECDEC7E/5EAE3E26" Ref="C50"  Part="1"
-F 0 "C6" H 6992 5496 50  0000 L CNN
+F 0 "C50" H 6992 5496 50  0000 L CNN
 F 1 "100nF" H 6992 5405 50  0000 L CNN
 F 2 "alexios:SMD_0805_2012Metric_Pad1.15x1.40mm_HandSolder" H 6900 5450 50  0001 C CNN
@@
 AR Path="/5ECDEC6E/5EAE37CE" Ref="C45"  Part="1"
 AR Path="/5ECDEC7E/5EAE37CE" Ref="C49"  Part="1"
-F 0 "C5" H 5959 5496 50  0000 R CNN
+F 0 "C49" H 5959 5496 50  0000 R CNN
 F 1 "100nF" H 5959 5405 50  0000 R CNN
 F 2 "alexios:SMD_0805_2012Metric_Pad1.15x1.40mm_HandSolder" H 6050 5450 50  0001 C CNN

Commit message: Fine tuned board, fixed issues, ready for plotting.
Other:
- note added: "16×512kbit SRAM Bank"
Changed lines of the file:
@@
 $Descr A4 11693 8268
 encoding utf-8
-Sheet 10 14
+Sheet 8 14
 Title ""
 Date ""
@@
 AR Path="/5ECDEC6E/5EACCD3C" Ref="U26"  Part="1"
 AR Path="/5ECDEC7E/5EACCD3C" Ref="U28"  Part="1"
-F 0 "U28" H 6500 4517 50  0000 C CNN
+F 0 "U18" H 6500 4517 50  0000 C CNN
 F 1 "IS61C5128AL" H 6500 4426 50  0000 C CNN
 F 2 "alexios:SOJ-36_10.16x23.49mm_P1.27mm" V 6400 3375 50  0001 C CNN
@@
 AR Path="/5ECDEC6E/5EACCD43" Ref="U25"  Part="1"
 AR Path="/5ECDEC7E/5EACCD43" Ref="U27"  Part="1"
-F 0 "U27" H 4600 4517 50  0000 C CNN
+F 0 "U17" H 4600 4517 50  0000 C CNN
 F 1 "IS61C5128AL" H 4600 4426 50  0000 C CNN
 F 2 "alexios:SOJ-36_10.16x23.49mm_P1.27mm" V 4500 3375 50  0001 C CNN
@@
 AR Path="/5ECDEC6E/5EAD7016" Ref="U25"  Part="2"
 AR Path="/5ECDEC7E/5EAD7016" Ref="U27"  Part="2"
-F 0 "U27" H 4575 5917 50  0000 C CNN
+F 0 "U17" H 4575 5917 50  0000 C CNN
 F 1 "IS61C5128AL" H 4575 5826 50  0000 C CNN
 F 2 "alexios:SOJ-36_10.16x23.49mm_P1.27mm" V 4500 5675 50  0001 C CNN
@@
 AR Path="/5ECDEC6E/5EAD85F7" Ref="U26"  Part="2"
 AR Path="/5ECDEC7E/5EAD85F7" Ref="U28"  Part="2"
-F 0 "U28" H 6475 5917 50  0000 C CNN
+F 0 "U18" H 6475 5917 50  0000 C CNN
 F 1 "IS61C5128AL" H 6475 5826 50  0000 C CNN
 F 2 "alexios:SOJ-36_10.16x23.49mm_P1.27mm" V 6400 5675 50  0001 C CNN
@@
 AR Path="/5ECDEC6E/5EAE1505" Ref="C43"  Part="1"
 AR Path="/5ECDEC7E/5EAE1505" Ref="C47"  Part="1"
-F 0 "C47" H 4059 5496 50  0000 R CNN
+F 0 "C27" H 4059 5496 50  0000 R CNN
 F 1 "100nF" H 4059 5405 50  0000 R CNN
 F 2 "alexios:SMD_0805_2012Metric_Pad1.15x1.40mm_HandSolder" H 4150 5450 50  0001 C CNN
@@
 AR Path="/5ECDEC6E/5EAE33D6" Ref="C44"  Part="1"
 AR Path="/5ECDEC7E/5EAE33D6" Ref="C48"  Part="1"
-F 0 "C48" H 5092 5496 50  0000 L CNN
+F 0 "C28" H 5092 5496 50  0000 L CNN
 F 1 "100nF" H 5092 5405 50  0000 L CNN
 F 2 "alexios:SMD_0805_2012Metric_Pad1.15x1.40mm_HandSolder" H 5000 5450 50  0001 C CNN
@@
 AR Path="/5ECDEC6E/5EAE3E26" Ref="C46"  Part="1"
 AR Path="/5ECDEC7E/5EAE3E26" Ref="C50"  Part="1"
-F 0 "C50" H 6992 5496 50  0000 L CNN
+F 0 "C30" H 6992 5496 50  0000 L CNN
 F 1 "100nF" H 6992 5405 50  0000 L CNN
 F 2 "alexios:SMD_0805_2012Metric_Pad1.15x1.40mm_HandSolder" H 6900 5450 50  0001 C CNN
@@
 AR Path="/5ECDEC6E/5EAE37CE" Ref="C45"  Part="1"
 AR Path="/5ECDEC7E/5EAE37CE" Ref="C49"  Part="1"
-F 0 "C49" H 5959 5496 50  0000 R CNN
+F 0 "C29" H 5959 5496 50  0000 R CNN
 F 1 "100nF" H 5959 5405 50  0000 R CNN
 F 2 "alexios:SMD_0805_2012Metric_Pad1.15x1.40mm_HandSolder" H 6050 5450 50  0001 C CNN
@@
 	1    0    0    -1
 $EndComp
+Text Notes 7100 7000 0    198  ~ 40
+16×512kbit SRAM Bank
 Wire Bus Line
 	7300 2150 7300 4500

Commit message: Updating schematics with new page layout.
Other:
- note removed: "16×512kbit SRAM Bank"
Changed lines of the file:
@@
 EESchema Schematic File Version 4
 LIBS:mem-cache
-EELAYER 30 0
+EELAYER 26 0
 EELAYER END
 $Descr A4 11693 8268
 encoding utf-8
-Sheet 8 14
-Title ""
+Sheet 2 14
+Title "16×512kbit SRAM Bank"
 Date ""
-Rev ""
+Rev "1945"
 Comp ""
-Comment1 ""
+Comment1 "MEM"
 Comment2 ""
 Comment3 ""
@@
 AR Path="/5ECDEC6E/5EACCD3C" Ref="U26"  Part="1"
 AR Path="/5ECDEC7E/5EACCD3C" Ref="U28"  Part="1"
-F 0 "U18" H 6500 4517 50  0000 C CNN
+F 0 "U6" H 6500 4517 50  0000 C CNN
 F 1 "IS61C5128AL" H 6500 4426 50  0000 C CNN
 F 2 "alexios:SOJ-36_10.16x23.49mm_P1.27mm" V 6400 3375 50  0001 C CNN
@@
 AR Path="/5ECDEC6E/5EACCD43" Ref="U25"  Part="1"
 AR Path="/5ECDEC7E/5EACCD43" Ref="U27"  Part="1"
-F 0 "U17" H 4600 4517 50  0000 C CNN
+F 0 "U5" H 4600 4517 50  0000 C CNN
 F 1 "IS61C5128AL" H 4600 4426 50  0000 C CNN
 F 2 "alexios:SOJ-36_10.16x23.49mm_P1.27mm" V 4500 3375 50  0001 C CNN
@@
 AR Path="/5ECDEC6E/5EAD7016" Ref="U25"  Part="2"
 AR Path="/5ECDEC7E/5EAD7016" Ref="U27"  Part="2"
-F 0 "U17" H 4575 5917 50  0000 C CNN
+F 0 "U5" H 4575 5917 50  0000 C CNN
 F 1 "IS61C5128AL" H 4575 5826 50  0000 C CNN
 F 2 "alexios:SOJ-36_10.16x23.49mm_P1.27mm" V 4500 5675 50  0001 C CNN
@@
 AR Path="/5ECDEC6E/5EAD85F7" Ref="U26"  Part="2"
 AR Path="/5ECDEC7E/5EAD85F7" Ref="U28"  Part="2"
-F 0 "U18" H 6475 5917 50  0000 C CNN
+F 0 "U6" H 6475 5917 50  0000 C CNN
 F 1 "IS61C5128AL" H 6475 5826 50  0000 C CNN
 F 2 "alexios:SOJ-36_10.16x23.49mm_P1.27mm" V 6400 5675 50  0001 C CNN
@@
 AR Path="/5ECDEC6E/5EADE4AF" Ref="#PWR090"  Part="1"
 AR Path="/5ECDEC7E/5EADE4AF" Ref="#PWR098"  Part="1"
-F 0 "#PWR098" H 4150 5200 50  0001 C CNN
+F 0 "#PWR010" H 4150 5200 50  0001 C CNN
 F 1 "+5V" H 4165 5523 50  0000 C CNN
 F 2 "" H 4150 5350 50  0001 C CNN
@@
 AR Path="/5ECDEC6E/5EADE72D" Ref="#PWR092"  Part="1"
 AR Path="/5ECDEC7E/5EADE72D" Ref="#PWR0100"  Part="1"
-F 0 "#PWR0100" H 5000 5200 50  0001 C CNN
+F 0 "#PWR012" H 5000 5200 50  0001 C CNN
 F 1 "+5V" H 5015 5523 50  0000 C CNN
 F 2 "" H 5000 5350 50  0001 C CNN
@@
 AR Path="/5ECDEC6E/5EADE7CB" Ref="#PWR094"  Part="1"
 AR Path="/5ECDEC7E/5EADE7CB" Ref="#PWR0102"  Part="1"
-F 0 "#PWR0102" H 6050 5200 50  0001 C CNN
+F 0 "#PWR014" H 6050 5200 50  0001 C CNN
 F 1 "+5V" H 6065 5523 50  0000 C CNN
 F 2 "" H 6050 5350 50  0001 C CNN
@@
 AR Path="/5ECDEC6E/5EADE963" Ref="#PWR096"  Part="1"
 AR Path="/5ECDEC7E/5EADE963" Ref="#PWR0104"  Part="1"
-F 0 "#PWR0104" H 6900 5200 50  0001 C CNN
+F 0 "#PWR016" H 6900 5200 50  0001 C CNN
 F 1 "+5V" H 6915 5523 50  0000 C CNN
 F 2 "" H 6900 5350 50  0001 C CNN
@@
 AR Path="/5ECDEC6E/5EADEDDC" Ref="#PWR097"  Part="1"
 AR Path="/5ECDEC7E/5EADEDDC" Ref="#PWR0105"  Part="1"
-F 0 "#PWR0105" H 6900 5300 50  0001 C CNN
+F 0 "#PWR017" H 6900 5300 50  0001 C CNN
 F 1 "GND" H 6905 5377 50  0000 C CNN
 F 2 "" H 6900 5550 50  0001 C CNN
@@
 AR Path="/5ECDEC6E/5EADF1C4" Ref="#PWR095"  Part="1"
 AR Path="/5ECDEC7E/5EADF1C4" Ref="#PWR0103"  Part="1"
-F 0 "#PWR0103" H 6050 5300 50  0001 C CNN
+F 0 "#PWR015" H 6050 5300 50  0001 C CNN
 F 1 "GND" H 6055 5377 50  0000 C CNN
 F 2 "" H 6050 5550 50  0001 C CNN
@@
 AR Path="/5ECDEC6E/5EADF5B8" Ref="#PWR091"  Part="1"
 AR Path="/5ECDEC7E/5EADF5B8" Ref="#PWR099"  Part="1"
-F 0 "#PWR099" H 4150 5300 50  0001 C CNN
+F 0 "#PWR011" H 4150 5300 50  0001 C CNN
 F 1 "GND" H 4155 5377 50  0000 C CNN
 F 2 "" H 4150 5550 50  0001 C CNN
@@
 AR Path="/5ECDEC6E/5EADFE90" Ref="#PWR093"  Part="1"
 AR Path="/5ECDEC7E/5EADFE90" Ref="#PWR0101"  Part="1"
-F 0 "#PWR0101" H 5000 5300 50  0001 C CNN
+F 0 "#PWR013" H 5000 5300 50  0001 C CNN
 F 1 "GND" H 5005 5377 50  0000 C CNN
 F 2 "" H 5000 5550 50  0001 C CNN
@@
 AR Path="/5ECDEC6E/5EAE1505" Ref="C43"  Part="1"
 AR Path="/5ECDEC7E/5EAE1505" Ref="C47"  Part="1"
-F 0 "C27" H 4059 5496 50  0000 R CNN
+F 0 "C3" H 4059 5496 50  0000 R CNN
 F 1 "100nF" H 4059 5405 50  0000 R CNN
 F 2 "alexios:SMD_0805_2012Metric_Pad1.15x1.40mm_HandSolder" H 4150 5450 50  0001 C CNN
@@
 AR Path="/5ECDEC6E/5EAE33D6" Ref="C44"  Part="1"
 AR Path="/5ECDEC7E/5EAE33D6" Ref="C48"  Part="1"
-F 0 "C28" H 5092 5496 50  0000 L CNN
+F 0 "C4" H 5092 5496 50  0000 L CNN
 F 1 "100nF" H 5092 5405 50  0000 L CNN
 F 2 "alexios:SMD_0805_2012Metric_Pad1.15x1.40mm_HandSolder" H 5000 5450 50  0001 C CNN
@@
 AR Path="/5ECDEC6E/5EAE3E26" Ref="C46"  Part="1"
 AR Path="/5ECDEC7E/5EAE3E26" Ref="C50"  Part="1"
-F 0 "C30" H 6992 5496 50  0000 L CNN
+F 0 "C6" H 6992 5496 50  0000 L CNN
 F 1 "100nF" H 6992 5405 50  0000 L CNN
 F 2 "alexios:SMD_0805_2012Metric_Pad1.15x1.40mm_HandSolder" H 6900 5450 50  0001 C CNN
@@
 AR Path="/5ECDEC6E/5EAE37CE" Ref="C45"  Part="1"
 AR Path="/5ECDEC7E/5EAE37CE" Ref="C49"  Part="1"
-F 0 "C29" H 5959 5496 50  0000 R CNN
+F 0 "C5" H 5959 5496 50  0000 R CNN
 F 1 "100nF" H 5959 5405 50  0000 R CNN
 F 2 "alexios:SMD_0805_2012Metric_Pad1.15x1.40mm_HandSolder" H 6050 5450 50  0001 C CNN
@@
 	1    0    0    -1
 $EndComp
-Text Notes 7100 7000 0    198  ~ 40
-16×512kbit SRAM Bank
 Wire Bus Line
 	7300 2150 7300 4500
