File: kicad/cft/cft_microcode.sch (KiCad schematic (older format))
At the start: 20 parts, among them U1403 74AHC1G08, U1701 74AHC1G08, U1702 74HC161, U1703 74AHC1G00, U1901 SN74ACT1073, U1902 SN74ACT1073, U1903 SN74ACT1071

Commit message: Renamed FPO to FPD. Moved IN-RSVD to microcode sheet. Removed bus hold circuitry from signals already terminated by the DFP.
Parts:
- removed C1901, C1903: 10µF, Capacitor_SMD:C_0805_2012Metric, symbol Device:C_Small
- removed C1902: 100nF, Capacitor_SMD:C_0805_2012Metric, symbol Device:C_Small
- removed U1901, U1902: SN74ACT1073, symbol alexios:SN74ACT1073
- added R?: 4.7kΩ, Resistor_SMD:R_0805_2012Metric, symbol Device:R_Small
- added unit 2 of U1903
Connections:
- net +5V: now also U1903.10 (VCC), U1903.11 (VCC)
- net ACTION1: no longer U1903.1 (D1)
- net ACTION2: no longer U1903.2 (D2)
- net ACTION3: no longer U1903.5 (D3)
- net COND0: now also U1903.1 (D1)
- net COND1: now also U1903.2 (D2)
- net COND2: now also U1903.5 (D3)
- net COND3: now also U1903.6 (D4)
- net COND4: now also U1903.7 (D5)
- net GND: now also R?.1, U1903.3 (GND), U1903.4 (GND); no longer U1903.13 (D9), U1903.14 (D10)
- net IN-RSVD: now also R?.2
- net ~END: now also U1903.8 (D6); no longer U1903.12 (D8)
- net ~IO: no longer U1903.7 (D5)
- net ~MEM: no longer U1903.6 (D4)
- net ~R: no longer U1903.8 (D6)
- net ~WEN: no longer U1903.9 (D7)
- no-connect marks 3 -> 7
Other:
- note added: "~µCE~ enables microcode unit decoders\nunless the processor is resetting or halted.\n\nTODO: ~HALT~ may not be required here!\nWe need decoders to work during HALT\nif the DFP needs them."
- note removed: "~µCE~ enables microcode unit decoders unless\nthe processor is resetting or halted."
- moved on the sheet: C1904, U1903A

Commit message: Added uSE#, fine tuning of schematic.
Parts:
- removed R1701: 30Ω, Resistor_SMD:R_0805_2012Metric, symbol Device:R_Small
- removed unit 1 of U1703
- added C?: 100nF, Capacitor_SMD:C_0805_2012Metric, symbol Device:C_Small
- added R? (x2): 4.7kΩ, Resistor_SMD:R_0805_2012Metric, symbol Device:R_Small
- added U? (x2): 74LVC1G00, symbol alexios:74LVC1G00
Connections:
- net +5V: now also C?.1, R?.2, R?.2, U?.5 (VCC)
- net GND: now also C?.2, U?.3 (GND)
- net ~ENDEXT: now also R?.1
- net ~HALT: now also R?.1, U?.1
- net ~RESET: now also U?.2
- new net ~µSE: U?.4
Other:
- note added: "(pulled up by the Wait State Handler circuitry)"
- note added: "High = Fetch.\nLow = Execute.\nThis is for the benefit of the front panel only."
- note added: "Note: The DFP adds bus hold\nto all other outputs."
- note added: "The Microcode Store is enabled\nwhen ~RESET~ and ~HALT~\nare both deasserted."
- note removed: "High = fetch. Low = Execute.\nThis is for the benefit of the front panel only."
- note removed: "~µCE~ enables microcode unit decoders\nunless the processor is resetting or halted.\n\nTODO: ~HALT~ may not be required here!\nWe need decoders to work during HALT\nif the DFP needs them."
- moved on the sheet: C1702, C1904, RN?, SW?, U1703B, U1903B, U?A

Commit message: Renamed some signals
Changed lines of the file:
@@
 IR15
 Text HLabel 950  4650 0    50   Input ~ 0
-~IRQSUC
+~IRQSµC
 Text HLabel 950  4750 0    50   Input ~ 0
 ~RSTHOLD
@@
 	950  4750 1900 4750
 Text Label 1900 4650 2    50   ~ 0
-~IRQSUC
+~IRQSµC
 Text Label 1900 4750 2    50   ~ 0
 ~RSTHOLD
@@
 F48 "IR14" I L 5450 4800 50
 F49 "IR15" I L 5450 4900 50
-F50 "~IRQSUC" I L 5450 5000 50
+F50 "~IRQSµC" I L 5450 5000 50
 F51 "~RSTHOLD" I L 5450 5100 50
 $EndSheet
@@
 UPC3
 Text Label 5050 5000 0    50   ~ 0
-~IRQSUC
+~IRQSµC
 Text Label 5050 5100 0    50   ~ 0
 ~RSTHOLD
@@
 F17 "IR14" I L 2950 4800 50
 F18 "IR15" I L 2950 4900 50
-F19 "~IRQSUC" I L 2950 5000 50
+F19 "~IRQSµC" I L 2950 5000 50
 F20 "~RSTHOLD" I L 2950 5100 50
 F21 "RADDR0" O R 4100 3300 50
@@
 UPC3
 Text Label 2550 5000 0    50   ~ 0
-~IRQSUC
+~IRQSµC
 Text Label 2550 5100 0    50   ~ 0
 ~RSTHOLD

Commit message: Moved things around a bit
Parts:
- gave numbers to parts that had none: 9
- renumbered C1701 to C3101, C1703 to C3102, C1702 to C3103, C1904 to C3106, U1403 to U3002, U1702 to U3101, U1701 to U3103, U1703 to U3104, U1903 to U3106

Commit message: Removed widebus buffer from microcode store µAddr High
Parts:
- renumbered C3101 to C1701, C3103 to C1702, C3102 to C1703, C3106 to C1904, C3104 to C?, C3105 to C?, R3103 to R?, R3101 to R?, R3102 to R?, RN3101 to RN?, SW3101 to SW?, U3002 to U1403, U3103 to U1701, U3101 to U1702, U3104 to U1703, U3106 to U1903, U3102 to U?, U3105 to U?
