File: kicad/cft/alu.sch (KiCad schematic (older format))
At the start: 8 parts, among them U2209 74LVC1G08, U2601 74HC138, U2602 74HC138, U2603 74LVC1G08, U2604 74LVC2G157, U2605 74LVC1G08

Commit message: Moved things around a bit
Parts:
- renumbered C2601 to C1601, C2602 to C1602, U2601 to U1601, U2209 to U1602, U2602 to U1603, U2603 to U1604, U2604 to U1605, U2605 to U1606
Changed lines of the file:
@@
 EESchema Schematic File Version 4
 LIBS:cft-cache
-EELAYER 26 0
+EELAYER 30 0
 EELAYER END
 $Descr A4 11693 8268
@@
 B[0..15]
 $Comp
-L alexios:74HC138 U2601
+L alexios:74HC138 U1601
 U 1 1 5CFB457F
 P 2850 3150
-F 0 "U2601" H 2850 3817 50  0000 C CNN
+F 0 "U1601" H 2850 3817 50  0000 C CNN
 F 1 "74HC138" H 2850 3726 50  0000 C CNN
 F 2 "" H 2850 3150 50  0001 C CNN
@@
 	2400 1500 2600 1500
 $Comp
-L alexios:74LVC1G08 U2209
+L alexios:74LVC1G08 U1602
 U 2 1 5D2E632C
 P 2800 7250
-F 0 "U2209" H 2880 7196 50  0000 L CNN
+F 0 "U1602" H 2880 7196 50  0000 L CNN
 F 1 "74LVC1G08" H 2880 7105 50  0000 L CNN
 F 2 "" H 2450 7250 50  0001 C CNN
@@
 $EndComp
 $Comp
-L alexios:74HC138 U2601
+L alexios:74HC138 U1601
 U 2 1 5D2E73E6
 P 1400 7350
-F 0 "U2601" H 1580 7396 50  0000 L CNN
+F 0 "U1601" H 1580 7396 50  0000 L CNN
 F 1 "74HC138" H 1580 7305 50  0000 L CNN
 F 2 "" H 1400 7350 50  0001 C CNN
@@
 AR Path="/5DC89E19/5CF23BD4/5D31C83B" Ref="C?"  Part="1"
 AR Path="/5DC89E19/5CF5A95E/5D31C83B" Ref="C?"  Part="1"
-AR Path="/5DC89E19/5D31C83B" Ref="C2601"  Part="1"
-F 0 "C2601" H 959 7396 50  0000 R CNN
+AR Path="/5DC89E19/5D31C83B" Ref="C1601"  Part="1"
+F 0 "C1601" H 959 7396 50  0000 R CNN
 F 1 "100nF" H 959 7305 50  0000 R CNN
 F 2 "Capacitor_SMD:C_0805_2012Metric" H 1050 7350 50  0001 C CNN
@@
 AR Path="/5DC89E19/5CF23BD4/5D31C841" Ref="#PWR?"  Part="1"
 AR Path="/5DC89E19/5CF5A95E/5D31C841" Ref="#PWR?"  Part="1"
-AR Path="/5DC89E19/5D31C841" Ref="#PWR02602"  Part="1"
-F 0 "#PWR02602" H 1050 7200 50  0001 C CNN
+AR Path="/5DC89E19/5D31C841" Ref="#PWR01602"  Part="1"
+F 0 "#PWR01602" H 1050 7200 50  0001 C CNN
 F 1 "GND" H 1055 7277 50  0000 C CNN
 F 2 "" H 1050 7450 50  0001 C CNN
@@
 AR Path="/5DC89E19/5CF23BD4/5D31C848" Ref="#PWR?"  Part="1"
 AR Path="/5DC89E19/5CF5A95E/5D31C848" Ref="#PWR?"  Part="1"
-AR Path="/5DC89E19/5D31C848" Ref="#PWR02601"  Part="1"
-F 0 "#PWR02601" H 1050 7100 50  0001 C CNN
+AR Path="/5DC89E19/5D31C848" Ref="#PWR01601"  Part="1"
+F 0 "#PWR01601" H 1050 7100 50  0001 C CNN
 F 1 "+5V" H 1065 7423 50  0000 C CNN
 F 2 "" H 1050 7250 50  0001 C CNN
@@
 AR Path="/5DC89E19/5CF23BD4/5D31D8AA" Ref="C?"  Part="1"
 AR Path="/5DC89E19/5CF5A95E/5D31D8AA" Ref="C?"  Part="1"
-AR Path="/5DC89E19/5D31D8AA" Ref="C2602"  Part="1"
-F 0 "C2602" H 2259 7396 50  0000 R CNN
+AR Path="/5DC89E19/5D31D8AA" Ref="C1602"  Part="1"
+F 0 "C1602" H 2259 7396 50  0000 R CNN
 F 1 "100nF" H 2259 7305 50  0000 R CNN
 F 2 "Capacitor_SMD:C_0805_2012Metric" H 2350 7350 50  0001 C CNN
@@
 AR Path="/5DC89E19/5CF23BD4/5D31D8B0" Ref="#PWR?"  Part="1"
 AR Path="/5DC89E19/5CF5A95E/5D31D8B0" Ref="#PWR?"  Part="1"
-AR Path="/5DC89E19/5D31D8B0" Ref="#PWR02604"  Part="1"
-F 0 "#PWR02604" H 2350 7200 50  0001 C CNN
+AR Path="/5DC89E19/5D31D8B0" Ref="#PWR01604"  Part="1"
+F 0 "#PWR01604" H 2350 7200 50  0001 C CNN
 F 1 "GND" H 2355 7277 50  0000 C CNN
 F 2 "" H 2350 7450 50  0001 C CNN
@@
 AR Path="/5DC89E19/5CF23BD4/5D31D8B6" Ref="#PWR?"  Part="1"
 AR Path="/5DC89E19/5CF5A95E/5D31D8B6" Ref="#PWR?"  Part="1"
-AR Path="/5DC89E19/5D31D8B6" Ref="#PWR02603"  Part="1"
-F 0 "#PWR02603" H 2350 7100 50  0001 C CNN
+AR Path="/5DC89E19/5D31D8B6" Ref="#PWR01603"  Part="1"
+F 0 "#PWR01603" H 2350 7100 50  0001 C CNN
 F 1 "+5V" H 2365 7423 50  0000 C CNN
 F 2 "" H 2350 7250 50  0001 C CNN
@@
 	4650 5050 4650 2250
 $Comp
-L alexios:74LVC1G08 U2603
+L alexios:74LVC1G08 U1604
 U 1 1 5D2D7C39
 P 3050 2300
-F 0 "U2603" H 2975 2033 50  0000 C CNN
+F 0 "U1604" H 2975 2033 50  0000 C CNN
 F 1 "74LVC1G08" H 2975 2124 50  0000 C CNN
 F 2 "" H 2700 2300 50  0001 C CNN
@@
 ~RESET
 $Comp
-L alexios:74LVC2G157 U2604
+L alexios:74LVC2G157 U1605
 U 1 1 5D8C718E
 P 8950 5700
-F 0 "U2604" H 8950 6067 50  0000 C CNN
+F 0 "U1605" H 8950 6067 50  0000 C CNN
 F 1 "74LVC2G157" H 8950 5976 50  0000 C CNN
 F 2 "" H 8850 5825 50  0001 C CNN
@@
 	6850 5700 8600 5700
 $Comp
-L power:GND #PWR02605
+L power:GND #PWR01605
 U 1 1 5D8FFD85
 P 8600 5900
-F 0 "#PWR02605" H 8600 5650 50  0001 C CNN
+F 0 "#PWR01605" H 8600 5650 50  0001 C CNN
 F 1 "GND" H 8605 5727 50  0000 C CNN
 F 2 "" H 8600 5900 50  0001 C CNN
@@
 	8600 5800 7900 5800
 $Comp
-L alexios:74LVC1G08 U2605
+L alexios:74LVC1G08 U1606
 U 1 1 5D94DBE2
 P 9050 5100
-F 0 "U2605" H 8975 5367 50  0000 C CNN
+F 0 "U1606" H 8975 5367 50  0000 C CNN
 F 1 "74LVC1G08" H 8975 5276 50  0000 C CNN
 F 2 "" H 8700 5100 50  0001 C CNN
@@
 SRU
 $Comp
-L alexios:74HC138 U2602
+L alexios:74HC138 U1603
 U 1 1 5DA9723E
 P 2850 4550
-F 0 "U2602" H 2850 5217 50  0000 C CNN
+F 0 "U1603" H 2850 5217 50  0000 C CNN
 F 1 "74HC138" H 2850 5126 50  0000 C CNN
 F 2 "" H 2850 4550 50  0001 C CNN

Commit message: Removed widebus buffer from microcode store µAddr High
Parts:
- added U? (x8): 74HC253, symbol alexios:74HC253
- added U?: 74LVC1G08, symbol alexios:74LVC1G08
- added U?: 74LVC1G32, symbol alexios:74LVC1G32
- added U?: 74LVC1G86, symbol alexios:74LVC1G86
- added U?: 74LVC1G04, symbol alexios:74LVC1G04
- renumbered C1601 to C2601, C1602 to C2602, U1602 to U2209, U1601 to U2601, U1603 to U2602, U1604 to U2603, U1605 to U2604, U1606 to U2605
Connections:
- net WADDR0: now also U?.1, U?.1, U?.1, U?.2
- net WADDR1: now also U?.2, U?.2, U?.2
- new net CFG0: U?.10 (2C0), U?.4, U?.6 (1C0)
- new net CFG1: U?.11 (2C1), U?.4, U?.5 (1C1)
- new net CFG2: U?.12 (2C2), U?.4, U?.4 (1C2)
- new net CFG3: U?.13 (2C3), U?.3 (1C3), U?.4

Commit message: Fine tuning of schematics.
Parts:
- removed U? (x8): 74HC253, symbol alexios:74HC253
- removed U?: 74LVC1G08, symbol alexios:74LVC1G08
- removed U?: 74LVC1G32, symbol alexios:74LVC1G32
- removed U?: 74LVC1G86, symbol alexios:74LVC1G86
- removed U?: 74LVC1G04, symbol alexios:74LVC1G04
Changed lines of the file:
@@
 $Descr A4 11693 8268
 encoding utf-8
-Sheet 16 34
+Sheet 14 34
 Title ""
 Date ""
@@
 Text Notes 8300 1150 0    100  ~ 20
 Redo these!
-$Comp
-L alexios:74HC253 U?
-U 1 1 5DF86F64
-P 16800 2550
-F 0 "U?" H 16800 3517 50  0000 C CNN
-F 1 "74HC253" H 16800 3426 50  0000 C CNN
-F 2 "" H 17100 3150 50  0001 C CNN
-F 3 "https://assets.nexperia.com/documents/data-sheet/74HC_HCT253.pdf" H 17100 3150 50  0001 C CNN
-	1    16800 2550
-	1    0    0    -1
-$EndComp
-$Comp
-L alexios:74HC253 U?
-U 1 1 5DF86FFA
-P 16800 4600
-F 0 "U?" H 16800 5567 50  0000 C CNN
-F 1 "74HC253" H 16800 5476 50  0000 C CNN
-F 2 "" H 17100 5200 50  0001 C CNN
-F 3 "https://assets.nexperia.com/documents/data-sheet/74HC_HCT253.pdf" H 17100 5200 50  0001 C CNN
-	1    16800 4600
-	1    0    0    -1
-$EndComp
-$Comp
-L alexios:74HC253 U?
-U 1 1 5DF87586
-P 18800 2550
-F 0 "U?" H 18800 3517 50  0000 C CNN
-F 1 "74HC253" H 18800 3426 50  0000 C CNN
-F 2 "" H 19100 3150 50  0001 C CNN
-F 3 "https://assets.nexperia.com/documents/data-sheet/74HC_HCT253.pdf" H 19100 3150 50  0001 C CNN
-	1    18800 2550
-	1    0    0    -1
-$EndComp
-$Comp
-L alexios:74HC253 U?
-U 1 1 5DF8758D
-P 18800 4600
-F 0 "U?" H 18800 5567 50  0000 C CNN
-F 1 "74HC253" H 18800 5476 50  0000 C CNN
-F 2 "" H 19100 5200 50  0001 C CNN
-F 3 "https://assets.nexperia.com/documents/data-sheet/74HC_HCT253.pdf" H 19100 5200 50  0001 C CNN
-	1    18800 4600
-	1    0    0    -1
-$EndComp
-$Comp
-L alexios:74HC253 U?
-U 1 1 5DF8A249
-P 20800 2550
-F 0 "U?" H 20800 3517 50  0000 C CNN
-F 1 "74HC253" H 20800 3426 50  0000 C CNN
-F 2 "" H 21100 3150 50  0001 C CNN
-F 3 "https://assets.nexperia.com/documents/data-sheet/74HC_HCT253.pdf" H 21100 3150 50  0001 C CNN
-	1    20800 2550
-	1    0    0    -1
-$EndComp
-$Comp
-L alexios:74HC253 U?
-U 1 1 5DF8A250
-P 20800 4600
-F 0 "U?" H 20800 5567 50  0000 C CNN
-F 1 "74HC253" H 20800 5476 50  0000 C CNN
-F 2 "" H 21100 5200 50  0001 C CNN
-F 3 "https://assets.nexperia.com/documents/data-sheet/74HC_HCT253.pdf" H 21100 5200 50  0001 C CNN
-	1    20800 4600
-	1    0    0    -1
-$EndComp
-$Comp
-L alexios:74HC253 U?
-U 1 1 5DF8CF0E
-P 22800 2550
-F 0 "U?" H 22800 3517 50  0000 C CNN
-F 1 "74HC253" H 22800 3426 50  0000 C CNN
-F 2 "" H 23100 3150 50  0001 C CNN
-F 3 "https://assets.nexperia.com/documents/data-sheet/74HC_HCT253.pdf" H 23100 3150 50  0001 C CNN
-	1    22800 2550
-	1    0    0    -1
-$EndComp
-$Comp
-L alexios:74HC253 U?
-U 1 1 5DF8CF15
-P 22800 4600
-F 0 "U?" H 22800 5567 50  0000 C CNN
-F 1 "74HC253" H 22800 5476 50  0000 C CNN
-F 2 "" H 23100 5200 50  0001 C CNN
-F 3 "https://assets.nexperia.com/documents/data-sheet/74HC_HCT253.pdf" H 23100 5200 50  0001 C CNN
-	1    22800 4600
-	1    0    0    -1
-$EndComp
-Wire Wire Line
-	12700 1850 13300 1850
-Wire Wire Line
-	12700 1950 13200 1950
-Text Label 12700 1850 0    50   ~ 0
-WADDR0
-Text Label 12700 1950 0    50   ~ 0
-WADDR1
-$Comp
-L alexios:74LVC1G08 U?
-U 1 1 5DFEC96B
-P 13700 1900
-F 0 "U?" H 13625 2167 50  0000 C CNN
-F 1 "74LVC1G08" H 13625 2076 50  0000 C CNN
-F 2 "" H 13350 1900 50  0001 C CNN
-F 3 "https://assets.nexperia.com/documents/data-sheet/74LVC1G08.pdf" H 13350 1900 50  0001 C CNN
-	1    13700 1900
-	1    0    0    -1
-$EndComp
-$Comp
-L alexios:74LVC1G32 U?
-U 1 1 5DFEFA2E
-P 13600 2350
-F 0 "U?" H 13650 2617 50  0000 C CNN
-F 1 "74LVC1G32" H 13650 2526 50  0000 C CNN
-F 2 "" H 13710 2330 50  0001 C CNN
-F 3 "http://www.ti.com/lit/sg/scyt129e/scyt129e.pdf" H 13710 2330 50  0001 C CNN
-	1    13600 2350
-	1    0    0    -1
-$EndComp
-$Comp
-L alexios:74LVC1G86 U?
-U 1 1 5DFEFB91
-P 13650 2700
-F 0 "U?" H 13650 2868 50  0000 C CNN
-F 1 "74LVC1G86" H 13650 2777 50  0000 C CNN
-F 2 "" H 13590 3010 50  0001 C CNN
-F 3 "https://assets.nexperia.com/documents/data-sheet/74LVC1G86.pdf" H 13590 3010 50  0001 C CNN
-	1    13650 2700
-	1    0    0    -1
-$EndComp
-$Comp
-L alexios:74LVC1G04 U?
-U 1 1 5DFEFCD3
-P 13700 3300
-F 0 "U?" H 13650 3567 50  0000 C CNN
-F 1 "74LVC1G04" H 13650 3476 50  0000 C CNN
-F 2 "" H 13700 3300 50  0001 C CNN
-F 3 "https://assets.nexperia.com/documents/data-sheet/74LVC1G04.pdf" H 13700 3300 50  0001 C CNN
-	1    13700 3300
-	1    0    0    -1
-$EndComp
-Wire Wire Line
-	13850 1900 14400 1900
-Text Label 14400 1900 2    50   ~ 0
-CFG0
-Wire Wire Line
-	13900 2350 14400 2350
-Text Label 14400 2350 2    50   ~ 0
-CFG1
-Wire Wire Line
-	13900 2800 14400 2800
-Text Label 14400 2800 2    50   ~ 0
-CFG2
-Wire Wire Line
-	13900 3300 14400 3300
-Text Label 14400 3300 2    50   ~ 0
-CFG3
-Wire Wire Line
-	13300 1850 13300 2300
-Wire Wire Line
-	13300 3300 13400 3300
-Connection ~ 13300 1850
-Wire Wire Line
-	13300 1850 13400 1850
-Wire Wire Line
-	13400 2750 13300 2750
-Connection ~ 13300 2750
-Wire Wire Line
-	13300 2750 13300 3300
-Wire Wire Line
-	13400 2300 13300 2300
-Connection ~ 13300 2300
-Wire Wire Line
-	13300 2300 13300 2750
-Wire Wire Line
-	13200 1950 13200 2400
-Wire Wire Line
-	13200 2850 13400 2850
-Connection ~ 13200 1950
-Wire Wire Line
-	13200 1950 13400 1950
-Wire Wire Line
-	13400 2400 13200 2400
-Connection ~ 13200 2400
-Wire Wire Line
-	13200 2400 13200 2850
-Wire Wire Line
-	16300 1850 16000 1850
-Wire Wire Line
-	16300 1950 16000 1950
-Wire Wire Line
-	16300 2050 16000 2050
-Wire Wire Line
-	16300 2150 16000 2150
-Text Label 16050 1850 0    50   ~ 0
-CFG0
-Text Label 16050 1950 0    50   ~ 0
-CFG1
-Text Label 16050 2050 0    50   ~ 0
-CFG2
-Text Label 16050 2150 0    50   ~ 0
-CFG3
-Entry Wire Line
-	15900 1750 16000 1850
-Entry Wire Line
-	15900 1850 16000 1950
-Entry Wire Line
-	15900 1950 16000 2050
-Entry Wire Line
-	15900 2050 16000 2150
-Wire Wire Line
-	16300 2550 16000 2550
-Wire Wire Line
-	16300 2650 16000 2650
-Wire Wire Line
-	16300 2750 16000 2750
-Wire Wire Line
-	16300 2850 16000 2850
-Text Label 16050 2550 0    50   ~ 0
-CFG0
-Text Label 16050 2650 0    50   ~ 0
-CFG1
-Text Label 16050 2750 0    50   ~ 0
-CFG2
-Text Label 16050 2850 0    50   ~ 0
-CFG3
-Entry Wire Line
-	15900 2450 16000 2550
-Entry Wire Line
-	15900 2550 16000 2650
-Entry Wire Line
-	15900 2650 16000 2750
-Entry Wire Line
-	15900 2750 16000 2850
-Wire Wire Line
-	16300 3250 15900 3250
-Wire Wire Line
-	16300 3350 15900 3350
 Wire Bus Line
 	3750 1650 5700 1650

Commit message: Working on ALU.
Parts:
- U2601: value 74HC138 -> 74AC138
Connections:
- net labels added: X0, X1, X2, X3, X4, X5, ~ROMCE
- wire segments 72 -> 80
- no-connect marks 10 -> 15
Other:
- note added: "1X0XX\nX1X00\n----\n11000"
- note added: "Base\n~Y4~\n\nFinal"
- note added: "NOTE: Use 74AC!"
- note added: "WADDR=1x0xx"
- note removed: "WADDR=10xxx"
- moved on the sheet: U2601A, U2602A
