File: kicad/cft/alu_reg.sch (KiCad schematic (older format))
At the start: 18 parts, among them U1519 74HC541, U1520 74HC541, U3301 74HC574, U3302 74HC574, U3303 74HC574, U3304 74HC574, U3305 74HC541, U3306 74HC541

Commit message: Moved things around a bit
Parts:
- renumbered C3301 to C2301, C3302 to C2302, C3303 to C2303, C3304 to C2304, C3305 to C2305, C3306 to C2306, RN3301 to RN2301, RN3302 to RN2302, RN3303 to RN2303, RN3304 to RN2304, U3301 to U2301, U3302 to U2302, U3303 to U2303, U3304 to U2304, U3305 to U2305, U3306 to U2306, U1519 to U2307, U1520 to U2308

Commit message: Removed widebus buffer from microcode store µAddr High
Parts:
- renumbered C2301 to C3301, C2302 to C3302, C2303 to C3303, C2304 to C3304, C2305 to C3305, C2306 to C3306, RN2301 to RN3301, RN2302 to RN3302, RN2303 to RN3303, RN2304 to RN3304, U2307 to U1519, U2308 to U1520, U2301 to U3301, U2302 to U3302, U2303 to U3303, U2304 to U3304, U2305 to U3305, U2306 to U3306
