File: kicad/cft/cpu_microcode_store.sch (KiCad schematic (older format))
At the start: 15 parts, among them U2101 29F040, U2102 29F040, U2103 29F040

Commit message: Renamed µCE# to µSE#.
Connections:
- net ~µCE renamed ~µSE
Changed lines of the file:
@@
 $Descr A4 11693 8268
 encoding utf-8
-Sheet 21 35
+Sheet 33 35
 Title ""
 Date ""
@@
 ~END
 Text HLabel 1150 4800 0    50   Input ~ 0
-~µCE
+~µSE
 Text Label 2250 4800 2    50   ~ 0
-~µCE
+~µSE
 Wire Wire Line
 	6000 4800 6000 4650

Commit message: Renamed some signals
Connections:
- net ~IRQSUC renamed ~IRQSµC
Changed lines of the file:
@@
 UPC3
 Text Label 4950 4150 0    50   ~ 0
-~IRQSUC
+~IRQSµC
 Text Label 4950 4250 0    50   ~ 0
 ~RSTHOLD
@@
 ~RSTHOLD
 Text Label 8000 4150 0    50   ~ 0
-~IRQSUC
+~IRQSµC
 Text Label 8000 2750 0    50   ~ 0
 UPC3
@@
 IR15
 Text HLabel 1100 4150 0    50   Input ~ 0
-~IRQSUC
+~IRQSµC
 Text HLabel 1100 4250 0    50   Input ~ 0
 ~RSTHOLD
@@
 UPC3
 Text Label 2200 4150 2    50   ~ 0
-~IRQSUC
+~IRQSµC
 Text Label 2200 4250 2    50   ~ 0
 ~RSTHOLD

Commit message: Moved things around a bit
Parts:
- renumbered C2101 to C3301, C2102 to C3302, C2103 to C3303, C2104 to C3304, C2105 to C3305, C2106 to C3306, RN2101 to RN3301, RN2102 to RN3302, RN2103 to RN3303, RN2104 to RN3304, RN2105 to RN3305, RN2106 to RN3306, U2101 to U3301, U2102 to U3302, U2103 to U3303

Commit message: Removed widebus buffer from microcode store µAddr High
Parts:
- renumbered C3301 to C2101, C3302 to C2102, C3303 to C2103, C3304 to C2104, C3305 to C2105, C3306 to C2106, RN3301 to RN2101, RN3302 to RN2102, RN3303 to RN2103, RN3304 to RN2104, RN3305 to RN2105, RN3306 to RN2106, U3301 to U2101, U3302 to U2102, U3303 to U2103
