File: kicad/cft/cft-alu/alu.sch (KiCad schematic (older format))
At the start: 8 parts, among them U2209 74LVC1G08, U2601 74HC138, U2602 74HC138, U2603 74LVC1G08, U2604 74LVC2G157, U2605 74LVC1G08

Commit message: Working on ALU layout.
Parts:
- C3: renamed from C2601; footprint alexios:C_SMD_0805_2012Metric_Pad1.15x1.40mm_HandSolder -> Capacitor_SMD:C_0805_2012Metric
- C4: renamed from C2602; footprint alexios:C_SMD_0805_2012Metric_Pad1.15x1.40mm_HandSolder -> Capacitor_SMD:C_0805_2012Metric
- U2: renamed from U2601; value 74HC138 -> 74AC138
- U5: renamed from U2604; footprint Housings_SSOP:SSOP-8_2.95x2.8mm_Pitch0.65mm -> Package_SO:TSSOP-8_3x3mm_P0.65mm
- renumbered U2603 to U1, U2602 to U3, U2605 to U4, U2209 to U6
Connections:
- net labels added: FL-IN, X0, X1, X2, X3, X4, X5, ~ROMCE
- net labels removed: ~READ-ALU-AND, ~READ-ALU-OR
- wire segments 72 -> 74
- no-connect marks 10 -> 15
Other:
- note added: "1X0XX\nX1X00\n----\n11000"
- note added: "Base\n~Y4~\n\nFinal"
- note added: "NOTE: Use 74AC!"
- note added: "WADDR=1x0xx"
- note removed: "ADD"
- note removed: "AND"
- note removed: "NOT"
- note removed: "OR"
- note removed: "WADDR=10xxx"
- note removed: "XOR"
- moved on the sheet: U2A, U3A
