File: kicad/cft/cft-alu/alu_and.sch (KiCad schematic (older format))
At the start: 14 parts, among them U1507 74HC541, U1508 74HC541, U2801 74HC08, U2802 74HC08, U2803 74HC08, U2804 74HC08, U2805 74HC541, U2806 74HC541

Commit message: Working on ALU layout.
Parts:
- C2801, C2802, C2803, C2804, C2805, C2806: footprint alexios:C_SMD_0805_2012Metric_Pad1.15x1.40mm_HandSolder -> Capacitor_SMD:C_0805_2012Metric
- U1507, U1508, U2805, U2806: footprint alexios:SOIC-20W -> (none)
- U2801, U2802, U2803, U2804: footprint alexios:SOIC-14 -> (none)
Changed lines of the file:
@@
 EESchema Schematic File Version 4
-LIBS:cft-alu-cache
+LIBS:cft-cache
 EELAYER 30 0
 EELAYER END
 $Descr A4 11693 8268
 encoding utf-8
-Sheet 4 11
+Sheet 16 35
 Title ""
 Date ""
@@
 F 0 "C2806" H 10109 5846 50  0000 R CNN
 F 1 "100nF" H 10109 5755 50  0000 R CNN
-F 2 "alexios:C_SMD_0805_2012Metric_Pad1.15x1.40mm_HandSolder" H 10200 5800 50  0001 C CNN
+F 2 "Capacitor_SMD:C_0805_2012Metric" H 10200 5800 50  0001 C CNN
 F 3 "~" H 10200 5800 50  0001 C CNN
 	1    10200 5800
@@
 F 0 "C2805" H 10109 5096 50  0000 R CNN
 F 1 "100nF" H 10109 5005 50  0000 R CNN
-F 2 "alexios:C_SMD_0805_2012Metric_Pad1.15x1.40mm_HandSolder" H 10200 5050 50  0001 C CNN
+F 2 "Capacitor_SMD:C_0805_2012Metric" H 10200 5050 50  0001 C CNN
 F 3 "~" H 10200 5050 50  0001 C CNN
 	1    10200 5050
@@
 F 0 "C2804" H 10109 4346 50  0000 R CNN
 F 1 "100nF" H 10109 4255 50  0000 R CNN
-F 2 "alexios:C_SMD_0805_2012Metric_Pad1.15x1.40mm_HandSolder" H 10200 4300 50  0001 C CNN
+F 2 "Capacitor_SMD:C_0805_2012Metric" H 10200 4300 50  0001 C CNN
 F 3 "~" H 10200 4300 50  0001 C CNN
 	1    10200 4300
@@
 F 0 "C2803" H 10109 3596 50  0000 R CNN
 F 1 "100nF" H 10109 3505 50  0000 R CNN
-F 2 "alexios:C_SMD_0805_2012Metric_Pad1.15x1.40mm_HandSolder" H 10200 3550 50  0001 C CNN
+F 2 "Capacitor_SMD:C_0805_2012Metric" H 10200 3550 50  0001 C CNN
 F 3 "~" H 10200 3550 50  0001 C CNN
 	1    10200 3550
@@
 F 0 "C2802" H 10109 2846 50  0000 R CNN
 F 1 "100nF" H 10109 2755 50  0000 R CNN
-F 2 "alexios:C_SMD_0805_2012Metric_Pad1.15x1.40mm_HandSolder" H 10200 2800 50  0001 C CNN
+F 2 "Capacitor_SMD:C_0805_2012Metric" H 10200 2800 50  0001 C CNN
 F 3 "~" H 10200 2800 50  0001 C CNN
 	1    10200 2800
@@
 F 0 "C2801" H 10109 2096 50  0000 R CNN
 F 1 "100nF" H 10109 2005 50  0000 R CNN
-F 2 "alexios:C_SMD_0805_2012Metric_Pad1.15x1.40mm_HandSolder" H 10200 2050 50  0001 C CNN
+F 2 "Capacitor_SMD:C_0805_2012Metric" H 10200 2050 50  0001 C CNN
 F 3 "~" H 10200 2050 50  0001 C CNN
 	1    10200 2050
@@
 F 0 "U1508" H 10730 5846 50  0000 L CNN
 F 1 "74HC541" H 10730 5755 50  0000 L CNN
-F 2 "alexios:SOIC-20W" H 10550 5800 50  0001 C CNN
+F 2 "" H 10550 5800 50  0001 C CNN
 F 3 "https://assets.nexperia.com/documents/data-sheet/74HC_HCT541.pdf" H 10550 5800 50  0001 C CNN
 	2    10550 5800
@@
 F 0 "U1507" H 10730 5096 50  0000 L CNN
 F 1 "74HC541" H 10730 5005 50  0000 L CNN
-F 2 "alexios:SOIC-20W" H 10550 5050 50  0001 C CNN
+F 2 "" H 10550 5050 50  0001 C CNN
 F 3 "https://assets.nexperia.com/documents/data-sheet/74HC_HCT541.pdf" H 10550 5050 50  0001 C CNN
 	2    10550 5050
@@
 F 0 "U2806" H 6750 2850 50  0000 C CNN
 F 1 "74HC541" H 6750 2750 50  0000 C CNN
-F 2 "alexios:SOIC-20W" H 6750 3550 50  0001 C CNN
+F 2 "" H 6750 3550 50  0001 C CNN
 F 3 "https://assets.nexperia.com/documents/data-sheet/74HC_HCT541.pdf" H 6750 3550 50  0001 C CNN
 	1    6750 3550
@@
 F 0 "U2805" H 6750 2867 50  0000 C CNN
 F 1 "74HC541" H 6750 2776 50  0000 C CNN
-F 2 "alexios:SOIC-20W" H 6750 2100 50  0001 C CNN
+F 2 "" H 6750 2100 50  0001 C CNN
 F 3 "https://assets.nexperia.com/documents/data-sheet/74HC_HCT541.pdf" H 6750 2100 50  0001 C CNN
 	1    6750 2100
@@
 F 0 "U2804" H 4750 4700 50  0000 C CNN
 F 1 "74HC08" H 4575 4734 50  0001 C CNN
-F 2 "alexios:SOIC-14" H 4650 4500 50  0001 C CNN
+F 2 "" H 4650 4500 50  0001 C CNN
 F 3 "http://www.ti.com/lit/gpn/sn74LS08" H 4650 4500 50  0001 C CNN
 	4    4450 4950
@@
 F 0 "U2804" H 4750 4450 50  0000 C CNN
 F 1 "74HC08" H 4575 4484 50  0001 C CNN
-F 2 "alexios:SOIC-14" H 4650 4250 50  0001 C CNN
+F 2 "" H 4650 4250 50  0001 C CNN
 F 3 "http://www.ti.com/lit/gpn/sn74LS08" H 4650 4250 50  0001 C CNN
 	3    4450 4700
@@
 F 0 "U2804" H 4750 4200 50  0000 C CNN
 F 1 "74HC08" H 4575 4234 50  0001 C CNN
-F 2 "alexios:SOIC-14" H 4650 4000 50  0001 C CNN
+F 2 "" H 4650 4000 50  0001 C CNN
 F 3 "http://www.ti.com/lit/gpn/sn74LS08" H 4650 4000 50  0001 C CNN
 	2    4450 4450
@@
 F 0 "U2804" H 4750 3950 50  0000 C CNN
 F 1 "74HC08" H 4575 3984 50  0001 C CNN
-F 2 "alexios:SOIC-14" H 4650 3750 50  0001 C CNN
+F 2 "" H 4650 3750 50  0001 C CNN
 F 3 "http://www.ti.com/lit/gpn/sn74LS08" H 4650 3750 50  0001 C CNN
 	1    4450 4200
@@
 F 0 "U2803" H 4750 3700 50  0000 C CNN
 F 1 "74HC08" H 4575 3734 50  0001 C CNN
-F 2 "alexios:SOIC-14" H 4650 3500 50  0001 C CNN
+F 2 "" H 4650 3500 50  0001 C CNN
 F 3 "http://www.ti.com/lit/gpn/sn74LS08" H 4650 3500 50  0001 C CNN
 	4    4450 3950
@@
 F 0 "U2803" H 4750 3450 50  0000 C CNN
 F 1 "74HC08" H 4575 3484 50  0001 C CNN
-F 2 "alexios:SOIC-14" H 4650 3250 50  0001 C CNN
+F 2 "" H 4650 3250 50  0001 C CNN
 F 3 "http://www.ti.com/lit/gpn/sn74LS08" H 4650 3250 50  0001 C CNN
 	3    4450 3700
@@
 F 0 "U2803" H 4750 3200 50  0000 C CNN
 F 1 "74HC08" H 4575 3234 50  0001 C CNN
-F 2 "alexios:SOIC-14" H 4650 3000 50  0001 C CNN
+F 2 "" H 4650 3000 50  0001 C CNN
 F 3 "http://www.ti.com/lit/gpn/sn74LS08" H 4650 3000 50  0001 C CNN
 	2    4450 3450
@@
 F 0 "U2803" H 4750 2950 50  0000 C CNN
 F 1 "74HC08" H 4575 2984 50  0001 C CNN
-F 2 "alexios:SOIC-14" H 4650 2750 50  0001 C CNN
+F 2 "" H 4650 2750 50  0001 C CNN
 F 3 "http://www.ti.com/lit/gpn/sn74LS08" H 4650 2750 50  0001 C CNN
 	1    4450 3200
@@
 F 0 "U2802" H 4750 2700 50  0000 C CNN
 F 1 "74HC08" H 4575 2734 50  0001 C CNN
-F 2 "alexios:SOIC-14" H 4650 2500 50  0001 C CNN
+F 2 "" H 4650 2500 50  0001 C CNN
 F 3 "http://www.ti.com/lit/gpn/sn74LS08" H 4650 2500 50  0001 C CNN
 	4    4450 2950
@@
 F 0 "U2802" H 4750 2450 50  0000 C CNN
 F 1 "74HC08" H 4575 2484 50  0001 C CNN
-F 2 "alexios:SOIC-14" H 4650 2250 50  0001 C CNN
+F 2 "" H 4650 2250 50  0001 C CNN
 F 3 "http://www.ti.com/lit/gpn/sn74LS08" H 4650 2250 50  0001 C CNN
 	3    4450 2700
@@
 F 0 "U2802" H 4750 2200 50  0000 C CNN
 F 1 "74HC08" H 4575 2234 50  0001 C CNN
-F 2 "alexios:SOIC-14" H 4650 2000 50  0001 C CNN
+F 2 "" H 4650 2000 50  0001 C CNN
 F 3 "http://www.ti.com/lit/gpn/sn74LS08" H 4650 2000 50  0001 C CNN
 	2    4450 2450
@@
 F 0 "U2802" H 4750 1950 50  0000 C CNN
 F 1 "74HC08" H 4575 1984 50  0001 C CNN
-F 2 "alexios:SOIC-14" H 4650 1750 50  0001 C CNN
+F 2 "" H 4650 1750 50  0001 C CNN
 F 3 "http://www.ti.com/lit/gpn/sn74LS08" H 4650 1750 50  0001 C CNN
 	1    4450 2200
@@
 F 0 "U2801" H 4750 1700 50  0000 C CNN
 F 1 "74HC08" H 4575 1734 50  0001 C CNN
-F 2 "alexios:SOIC-14" H 4650 1500 50  0001 C CNN
+F 2 "" H 4650 1500 50  0001 C CNN
 F 3 "http://www.ti.com/lit/gpn/sn74LS08" H 4650 1500 50  0001 C CNN
 	4    4450 1950
@@
 F 0 "U2801" H 4750 1450 50  0000 C CNN
 F 1 "74HC08" H 4575 1484 50  0001 C CNN
-F 2 "alexios:SOIC-14" H 4650 1250 50  0001 C CNN
+F 2 "" H 4650 1250 50  0001 C CNN
 F 3 "http://www.ti.com/lit/gpn/sn74LS08" H 4650 1250 50  0001 C CNN
 	3    4450 1700
@@
 F 0 "U2801" H 4750 1200 50  0000 C CNN
 F 1 "74HC08" H 4575 1234 50  0001 C CNN
-F 2 "alexios:SOIC-14" H 4650 1000 50  0001 C CNN
+F 2 "" H 4650 1000 50  0001 C CNN
 F 3 "http://www.ti.com/lit/gpn/sn74LS08" H 4650 1000 50  0001 C CNN
 	2    4450 1450
@@
 F 0 "U2801" H 4575 1075 50  0000 C CNN
 F 1 "74HC08" H 4575 984 50  0000 C CNN
-F 2 "alexios:SOIC-14" H 4650 750 50  0001 C CNN
+F 2 "" H 4650 750 50  0001 C CNN
 F 3 "http://www.ti.com/lit/gpn/sn74LS08" H 4650 750 50  0001 C CNN
 	1    4450 1200
@@
 F 0 "U2801" H 10730 996 50  0000 L CNN
 F 1 "74HC08" H 10730 905 50  0000 L CNN
-F 2 "alexios:SOIC-14" H 10600 1050 50  0001 C CNN
+F 2 "" H 10600 1050 50  0001 C CNN
 F 3 "http://www.ti.com/lit/gpn/sn74LS08" H 10600 1050 50  0001 C CNN
 	5    10400 1500
@@
 F 0 "U2802" H 10730 1746 50  0000 L CNN
 F 1 "74HC08" H 10730 1655 50  0000 L CNN
-F 2 "alexios:SOIC-14" H 10600 1800 50  0001 C CNN
+F 2 "" H 10600 1800 50  0001 C CNN
 F 3 "http://www.ti.com/lit/gpn/sn74LS08" H 10600 1800 50  0001 C CNN
 	5    10400 2250
@@
 F 0 "U2803" H 10730 2496 50  0000 L CNN
 F 1 "74HC08" H 10730 2405 50  0000 L CNN
-F 2 "alexios:SOIC-14" H 10600 2550 50  0001 C CNN
+F 2 "" H 10600 2550 50  0001 C CNN
 F 3 "http://www.ti.com/lit/gpn/sn74LS08" H 10600 2550 50  0001 C CNN
 	5    10400 3000
@@
 F 0 "U2804" H 10730 3246 50  0000 L CNN
 F 1 "74HC08" H 10730 3155 50  0000 L CNN
-F 2 "alexios:SOIC-14" H 10600 3300 50  0001 C CNN
+F 2 "" H 10600 3300 50  0001 C CNN
 F 3 "http://www.ti.com/lit/gpn/sn74LS08" H 10600 3300 50  0001 C CNN
 	5    10400 3750
