File: kicad/cft/cft-alu/alu_port_b.sch (KiCad schematic (older format))
At the start: 10 parts, among them U26 74HC574, U27 74HC541, U28 74HC574, U29 74HC541

Commit message: Simplified the SRU, working through DRC.
Parts:
- removed U?: 74LVC1G74, symbol alexios:74LVC1G74
- gave numbers to parts that had none: 1
Changed lines of the file:
@@
 EESchema Schematic File Version 4
-EELAYER 30 0
+LIBS:cft-alu-cache
+EELAYER 26 0
 EELAYER END
 $Descr A4 11693 8268
@@
 AR Path="/5DC89E19/5EDE4D1C" Ref="U?"  Part="1"
 AR Path="/5EDE4D1C" Ref="U?"  Part="1"
-F 0 "U?" H 2075 2683 50  0000 C CNN
+AR Path="/5DEA5E6C/5EDE4D1C" Ref="U2"  Part="1"
+F 0 "U2" H 2075 2683 50  0000 C CNN
 F 1 "74LVC1G08" H 2075 2774 50  0000 C CNN
 F 2 "alexios:SOT-23-5_HandSoldering" H 1800 2950 50  0001 C CNN
@@
 Wire Wire Line
 	2550 2950 2550 3500
-$Comp
-L alexios:74LVC1G74 U?
-U 1 1 5EDFB6F3
-P 5050 5800
-F 0 "U?" H 5050 6217 50  0000 C CNN
-F 1 "74LVC1G74" H 5050 6126 50  0000 C CNN
-F 2 "" H 5500 5800 50  0001 C CNN
-F 3 "https://assets.nexperia.com/documents/data-sheet/74LVC1G74.pdf" H 5500 5800 50  0001 C CNN
-	1    5050 5800
-	1    0    0    -1
-$EndComp
-Wire Wire Line
-	5500 5650 9250 5650
-Text HLabel 9250 5650 2    50   Output ~ 0
-B16
-Text Label 5750 5650 0    50   ~ 0
-B16
-Wire Wire Line
-	4600 5950 1350 5950
-Text HLabel 1350 5950 0    50   Input ~ 0
-~RESET
-$Comp
-L power:+5V #PWR?
-U 1 1 5EE2085B
-P 4550 5600
-F 0 "#PWR?" H 4550 5450 50  0001 C CNN
-F 1 "+5V" H 4565 5773 50  0000 C CNN
-F 2 "" H 4550 5600 50  0001 C CNN
-F 3 "" H 4550 5600 50  0001 C CNN
-	1    4550 5600
-	1    0    0    -1
-$EndComp
-Wire Wire Line
-	4550 5600 4550 5650
-Wire Wire Line
-	4550 5650 4600 5650
-Wire Wire Line
-	4600 5750 1350 5750
 Wire Bus Line
 	8550 2000 8550 4450

Commit message: Switched ALU ROMs to 55ns 1MBit devices.
Parts:
- added C33: 100nF, alexios:C_SMD_0805_2012Metric_Pad1.15x1.40mm_HandSolder, symbol Device:C_Small
- added unit 2 of U4
- renumbered U2 to U4
Connections:
- net +5V: now also C33.1, U4.5 (VCC)
- net GND: now also C33.2, U4.3 (GND)
Other:
- moved on the sheet: C27, C28, C29, C30, U26B, U27B, U28B, U29B

Commit message: Cleaning up ALU schematics.
Other:
- note removed: "ALU Port B"
Changed lines of the file:
@@
 encoding utf-8
 Sheet 5 9
-Title "Arithmetic & Logic Unit"
+Title "ALU B Register/Port"
 Date "2019-11-17"
 Rev ""
@@
 Text Label 2650 3600 0    50   ~ 0
 ~READ-ALU-B
-Text Notes 7100 7000 0    197  ~ 39
-ALU Port B
 Text Label 7050 3250 2    50   ~ 0
 ~READ-ALU-B

Commit message: Verifying schematics and ALU PCB match Verilog description.
Connections:
- net BCP renamed CP
Other:
- moved on the sheet: U4A
Changed lines of the file:
@@
 Entry Wire Line
 	6050 3950 5950 3850
-Text Label 4200 3250 0    50   ~ 0
-BCP
-Text Label 4200 4750 0    50   ~ 0
-BCP
 Text Label 4200 2350 0    50   ~ 0
 IBUS0
@@
 	5600 3050 5950 3050
 Entry Bus Bus
-	3900 1900 4000 2000
-Entry Bus Bus
 	6050 5200 6150 5300
 Wire Bus Line
-	3900 1900 2550 1900
-Wire Bus Line
 	6150 5300 9250 5300
-Wire Wire Line
-	2550 3500 3850 3500
-Wire Wire Line
-	3850 4750 3850 3500
 Wire Wire Line
 	3850 4750 4600 4750
@@
 Text Label 4000 4100 1    50   ~ 0
 IBUS[0..15]
-Text Label 2650 1900 0    50   ~ 0
-IBUS[0..15]
-Text HLabel 2550 1900 0    50   BiDi ~ 0
-IBUS[0..15]
-Text Label 2650 3500 0    50   ~ 0
-BCP
-Text HLabel 1300 2900 0    50   Input ~ 0
+Text HLabel 1800 3200 0    50   Input ~ 0
 ~WRITE-ALU-B
 Text Label 9150 5300 2    50   ~ 0
@@
 Entry Bus Bus
 	4000 2000 4100 1900
-Wire Bus Line
-	4100 1900 8450 1900
 Entry Bus Bus
 	8450 1900 8550 2000
@@
 Entry Wire Line
 	8450 2350 8550 2250
-Text HLabel 1300 3600 0    50   Input ~ 0
-~READ-ALU-B
 $Comp
 L Device:C_Small C?
@@
 Connection ~ 3850 7350
 Connection ~ 3850 7150
-Wire Wire Line
-	3850 3250 3850 3500
 Text Label 5900 2350 2    50   ~ 0
 B0
@@
 Text Label 5900 4550 2    50   ~ 0
 B15
-Connection ~ 3850 3500
-Wire Wire Line
-	1300 3600 6400 3600
 Connection ~ 6400 3600
 Wire Wire Line
 	6400 3600 6400 3250
-Text Label 2650 3600 0    50   ~ 0
-~READ-ALU-B
 Text Label 7050 3250 2    50   ~ 0
 ~READ-ALU-B
@@
 L alexios:74LVC1G08 U?
 U 1 1 5EDE4D1C
-P 2150 2950
+P 2800 3250
 AR Path="/5DC89E19/5EDE4D1C" Ref="U?"  Part="1"
 AR Path="/5EDE4D1C" Ref="U?"  Part="1"
 AR Path="/5DEA5E6C/5EDE4D1C" Ref="U4"  Part="1"
-F 0 "U4" H 2075 2683 50  0000 C CNN
-F 1 "74LVC1G08" H 2075 2774 50  0000 C CNN
-F 2 "alexios:SOT-23-5_HandSoldering" H 1800 2950 50  0001 C CNN
-F 3 "https://assets.nexperia.com/documents/data-sheet/74LVC1G08.pdf" H 1800 2950 50  0001 C CNN
-	1    2150 2950
-	1    0    0    -1
-$EndComp
-Text Label 1300 3000 0    50   ~ 0
+F 0 "U4" H 2725 3517 50  0000 C CNN
+F 1 "74LVC1G08" H 2725 3426 50  0000 C CNN
+F 2 "alexios:SOT-23-5_HandSoldering" H 2450 3250 50  0001 C CNN
+F 3 "https://assets.nexperia.com/documents/data-sheet/74LVC1G08.pdf" H 2450 3250 50  0001 C CNN
+	1    2800 3250
+	1    0    0    -1
+$EndComp
+Text Label 1850 3300 0    50   ~ 0
 BCP-SRU
 Wire Wire Line
-	1300 2900 1850 2900
-Wire Wire Line
-	1850 3000 1300 3000
-Text Label 1300 2900 0    50   ~ 0
+	1800 3200 2500 3200
+Wire Wire Line
+	2500 3300 1800 3300
+Text Label 1850 3200 0    50   ~ 0
 ~WRITE-ALU-B
-Text HLabel 1300 3000 0    50   Input ~ 0
+Text HLabel 1800 3300 0    50   Input ~ 0
 BCP-SRU
-Wire Wire Line
-	2300 2950 2550 2950
-Wire Wire Line
-	2550 2950 2550 3500
 $Comp
 L alexios:74LVC1G08 U?
@@
 Connection ~ 1000 7150
 Connection ~ 1000 7350
+Connection ~ 3850 3250
+Wire Wire Line
+	3850 3250 3850 4750
+Wire Wire Line
+	2950 3250 3850 3250
+Text Label 1850 3600 0    50   ~ 0
+~READ-ALU-B
+Wire Bus Line
+	4100 1900 8450 1900
+Text HLabel 1800 1900 0    50   BiDi ~ 0
+IBUS[0..15]
+Entry Bus Bus
+	3900 1900 4000 2000
+Wire Bus Line
+	3900 1900 1800 1900
+Text Label 1850 1900 0    50   ~ 0
+IBUS[0..15]
+Text HLabel 1800 3600 0    50   Input ~ 0
+~READ-ALU-B
+Wire Wire Line
+	1800 3600 6400 3600
 Wire Bus Line
 	8550 2000 8550 4450
@@
 Wire Bus Line
 	4000 2000 4000 4450
+Text Label 4200 4750 0    50   ~ 0
+CP
+Text Label 4200 3250 0    50   ~ 0
+CP
+Text Label 3150 3250 0    50   ~ 0
+CP
 $EndSCHEMATC

Commit message: Fine-tunint ALU board.
Connections:
- net BCP-SRU renamed BCP
Changed lines of the file:
@@
 $EndComp
 Text Label 1850 3300 0    50   ~ 0
-BCP-SRU
+BCP
 Wire Wire Line
 	1800 3200 2500 3200
@@
 ~WRITE-ALU-B
 Text HLabel 1800 3300 0    50   Input ~ 0
-BCP-SRU
+BCP
 $Comp
 L alexios:74LVC1G08 U?
@@
 Wire Wire Line
 	1800 3600 6400 3600
+Text Label 4200 4750 0    50   ~ 0
+CP
+Text Label 4200 3250 0    50   ~ 0
+CP
+Text Label 3150 3250 0    50   ~ 0
+CP
 Wire Bus Line
 	8550 2000 8550 4450
@@
 Wire Bus Line
 	4000 2000 4000 4450
-Text Label 4200 4750 0    50   ~ 0
-CP
-Text Label 4200 3250 0    50   ~ 0
-CP
-Text Label 3150 3250 0    50   ~ 0
-CP
 $EndSCHEMATC
