File: kicad/cft/cft-alu/cft-alu.kicad_pcb (KiCad board)
At the start: 2 copper layers, 131.9 x 164.6 mm, 125 parts, among them P1 CFT-2019-Bus, U1 29W010, U10 74AC191, U11 74HC04, U12 74AC86, U13 74AC541, U14 74AC541, U15 74AC253, U16 74LVC2G157, U17 74LVC2G157, U18 74LVC1G04, U19 74LVC1G86, U2 29W010, U20 74LVC1G0832, U22 74HC08, U23 74AC74, U24 74LVC2G157, U25 74LVC1G08, U26 74HC574, U27 74HC541, U28 74HC574, U29 74HC541, U3 29W010, U30 74HC574, U31 74HC574, U32 74HC32, U33 74AC74, U34 74HC253, U35 74LVC1G08, U36 74LVC1G08, U37 74LVC1G32, U38 74LVC1G11, U39 74AC138, U4 74LVC1G08, U40 74HC138, U41 74HC138, U42 74HC138, U43 74HC573, U44 74LVC1G32, U45 74LVC1G32, U47 74LVC1G08, U48 74LVC1G04, U49 74LVC1G74, U5 74HC541, U6 74HC541, U7 74AUC1G74, U8 74AC541, U9 74AC541

Commit message: Verifying schematics and ALU PCB match Verilog description.
Connections:
- net /Port B/BCP renamed /Port B/CP
- net /sheet5DE3C026/REGCP renamed /sheet5DE3C026/REGLE
- U19 pad 1: /sheet5DE3C026/FLOUT -> /FLOUT-ROM
- U19 pad 4: /FLOUT-ROM -> Net-(U19-Pad4)
- U23 pad 1: /~RESET -> /~RSTHOLD
- U23 pad 13: /~RESET -> /~RSTHOLD
- U3 pad 20: /sheet5DE3C026/FLOUT -> /FLOUT-ROM
- U34 pad 4: /FLOUT-ROM -> Net-(U19-Pad4)
- U36 pad 2: /BCP-SRU -> /Link Register (L)/BCP
- U39 pad 5: /T34 -> GND
- U4 pad 2: /BCP-SRU -> /Port B/BCP-SRU
- U42 pad 10: Net-(U42-Pad10) -> /~WRITE-ALU-B
- U42 pad 11: /~WRITE-ALU-B -> Net-(U42-Pad11)
Routing:
- net /sheet5DE3C026/FLOUT: track 102.5 -> 0.00 mm, vias 1 -> 0
- net /~RESET: track 198.6 -> 142.3 mm, vias 8 -> 5
- net Net-(U19-Pad4): track 0.00 -> 51.5 mm, vias 0 -> 2
- net /FLOUT-ROM: track 51.5 -> 102.5 mm, vias 2 -> 1
- net /~RSTHOLD: track 319.3 -> 338.2 mm, vias 10 -> 12
- net GND: track 195.1 -> 197.7 mm, vias 458 -> 459
- net /~WRITE-ALU-B: track 105.2 -> 103.9 mm
- net /T34: track 101.7 -> 101.2 mm

Commit message: Fine-tunint ALU board.
Parts:
- moved TP9 0.31 mm to (126.0, 165.2)
Connections:
- TP9 pad 1: /BCP-SRU -> /BCP
- U20 pad 4: /BCP-SRU -> /BCP
- U36 pad 2: /Link Register (L)/BCP -> /BCP
- U4 pad 2: /Port B/BCP-SRU -> /BCP
- U7 pad 1: /sheet5DF75CCD/CLK3 -> /CLK3
Routing:
- net /CLK3: track 0.00 -> 142.3 mm, vias 0 -> 6
- net /BCP-SRU: track 41.2 -> 0.00 mm
- net /BCP: track 0.00 -> 40.8 mm
- net GND: track 197.7 -> 213.2 mm, vias 459 -> 458
- net /CLK2: track 164.4 -> 153.3 mm, vias 5 -> 3
- net /T34: track 101.2 -> 91.4 mm, vias 4 -> 1
- net /Port A/A8: track 111.1 -> 104.4 mm
- net +5V: track 1531.5 -> 1529.7 mm
- net /sheet5DE3C026/OP2: track 141.1 -> 142.0 mm
- net /~READ-ALU-B: track 117.4 -> 116.6 mm
- net /~ALU-OP: track 108.3 -> 109.0 mm
- net /CLK4: track 283.8 -> 284.3 mm
- net /Port B/B0: track 232.5 -> 233.0 mm

Commit message: Cleaning up schematics, added notes, fine-tuned ALU PCB.
Parts:
- added C48: 100nF, alexios:C_SMD_0805_2012Metric_Pad1.15x1.40mm_HandSolder, F.Cu at (60.1, 195.3)
- added C53: 100nF, alexios:C_SMD_0805_2012Metric_Pad1.15x1.40mm_HandSolder, F.Cu at (70.4, 190.2)
- added JP2: SolderJumper_2_Open, Jumper:SolderJumper-2_P1.3mm_Open_RoundedPad1.0x1.5mm, F.Cu at (72.5, 194.3)
- added R3: 0Ω, alexios:R_SMD_0805_2012Metric_Pad1.15x1.40mm_HandSolder, F.Cu at (73.0, 174.5)
- added R4: 0Ω, alexios:R_SMD_0805_2012Metric_Pad1.15x1.40mm_HandSolder, F.Cu at (73.0, 179.1)
- added R5: 0Ω, alexios:R_SMD_0805_2012Metric_Pad1.15x1.40mm_HandSolder, B.Cu at (85.8, 178.1)
- added R6: 0Ω, alexios:R_SMD_0805_2012Metric_Pad1.15x1.40mm_HandSolder, B.Cu at (96.2, 177.4)
- added R7: 0Ω, alexios:R_SMD_0805_2012Metric_Pad1.15x1.40mm_HandSolder, B.Cu at (68.1, 184.8)
- added U21: 74LVC1G04, alexios:SOT-23-5_HandSoldering, F.Cu at (65.4, 189.2)
- added U46: ICS501, alexios:SOIC-8, F.Cu at (62.8, 193.0)
- moved TP5 13.7 mm to (87.0, 176.4)
- moved TP7 13.7 mm to (87.0, 178.5)
- moved C50 2.84 mm to (166.8, 69.6)
- moved U48 2.84 mm to (162.0, 68.6)
- moved C51 1.27 mm to (166.7, 74.7)
- moved U47 1.27 mm to (161.8, 73.7)
- moved TP6 0.98 mm to (87.0, 180.6)
- moved JP1 0.38 mm to (86.9, 182.0)
- moved C10 0.13 mm to (154.6, 181.6)
Connections:
- TP6 pad 1: /sheet5DF75CCD/x4CLK -> Net-(R5-Pad2)
- U10 pad 12: /sheet5DF75CCD/TC -> Net-(R6-Pad2)
- U11 pad 4: Net-(U11-Pad4) -> Net-(R3-Pad2)
- U11 pad 8: Net-(U11-Pad8) -> Net-(R4-Pad2)
- U12 pad 1: Net-(U11-Pad4) -> Net-(R3-Pad1)
- U12 pad 4: Net-(U11-Pad8) -> Net-(R4-Pad1)
- U12 pad 8: /sheet5DF75CCD/x4CLK -> Net-(R5-Pad2)
Routing:
- net +5V: track 1529.7 -> 1605.0 mm
- net /sheet5DF75CCD/x4CLK: track 31.2 -> 49.0 mm, vias 3 -> 5
- net Net-(U11-Pad4): track 15.5 -> 0.00 mm
- net Net-(U11-Pad8): track 13.5 -> 0.00 mm
- net /CLK4: track 284.3 -> 296.5 mm, vias 9 -> 10
- net Net-(R3-Pad2): track 0.00 -> 9.99 mm
- net Net-(U21-Pad2): track 0.00 -> 9.84 mm
- net Net-(R4-Pad1): track 0.00 -> 8.20 mm
- net Net-(R7-Pad2): track 0.00 -> 6.88 mm, vias 0 -> 1
- net Net-(R5-Pad2): track 0.00 -> 5.09 mm, vias 0 -> 1
- net Net-(R6-Pad2): track 0.00 -> 3.86 mm, vias 0 -> 1
- net /~ALU-OP: track 109.0 -> 105.4 mm
- net Net-(R3-Pad1): track 0.00 -> 3.48 mm
- net Net-(R4-Pad2): track 0.00 -> 3.41 mm
- net /Decoders/ACP: track 63.8 -> 60.6 mm
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Other:
- board text added: "Install U11 & U12 or U46 & U21. JP2 tristates PLL if bridged."
- board text added: "PLL"
- board text added: "×2CLK"
- board text added: "×4CLK"
- board text added: "×4CLK terminating resistors. Install R5 or R7 only!"
- board text removed: "x4CLK"

Commit message: Wrapping up ALU PCB.
Parts:
- added G***: LOGO, alexios:CFT, B.Cu at (149.8, 197.0)
- added G***: LOGO, alexios:CFT, F.Cu at (171.7, 125.7)
- added REF**: ESD-Logo_8.9x8mm_SilkScreen, Symbol:ESD-Logo_8.9x8mm_SilkScreen, B.Cu at (171.6, 124.8)
- added REF**: WEEE-Logo_5.6x8mm_SilkScreen, Symbol:WEEE-Logo_5.6x8mm_SilkScreen, B.Cu at (173.9, 69.2)
- added REF**: KiCad-Logo2_6mm_SilkScreen, Symbol:KiCad-Logo2_6mm_SilkScreen, B.Cu at (67.1, 79.0)
- added REF**: SIGNATURESILK, alexios:SIGNATURE, F.Cu at (171.9, 79.8)
- added REF**: QRCODE-CFT, alexios:QRCODE-CFT, B.Cu at (114.3, 98.3)
Routing:
- net +5V: track 1605.0 -> 1631.3 mm
- net GND: track 211.0 -> 211.3 mm, vias 461 -> 753
Other:
- board text added: "Address Latch"
- board text added: "WARNING: THIS IS NOT PCI EXPRESS. Do not plug into PCI Express receptacles, not even extension cables. Damage may occur."
- board text added: "www.bedroomlan.org/cft"
- board text added: "© 2020 Alexios Chouchoulas"

Commit message: Fine-tuning ALU board.
Parts:
- moved C4 1.99 mm to (61.9, 133.7)
Routing:
- net +5V: track 1631.3 -> 1330.8 mm, vias 19 -> 23
- net GND: track 211.3 -> 213.6 mm, vias 753 -> 747
- net /sheet5DE3C026/Y13: track 99.1 -> 99.7 mm
Other:
- board text added: "Distance counter"
- board text removed: "Distance"

Commit message: Fine-tuning ALU and CTL boards.
Other:
- board text added: "2020"
Changed lines of the file:
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@@
   (general
     (thickness 1.6)
-    (drawings 44)
+    (drawings 49)
     (tracks 3803)
     (zones 0)
@@
   )
   (setup
-    (last_trace_width 0.6096)
+    (last_trace_width 0.1778)
     (user_trace_width 0.1778)
     (user_trace_width 0.6096)
@@
       ))
   )
+  (gr_line (start 174.022 184.404) (end 174.022 187.706) (layer F.SilkS) (width 0.3048))
+  (gr_line (start 174.022 187.706) (end 166.402 187.706) (layer F.SilkS) (width 0.3048))
+  (gr_line (start 166.402 187.706) (end 166.402 184.404) (layer F.SilkS) (width 0.3048))
+  (gr_line (start 166.402 184.404) (end 174.022 184.404) (layer F.SilkS) (width 0.3048))
+  (gr_text 2020 (at 170.212 186.055) (layer F.SilkS)
+    (effects (font (size 1.66 1.66) (thickness 0.3)))
+  )
   (gr_text "Address Latch" (at 99.219 134.112) (layer F.SilkS)

Commit message: Checks passing, updating schematics.
Parts:
- removed G*** (x2): LOGO, alexios:CFT
- removed the REF** at (171.6, 124.8)
- removed the REF** at (173.9, 69.2)
- removed the REF** at (67.1, 79.0)
- removed the REF** at (171.9, 79.8)
- removed the REF** at (114.3, 98.3)
- added JP3: Jumper_NC_Small, Jumper:SolderJumper-2_P1.3mm_Bridged_RoundedPad1.0x1.5mm, F.Cu at (31.8, 74.8)
- added JP4: Jumper_NC_Small, Jumper:SolderJumper-2_P1.3mm_Bridged_RoundedPad1.0x1.5mm, F.Cu at (36.1, 74.8)
Connections:
- U40 pad 4: /T34 -> /Decoders/CLK4
- U41 pad 4: /T34 -> Net-(JP3-Pad2)
- U42 pad 4: /T34 -> Net-(JP4-Pad2)

Commit message: Synced schematics with recent timing changes.
Parts:
- removed C36: 100nF, alexios:C_SMD_0805_2012Metric_Pad1.15x1.40mm_HandSolder
- removed U36: 74LVC1G08, alexios:SOT-23-5_HandSoldering
- U35: value 74LVC1G08 -> 74LVC1G11; footprint alexios:SOT-23-5_HandSoldering -> alexios:SOT-23-6_Handsoldering
- moved U35 25.4 mm to (131.9, 164.2)
Connections:
- JP4 pad 1: /T34 -> /CLK4
- U35 pad 1: /~FLAGWE -> /BCP
- U35 pad 2: /~SETL-ROM -> GND
- U35 pad 3: GND -> /~SETL-ROM
- U35 pad 4: Net-(U35-Pad4) -> /Link Register (L)/CLKL
- U40 pad 4: /Decoders/CLK4 -> /CLK4
Routing:
- net Net-(U35-Pad4): track 33.9 -> 0.00 mm, vias 2 -> 0
- net /BCP: track 40.8 -> 69.1 mm, vias 0 -> 2
- net GND: track 213.6 -> 212.3 mm, vias 747 -> 746
