File: kicad/cft/cft-dfp/cft_dfp_abpod.sch (KiCad schematic (older format))
At the start: 12 parts, among them U601 74HC574, U602 74HC574, U603 74HC574, U604 74HC574, U605 74HC574, U606 74HC574

Commit message: Verifying footprints.
Parts:
- U601, U602, U603, U604, U605, U606: Verified (none) -> Yes
Changed lines of the file:
@@
 $Descr A4 11693 8268
 encoding utf-8
-Sheet 6 13
+Sheet 5 13
 Title ""
 Date ""
@@
 F 2 "alexios:SOIC-20W" H 900 6650 50  0001 C CNN
 F 3 "http://www.ti.com/lit/gpn/sn74LS574" H 900 6650 50  0001 C CNN
+F 4 "Yes" H 0   0   50  0001 C CNN "Verified"
 	2    1200 6700
 	1    0    0    -1
@@
 F 2 "alexios:SOIC-20W" H 3800 6650 50  0001 C CNN
 F 3 "http://www.ti.com/lit/gpn/sn74LS574" H 3800 6650 50  0001 C CNN
+F 4 "Yes" H 0   0   50  0001 C CNN "Verified"
 	2    4100 6700
 	1    0    0    -1
@@
 F 2 "alexios:SOIC-20W" H 7050 3100 50  0001 C CNN
 F 3 "http://www.ti.com/lit/gpn/sn74LS574" H 7050 3100 50  0001 C CNN
+F 4 "Yes" H 0   0   50  0001 C CNN "Verified"
 	1    7350 3150
 	1    0    0    -1
@@
 F 2 "alexios:SOIC-20W" H 7050 1650 50  0001 C CNN
 F 3 "http://www.ti.com/lit/gpn/sn74LS574" H 7050 1650 50  0001 C CNN
+F 4 "Yes" H 0   0   50  0001 C CNN "Verified"
 	1    7350 1700
 	1    0    0    -1
@@
 F 2 "alexios:SOIC-20W" H 4800 3100 50  0001 C CNN
 F 3 "http://www.ti.com/lit/gpn/sn74LS574" H 4800 3100 50  0001 C CNN
+F 4 "Yes" H 0   0   50  0001 C CNN "Verified"
 	1    5100 3150
 	1    0    0    -1
@@
 F 2 "alexios:SOIC-20W" H 4800 1650 50  0001 C CNN
 F 3 "http://www.ti.com/lit/gpn/sn74LS574" H 4800 1650 50  0001 C CNN
+F 4 "Yes" H 5100 1700 50  0001 C CNN "Verified"
 	1    5100 1700
 	1    0    0    -1
@@
 F 2 "alexios:SOIC-20W" H 4800 4550 50  0001 C CNN
 F 3 "http://www.ti.com/lit/gpn/sn74LS574" H 4800 4550 50  0001 C CNN
+F 4 "Yes" H 0   0   50  0001 C CNN "Verified"
 	1    5100 4600
 	1    0    0    -1
@@
 F 2 "alexios:SOIC-20W" H 7050 4550 50  0001 C CNN
 F 3 "http://www.ti.com/lit/gpn/sn74LS574" H 7050 4550 50  0001 C CNN
+F 4 "Yes" H 0   0   50  0001 C CNN "Verified"
 	1    7350 4600
 	1    0    0    -1
@@
 F 2 "alexios:SOIC-20W" H 900 7350 50  0001 C CNN
 F 3 "http://www.ti.com/lit/gpn/sn74LS574" H 900 7350 50  0001 C CNN
+F 4 "Yes" H 0   0   50  0001 C CNN "Verified"
 	2    1200 7400
 	1    0    0    -1
@@
 F 2 "alexios:SOIC-20W" H 2350 7350 50  0001 C CNN
 F 3 "http://www.ti.com/lit/gpn/sn74LS574" H 2350 7350 50  0001 C CNN
+F 4 "Yes" H 0   0   50  0001 C CNN "Verified"
 	2    2650 7400
 	1    0    0    -1
@@
 F 2 "alexios:SOIC-20W" H 3800 7350 50  0001 C CNN
 F 3 "http://www.ti.com/lit/gpn/sn74LS574" H 3800 7350 50  0001 C CNN
+F 4 "Yes" H 0   0   50  0001 C CNN "Verified"
 	2    4100 7400
 	1    0    0    -1
@@
 F 2 "alexios:SOIC-20W" H 2350 6650 50  0001 C CNN
 F 3 "http://www.ti.com/lit/gpn/sn74LS574" H 2350 6650 50  0001 C CNN
+F 4 "Yes" H 0   0   50  0001 C CNN "Verified"
 	2    2650 6700
 	1    0    0    -1

Commit message: Changed 0805 footprints to my own version.
Parts:
- C601, C602, C603, C604, C605, C606: footprint Capacitor_SMD:C_0805_2012Metric_Pad1.15x1.40mm_HandSolder -> alexios:SMD_0805_2012Metric_Pad1.15x1.40mm_HandSolder
Changed lines of the file:
@@
 F 0 "C601" H 759 6746 50  0000 R CNN
 F 1 "100nF" H 759 6655 50  0000 R CNN
-F 2 "Capacitor_SMD:C_0805_2012Metric_Pad1.15x1.40mm_HandSolder" H 850 6700 50  0001 C CNN
+F 2 "alexios:SMD_0805_2012Metric_Pad1.15x1.40mm_HandSolder" H 850 6700 50  0001 C CNN
 F 3 "~" H 850 6700 50  0001 C CNN
 	1    850  6700
@@
 F 0 "C605" H 3659 6746 50  0000 R CNN
 F 1 "100nF" H 3659 6655 50  0000 R CNN
-F 2 "Capacitor_SMD:C_0805_2012Metric_Pad1.15x1.40mm_HandSolder" H 3750 6700 50  0001 C CNN
+F 2 "alexios:SMD_0805_2012Metric_Pad1.15x1.40mm_HandSolder" H 3750 6700 50  0001 C CNN
 F 3 "~" H 3750 6700 50  0001 C CNN
 	1    3750 6700
@@
 F 0 "C602" H 759 7446 50  0000 R CNN
 F 1 "100nF" H 759 7355 50  0000 R CNN
-F 2 "Capacitor_SMD:C_0805_2012Metric_Pad1.15x1.40mm_HandSolder" H 850 7400 50  0001 C CNN
+F 2 "alexios:SMD_0805_2012Metric_Pad1.15x1.40mm_HandSolder" H 850 7400 50  0001 C CNN
 F 3 "~" H 850 7400 50  0001 C CNN
 	1    850  7400
@@
 F 0 "C604" H 2209 7446 50  0000 R CNN
 F 1 "100nF" H 2209 7355 50  0000 R CNN
-F 2 "Capacitor_SMD:C_0805_2012Metric_Pad1.15x1.40mm_HandSolder" H 2300 7400 50  0001 C CNN
+F 2 "alexios:SMD_0805_2012Metric_Pad1.15x1.40mm_HandSolder" H 2300 7400 50  0001 C CNN
 F 3 "~" H 2300 7400 50  0001 C CNN
 	1    2300 7400
@@
 F 0 "C606" H 3659 7446 50  0000 R CNN
 F 1 "100nF" H 3659 7355 50  0000 R CNN
-F 2 "Capacitor_SMD:C_0805_2012Metric_Pad1.15x1.40mm_HandSolder" H 3750 7400 50  0001 C CNN
+F 2 "alexios:SMD_0805_2012Metric_Pad1.15x1.40mm_HandSolder" H 3750 7400 50  0001 C CNN
 F 3 "~" H 3750 7400 50  0001 C CNN
 	1    3750 7400
@@
 F 0 "C603" H 2209 6746 50  0000 R CNN
 F 1 "100nF" H 2209 6655 50  0000 R CNN
-F 2 "Capacitor_SMD:C_0805_2012Metric_Pad1.15x1.40mm_HandSolder" H 2300 6700 50  0001 C CNN
+F 2 "alexios:SMD_0805_2012Metric_Pad1.15x1.40mm_HandSolder" H 2300 6700 50  0001 C CNN
 F 3 "~" H 2300 6700 50  0001 C CNN
 	1    2300 6700
