File: kicad/cft/cft-dfp/cft_dsp_ucvpod.sch (KiCad schematic (older format))
At the start: 6 parts, among them U1001 74HC574, U1002 74HC574, U1003 74HC574

Commit message: Rework DFP schematics for Revision B
Connections:
- net ~µCVOE renamed ~CVOE
Changed lines of the file:
@@
 $Descr A4 11693 8268
 encoding utf-8
-Sheet 9 13
+Sheet 9 14
 Title "Control Unit Pod"
 Date "2019-11-17"
@@
 µCVCPL
 Text HLabel 3400 2950 0    50   Input ~ 0
-~µCVOE
+~CVOE
 Wire Wire Line
 	4600 2950 3400 2950
@@
 	5000 4400 4600 4400
 Text Label 3500 2950 0    50   ~ 0
-~µCVOE
+~CVOE
 Wire Wire Line
 	5000 2950 4600 2950
@@
 µCVCPH
 Text Label 4950 2950 2    50   ~ 0
-~µCVOE
+~CVOE
 Text Label 4950 4400 2    50   ~ 0
-~µCVOE
+~CVOE
 Text Label 4950 5850 2    50   ~ 0
-~µCVOE
+~CVOE
 Entry Wire Line
 	4500 4850 4400 4750

Commit message: Work on DFP schematics
Changed lines of the file:
@@
 $Descr A4 11693 8268
 encoding utf-8
-Sheet 9 14
+Sheet 9 15
 Title "Control Unit Pod"
 Date "2019-11-17"
@@
 AR Path="/5D42FF4D/5D492997" Ref="U?"  Part="1"
 AR Path="/5E6A6F4A/5D492997" Ref="U1002"  Part="1"
-F 0 "U1002" H 5500 4667 50  0000 C CNN
+F 0 "U?" H 5500 4667 50  0000 C CNN
 F 1 "74HC574" H 5500 4576 50  0000 C CNN
 F 2 "alexios:SOIC-20W" H 5200 3850 50  0001 C CNN
@@
 AR Path="/5D42FF4D/5D49299E" Ref="U?"  Part="1"
 AR Path="/5E6A6F4A/5D49299E" Ref="U1001"  Part="1"
-F 0 "U1001" H 5500 3217 50  0000 C CNN
+F 0 "U?" H 5500 3217 50  0000 C CNN
 F 1 "74HC574" H 5500 3126 50  0000 C CNN
 F 2 "alexios:SOIC-20W" H 5200 2400 50  0001 C CNN
@@
 AR Path="/5D42FF4D/5D4929F9" Ref="U?"  Part="1"
 AR Path="/5E6A6F4A/5D4929F9" Ref="U1003"  Part="1"
-F 0 "U1003" H 5500 6117 50  0000 C CNN
+F 0 "U?" H 5500 6117 50  0000 C CNN
 F 1 "74HC574" H 5500 6026 50  0000 C CNN
 F 2 "alexios:SOIC-20W" H 5200 5300 50  0001 C CNN
@@
 AR Path="/5D42FF4D/5D49B81E" Ref="#PWR?"  Part="1"
 AR Path="/5E6A6F4A/5D49B81E" Ref="#PWR01006"  Part="1"
-F 0 "#PWR01006" H 3850 7250 50  0001 C CNN
+F 0 "#PWR?" H 3850 7250 50  0001 C CNN
 F 1 "GND" H 3855 7327 50  0000 C CNN
 F 2 "" H 3850 7500 50  0001 C CNN
@@
 AR Path="/5D42FF4D/5D49B824" Ref="#PWR?"  Part="1"
 AR Path="/5E6A6F4A/5D49B824" Ref="#PWR01005"  Part="1"
-F 0 "#PWR01005" H 3850 7150 50  0001 C CNN
+F 0 "#PWR?" H 3850 7150 50  0001 C CNN
 F 1 "+5V" H 3865 7473 50  0000 C CNN
 F 2 "" H 3850 7300 50  0001 C CNN
@@
 AR Path="/5D42FF4D/5D49B82A" Ref="C?"  Part="1"
 AR Path="/5E6A6F4A/5D49B82A" Ref="C1003"  Part="1"
-F 0 "C1003" H 3759 7446 50  0000 R CNN
+F 0 "C?" H 3759 7446 50  0000 R CNN
 F 1 "100nF" H 3759 7355 50  0000 R CNN
 F 2 "alexios:SMD_0805_2012Metric_Pad1.15x1.40mm_HandSolder" H 3850 7400 50  0001 C CNN
@@
 AR Path="/5D42FF4D/5D49B831" Ref="U?"  Part="2"
 AR Path="/5E6A6F4A/5D49B831" Ref="U1003"  Part="2"
-F 0 "U1003" H 4379 7446 50  0000 L CNN
+F 0 "U?" H 4379 7446 50  0000 L CNN
 F 1 "74HC574" H 4379 7355 50  0000 L CNN
 F 2 "alexios:SOIC-20W" H 3900 7350 50  0001 C CNN
@@
 AR Path="/5D42FF4D/5D49B815" Ref="U?"  Part="2"
 AR Path="/5E6A6F4A/5D49B815" Ref="U1002"  Part="2"
-F 0 "U1002" H 2929 7446 50  0000 L CNN
+F 0 "U?" H 2929 7446 50  0000 L CNN
 F 1 "74HC574" H 2929 7355 50  0000 L CNN
 F 2 "alexios:SOIC-20W" H 2450 7350 50  0001 C CNN
@@
 AR Path="/5D42FF4D/5D49B80E" Ref="C?"  Part="1"
 AR Path="/5E6A6F4A/5D49B80E" Ref="C1002"  Part="1"
-F 0 "C1002" H 2309 7446 50  0000 R CNN
+F 0 "C?" H 2309 7446 50  0000 R CNN
 F 1 "100nF" H 2309 7355 50  0000 R CNN
 F 2 "alexios:SMD_0805_2012Metric_Pad1.15x1.40mm_HandSolder" H 2400 7400 50  0001 C CNN
@@
 AR Path="/5D42FF4D/5D49B808" Ref="#PWR?"  Part="1"
 AR Path="/5E6A6F4A/5D49B808" Ref="#PWR01003"  Part="1"
-F 0 "#PWR01003" H 2400 7150 50  0001 C CNN
+F 0 "#PWR?" H 2400 7150 50  0001 C CNN
 F 1 "+5V" H 2415 7473 50  0000 C CNN
 F 2 "" H 2400 7300 50  0001 C CNN
@@
 AR Path="/5D42FF4D/5D49B802" Ref="#PWR?"  Part="1"
 AR Path="/5E6A6F4A/5D49B802" Ref="#PWR01004"  Part="1"
-F 0 "#PWR01004" H 2400 7250 50  0001 C CNN
+F 0 "#PWR?" H 2400 7250 50  0001 C CNN
 F 1 "GND" H 2405 7327 50  0000 C CNN
 F 2 "" H 2400 7500 50  0001 C CNN
@@
 AR Path="/5D42FF4D/5D49B7F9" Ref="U?"  Part="2"
 AR Path="/5E6A6F4A/5D49B7F9" Ref="U1001"  Part="2"
-F 0 "U1001" H 1479 7446 50  0000 L CNN
+F 0 "U?" H 1479 7446 50  0000 L CNN
 F 1 "74HC574" H 1479 7355 50  0000 L CNN
 F 2 "alexios:SOIC-20W" H 1000 7350 50  0001 C CNN
@@
 AR Path="/5D42FF4D/5D49B7F2" Ref="C?"  Part="1"
 AR Path="/5E6A6F4A/5D49B7F2" Ref="C1001"  Part="1"
-F 0 "C1001" H 859 7446 50  0000 R CNN
+F 0 "C?" H 859 7446 50  0000 R CNN
 F 1 "100nF" H 859 7355 50  0000 R CNN
 F 2 "alexios:SMD_0805_2012Metric_Pad1.15x1.40mm_HandSolder" H 950 7400 50  0001 C CNN
@@
 AR Path="/5D42FF4D/5D49B7EC" Ref="#PWR?"  Part="1"
 AR Path="/5E6A6F4A/5D49B7EC" Ref="#PWR01001"  Part="1"
-F 0 "#PWR01001" H 950 7150 50  0001 C CNN
+F 0 "#PWR?" H 950 7150 50  0001 C CNN
 F 1 "+5V" H 965 7473 50  0000 C CNN
 F 2 "" H 950 7300 50  0001 C CNN
@@
 AR Path="/5D42FF4D/5D49B7E6" Ref="#PWR?"  Part="1"
 AR Path="/5E6A6F4A/5D49B7E6" Ref="#PWR01002"  Part="1"
-F 0 "#PWR01002" H 950 7250 50  0001 C CNN
+F 0 "#PWR?" H 950 7250 50  0001 C CNN
 F 1 "GND" H 955 7327 50  0000 C CNN
 F 2 "" H 950 7500 50  0001 C CNN
