File: kicad/cft/cft-dfp/cft-dfp-scan.sch (KiCad schematic (older format))
At the start: 14 parts, among them U33 74LVC1G00, U34 74HC138, U35 74LVC1G04, U36 74HC154, U37 74HC154, U38 74HC540, U39 74HC139

Commit message: Work on DFP
Parts:
- added R901, R902, R903, R904, R905: 1kΩ?, alexios:R_SMD_0805_2012Metric_Pad1.15x1.40mm_HandSolder, symbol Device:R_Small
Connections:
- wire segments 103 -> 108
Other:
- moved on the sheet: U33A, U34A
Changed lines of the file:
@@
 Module A, Row 1 (µCV high)
 Wire Wire Line
-	2800 1200 3100 1200
-Entry Wire Line
-	2700 1000 2800 1100
-Entry Wire Line
-	2700 1100 2800 1200
-Wire Wire Line
-	2800 1100 3100 1100
-Wire Wire Line
-	2800 1300 3100 1300
-Entry Wire Line
-	2700 1200 2800 1300
-Text Label 2900 1100 0    50   ~ 0
+	2150 1200 2450 1200
+Entry Wire Line
+	2050 1000 2150 1100
+Entry Wire Line
+	2050 1100 2150 1200
+Wire Wire Line
+	2150 1100 2450 1100
+Wire Wire Line
+	2150 1300 2450 1300
+Entry Wire Line
+	2050 1200 2150 1300
+Text Label 2250 1100 0    50   ~ 0
 FPA2
-Text Label 2900 1200 0    50   ~ 0
+Text Label 2250 1200 0    50   ~ 0
 FPA3
-Text Label 2900 1300 0    50   ~ 0
+Text Label 2250 1300 0    50   ~ 0
 FPA4
 Text Label 7050 5050 0    50   ~ 0
@@
 Text Label 7500 4650 2    50   ~ 0
 ~FPOE20
-Text Label 1550 3150 2    50   ~ 0
+Text Label 900  3150 2    50   ~ 0
 ~PANELEN
-Text HLabel 1100 3150 0    50   Input ~ 0
+Text HLabel 450  3150 0    50   Input ~ 0
 ~PANELEN
 Entry Wire Line
-	2700 1700 2800 1800
-Entry Wire Line
-	2700 1800 2800 1900
-Wire Wire Line
-	2800 1800 3100 1800
-Wire Wire Line
-	2800 1900 3100 1900
-Text Label 2900 1900 0    50   ~ 0
+	2050 1700 2150 1800
+Entry Wire Line
+	2050 1800 2150 1900
+Wire Wire Line
+	2150 1800 2450 1800
+Wire Wire Line
+	2150 1900 2450 1900
+Text Label 2250 1900 0    50   ~ 0
 FPA7
-Text Label 2900 1800 0    50   ~ 0
+Text Label 2250 1800 0    50   ~ 0
 FPA6
-Text Notes 2950 2750 0    50   ~ 0
+Text Notes 2300 2750 0    50   ~ 0
 ROW₁ to ROW₅ are decoded strobes\nfor the front panel modules. The\nappropriate module is enabled for\nwriting using address FA₀–FA₁ and\nthe desired 8-bit register on that\nmodule is clocked using the ~ROW~\nstrobes.
-Text Notes 2950 3800 0    50   ~ 0
+Text Notes 2300 3800 0    50   ~ 0
 When ~PANELEN~ is de-asserted,\nthe MCU can control the front panel\nlights directly.\n\n~PANELEN~ should ALWAYS be\nde-asserted when writing to MCU\naddresses &00–&03F.
 Wire Wire Line
-	3100 1700 3050 1700
+	2450 1700 2400 1700
 Wire Notes Line width 24 style solid
-	2850 3000 1100 3000
+	2200 3000 450  3000
 Wire Notes Line width 24 style solid
-	1100 900  2850 900
-Text Notes 1200 1750 0    63   ~ 13
+	450  900  2200 900
+Text Notes 550  1750 0    63   ~ 13
 Erratum, rev. A (1930)
 Wire Notes Line width 24 style solid
-	1100 3000 1100 900
-Text Label 1750 1450 0    50   ~ 0
+	450  3000 450  900
+Text Label 1100 1450 0    50   ~ 0
 ~SCANEN
-Text Label 1750 1350 0    50   ~ 0
+Text Label 1100 1350 0    50   ~ 0
 ~WR
-Text HLabel 1650 1450 0    50   Input ~ 0
+Text HLabel 1000 1450 0    50   Input ~ 0
 ~SCANEN
-Text HLabel 1650 1350 0    50   Input ~ 0
+Text HLabel 1000 1350 0    50   Input ~ 0
 ~WR
 Wire Wire Line
-	2100 1450 1650 1450
-Wire Wire Line
-	2100 1350 1650 1350
+	1450 1450 1000 1450
+Wire Wire Line
+	1450 1350 1000 1350
 Wire Notes Line width 24 style solid
-	2850 3000 2850 900
-Text Notes 1200 2900 0    50   ~ 0
+	2200 3000 2200 900
+Text Notes 550  2900 0    50   ~ 0
 In XMem mode, the Atmega drives its\naddress bus all the time, but the '138\ndecoder in Rev. A of the board isn't\ngated, so the front panel shows the\ninner workings of the Atmega instead\nof the CFT!\n\nU1202 should be gated such that it\nstrobes ~ROWx~ when either ~SCANEN~ or\nthe Atmega's ~WR~ signal is asserted.\n\nNote: this removes the (unused)\n‘snoop-update’ mode of the FP.
 Text Notes 6950 1100 2    50   ~ 10
@@
 	4500 700  4600 800
 Wire Bus Line
-	2800 700  4500 700
+	2150 700  4500 700
 Entry Bus Bus
-	2600 700  2700 800
-Text Label 1500 700  2    50   ~ 0
+	1950 700  2050 800
+Text Label 850  700  2    50   ~ 0
 FPA[0..7]
 Entry Bus Bus
-	2800 700  2700 800
+	2150 700  2050 800
 Wire Bus Line
-	1100 700  2600 700
-Text HLabel 1100 700  0    50   Input ~ 0
+	450  700  1950 700
+Text HLabel 450  700  0    50   Input ~ 0
 FPA[0..7]
 Text Label 4700 2150 0    50   ~ 0
@@
 	7050 5050 7600 5050
 Wire Wire Line
-	1100 3150 4450 3150
+	450  3150 4450 3150
 Wire Wire Line
 	4450 3650 4450 3150
@@
 Text Label 4450 3050 1    50   ~ 0
 ~PANELEN
-NoConn ~ 4100 1600
-NoConn ~ 4100 1700
-NoConn ~ 4100 1800
-Wire Wire Line
-	2550 1400 3050 1400
-Wire Wire Line
-	3050 1400 3050 1700
+NoConn ~ 3450 1700
+NoConn ~ 3450 1800
+Wire Wire Line
+	1900 1400 2400 1400
+Wire Wire Line
+	2400 1400 2400 1700
 Text HLabel 1200 6450 0    50   Input ~ 0
 MFD0
@@
 L alexios:74LVC1G00 U33
 U 1 1 6AFE1F5D
-P 2400 1400
-F 0 "U33" H 2325 1667 50  0000 C CNN
-F 1 "74LVC1G00" H 2325 1576 50  0000 C CNN
-F 2 "alexios:SOT-23-5_HandSoldering" H 2050 1400 50  0001 C CNN
-F 3 "https://assets.nexperia.com/documents/data-sheet/74LVC1G00.pdf" H 2050 1400 50  0001 C CNN
-	1    2400 1400
-	1    0    0    -1
-$EndComp
-$Comp
-L alexios:74HC138 U34
-U 1 1 6AFE3EEE
-P 3600 1500
-F 0 "U34" H 3600 2167 50  0000 C CNN
-F 1 "74HC138" H 3600 2076 50  0000 C CNN
-F 2 "alexios:DIP-16_W7.62mm_Socket" H 3600 1500 50  0001 C CNN
-F 3 "https://assets.nexperia.com/documents/data-sheet/74HC_HCT138.pdf" H 3600 1500 50  0001 C CNN
-F 4 "Yes" H 3525 675 50  0001 C CNN "Verified"
-	1    3600 1500
+P 1750 1400
+F 0 "U33" H 1675 1667 50  0000 C CNN
+F 1 "74LVC1G00" H 1675 1576 50  0000 C CNN
+F 2 "alexios:SOT-23-5_HandSoldering" H 1400 1400 50  0001 C CNN
+F 3 "https://assets.nexperia.com/documents/data-sheet/74LVC1G00.pdf" H 1400 1400 50  0001 C CNN
+	1    1750 1400
 	1    0    0    -1
 $EndComp
@@
 Text Label 7500 5550 2    50   ~ 0
 FPD[0..7]
-Wire Wire Line
-	4100 1100 4400 1100
-Wire Wire Line
-	4100 1200 4400 1200
-Wire Wire Line
-	4100 1300 4400 1300
-Wire Wire Line
-	4100 1400 4400 1400
-Wire Wire Line
-	4100 1500 4400 1500
-Text Label 4400 1100 2    50   ~ 0
+Text Label 4300 1100 2    50   ~ 0
 ~ROW1
-Text Label 4400 1200 2    50   ~ 0
+Text Label 4300 1200 2    50   ~ 0
 ~ROW2
-Text Label 4400 1300 2    50   ~ 0
+Text Label 4300 1300 2    50   ~ 0
 ~ROW3
-Text Label 4400 1400 2    50   ~ 0
+Text Label 4300 1400 2    50   ~ 0
 ~ROW4
-Text Label 4400 1500 2    50   ~ 0
+Text Label 4300 1500 2    50   ~ 0
 ~ROW5
 Text HLabel 1200 6550 0    50   Input ~ 0
@@
 Wire Wire Line
 	1300 6550 1800 6550
+NoConn ~ 3450 1600
+$Comp
+L alexios:74HC138 U34
+U 1 1 6AFE3EEE
+P 2950 1500
+F 0 "U34" H 2950 2167 50  0000 C CNN
+F 1 "74HC138" H 2950 2076 50  0000 C CNN
+F 2 "alexios:DIP-16_W7.62mm_Socket" H 2950 1500 50  0001 C CNN
+F 3 "https://assets.nexperia.com/documents/data-sheet/74HC_HCT138.pdf" H 2950 1500 50  0001 C CNN
+F 4 "Yes" H 2875 675 50  0001 C CNN "Verified"
+	1    2950 1500
+	1    0    0    -1
+$EndComp
+Wire Wire Line
+	3450 1500 3550 1500
+Wire Wire Line
+	3450 1100 3550 1100
+Wire Wire Line
+	3450 1200 3550 1200
+Wire Wire Line
+	3450 1300 3550 1300
+Wire Wire Line
+	3450 1400 3550 1400
+$Comp
+L Device:R_Small R?
+U 1 1 64196A39
+P 3650 1100
+AR Path="/614F5B8D/64196A39" Ref="R?"  Part="1"
+AR Path="/65BD1B6F/64196A39" Ref="R901"  Part="1"
+F 0 "R901" V 3600 1200 50  0000 L CNN
+F 1 "1kΩ?" V 3550 1100 50  0000 C CNN
+F 2 "alexios:R_SMD_0805_2012Metric_Pad1.15x1.40mm_HandSolder" H 3650 1100 50  0001 C CNN
+F 3 "~" H 3650 1100 50  0001 C CNN
+	1    3650 1100
+	0    1    1    0
+$EndComp
+Wire Wire Line
+	3750 1100 4300 1100
+$Comp
+L Device:R_Small R?
+U 1 1 642B7233
+P 3650 1200
+AR Path="/614F5B8D/642B7233" Ref="R?"  Part="1"
+AR Path="/65BD1B6F/642B7233" Ref="R902"  Part="1"
+F 0 "R902" V 3600 1300 50  0000 L CNN
+F 1 "1kΩ?" V 3550 1200 50  0001 C CNN
+F 2 "alexios:R_SMD_0805_2012Metric_Pad1.15x1.40mm_HandSolder" H 3650 1200 50  0001 C CNN
+F 3 "~" H 3650 1200 50  0001 C CNN
+	1    3650 1200
+	0    1    1    0
+$EndComp
+Wire Wire Line
+	3750 1200 4300 1200
+Wire Wire Line
+	3750 1300 4300 1300
+Wire Wire Line
+	3750 1400 4300 1400
+Wire Wire Line
+	3750 1500 4300 1500
+$Comp
+L Device:R_Small R?
+U 1 1 644F91ED
+P 3650 1300
+AR Path="/614F5B8D/644F91ED" Ref="R?"  Part="1"
+AR Path="/65BD1B6F/644F91ED" Ref="R903"  Part="1"
+F 0 "R903" V 3600 1400 50  0000 L CNN
+F 1 "1kΩ?" V 3550 1300 50  0001 C CNN
+F 2 "alexios:R_SMD_0805_2012Metric_Pad1.15x1.40mm_HandSolder" H 3650 1300 50  0001 C CNN
+F 3 "~" H 3650 1300 50  0001 C CNN
+	1    3650 1300
+	0    1    1    0
+$EndComp
+$Comp
+L Device:R_Small R?
+U 1 1 644F9382
+P 3650 1400
+AR Path="/614F5B8D/644F9382" Ref="R?"  Part="1"
+AR Path="/65BD1B6F/644F9382" Ref="R904"  Part="1"
+F 0 "R904" V 3600 1500 50  0000 L CNN
+F 1 "1kΩ?" V 3550 1400 50  0001 C CNN
+F 2 "alexios:R_SMD_0805_2012Metric_Pad1.15x1.40mm_HandSolder" H 3650 1400 50  0001 C CNN
+F 3 "~" H 3650 1400 50  0001 C CNN
+	1    3650 1400
+	0    1    1    0
+$EndComp
+$Comp
+L Device:R_Small R?
+U 1 1 644F94C4
+P 3650 1500
+AR Path="/614F5B8D/644F94C4" Ref="R?"  Part="1"
+AR Path="/65BD1B6F/644F94C4" Ref="R905"  Part="1"
+F 0 "R905" V 3600 1600 50  0000 L CNN
+F 1 "1kΩ?" V 3550 1500 50  0001 C CNN
+F 2 "alexios:R_SMD_0805_2012Metric_Pad1.15x1.40mm_HandSolder" H 3650 1500 50  0001 C CNN
+F 3 "~" H 3650 1500 50  0001 C CNN
+	1    3650 1500
+	0    1    1    0
+$EndComp
 Wire Bus Line
-	2700 800  2700 1800
+	2050 800  2050 1800
 Wire Bus Line
 	3150 4700 3150 5450

Commit message: Add decoder GALs and route signals.
Parts:
- removed C56, C57, C60: 100nF, alexios:C_SMD_0805_2012Metric_Pad1.15x1.40mm_HandSolder, symbol Device:C_Small
- removed U35: 74LVC1G04, alexios:SOT-23-5_HandSoldering, symbol alexios:74LVC1G04
- removed U36, U37: 74HC154, alexios:DIP-24_W7.62mm_Socket, symbol alexios:74HC154
- removed U39: 74HC139, alexios:DIP-16_W7.62mm_Socket, symbol alexios:74HC139
- added C1901, C1902, C1903, C1904: 100nF, alexios:C_SMD_0805_2012Metric_Pad1.15x1.40mm_HandSolder, symbol Device:C_Small
- added U1901, U1902, U1903, U1904: ATF16V8B, alexios:DIP-20_W7.62mm_Socket, symbol alexios:ATF16V8B
Connections:
- net labels added: FPA5
- wire segments 108 -> 176
- no-connect marks 5 -> 9
Other:
- note added: "Note: discontinuity here"

Commit message: Route DFP board
Other:
- moved on the sheet: C1901, C1902, C1903, C1904, U1901B, U1902B, U1903B, U1904B

Commit message: Route DFP board
Parts:
- renumbered C59 to C38
Changed lines of the file:
@@
 $Descr A4 11693 8268
 encoding utf-8
-Sheet 19 20
+Sheet 18 19
 Title "Front Panel Light Scanner"
 Date "2019-11-17"
@@
 AR Path="/60757845/607964B6/6AEB8989" Ref="C?"  Part="1"
 AR Path="/64FC7999/650046D0/6AEB8989" Ref="C?"  Part="1"
-AR Path="/65BD1B6F/6AEB8989" Ref="C59"  Part="1"
-F 0 "C59" H 4309 6146 50  0000 R CNN
+AR Path="/65BD1B6F/6AEB8989" Ref="C38"  Part="1"
+F 0 "C38" H 4309 6146 50  0000 R CNN
 F 1 "100nF" H 4309 6055 50  0000 R CNN
 F 2 "alexios:C_SMD_0805_2012Metric_Pad1.15x1.40mm_HandSolder" H 4400 6100 50  0001 C CNN

Commit message: Route DFP board
Parts:
- renumbered C54 to C33, C55 to C34
Connections:
- net labels added: ~AUTOSCAN
- net labels removed: ~SCANEN
- wire segments 176 -> 166
Changed lines of the file:
@@
 AR Path="/60757845/607964B6/62ECDEB3" Ref="C?"  Part="1"
 AR Path="/64FC7999/650046D0/62ECDEB3" Ref="C?"  Part="1"
-AR Path="/65BD1B6F/62ECDEB3" Ref="C54"  Part="1"
-F 0 "C54" H 5709 6196 50  0000 R CNN
+AR Path="/65BD1B6F/62ECDEB3" Ref="C33"  Part="1"
+F 0 "C33" H 5709 6196 50  0000 R CNN
 F 1 "100nF" H 5709 6105 50  0000 R CNN
 F 2 "alexios:C_SMD_0805_2012Metric_Pad1.15x1.40mm_HandSolder" H 5800 6150 50  0001 C CNN
@@
 AR Path="/60757845/607964B6/62EDD3ED" Ref="C?"  Part="1"
 AR Path="/64FC7999/650046D0/62EDD3ED" Ref="C?"  Part="1"
-AR Path="/65BD1B6F/62EDD3ED" Ref="C55"  Part="1"
-F 0 "C55" H 5709 6946 50  0000 R CNN
+AR Path="/65BD1B6F/62EDD3ED" Ref="C34"  Part="1"
+F 0 "C34" H 5709 6946 50  0000 R CNN
 F 1 "100nF" H 5709 6855 50  0000 R CNN
 F 2 "alexios:C_SMD_0805_2012Metric_Pad1.15x1.40mm_HandSolder" H 5800 6900 50  0001 C CNN
@@
 Wire Notes Line width 24 style solid
 	450  3000 450  900
-Text Label 1100 1450 0    50   ~ 0
-~SCANEN
-Text Label 1100 1350 0    50   ~ 0
+Text Label 1050 1450 0    50   ~ 0
+~AUTOSCAN
+Text Label 1050 1350 0    50   ~ 0
 ~WR
 Text HLabel 1000 1450 0    50   Input ~ 0
-~SCANEN
+~AUTOSCAN
 Text HLabel 1000 1350 0    50   Input ~ 0
 ~WR
@@
 Wire Wire Line
 	2800 6450 3250 6450
-Text Label 1500 7350 0    50   ~ 0
-~FPOE14
-Wire Wire Line
-	1800 7350 1500 7350
-Text Label 1500 6750 0    50   ~ 0
-~FPOE13
-Text Label 1500 7150 0    50   ~ 0
-MFD1
-Text Label 1500 7050 0    50   ~ 0
-MFD0
-Text Label 1500 6550 0    50   ~ 0
-MFD1
-Text Label 1500 6450 0    50   ~ 0
-MFD0
-Wire Wire Line
-	1800 6750 1500 6750
-Wire Wire Line
-	1200 6550 1300 6550
 Text HLabel 3250 6450 2    50   Output ~ 0
 ~ORHOE
@@
 Text HLabel 3250 7250 2    50   Output ~ 0
 ~FPSPLOE~
-Wire Wire Line
-	1400 6450 1400 7050
-Wire Wire Line
-	1400 7050 1800 7050
-Connection ~ 1400 6450
-Wire Wire Line
-	1400 6450 1800 6450
-Wire Wire Line
-	1300 7150 1800 7150
 Text Notes 6100 800  0    100  ~ 20
 Front-Panel Address Decoder
@@
 Text HLabel 1200 6550 0    50   Input ~ 0
 MFD1
-Wire Wire Line
-	1200 6450 1400 6450
-Wire Wire Line
-	1300 6550 1300 7150
-Connection ~ 1300 6550
-Wire Wire Line
-	1300 6550 1800 6550
 NoConn ~ 3450 1600
 $Comp
@@
 Wire Wire Line
 	4900 11300 4150 11300
+Text Label 3950 12950 2    50   ~ 0
+~FPOE15
+Text Label 3950 13050 2    50   ~ 0
+~FPOE16
+Entry Wire Line
+	3950 12650 4050 12550
+Text Label 3950 12650 2    50   ~ 0
+~FPOE12
 Wire Bus Line
 	2050 800  2050 1800
@@
 Wire Bus Line
 	6750 1200 6750 4850
-Text Label 3950 12950 2    50   ~ 0
-~FPOE15
-Text Label 3950 13050 2    50   ~ 0
-~FPOE16
-Entry Wire Line
-	3950 12650 4050 12550
-Text Label 3950 12650 2    50   ~ 0
-~FPOE12
 $EndSCHEMATC

Commit message: Rearrange front panel modules, add MFD2 and AB/DB to panel v.11
Connections:
- wire segments 166 -> 164
- no-connect marks 9 -> 5
Other:
- note added: "Checked for Panel v.11."
Changed lines of the file:
@@
 	4450 3150 4450 1950
 Wire Wire Line
-	1400 5500 1800 5500
-Text Label 1400 4800 0    50   ~ 0
+	1350 5500 1800 5500
+Text Label 1350 4700 0    50   ~ 0
 ~LED-STOP
-Text Label 1400 4600 0    50   ~ 0
+Text Label 1350 5200 0    50   ~ 0
 ~RSTHOLD
-Text Label 1400 5200 0    50   ~ 0
+Text Label 1350 5300 0    50   ~ 0
 ~IRQS
-Text Label 1400 4700 0    50   ~ 0
+Text Label 1350 4600 0    50   ~ 0
 STEP∕~RUN
 Wire Wire Line
-	1750 5600 1750 5300
-Wire Wire Line
 	1800 5600 1750 5600
-Wire Wire Line
-	1750 5300 1800 5300
-Connection ~ 1750 5600
 Wire Wire Line
 	1750 5650 1750 5600
@@
 	1    0    0    -1
 $EndComp
-Text Label 1400 5100 0    50   ~ 0
+Text Label 1350 5000 0    50   ~ 0
 ~LED-EXEC
-Text Label 1400 5000 0    50   ~ 0
+Text Label 1350 4900 0    50   ~ 0
 ~LED-FETCH
-Text Label 1400 4900 0    50   ~ 0
+Text Label 1350 4800 0    50   ~ 0
 ~WS
 Text Label 3000 5300 2    50   ~ 0
@@
 Text Label 3000 4600 2    50   ~ 0
 FPD0
-Text Label 1400 5500 0    50   ~ 0
+Text Label 1350 5500 0    50   ~ 0
 ~FPOE16
 Text Notes 1500 4250 0    100  ~ 20
 State Lights (~FPOE16~)
 Wire Wire Line
-	1300 4600 1800 4600
-Wire Wire Line
-	1300 4700 1800 4700
-Wire Wire Line
-	1300 4800 1800 4800
-Wire Wire Line
-	1300 4900 1800 4900
-Wire Wire Line
-	1300 5000 1800 5000
-Wire Wire Line
-	1300 5100 1800 5100
-Wire Wire Line
-	1300 5200 1800 5200
-Text HLabel 1300 4600 0    50   Input ~ 0
+	1250 5200 1800 5200
+Wire Wire Line
+	1250 4600 1800 4600
+Wire Wire Line
+	1250 4700 1800 4700
+Wire Wire Line
+	1250 4800 1800 4800
+Wire Wire Line
+	1250 4900 1800 4900
+Wire Wire Line
+	1250 5000 1800 5000
+Wire Wire Line
+	1250 5300 1800 5300
+Text HLabel 1250 5200 0    50   Input ~ 0
 ~RSTHOLD
-Text HLabel 1300 4700 0    50   Input ~ 0
+Text HLabel 1250 4600 0    50   Input ~ 0
 STEP∕~RUN
-Text HLabel 1300 4800 0    50   Input ~ 0
+Text HLabel 1250 4700 0    50   Input ~ 0
 ~LED-STOP
-Text HLabel 1300 4900 0    50   Input ~ 0
+Text HLabel 1250 4800 0    50   Input ~ 0
 ~WS
-Text HLabel 1300 5000 0    50   Input ~ 0
+Text HLabel 1250 4900 0    50   Input ~ 0
 ~LED-FETCH
-Text HLabel 1300 5100 0    50   Input ~ 0
+Text HLabel 1250 5000 0    50   Input ~ 0
 ~LED-EXEC
-Text HLabel 1300 5200 0    50   Input ~ 0
+Text HLabel 1250 5300 0    50   Input ~ 0
 ~IRQS
 $Comp
@@
 Wire Wire Line
 	2400 9950 2750 9950
-Text Label 2400 10350 0    50   ~ 0
-~PANELEN
 Wire Wire Line
 	2750 9650 2400 9650
@@
 Text Label 2400 9650 0    50   ~ 0
 FPA1
-Wire Wire Line
-	2400 10350 2750 10350
 Wire Wire Line
 	2750 10050 2400 10050
@@
 Wire Wire Line
 	2400 11500 2750 11500
-Text Label 2400 11900 0    50   ~ 0
-~PANELEN
 Wire Wire Line
 	2750 11200 2400 11200
@@
 Text Label 2400 11200 0    50   ~ 0
 FPA1
-Wire Wire Line
-	2400 11900 2750 11900
 Wire Wire Line
 	2750 11600 2400 11600
@@
 Wire Wire Line
 	2400 13050 2750 13050
-Text Label 2400 13450 0    50   ~ 0
-~PANELEN
 Wire Wire Line
 	2750 12750 2400 12750
@@
 FPA1
 Wire Wire Line
-	2400 13450 2750 13450
-Wire Wire Line
 	2750 13150 2400 13150
 Text Label 2400 13150 0    50   ~ 0
@@
 Text Label 2400 13250 0    50   ~ 0
 MFD0
-Text Label 2400 13350 0    50   ~ 0
-MFD1
 Wire Wire Line
 	2750 13350 2400 13350
@@
 Wire Wire Line
 	2400 14650 2750 14650
-Text Label 2400 15050 0    50   ~ 0
-~PANELEN
 Wire Wire Line
 	2750 14350 2400 14350
@@
 Text Label 2400 14350 0    50   ~ 0
 FPA1
-Wire Wire Line
-	2400 15050 2750 15050
 Wire Wire Line
 	2750 14750 2400 14750
@@
 Entry Wire Line
 	3950 14350 4050 14250
-NoConn ~ 2750 10450
-NoConn ~ 2750 12000
-NoConn ~ 2750 13550
-NoConn ~ 2750 15150
 Text Notes 4100 11500 0    50   ~ 0
 Note: discontinuity here
@@
 Text Label 3950 12650 2    50   ~ 0
 ~FPOE12
+$Comp
+L power:+5V #PWR0128
+U 1 1 61BD34DB
+P 1800 5100
+F 0 "#PWR0128" H 1800 4950 50  0001 C CNN
+F 1 "+5V" V 1815 5228 50  0000 L CNN
+F 2 "" H 1800 5100 50  0001 C CNN
+F 3 "" H 1800 5100 50  0001 C CNN
+	1    1800 5100
+	0    -1   -1   0
+$EndComp
+Text Notes 2000 5800 0    50   ~ 0
+Checked for Panel v.11.
+Text Label 2400 13350 0    50   ~ 0
+MFD1
+Wire Wire Line
+	2400 15050 2750 15050
+Text Label 2400 15050 0    50   ~ 0
+~PANELEN
+Wire Wire Line
+	2400 13450 2750 13450
+Text Label 2400 13450 0    50   ~ 0
+~PANELEN
+Wire Wire Line
+	2400 11900 2750 11900
+Text Label 2400 11900 0    50   ~ 0
+~PANELEN
 Wire Bus Line
-	2050 800  2050 1800
+	4050 9350 4050 14850
 Wire Bus Line
 	3150 4700 3150 5450
@@
 	4600 800  4600 3250
 Wire Bus Line
-	4050 9350 4050 14850
+	6750 1200 6750 4850
 Wire Bus Line
-	6750 1200 6750 4850
+	2050 800  2050 1800
+Wire Wire Line
+	2400 10350 2750 10350
+Text Label 2400 10350 0    50   ~ 0
+~PANELEN
 $EndSCHEMATC
