File: kicad/cft/cft-backplane/cft-backplane.kicad_pcb (KiCad board)
At the start: 4 copper layers, 131.9 x 165.1 mm, 73 parts, among them J1 Conn_02x20_Top_Bottom, J10 Conn_02x04_Top_Bottom, J11 Conn_01x04, J12 Conn_01x04, J13 Conn_01x04, J14 Conn_01x04, J15 Conn_01x03, J2 Conn_02x20_Top_Bottom, J3 Conn_02x20_Top_Bottom, J4 Conn_02x20_Top_Bottom, J5 Conn_02x20_Top_Bottom, J6 Conn_02x20_Top_Bottom, J7 Conn_02x20_Top_Bottom, J8 Conn_02x20_Top_Bottom, J9 Conn_02x02_Top_Bottom

Commit message: Added Mini-Fit Jr. 3D models.
Parts:
- moved REF** 4.44 mm to (155.1, 75.1)
Changed lines of the file:
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@@
-(kicad_pcb (version 20171130) (host pcbnew 5.1.2-f72e74a~84~ubuntu18.04.1)
+(kicad_pcb (version 20171130) (host pcbnew 5.1.4-e60b266~84~ubuntu18.04.1)
   (general
     (thickness 1.6)
@@
     (35 F.Paste user hide)
     (36 B.SilkS user)
-    (37 F.SilkS user hide)
+    (37 F.SilkS user)
     (38 B.Mask user hide)
     (39 F.Mask user)
@@
   )
   (module Symbol:WEEE-Logo_5.6x8mm_SilkScreen (layer B.Cu)
-    (at 155.095 70.7 180)
+    (at 155.06 75.14 180)
     (descr "Waste Electrical and Electronic Equipment Directive")
     (tags "Logo WEEE")
@@
       (rotate (xyz 0 0 0))
     )
+    (model /home/alexios/PROJECTS/HARDWARE/cft/kicad/alexios.pretty/Molex_Mini-Fit_Jr_5566-04A2_2x02_P4.20mm_Vertical.wrl
+      (offset (xyz 2.1 -2.55 0))
+      (scale (xyz 0.395 0.395 0.395))
+      (rotate (xyz 0 0 0))
+    )
   )
   (module Connector_IDC:IDC-Header_2x20_P2.54mm_Vertical (layer B.Cu)
@@
     (pad "" np_thru_hole circle (at -4.7 -5.04 270) (size 3 3) (drill 3) (layers *.Cu *.Mask))
     (pad "" np_thru_hole circle (at 17.3 -5.04 270) (size 3 3) (drill 3) (layers *.Cu *.Mask))
-    (model ${KISYS3DMOD}/Connector_Molex.3dshapes/Molex_Mini-Fit_Jr_5566-08A2_2x04_P4.20mm_Vertical.wrl
-      (at (xyz 0 0 0))
-      (scale (xyz 1 1 1))
-      (rotate (xyz 0 0 0))
+    (model /home/alexios/PROJECTS/HARDWARE/cft/kicad/alexios.pretty/Molex_Mini-Fit_Jr_5566-08A2_2x04_P4.20mm_Vertical.wrl
+      (offset (xyz 6.3 -2.6 0))
+      (scale (xyz 0.395 0.395 0.395))
+      (rotate (xyz 0 0 180))
     )
   )

Commit message: Revision 1922 has a short. Fixed issue and stepped revision.
Parts:
- removed G*** (x2): LOGO, alexios:CFT
- removed REF** (x2): SIGNATURESILK, alexios:SIGNATURE
- removed REF** (x12): MountingHole_2.2mm_M2, MountingHole:MountingHole_2.2mm_M2
- removed REF**: WEEE-Logo_5.6x8mm_SilkScreen, Symbol:WEEE-Logo_5.6x8mm_SilkScreen
- removed REF**: QRCODE-CFT, alexios:QRCODE-CFT
- removed REF** (x6): MountingHole_3.2mm_M3_DIN965, MountingHole:MountingHole_3.2mm_M3_DIN965
- removed REF** (x2): OSHW-Logo2_14.6x12mm_SilkScreen, Symbol:OSHW-Logo2_14.6x12mm_SilkScreen
Connections:
- SLOT1 pad A73: /Slot/A72 -> /Slot/A73
- SLOT2 pad A73: /Slot/A72 -> /Slot/A73
- SLOT3 pad A73: /Slot/A72 -> /Slot/A73
- SLOT4 pad A73: /Slot/A72 -> /Slot/A73
- SLOT5 pad A73: /Slot/A72 -> /Slot/A73
- SLOT6 pad A73: /Slot/A72 -> /Slot/A73
- SLOT7 pad A73: /Slot/A72 -> /Slot/A73
- SLOT8 pad A73: /Slot/A72 -> /Slot/A73
Routing:
- net /Slot/A72: track 310.4 -> 154.5 mm
- net /Slot/A73: track 0.00 -> 154.4 mm
Other:
- board text added: "1945"

Commit message: Documenting Backplane issue with pins A72 and A73.
Connections:
- SLOT1 pad A72: /Slot/A72 -> GND
- SLOT1 pad A73: /Slot/A73 -> GND
- SLOT2 pad A72: /Slot/A72 -> GND
- SLOT2 pad A73: /Slot/A73 -> GND
- SLOT3 pad A72: /Slot/A72 -> GND
- SLOT3 pad A73: /Slot/A73 -> GND
- SLOT4 pad A72: /Slot/A72 -> GND
- SLOT4 pad A73: /Slot/A73 -> GND
- SLOT5 pad A72: /Slot/A72 -> GND
- SLOT5 pad A73: /Slot/A73 -> GND
- SLOT6 pad A72: /Slot/A72 -> GND
- SLOT6 pad A73: /Slot/A73 -> GND
- SLOT7 pad A72: /Slot/A72 -> GND
- SLOT7 pad A73: /Slot/A73 -> GND
- SLOT8 pad A72: /Slot/A72 -> GND
- SLOT8 pad A73: /Slot/A73 -> GND
Routing:
- net /Slot/A72: track 154.5 -> 0.00 mm
- net /Slot/A73: track 154.4 -> 0.00 mm
- net GND: track 0.00 -> 44.1 mm
- net /Slot/B73: track 171.5 -> 170.1 mm
- net /Slot/B69: track 164.4 -> 163.0 mm
- net /Slot/B65: track 158.2 -> 156.8 mm
Other:
- board text added: "CFT 8-Slot Backplane"
- board text added: "Caution"
- board text added: "This revision connects pins A72 and A73 to ground. This was done because of an error in revision 1922 where two pins were shorted by a misplaced segment of copper in layer 3."

Commit message: Added missing parts to revision 1945
Parts:
- added G***: LOGO, alexios:CFT, F.Cu at (40.0, 77.8)
- added REF**: OSHW-Logo2_14.6x12mm_SilkScreen, Symbol:OSHW-Logo2_14.6x12mm_SilkScreen, B.Cu at (44.0, 52.9)
- added REF**: MountingHole_2.2mm_M2, MountingHole:MountingHole_2.2mm_M2, F.Cu at (152.6, 148.5)
- added REF**: MountingHole_2.2mm_M2, MountingHole:MountingHole_2.2mm_M2, F.Cu at (146.6, 28.5)
- added REF**: MountingHole_2.2mm_M2, MountingHole:MountingHole_2.2mm_M2, F.Cu at (146.6, 68.5)
- added REF**: MountingHole_2.2mm_M2, MountingHole:MountingHole_2.2mm_M2, F.Cu at (146.6, 128.5)
- added REF**: MountingHole_2.2mm_M2, MountingHole:MountingHole_2.2mm_M2, F.Cu at (146.6, 148.5)
- added REF**: MountingHole_2.2mm_M2, MountingHole:MountingHole_2.2mm_M2, F.Cu at (146.6, 168.5)
- added REF**: MountingHole_2.2mm_M2, MountingHole:MountingHole_2.2mm_M2, F.Cu at (152.6, 168.5)
- added REF**: WEEE-Logo_5.6x8mm_SilkScreen, Symbol:WEEE-Logo_5.6x8mm_SilkScreen, B.Cu at (155.1, 75.1)
- added REF**: QRCODE-CFT, alexios:QRCODE-CFT, B.Cu at (50.3, 40.3)
- added REF**: MountingHole_3.2mm_M3_DIN965, MountingHole:MountingHole_3.2mm_M3_DIN965, F.Cu at (157.3, 107.9)
- added REF**: OSHW-Logo2_14.6x12mm_SilkScreen, Symbol:OSHW-Logo2_14.6x12mm_SilkScreen, F.Cu at (39.5, 31.3)
- added REF**: MountingHole_3.2mm_M3_DIN965, MountingHole:MountingHole_3.2mm_M3_DIN965, F.Cu at (35.7, 179.4)
- added REF**: MountingHole_3.2mm_M3_DIN965, MountingHole:MountingHole_3.2mm_M3_DIN965, F.Cu at (37.6, 107.9)
- added REF**: MountingHole_3.2mm_M3_DIN965, MountingHole:MountingHole_3.2mm_M3_DIN965, F.Cu at (37.6, 47.9)
- added REF**: MountingHole_3.2mm_M3_DIN965, MountingHole:MountingHole_3.2mm_M3_DIN965, F.Cu at (157.3, 47.9)
- added REF**: MountingHole_3.2mm_M3_DIN965, MountingHole:MountingHole_3.2mm_M3_DIN965, F.Cu at (157.3, 179.4)
- added REF**: SIGNATURESILK, alexios:SIGNATURE, F.Cu at (149.4, 141.8)
- added REF**: SIGNATURESILK, alexios:SIGNATURE, B.Cu at (159.8, 38.4)
- added REF**: MountingHole_2.2mm_M2, MountingHole:MountingHole_2.2mm_M2, F.Cu at (146.6, 88.5)
- added REF**: MountingHole_2.2mm_M2, MountingHole:MountingHole_2.2mm_M2, F.Cu at (152.6, 88.5)
- added REF**: MountingHole_2.2mm_M2, MountingHole:MountingHole_2.2mm_M2, F.Cu at (152.6, 28.5)
- added REF**: MountingHole_2.2mm_M2, MountingHole:MountingHole_2.2mm_M2, F.Cu at (152.6, 68.5)
- added REF**: MountingHole_2.2mm_M2, MountingHole:MountingHole_2.2mm_M2, F.Cu at (152.6, 128.5)
Other:
- board text added: "CFT Backplane 2 Rev B"
- board text added: "CFT Backplane 2.1"
- board text removed: "CFT Backplane 2 Rev A"
- board text removed: "CFT Backplane 2.0"

Commit message: Updating schematics with new page layout.
Other:
- board text removed: "CFT 8-Slot Backplane"
Changed lines of the file:
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@@
-(kicad_pcb (version 20171130) (host pcbnew 5.1.4-e60b266~84~ubuntu18.04.1)
+(kicad_pcb (version 20171130) (host pcbnew 5.0.2+dfsg1-1~bpo9+1)
   (general
     (thickness 1.6)
-    (drawings 266)
+    (drawings 265)
     (tracks 8341)
     (zones 0)
@@
   (title_block
     (title "CFT 8 Slot Backplane")
+    (date 2019-11-13)
+    (rev 1945)
+    (comment 1 BPL)
+    (comment 2 "1922: Manufactured, A72 & A73 shorted by mistake.")
+    (comment 3 "1945: Reassigns A72 & A73 to GND")
   )
   (layers
@@
     (46 B.CrtYd user)
     (47 F.CrtYd user)
-    (48 B.Fab user)
-    (49 F.Fab user)
+    (48 B.Fab user hide)
+    (49 F.Fab user hide)
   )
   (setup
@@
     (zone_45_only yes)
     (trace_min 0.127)
+    (segment_width 0.2)
+    (edge_width 0.05)
     (via_size 0.6096)
     (via_drill 0.4)
@@
     (uvia_min_size 0.2)
     (uvia_min_drill 0.1)
-    (edge_width 0.05)
-    (segment_width 0.2)
     (pcb_text_width 0.3)
     (pcb_text_size 1.5 1.5)
@@
     (effects (font (size 3 3) (thickness 0.6)))
   )
-  (gr_text "CFT 8-Slot Backplane" (at 223.43 174.38) (layer Dwgs.User)
-    (effects (font (size 5 5) (thickness 1)))
-  )
   (gr_line (start 155.984 151.726) (end 155.984 143.471) (layer F.SilkS) (width 0.3048))
