File: kicad/cft/cft-backplane/slot.sch (KiCad schematic (older format))
At the start: 1 part, among them J1 DIN-41612-3x32-Bauform-C

Commit message: Work on backplane
Parts:
- added H1, H2: MountingHole_Pad, MountingHole:MountingHole_2.7mm_M2.5_ISO14580_Pad, symbol Mechanical:MountingHole_Pad
Connections:
- new net GND: H1.1, H2.1
Changed lines of the file:
@@
 $Descr A4 11693 8268
 encoding utf-8
-Sheet 2 13
+Sheet 3 13
 Title ""
 Date ""
@@
 AR Path="/85A9A356/66BD4109" Ref="J11"  Part="1"
 AR Path="/85AAD6B0/66BD4109" Ref="J12"  Part="1"
-F 0 "J1" H 4950 5100 50  0000 C CNN
+F 0 "J2" H 4950 5100 50  0000 C CNN
 F 1 "DIN-41612-3x32-Bauform-C" H 4800 1600 50  0000 L CNN
 F 2 "alexios:DIN41612_C_3x32_Female_Vertical_THT" H 4925 0   50  0001 C CNN
@@
 	1    0    0    -1
 $EndComp
-Text Label 4500 5000 0    50   ~ 0
-A32
-Text Label 4500 4900 0    50   ~ 0
-A31
 Text Label 4500 4800 0    50   ~ 0
 A30
@@
 AR Path="/85A9A356/6DF9D4CB" Ref="J11"  Part="3"
 AR Path="/85AAD6B0/6DF9D4CB" Ref="J12"  Part="3"
-F 0 "J1" H 7250 5100 50  0000 L CNN
+F 0 "J2" H 7250 5100 50  0000 L CNN
 F 1 "DIN-41612-3x32-Bauform-C" H 7530 3305 50  0001 L CNN
 F 2 "alexios:DIN41612_C_3x32_Female_Vertical_THT" H 7325 0   50  0001 C CNN
@@
 AR Path="/85A9A356/6D6BB2B9" Ref="J11"  Part="2"
 AR Path="/85AAD6B0/6D6BB2B9" Ref="J12"  Part="2"
-F 0 "J1" H 6150 5100 50  0000 C CNN
+F 0 "J2" H 6150 5100 50  0000 C CNN
 F 1 "DIN-41612-3x32-Bauform-C" H 6330 3305 50  0001 L CNN
 F 2 "alexios:DIN41612_C_3x32_Female_Vertical_THT" H 6125 0   50  0001 C CNN
@@
 $EndComp
 Wire Wire Line
-	4500 5000 4650 5000
-Wire Wire Line
-	4500 4900 4650 4900
-Wire Wire Line
 	4500 4800 4650 4800
 Wire Wire Line
@@
 Entry Wire Line
 	4400 4600 4500 4700
-Entry Wire Line
-	4400 4700 4500 4800
-Entry Wire Line
-	4400 4800 4500 4900
-Entry Wire Line
-	4400 4900 4500 5000
 Entry Wire Line
 	5600 1800 5700 1900
@@
 Text HLabel 6550 1500 0    50   UnSpc ~ 0
 C[1..32]
+$Comp
+L Mechanical:MountingHole_Pad H1
+U 1 1 85E2059E
+P 9050 2050
+AR Path="/6199673B/85E2059E" Ref="H1"  Part="1"
+AR Path="/859EF273/85E2059E" Ref="H3"  Part="1"
+AR Path="/85A02236/85E2059E" Ref="H5"  Part="1"
+AR Path="/85A150E4/85E2059E" Ref="H7"  Part="1"
+AR Path="/85A27F74/85E2059E" Ref="H9"  Part="1"
+AR Path="/85A3ADD9/85E2059E" Ref="H11"  Part="1"
+AR Path="/85A4DD82/85E2059E" Ref="H13"  Part="1"
+AR Path="/85A60DD6/85E2059E" Ref="H15"  Part="1"
+AR Path="/85A73EB4/85E2059E" Ref="H17"  Part="1"
+AR Path="/85A8707D/85E2059E" Ref="H19"  Part="1"
+AR Path="/85A9A356/85E2059E" Ref="H21"  Part="1"
+AR Path="/85AAD6B0/85E2059E" Ref="H23"  Part="1"
+F 0 "H3" H 9150 2099 50  0000 L CNN
+F 1 "MountingHole_Pad" H 9150 2008 50  0000 L CNN
+F 2 "MountingHole:MountingHole_2.7mm_M2.5_ISO14580_Pad" H 9050 2050 50  0001 C CNN
+F 3 "~" H 9050 2050 50  0001 C CNN
+	1    9050 2050
+	1    0    0    -1
+$EndComp
+$Comp
+L power:GND #PWR05
+U 1 1 85E20FCF
+P 9050 2150
+AR Path="/6199673B/85E20FCF" Ref="#PWR05"  Part="1"
+AR Path="/859EF273/85E20FCF" Ref="#PWR07"  Part="1"
+AR Path="/85A02236/85E20FCF" Ref="#PWR09"  Part="1"
+AR Path="/85A150E4/85E20FCF" Ref="#PWR011"  Part="1"
+AR Path="/85A27F74/85E20FCF" Ref="#PWR013"  Part="1"
+AR Path="/85A3ADD9/85E20FCF" Ref="#PWR015"  Part="1"
+AR Path="/85A4DD82/85E20FCF" Ref="#PWR017"  Part="1"
+AR Path="/85A60DD6/85E20FCF" Ref="#PWR019"  Part="1"
+AR Path="/85A73EB4/85E20FCF" Ref="#PWR021"  Part="1"
+AR Path="/85A8707D/85E20FCF" Ref="#PWR023"  Part="1"
+AR Path="/85A9A356/85E20FCF" Ref="#PWR025"  Part="1"
+AR Path="/85AAD6B0/85E20FCF" Ref="#PWR027"  Part="1"
+F 0 "#PWR07" H 9050 1900 50  0001 C CNN
+F 1 "GND" H 9055 1977 50  0000 C CNN
+F 2 "" H 9050 2150 50  0001 C CNN
+F 3 "" H 9050 2150 50  0001 C CNN
+	1    9050 2150
+	1    0    0    -1
+$EndComp
+$Comp
+L Mechanical:MountingHole_Pad H2
+U 1 1 85E2263F
+P 9050 2550
+AR Path="/6199673B/85E2263F" Ref="H2"  Part="1"
+AR Path="/859EF273/85E2263F" Ref="H4"  Part="1"
+AR Path="/85A02236/85E2263F" Ref="H6"  Part="1"
+AR Path="/85A150E4/85E2263F" Ref="H8"  Part="1"
+AR Path="/85A27F74/85E2263F" Ref="H10"  Part="1"
+AR Path="/85A3ADD9/85E2263F" Ref="H12"  Part="1"
+AR Path="/85A4DD82/85E2263F" Ref="H14"  Part="1"
+AR Path="/85A60DD6/85E2263F" Ref="H16"  Part="1"
+AR Path="/85A73EB4/85E2263F" Ref="H18"  Part="1"
+AR Path="/85A8707D/85E2263F" Ref="H20"  Part="1"
+AR Path="/85A9A356/85E2263F" Ref="H22"  Part="1"
+AR Path="/85AAD6B0/85E2263F" Ref="H24"  Part="1"
+F 0 "H4" H 9150 2599 50  0000 L CNN
+F 1 "MountingHole_Pad" H 9150 2508 50  0000 L CNN
+F 2 "MountingHole:MountingHole_2.7mm_M2.5_ISO14580_Pad" H 9050 2550 50  0001 C CNN
+F 3 "~" H 9050 2550 50  0001 C CNN
+	1    9050 2550
+	1    0    0    -1
+$EndComp
+$Comp
+L power:GND #PWR06
+U 1 1 85E22645
+P 9050 2650
+AR Path="/6199673B/85E22645" Ref="#PWR06"  Part="1"
+AR Path="/859EF273/85E22645" Ref="#PWR08"  Part="1"
+AR Path="/85A02236/85E22645" Ref="#PWR010"  Part="1"
+AR Path="/85A150E4/85E22645" Ref="#PWR012"  Part="1"
+AR Path="/85A27F74/85E22645" Ref="#PWR014"  Part="1"
+AR Path="/85A3ADD9/85E22645" Ref="#PWR016"  Part="1"
+AR Path="/85A4DD82/85E22645" Ref="#PWR018"  Part="1"
+AR Path="/85A60DD6/85E22645" Ref="#PWR020"  Part="1"
+AR Path="/85A73EB4/85E22645" Ref="#PWR022"  Part="1"
+AR Path="/85A8707D/85E22645" Ref="#PWR024"  Part="1"
+AR Path="/85A9A356/85E22645" Ref="#PWR026"  Part="1"
+AR Path="/85AAD6B0/85E22645" Ref="#PWR028"  Part="1"
+F 0 "#PWR08" H 9050 2400 50  0001 C CNN
+F 1 "GND" H 9055 2477 50  0000 C CNN
+F 2 "" H 9050 2650 50  0001 C CNN
+F 3 "" H 9050 2650 50  0001 C CNN
+	1    9050 2650
+	1    0    0    -1
+$EndComp
+Entry Wire Line
+	4400 4700 4500 4800
 Wire Bus Line
-	4400 1600 4400 4900
+	6800 1600 6800 4900
 Wire Bus Line
 	5600 1600 5600 4900
 Wire Bus Line
-	6800 1600 6800 4900
+	4400 1600 4400 4900
+Entry Wire Line
+	4400 4800 4500 4900
+Entry Wire Line
+	4400 4900 4500 5000
+Wire Wire Line
+	4500 4900 4650 4900
+Wire Wire Line
+	4500 5000 4650 5000
+Text Label 4500 4900 0    50   ~ 0
+A31
+Text Label 4500 5000 0    50   ~ 0
+A32
 $EndSCHEMATC

Commit message: Work on backplane
Changed lines of the file:
@@
 $Descr A4 11693 8268
 encoding utf-8
-Sheet 3 13
+Sheet 2 13
 Title ""
 Date ""
@@
 AR Path="/85A9A356/66BD4109" Ref="J11"  Part="1"
 AR Path="/85AAD6B0/66BD4109" Ref="J12"  Part="1"
-F 0 "J2" H 4950 5100 50  0000 C CNN
+F 0 "J1" H 4950 5100 50  0000 C CNN
 F 1 "DIN-41612-3x32-Bauform-C" H 4800 1600 50  0000 L CNN
 F 2 "alexios:DIN41612_C_3x32_Female_Vertical_THT" H 4925 0   50  0001 C CNN
@@
 AR Path="/85A9A356/6DF9D4CB" Ref="J11"  Part="3"
 AR Path="/85AAD6B0/6DF9D4CB" Ref="J12"  Part="3"
-F 0 "J2" H 7250 5100 50  0000 L CNN
+F 0 "J1" H 7250 5100 50  0000 L CNN
 F 1 "DIN-41612-3x32-Bauform-C" H 7530 3305 50  0001 L CNN
 F 2 "alexios:DIN41612_C_3x32_Female_Vertical_THT" H 7325 0   50  0001 C CNN
@@
 AR Path="/85A9A356/6D6BB2B9" Ref="J11"  Part="2"
 AR Path="/85AAD6B0/6D6BB2B9" Ref="J12"  Part="2"
-F 0 "J2" H 6150 5100 50  0000 C CNN
+F 0 "J1" H 6150 5100 50  0000 C CNN
 F 1 "DIN-41612-3x32-Bauform-C" H 6330 3305 50  0001 L CNN
 F 2 "alexios:DIN41612_C_3x32_Female_Vertical_THT" H 6125 0   50  0001 C CNN
@@
 AR Path="/85A9A356/85E2059E" Ref="H21"  Part="1"
 AR Path="/85AAD6B0/85E2059E" Ref="H23"  Part="1"
-F 0 "H3" H 9150 2099 50  0000 L CNN
+F 0 "H1" H 9150 2099 50  0000 L CNN
 F 1 "MountingHole_Pad" H 9150 2008 50  0000 L CNN
 F 2 "MountingHole:MountingHole_2.7mm_M2.5_ISO14580_Pad" H 9050 2050 50  0001 C CNN
@@
 AR Path="/85A9A356/85E20FCF" Ref="#PWR025"  Part="1"
 AR Path="/85AAD6B0/85E20FCF" Ref="#PWR027"  Part="1"
-F 0 "#PWR07" H 9050 1900 50  0001 C CNN
+F 0 "#PWR027" H 9050 1900 50  0001 C CNN
 F 1 "GND" H 9055 1977 50  0000 C CNN
 F 2 "" H 9050 2150 50  0001 C CNN
@@
 AR Path="/85A9A356/85E2263F" Ref="H22"  Part="1"
 AR Path="/85AAD6B0/85E2263F" Ref="H24"  Part="1"
-F 0 "H4" H 9150 2599 50  0000 L CNN
+F 0 "H2" H 9150 2599 50  0000 L CNN
 F 1 "MountingHole_Pad" H 9150 2508 50  0000 L CNN
 F 2 "MountingHole:MountingHole_2.7mm_M2.5_ISO14580_Pad" H 9050 2550 50  0001 C CNN
@@
 AR Path="/85A9A356/85E22645" Ref="#PWR026"  Part="1"
 AR Path="/85AAD6B0/85E22645" Ref="#PWR028"  Part="1"
-F 0 "#PWR08" H 9050 2400 50  0001 C CNN
+F 0 "#PWR028" H 9050 2400 50  0001 C CNN
 F 1 "GND" H 9055 2477 50  0000 C CNN
 F 2 "" H 9050 2650 50  0001 C CNN
@@
 Entry Wire Line
 	4400 4700 4500 4800
+Entry Wire Line
+	4400 4800 4500 4900
+Entry Wire Line
+	4400 4900 4500 5000
+Wire Wire Line
+	4500 4900 4650 4900
+Wire Wire Line
+	4500 5000 4650 5000
+Text Label 4500 4900 0    50   ~ 0
+A31
+Text Label 4500 5000 0    50   ~ 0
+A32
 Wire Bus Line
 	6800 1600 6800 4900
@@
 Wire Bus Line
 	4400 1600 4400 4900
-Entry Wire Line
-	4400 4800 4500 4900
-Entry Wire Line
-	4400 4900 4500 5000
-Wire Wire Line
-	4500 4900 4650 4900
-Wire Wire Line
-	4500 5000 4650 5000
-Text Label 4500 4900 0    50   ~ 0
-A31
-Text Label 4500 5000 0    50   ~ 0
-A32
 $EndSCHEMATC

Commit message: Split backplanesl; route processor backplane
Parts:
- removed J1: DIN-41612-3x32-Bauform-C, alexios:DIN41612_C_3x32_Female_Vertical_THT, symbol alexios:DIN-41612-3x32-Bauform-C
- added J5: DIN-41612-3x32-Bauform-C, alexios:DIN41612_C_3x32_Female_Vertical_THT, symbol alexios:DIN-41612-3x32-Bauform-C
Connections:
- net A1: now also J5.A1
- net A2: now also J5.A2
- net A23: now also J5.A23
- net A24: now also J5.A24
- net A25: now also J5.A25
- net A26: now also J5.A26
- net A27: now also J5.A27
- net A28: now also J5.A28
- net A29: now also J5.A29
- net A30: now also J5.A30
- net A31: now also J5.A31
- net A32: now also J5.A32
- net B1: now also J5.B1
- net B10: now also J5.B10
- net B11: now also J5.B11
- net B12: now also J5.B12
- net B13: now also J5.B13
- net B14: now also J5.B14
- net B15: now also J5.B15
- net B16: now also J5.B16
- net B17: now also J5.B17
- net B18: now also J5.B18
- net B19: now also J5.B19
- net B2: now also J5.B2
- net B20: now also J5.B20
- net B21: now also J5.B21
- net B22: now also J5.B22
- net B3: now also J5.B3
- net B31: now also J5.B31
- net B32: now also J5.B32
- net B4: now also J5.B4
- net B5: now also J5.B5
- net B6: now also J5.B6
- net B7: now also J5.B7
- net B8: now also J5.B8
- net B9: now also J5.B9
- net C1: now also J5.C1
- net C10: now also J5.C10
- net C11: now also J5.C11
- net C13: now also J5.C13
- net C14: now also J5.C14
- net C15: now also J5.C15
- net C16: now also J5.C16
- net C17: now also J5.C17
- net C18: now also J5.C18
- net C19: now also J5.C19
- net C2: now also J5.C2
- net C20: now also J5.C20
- net C21: now also J5.C21
- net C22: now also J5.C22
- net C23: now also J5.C23
- net C24: now also J5.C24
- net C25: now also J5.C25
- net C26: now also J5.C26
- net C27: now also J5.C27
- net C28: now also J5.C28
- net C29: now also J5.C29
- net C3: now also J5.C3
- net C30: now also J5.C30
- net C31: now also J5.C31
- net C32: now also J5.C32
- net C4: now also J5.C4
- net C6: now also J5.C6
- net C7: now also J5.C7
- net C8: now also J5.C8
- net C9: now also J5.C9
- no-connect marks 0 -> 30

Commit message: Work on Peripheral Backplane
Connections:
- net B23: now reaches J5.B23
- net B24: now reaches J5.B24
- net B25: now reaches J5.B25
- net B26: now reaches J5.B26
- net B27: now reaches J5.B27
- net B28: now reaches J5.B28
- net B29: now reaches J5.B29
- net B30: now reaches J5.B30
- net C12: now reaches J5.C12
- net C5: now reaches J5.C5
- net A10: now reaches J5.A10
- net A11: now reaches J5.A11
- net A12: now reaches J5.A12
- net A13: now reaches J5.A13
- net A14: now reaches J5.A14
- net A15: now reaches J5.A15
- net A16: now reaches J5.A16
- net A17: now reaches J5.A17
- net A18: now reaches J5.A18
- net A19: now reaches J5.A19
- net A20: now reaches J5.A20
- net A21: now reaches J5.A21
- net A22: now reaches J5.A22
- net A3: now reaches J5.A3
- net A4: now reaches J5.A4
- net A5: now reaches J5.A5
- net A6: now reaches J5.A6
- net A7: now reaches J5.A7
- net A8: now reaches J5.A8
- net A9: now reaches J5.A9
- no-connect marks 30 -> 0
Changed lines of the file:
@@
 $Descr A4 11693 8268
 encoding utf-8
-Sheet 13 13
+Sheet 9 13
 Title "Single DIN 41612 Slot"
 Date ""
@@
 AR Path="/61A07546/85E2059E" Ref="H5"  Part="1"
 AR Path="/61A07551/85E2059E" Ref="H7"  Part="1"
-F 0 "H7" H 9150 2099 50  0000 L CNN
+F 0 "H23" H 9150 2099 50  0000 L CNN
 F 1 "MountingHole_Pad" H 9150 2008 50  0000 L CNN
 F 2 "MountingHole:MountingHole_2.7mm_M2.5_ISO14580_Pad" H 9050 2050 50  0001 C CNN
@@
 AR Path="/61A07546/85E2263F" Ref="H6"  Part="1"
 AR Path="/61A07551/85E2263F" Ref="H8"  Part="1"
-F 0 "H8" H 9150 2599 50  0000 L CNN
+F 0 "H24" H 9150 2599 50  0000 L CNN
 F 1 "MountingHole_Pad" H 9150 2508 50  0000 L CNN
 F 2 "MountingHole:MountingHole_2.7mm_M2.5_ISO14580_Pad" H 9050 2550 50  0001 C CNN
@@
 AR Path="/61A07546/619501C5" Ref="J2"  Part="3"
 AR Path="/61A07551/619501C5" Ref="J1"  Part="3"
-F 0 "J1" H 7250 5450 50  0000 L CNN
+F 0 "J12" H 7250 5450 50  0000 L CNN
 F 1 "DIN-41612-3x32-Bauform-C" H 7530 3655 50  0001 L CNN
 F 2 "alexios:DIN41612_C_3x32_Female_Vertical_THT" H 7325 350 50  0001 C CNN
@@
 AR Path="/61A07546/619501F3" Ref="J2"  Part="1"
 AR Path="/61A07551/619501F3" Ref="J1"  Part="1"
-F 0 "J1" H 3950 5450 50  0000 C CNN
+F 0 "J12" H 3950 5450 50  0000 C CNN
 F 1 "DIN-41612-3x32-Bauform-C" H 3800 1950 50  0000 L CNN
 F 2 "alexios:DIN41612_C_3x32_Female_Vertical_THT" H 3925 350 50  0001 C CNN
@@
 Text Label 6900 5350 0    50   ~ 0
 C32
-NoConn ~ 3650 2450
-NoConn ~ 3650 2550
-NoConn ~ 3650 2650
-NoConn ~ 3650 2750
-NoConn ~ 3650 2850
-NoConn ~ 3650 2950
-NoConn ~ 3650 3050
-NoConn ~ 3650 3150
-NoConn ~ 3650 3250
-NoConn ~ 3650 3350
-NoConn ~ 3650 3450
-NoConn ~ 3650 3550
-NoConn ~ 3650 3650
-NoConn ~ 3650 3750
-NoConn ~ 3650 3850
-NoConn ~ 3650 3950
-NoConn ~ 3650 4050
-NoConn ~ 3650 4150
-NoConn ~ 3650 4250
-NoConn ~ 3650 4350
-NoConn ~ 7050 2650
-NoConn ~ 7050 3350
 $Comp
 L alexios:DIN-41612-3x32-Bauform-C J?
@@
 AR Path="/61A07546/619501A7" Ref="J2"  Part="2"
 AR Path="/61A07551/619501A7" Ref="J1"  Part="2"
-F 0 "J1" H 5650 5450 50  0000 C CNN
+F 0 "J12" H 5650 5450 50  0000 C CNN
 F 1 "DIN-41612-3x32-Bauform-C" H 5830 3655 50  0001 L CNN
 F 2 "alexios:DIN41612_C_3x32_Female_Vertical_THT" H 5625 350 50  0001 C CNN
@@
 	1    0    0    -1
 $EndComp
-NoConn ~ 5350 4450
-NoConn ~ 5350 4550
-NoConn ~ 5350 4650
-NoConn ~ 5350 4750
-NoConn ~ 5350 4850
-NoConn ~ 5350 4950
-NoConn ~ 5350 5050
-NoConn ~ 5350 5150
+Wire Wire Line
+	3650 2450 3000 2450
+Wire Wire Line
+	3650 2550 3000 2550
+Wire Wire Line
+	3650 2650 3000 2650
+Wire Wire Line
+	3650 2750 3000 2750
+Wire Wire Line
+	3650 2850 3000 2850
+Wire Wire Line
+	3650 2950 3000 2950
+Wire Wire Line
+	3650 3050 3000 3050
+Wire Wire Line
+	3650 3150 3000 3150
+Wire Wire Line
+	3650 3250 3000 3250
+Wire Wire Line
+	3650 3350 3000 3350
+Wire Wire Line
+	3650 3450 3000 3450
+Wire Wire Line
+	3650 3550 3000 3550
+Wire Wire Line
+	3650 3650 3000 3650
+Wire Wire Line
+	3650 3750 3000 3750
+Wire Wire Line
+	3650 3850 3000 3850
+Wire Wire Line
+	3650 3950 3000 3950
+Wire Wire Line
+	3650 4050 3000 4050
+Wire Wire Line
+	3650 4150 3000 4150
+Wire Wire Line
+	3650 4250 3000 4250
+Wire Wire Line
+	3650 4350 3000 4350
+Entry Wire Line
+	2900 2350 3000 2450
+Entry Wire Line
+	2900 2450 3000 2550
+Entry Wire Line
+	2900 2550 3000 2650
+Entry Wire Line
+	2900 2650 3000 2750
+Entry Wire Line
+	2900 2750 3000 2850
+Entry Wire Line
+	2900 2850 3000 2950
+Entry Wire Line
+	2900 2950 3000 3050
+Entry Wire Line
+	2900 3050 3000 3150
+Entry Wire Line
+	2900 3150 3000 3250
+Entry Wire Line
+	2900 3250 3000 3350
+Entry Wire Line
+	2900 3350 3000 3450
+Entry Wire Line
+	2900 3450 3000 3550
+Entry Wire Line
+	2900 3550 3000 3650
+Entry Wire Line
+	2900 3650 3000 3750
+Entry Wire Line
+	2900 3750 3000 3850
+Entry Wire Line
+	2900 3850 3000 3950
+Entry Wire Line
+	2900 3950 3000 4050
+Entry Wire Line
+	2900 4050 3000 4150
+Entry Wire Line
+	2900 4150 3000 4250
+Entry Wire Line
+	2900 4250 3000 4350
+Text Label 3500 2450 0    50   ~ 0
+A3
+Text Label 3500 2550 0    50   ~ 0
+A4
+Text Label 3500 2650 0    50   ~ 0
+A5
+Text Label 3500 2750 0    50   ~ 0
+A6
+Text Label 3500 2850 0    50   ~ 0
+A7
+Text Label 3500 2950 0    50   ~ 0
+A8
+Text Label 3500 3050 0    50   ~ 0
+A9
+Text Label 3500 3150 0    50   ~ 0
+A10
+Text Label 3500 3250 0    50   ~ 0
+A11
+Text Label 3500 3350 0    50   ~ 0
+A12
+Text Label 3500 3450 0    50   ~ 0
+A13
+Text Label 3500 3550 0    50   ~ 0
+A14
+Text Label 3500 3650 0    50   ~ 0
+A15
+Text Label 3500 3750 0    50   ~ 0
+A16
+Text Label 3500 3850 0    50   ~ 0
+A17
+Text Label 3500 3950 0    50   ~ 0
+A18
+Text Label 3500 4050 0    50   ~ 0
+A19
+Text Label 3500 4150 0    50   ~ 0
+A20
+Text Label 3500 4250 0    50   ~ 0
+A21
+Text Label 3500 4350 0    50   ~ 0
+A22
+Entry Wire Line
+	4600 4350 4700 4450
+Wire Wire Line
+	4700 4450 5350 4450
+Entry Wire Line
+	4600 4450 4700 4550
+Wire Wire Line
+	4700 4550 5350 4550
+Entry Wire Line
+	4600 4550 4700 4650
+Wire Wire Line
+	4700 4650 5350 4650
+Entry Wire Line
+	4600 4650 4700 4750
+Wire Wire Line
+	4700 4750 5350 4750
+Entry Wire Line
+	4600 4750 4700 4850
+Wire Wire Line
+	4700 4850 5350 4850
+Entry Wire Line
+	4600 4850 4700 4950
+Wire Wire Line
+	4700 4950 5350 4950
+Entry Wire Line
+	4600 4950 4700 5050
+Wire Wire Line
+	4700 5050 5350 5050
+Entry Wire Line
+	4600 5050 4700 5150
+Wire Wire Line
+	4700 5150 5350 5150
+Text Label 5350 4450 2    50   ~ 0
+B23
+Text Label 5350 4550 2    50   ~ 0
+B24
+Text Label 5350 4650 2    50   ~ 0
+B25
+Text Label 5350 4750 2    50   ~ 0
+B26
+Text Label 5350 4850 2    50   ~ 0
+B27
+Text Label 5350 4950 2    50   ~ 0
+B28
+Text Label 5350 5050 2    50   ~ 0
+B29
+Text Label 5350 5150 2    50   ~ 0
+B30
+Entry Wire Line
+	6300 2550 6400 2650
+Wire Wire Line
+	6400 2650 7050 2650
+Entry Wire Line
+	6300 3250 6400 3350
+Wire Wire Line
+	6400 3350 7050 3350
+Wire Bus Line
+	6300 1950 6300 5250
 Wire Bus Line
 	2900 1950 2900 5250
 Wire Bus Line
-	6300 1950 6300 5250
-Wire Bus Line
 	4600 1950 4600 5250
+Text Label 7000 2650 2    50   ~ 0
+C5
+Text Label 7050 3350 2    50   ~ 0
+C12
 $EndSCHEMATC
