File: kicad/cft/cft-pb0/cft_sbl.sch (KiCad schematic (older format))
At the start: 0 parts

Commit message: Recreated PB0 to test layout feasibility.
Parts:
- added C1, C2, C3, C4, C5, C6, C7, C8, C9: 100nF, Capacitor_SMD:C_0805_2012Metric, symbol Device:C_Small
- added R1, R2, R3: 4.7kΩ, Resistor_SMD:R_0805_2012Metric, symbol Device:R_Small
- added R4, R5, R6, R8: 10kΩ, Resistor_SMD:R_0805_2012Metric, symbol Device:R_Small
- added R7: 30Ω, alexios:R_SMD_0805_2012Metric_Pad1.15x1.40mm_HandSolder, symbol Device:R_Small
- added U1, U5: 74HC251, alexios:SOIC-16, symbol alexios:74HC251
- added U2: 74HC08, alexios:SOIC-14, symbol alexios:74HC08
- added U3, UU1: 74HC32, alexios:SOIC-14, symbol alexios:74HC32
- added U4: 74AHC1G86, alexios:SOT-23-5_HandSoldering, symbol alexios:74AHC1G86
- added U6: 74AHC1G04, alexios:SOT-23-5_HandSoldering, symbol alexios:74AHC1G04
- added U7: 74LVC1G11, alexios:SOT-23-6_Handsoldering, symbol alexios:74LVC1G11
- added U8: 74LVC1G74, symbol alexios:74LVC1G74
- added U9: 74LVC1G332, alexios:SOT-23-6_Handsoldering, symbol alexios:74LVC1G332
Connections:
- new net: R4.1, U5.4 (I0)
- new net: R6.1, U5.13 (I6)
- new net: R8.1, U8.6 (~CLR)
- new net: R7.2, U8.5 (Q)
- new net: R5.1, U5.3 (I1)
- new net: U3.8, U4.2
- new net +5V: C1.1, C2.1, C3.1, C4.1, C5.1, C6.1, C7.1, C8.1, C9.1, R1.1, R2.1, R3.1, R8.2, U1.16 (VCC), U2.14 (VCC), U3.12, U3.13, U3.14 (VCC), U4.5 (VCC), U5.16 (VCC), U6.5 (VCC), U7.5 (VCC), U8.8 (VCC), U9.5 (VCC)
- new net CLK4: U8.1 (CLK)
- new net COND0: U1.11 (S0), U5.11 (S0)
- new net COND1: U1.10 (S1), U5.10 (S1)
- new net COND2: U1.9 (S2), U5.9 (S2)
- new net COND3: U1.7 (~OE)
- new net FL: U2.5, U5.1 (I3)
- new net FN: U2.13, U5.14 (I5)
- new net FV: U2.2, U5.2 (I2)
- new net FZ: U2.10, U5.15 (I4)
- new net GND: C1.2, C2.2, C3.2, C4.2, C5.2, C6.2, C7.2, C8.2, C9.2, R4.2, R5.2, R6.2, U1.4 (I0), U1.8 (GND), U2.7 (GND), U3.7 (GND), U4.3 (GND), U5.8 (GND), U6.3 (GND), U7.2 (GND), U8.4 (GND), U9.2 (GND)
- new net IR0: U1.3 (I1), U2.1
- new net IR1: U1.2 (I2), U2.4
- new net IR2: U1.1 (I3), U2.9
- new net IR3: U1.15 (I4), U2.12
- new net IR4: U1.14 (I5), U4.1
- new net IR5: U1.13 (I6)
- new net IR6: U1.12 (I7)
- new net OP1-BRANCH: U4.4, U5.12 (I7)
- new net SKIPMUXLO: R2.2, U1.6 (~Y), U7.6
- new net SL: U2.6, UU1.4
- new net SN: U2.11, U3.1
- new net SV: U2.3, UU1.5
- new net SVL: U3.10, UU1.6
- new net SZ: U2.8, U3.2
- new net SZN: U3.3, U3.9
- new net ~COND3: U5.7 (~OE)
- new net ~RESET: U8.7 (~PRE)
- new net ~SKIP: R7.1
- new net ~SKIP1: R3.2, U5.6 (~Y), U7.1
- new net ~SKIP2: U7.4, U8.2 (D)
- new net ~SKIPEXT: R1.2, U7.3
- no-connect marks 0 -> 4
Other:
- note added: "Skip & Branch Unit"
- note added: "TODO: Check inversions here! E.g when IR0=1, we want to output 0!"
- note added: "TODO: Rearrange these?"
- note added: "TODO: add a gate here to avoid hazards\nbecause of ~COND3~ below?"
- note added: "Under Review! DO NOT IMPLEMENT"

Commit message: Checking board fit, fixed minor issues.
Parts:
- renumbered UU1 to U3
Changed lines of the file:
@@
 EESchema Schematic File Version 4
-LIBS:cft-cache
 EELAYER 30 0
 EELAYER END
@@
 P 3850 4950
 AR Path="/5F031629" Ref="UU?"  Part="1"
-AR Path="/5EFCF155/5F031629" Ref="UU1"  Part="2"
-F 0 "UU1" H 3850 5025 50  0000 C CNN
+AR Path="/5EFCF155/5F031629" Ref="U3"  Part="2"
+F 0 "U3" H 3850 5025 50  0000 C CNN
 F 1 "74HC32" H 3850 4934 50  0000 C CNN
 F 2 "alexios:SOIC-14" H 3850 4950 50  0001 C CNN

Commit message: New page layout
Other:
- note removed: "Skip & Branch Unit"
Changed lines of the file:
@@
 encoding utf-8
 Sheet 2 12
-Title "CFT Homebrew 16-bit Minicomputer"
+Title "Skip/Branch Unit"
 Date ""
 Rev ""
 Comp ""
-Comment1 ""
+Comment1 "CUB"
 Comment2 ""
 Comment3 ""
-Comment4 ""
+Comment4 "sbu.v"
 $EndDescr
 $Comp
@@
 Text Label 5650 2800 1    50   ~ 0
 FN
-Text Notes 7200 7000 0    197  ~ 39
-Skip & Branch Unit
 Wire Wire Line
 	5500 4650 7400 4650
@@
 	1    0    0    -1
 $EndComp
+Wire Notes Line style solid rgb(255, 11, 2)
+	6350 5150 7300 5150
+Wire Notes Line style solid rgb(255, 5, 1)
+	6350 5350 6350 5150
+Wire Notes Line style solid rgb(255, 11, 2)
+	6350 5350 7300 5350
+Wire Notes Line style solid rgb(255, 5, 1)
+	7300 5350 7300 5150
 Wire Bus Line
 	950  1500 6100 1500

Commit message: Working on PB0
Connections:
- net ~SKIP renamed ~COND
Changed lines of the file:
@@
 	9050 1100 9050 4800
 Text HLabel 10900 5800 2    50   Output ~ 0
-~SKIP
+~COND
 Text Label 9150 2550 1    50   ~ 0
 SKIPMUXLO
@@
 	9050 5300 9050 5900
 Text Label 10650 5800 0    50   ~ 0
-~SKIP
+~COND
 Wire Wire Line
 	10600 5800 10900 5800
@@
 	1    0    0    -1
 $EndComp
-Wire Notes Line style solid rgb(255, 11, 2)
+Wire Notes Line style solid rgb(255, 11, 0)
 	6350 5150 7300 5150
-Wire Notes Line style solid rgb(255, 5, 1)
+Wire Notes Line style solid rgb(255, 5, 0)
 	6350 5350 6350 5150
-Wire Notes Line style solid rgb(255, 11, 2)
+Wire Notes Line style solid rgb(255, 11, 0)
 	6350 5350 7300 5350
-Wire Notes Line style solid rgb(255, 5, 1)
+Wire Notes Line style solid rgb(255, 5, 0)
 	7300 5350 7300 5150
 Wire Bus Line

Commit message: Working on Control board (ex PB0)
Parts:
- U8: footprint (none) -> alexios:TSSOP-8_3x3mm_P0.65mm
Changed lines of the file:
@@
 EESchema Schematic File Version 4
 LIBS:cft-pb0-cache
-EELAYER 26 0
+EELAYER 30 0
 EELAYER END
 $Descr A4 11693 8268
 encoding utf-8
-Sheet 2 12
+Sheet 2 13
 Title "Skip/Branch Unit"
 Date ""
@@
 F 0 "U8" H 9950 6367 50  0000 C CNN
 F 1 "74LVC1G74" H 9950 6276 50  0000 C CNN
-F 2 "" H 10400 5950 50  0001 C CNN
+F 2 "alexios:TSSOP-8_3x3mm_P0.65mm" H 10400 5950 50  0001 C CNN
 F 3 "https://assets.nexperia.com/documents/data-sheet/74LVC1G74.pdf" H 10400 5950 50  0001 C CNN
 	1    9950 5950
@@
 F 0 "U8" H 5630 7446 50  0000 L CNN
 F 1 "74LVC1G74" H 5630 7355 50  0000 L CNN
-F 2 "" H 5900 7400 50  0001 C CNN
+F 2 "alexios:TSSOP-8_3x3mm_P0.65mm" H 5900 7400 50  0001 C CNN
 F 3 "https://assets.nexperia.com/documents/data-sheet/74LVC1G74.pdf" H 5900 7400 50  0001 C CNN
 	2    5450 7400
