File: kicad/cft/cft-bus/reg_mbr.sch (KiCad schematic (older format))
At the start: 22 parts, among them U14 74AHC1G125, U28 74HC670, U29 74HC670, U30 74HC541, U31 74HC139, U33 74HC670, U34 74HC670, U35 74LVC1G74, U36 74AHC1G125, U39 74HC139, U40 74LVC1G74

Commit message: A little work on the BUS card
Parts:
- added U?: 74AC161, symbol alexios:74AC161
Connections:
- net +5V: now also U?.10 (CET), U?.3 (D0), U?.4 (D1), U?.5 (D2), U?.6 (D3), U?.7 (CEP), U?.9 (~PE)
- new net FPR0: U?.14 (Q0)
- new net FPR1: U?.13 (Q1)
- new net FPR2: U?.12 (Q2)
- new net ~FPMBREN: U?.2 (CP)
- new net ~FPMBRR: U?.1 (~MR)
- no-connect marks 4 -> 6
Changed lines of the file:
@@
 Rev ""
 Comp ""
-Comment1 "CTL"
+Comment1 "BUS"
 Comment2 ""
 Comment3 ""
@@
 Text Notes 8250 2950 0    50   ~ 10
 Note
+$Sheet
+S 13400 1400 1150 1500
+U 5E647D2E
+F0 "4×8 bit file" 50
+F1 "regfile4x8.sch" 50
+F2 "WA0" I L 13400 2650 50
+F3 "WA1" I L 13400 2750 50
+F4 "RA0" I R 14550 2650 50
+F5 "RA1" I R 14550 2750 50
+F6 "~RE" I R 14550 2450 50
+F7 "~WE" I L 13400 2450 50
+F8 "IN0" I L 13400 1550 50
+F9 "IN1" I L 13400 1650 50
+F10 "IN2" I L 13400 1750 50
+F11 "IN3" I L 13400 1850 50
+F12 "IN4" I L 13400 1950 50
+F13 "IN5" I L 13400 2050 50
+F14 "IN6" I L 13400 2150 50
+F15 "IN7" I L 13400 2250 50
+F16 "OUT0" O R 14550 1550 50
+F17 "OUT1" O R 14550 1650 50
+F18 "OUT2" O R 14550 1750 50
+F19 "OUT3" O R 14550 1850 50
+F20 "OUT4" O R 14550 1950 50
+F21 "OUT5" O R 14550 2050 50
+F22 "OUT6" O R 14550 2150 50
+F23 "OUT7" O R 14550 2250 50
+$EndSheet
+Text Label 14700 1850 0    50   ~ 0
+AEXT3
+Text Label 14700 1750 0    50   ~ 0
+AEXT2
+Text Label 14700 1650 0    50   ~ 0
+AEXT1
+Text Label 14700 1550 0    50   ~ 0
+AEXT0
+Wire Wire Line
+	14550 1850 15000 1850
+Wire Wire Line
+	14550 1750 15000 1750
+Wire Wire Line
+	14550 1650 15000 1650
+Wire Wire Line
+	14550 1550 15000 1550
+Text Label 14700 1950 0    50   ~ 0
+AEXT4
+Text Label 14700 2050 0    50   ~ 0
+AEXT5
+Text Label 14700 2150 0    50   ~ 0
+AEXT6
+Text Label 14700 2250 0    50   ~ 0
+AEXT7
+Wire Wire Line
+	14550 1950 15000 1950
+Wire Wire Line
+	14550 2250 15000 2250
+Wire Wire Line
+	14550 2150 15000 2150
+Wire Wire Line
+	14550 2050 15000 2050
+Wire Wire Line
+	13400 1850 12950 1850
+Wire Wire Line
+	13400 1750 12950 1750
+Wire Wire Line
+	13400 1650 12950 1650
+Wire Wire Line
+	13400 1550 12950 1550
+Entry Wire Line
+	12950 1950 12850 1850
+Entry Wire Line
+	12950 2050 12850 1950
+Entry Wire Line
+	12950 2150 12850 2050
+Entry Wire Line
+	12950 2250 12850 2150
+Entry Wire Line
+	12950 1550 12850 1450
+Entry Wire Line
+	12950 1650 12850 1550
+Entry Wire Line
+	12950 1750 12850 1650
+Entry Wire Line
+	12950 1850 12850 1750
+Wire Wire Line
+	13400 1950 12950 1950
+Wire Wire Line
+	13400 2250 12950 2250
+Wire Wire Line
+	13400 2150 12950 2150
+Wire Wire Line
+	13400 2050 12950 2050
+Text Label 13050 1550 0    50   ~ 0
+IBUS0
+Text Label 13050 1650 0    50   ~ 0
+IBUS1
+Text Label 13050 1750 0    50   ~ 0
+IBUS2
+Text Label 13050 1850 0    50   ~ 0
+IBUS3
+Text Label 13050 1950 0    50   ~ 0
+IBUS4
+Text Label 13050 2050 0    50   ~ 0
+IBUS5
+Text Label 13050 2150 0    50   ~ 0
+IBUS6
+Text Label 13050 2250 0    50   ~ 0
+IBUS7
+Wire Wire Line
+	13400 2450 12950 2450
+Wire Wire Line
+	13400 2650 12950 2650
+Wire Wire Line
+	13400 2750 12950 2750
+Text Label 12950 2650 0    50   ~ 0
+SEL0
+Text Label 12950 2750 0    50   ~ 0
+SEL1
+Text Label 12950 2450 0    50   ~ 0
+~BANKW0
+Entry Wire Line
+	15000 1950 15100 1850
+Entry Wire Line
+	15000 2050 15100 1950
+Entry Wire Line
+	15000 2150 15100 2050
+Entry Wire Line
+	15000 2250 15100 2150
+Entry Wire Line
+	15000 1550 15100 1450
+Entry Wire Line
+	15000 1650 15100 1550
+Entry Wire Line
+	15000 1750 15100 1650
+Entry Wire Line
+	15000 1850 15100 1750
+Wire Wire Line
+	14550 2450 15000 2450
+Wire Wire Line
+	14550 2650 15000 2650
+Wire Wire Line
+	14550 2750 15000 2750
+Text Label 15000 2450 2    50   ~ 0
+~BANKR0
+Text Label 15000 2650 2    50   ~ 0
+IR0
+Text Label 15000 2750 2    50   ~ 0
+IR1
+$Comp
+L alexios:74AC161 U?
+U 1 1 5DF5E120
+P 13700 4950
+F 0 "U?" H 13700 5717 50  0000 C CNN
+F 1 "74AC161" H 13700 5626 50  0000 C CNN
+F 2 "" H 14000 5200 50  0001 C CNN
+F 3 "https://assets.nexperia.com/documents/data-sheet/74HC161.pdf" H 14000 5200 50  0001 C CNN
+	1    13700 4950
+	1    0    0    -1
+$EndComp
+Wire Wire Line
+	14200 4450 14650 4450
+Wire Wire Line
+	14200 4550 14650 4550
+Wire Wire Line
+	14200 4650 14650 4650
+Text Label 14650 4450 2    50   ~ 0
+FPR0
+Text Label 14650 4550 2    50   ~ 0
+FPR1
+Text Label 14650 4650 2    50   ~ 0
+FPR2
+NoConn ~ 14200 4750
+NoConn ~ 14200 4950
+Wire Wire Line
+	13200 5050 13100 5050
+$Comp
+L power:+5V #PWR?
+U 1 1 5DFAEFFD
+P 13100 4350
+F 0 "#PWR?" H 13100 4200 50  0001 C CNN
+F 1 "+5V" H 13115 4523 50  0000 C CNN
+F 2 "" H 13100 4350 50  0001 C CNN
+F 3 "" H 13100 4350 50  0001 C CNN
+	1    13100 4350
+	1    0    0    -1
+$EndComp
+Wire Wire Line
+	13200 5150 13100 5150
+Wire Wire Line
+	13200 5250 12700 5250
+Text Label 12700 5250 0    50   ~ 0
+~FPMBREN
+Wire Wire Line
+	13200 5450 12700 5450
+Text Label 12700 5450 0    50   ~ 0
+~FPMBRR
+Wire Wire Line
+	13100 5150 13100 5050
+Connection ~ 13100 5050
+Wire Wire Line
+	13100 5050 13100 4950
+Wire Wire Line
+	13200 4450 13100 4450
+Connection ~ 13100 4450
+Wire Wire Line
+	13100 4450 13100 4350
+Wire Wire Line
+	13200 4550 13100 4550
+Connection ~ 13100 4550
+Wire Wire Line
+	13100 4550 13100 4450
+Wire Wire Line
+	13200 4650 13100 4650
+Connection ~ 13100 4650
+Wire Wire Line
+	13100 4650 13100 4550
+Wire Wire Line
+	13200 4750 13100 4750
+Connection ~ 13100 4750
+Wire Wire Line
+	13100 4750 13100 4650
+Wire Wire Line
+	13200 4950 13100 4950
+Connection ~ 13100 4950
+Wire Wire Line
+	13100 4950 13100 4750
+Wire Bus Line
+	12850 1350 12850 2150
+Wire Bus Line
+	15100 1350 15100 2150
 Wire Bus Line
 	3700 800  3700 3300
@@
 Wire Bus Line
 	7650 1600 7650 4400
-$Sheet
-S 11900 1400 600  1300
-U 5E647D2E
-F0 "4×8 bit file" 50
-F1 "regfile4x8.sch" 50
-F2 "OUT[0..7]" T R 12500 1500 50
-F3 "IN[0..7]" T L 11900 1500 50
-$EndSheet
 $EndSCHEMATC

Commit message: Better FP support for MBR
Parts:
- removed C22, C23, C26, C27: 100nF, Capacitor_SMD:C_0805_2012Metric, symbol Device:C_Small
- removed U28, U29, U33, U34: 74HC670, alexios:SOIC-16, symbol alexios:74HC670
- added U? (x2): 74HC139, alexios:SOIC-16, symbol alexios:74HC139
- added U?: 74HC541, alexios:SOIC-20W, symbol alexios:74HC541
Connections:
- net +5V: now also U?.13 (A1), U?.14 (A0), U?.15 (E)
- net FPR2: now also U?.2 (A0)
- net GND: now also U?.1 (~G), U?.3 (A1)
- new net ~BANKFP0: U?.4 (Y0)
- new net ~BANKFP1: U?.5 (Y1)
- no-connect marks 6 -> 12
Other:
- moved on the sheet: C19, C21, C24, C25, R3, RN1, RN2, U14A, U30A, U30B, U31A, U31B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

Commit message: Work on BUS board.
Connections:
- net FPD0: now also U?.18 (Y0)
- net FPD1: now also U?.17 (Y1)
- net FPD2: now also U?.16 (Y2)
- net FPD3: now also U?.15 (Y3)
- net FPD4: now also U?.14 (Y4)
- net FPD5: now also U?.13 (Y5)
- net FPD6: now also U?.12 (Y6)
- net FPD7: now also U?.11 (Y7)
- net GND: now also U?.19 (~G2)
- net ~FPMBREN: now also U?.1 (~G1)
- net FPOD0: now reaches U?.2 (A0)
- net FPOD1: now reaches U?.3 (A1)
- net FPOD2: now reaches U?.4 (A2)
- net FPOD3: now reaches U?.5 (A3)
- net FPOD4: now reaches U?.6 (A4)
- net FPOD5: now reaches U?.7 (A5)
- net FPOD6: now reaches U?.8 (A6)
- net FPOD7: now reaches U?.9 (A7)
Other:
- note added: "Front Panel Shadow File"
- note added: "Main Register File"
- note added: "Register Reads"
- note added: "←"
- moved on the sheet: C19, C21, C24, C25, R3, RN1, RN2, U14A, U30A, U30B, U31A, U31B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

Commit message: Remap MBR to I/O space.
Other:
- note added: "Remapping to I/O space, redo stuff!"
Changed lines of the file:
@@
 Text Notes 7150 4950 0    198  ~ 0
 ←
+Text Notes 650  2300 0    198  ~ 0
+Remapping to I/O space, redo stuff!
 Wire Bus Line
 	8300 4550 8300 5450

Commit message: Reworking MBU to reduce chip count.
Parts:
- added U?: 74HC245, symbol alexios:74HC245
- added U?: IS61C64AL, Package_SO:SOJ-28_10.16x23.49mm_P1.27mm, symbol alexios:IS61C64AL
Connections:
- net AEXT0: now also U?.11 (D0), U?.2 (A0)
- net AEXT1: now also U?.12 (D1), U?.3 (A1)
- net AEXT2: now also U?.13 (D2), U?.4 (A2)
- net AEXT3: now also U?.15 (D3), U?.5 (A3)
- net AEXT4: now also U?.16 (D4), U?.6 (A4)
- net AEXT5: now also U?.17 (D5), U?.7 (A5)
- net AEXT6: now also U?.18 (D6), U?.8 (A6)
- net AEXT7: now also U?.19 (D7), U?.9 (A7)
- net GND: now also U?.2 (A12), U?.20 (~CE), U?.21 (A10), U?.23 (A11), U?.24 (A9), U?.25 (A8), U?.3 (A7), U?.4 (A6), U?.5 (A5), U?.6 (A4), U?.7 (A3)
- net IBUS0: now also U?.18 (B0)
- net IBUS1: now also U?.17 (B1)
- net IBUS2: now also U?.16 (B2)
- net IBUS3: now also U?.15 (B3)
- net IBUS4: now also U?.14 (B4)
- net IBUS5: now also U?.13 (B5)
- net IBUS6: now also U?.12 (B6)
- net IBUS7: now also U?.11 (B7)
- net SEL0: now also U?.10 (A0)
- net SEL1: now also U?.9 (A1)
- net SEL2: now also U?.8 (A2)
- net ~RMBR: now also U?.22 (~OE)
- net ~WMBR: now also U?.27 (~WE)
Other:
- note removed: "Remapping to I/O space, redo stuff!"

Commit message: (hopefully) Finalise MBU design.
Parts:
- removed C19, C21, C24, C25: 100nF, Capacitor_SMD:C_0805_2012Metric, symbol Device:C_Small
- removed R3: 4.7kΩ, Resistor_SMD:R_0805_2012Metric, symbol Device:R_Small
- removed RN1, RN2: 4.7kΩ, Resistor_THT:R_Array_SIP5, symbol Device:R_Network04
- removed U14, U36: 74AHC1G125, alexios:SOT-23-5_HandSoldering, symbol alexios:74AHC1G125
- removed U30, U?: 74HC541, alexios:SOIC-20W, symbol alexios:74HC541
- removed U31, U39, U? (x2): 74HC139, alexios:SOIC-16, symbol alexios:74HC139
- removed U35, U40: 74LVC1G74, alexios:TSSOP-8_3x3mm_P0.65mm, symbol alexios:74LVC1G74
- removed U?: 74AC161, symbol alexios:74AC161
- added C? (x10): 100nF, Capacitor_SMD:C_0805_2012Metric, symbol Device:C_Small
- added D? (x4): LED_ALT, symbol Device:LED_ALT
- added JP? (x3): Jumper_2_Open, symbol Jumper:Jumper_2_Open
- added JP?: Jumper_2_Bridged, symbol Jumper:Jumper_2_Bridged
- added JP?: Jumper_3_Bridged12, symbol Jumper:Jumper_3_Bridged12
- added R? (x4): 680Ω, symbol Device:R_Small
- added U? (x8): 74HC138, alexios:SOIC-16, symbol alexios:74HC138
- added U? (x2): 27C256, Package_DIP:DIP-28_W15.24mm, symbol alexios:27C256
- added U? (x5): 74AC32, symbol alexios:74AC32
- added U? (x4): 74AC244, symbol alexios:74AC244
- added U?: 74HC245, symbol alexios:74HC245
- added U?: IS61C64AL, Package_SO:SOJ-28_10.16x23.49mm_P1.27mm, symbol alexios:IS61C64AL
Connections:
- net +5V: now also C?.1, C?.1, C?.1, C?.1, C?.1, C?.1, C?.1, C?.1, C?.1, C?.1, R?.1, R?.1, R?.1, R?.1, U?.1 (A0), U?.1 (VPP), U?.14 (VCC), U?.16 (VCC), U?.16 (VCC), U?.16 (VCC), U?.16 (VCC), U?.2 (A1), U?.20 (VCC), U?.20 (VCC), U?.20 (VCC), U?.28 (VCC), U?.28 (VCC), U?.3 (A2)
- net GND: now also C?.2, C?.2, C?.2, C?.2, C?.2, C?.2, C?.2, C?.2, C?.2, C?.2, JP?.3 (B), U?.10 (GND), U?.10 (GND), U?.10 (GND), U?.11 (2A3), U?.11 (2A3), U?.13 (2A2), U?.14 (GND), U?.14 (GND), U?.15 (2A1), U?.17 (2A0), U?.20 (~CE), U?.22 (~OE), U?.27 (A14), U?.4 (~G2B), U?.4 (~G2B), U?.6 (1A2), U?.7 (GND), U?.8 (1A3), U?.8 (1A3), U?.8 (GND), U?.8 (GND), U?.8 (GND), U?.8 (GND)
- net IR0: now also U?.17 (2A0)
- net IR1: now also U?.15 (2A1)
- net IR2: now also U?.13 (2A2)
- net SEL0: now also U?.18 (1Y0), U?.18 (1Y0), U?.3 (2Y0), U?.3 (2Y0)
- net SEL1: now also U?.16 (1Y1), U?.16 (1Y1), U?.5 (2Y1), U?.5 (2Y1)
- net SEL2: now also U?.14 (1Y2), U?.14 (1Y2), U?.7 (2Y2), U?.7 (2Y2)
- net ~RMBR: now also JP?.2 (B), JP?.2 (B), JP?.2 (B), JP?.2 (B)
- net ~WMBR: now also U?.11
- net ~IBUSW: now reaches U?.1 (A→B)
- net ~IBUSW: now also U?.19 (D7)
- net ~IBUSEN: now reaches U?.19 (CE)
- net ~IBUSEN: now also U?.18 (D6)
- new net: JP?.1 (A), U?.1, U?.11 (D0), U?.2
- new net: U?.12, U?.12 (D1)
- new net: JP?.1 (A), U?.3, U?.4, U?.5
- new net: JP?.1 (A), U?.10, U?.6, U?.9
- new net: JP?.1 (A), U?.8
- new net: JP?.2 (C), U?.13
- new net: D?.2 (A), R?.2 (x4)
- new net AB0: U?.2 (1A0)
- new net AB1: U?.4 (1A1)
- new net AB2: U?.6 (1A2)
- new net AB3: U?.6 (G1)
- new net AB4: U?.1 (A0)
- new net AB5: U?.2 (A1)
- new net AB6: U?.3 (A2)
- new net AB7: U?.5 (~G2A)
- new net IR10: U?.2 (A12)
- new net IR11: U?.26 (A13)
- new net IR8: U?.21 (A10)
- new net IR9: U?.23 (A11)
- new net LED0: U?.12 (1Y3)
- new net LED1: D?.1 (K), U?.9 (2Y3)
- new net LED2: D?.1 (K), U?.12 (1Y3)
- new net LED3: D?.1 (K), U?.9 (2Y3)
- new net LED4: D?.1 (K)
- new net RADDR0: U?.1 (A0)
- new net RADDR1: U?.2 (A1)
- new net RADDR2: U?.3 (A2)
- new net RADDR3: U?.6 (G1)
- new net RADDR4: U?.5 (~G2A)
- new net WADDR0: U?.1 (A0), U?.2 (1A0), U?.25 (A8)
- new net WADDR1: U?.2 (A1), U?.24 (A9), U?.4 (1A1)
- new net WADDR2: U?.3 (A2), U?.6 (G1)
- new net WADDR3: U?.5 (~G2A), U?.6 (G1)
- new net WADDR4: U?.4 (~G2B), U?.5 (~G2A)
- new net WSTB: JP?.1 (A)
- new net ~IOMBR: U?.15 (~Y0), U?.8 (A2)
- new net ~R: U?.10 (A0)
- new net ~READ-FLAGS: U?.9 (~Y6)
- new net ~READ-MBP: U?.11 (~Y4), U?.7 (A3)
- new net ~READ-MBP+FLAGS: U?.10 (~Y5), U?.6 (A4)
- new net ~SYSDEV: U?.4 (~G2B)
- new net ~USE_AB: U?.1 (1OE), U?.13 (D2)
- new net ~USE_IR: U?.17 (D5), U?.19 (2OE)
- new net ~USE_WADDR: U?.1 (1OE), U?.16 (D4)
- new net ~USE_ZERO: U?.15 (D3), U?.19 (2OE)
- new net ~W: U?.9 (A1)
- new net ~WRITE-FLAGS: U?.9 (~Y6)
- new net ~WRITE-MBP: U?.11 (~Y4), U?.5 (A5)
- new net ~WRITE-MBP+FLAGS: U?.10 (~Y5), U?.4 (A6)
- new net ~WRITE-MBx-AR: U?.3 (A7), U?.7 (~Y7)
- no-connect marks 12 -> 24
Other:
- note added: "&008–&00F"
- note added: "Address Decoding"
- note added: "Address Multiplexer"
- note added: "Control ROM"
- note added: "Convenience outputs to the Flag Unit"
- note added: "IBus Transceiver"
- note added: "IOADDR=00:00001xxx"
- note added: "MUX LEDs"
- note added: "Optional 0–3×Tpd delay line"
- note added: "RADDR=01XXX"
- note added: "Register File"
- note added: "Strobe Synchronisation"
- note added: "WADDR=001XX"
- note added: "WADDR=01XXX"
- note added: "We only use 7 lines: bits 0–2 and 8–11."
- note removed: "After ~RESET~ and before ~BANKW0~ is asserted, drive AEXT₀₋₇ with &00 (~RAM~/ROM position set to ~RAM~)\nor &80 (set to ROM). Use pull-down resistors for most of the vector. After the first write to an MBR register,\nthis stops and random values can be expected to be present! So the minimum required registers should be\ninitialised as early as possible after reset."
- note removed: "Front Panel Shadow File"
- note removed: "High after ~BANKW0~\nasserted."
- note removed: "High after ~RESET~\nasserted."
- note removed: "MBn registers are accessed when:\n\n1. Write access when WADDR=00001 is selected (~WRITE-MBP+FLAGS~).\n2. Write access when WADDR=00011 is selected (~WRITE-MBn~).\n3. Read access when RADDR=00001 is selected (~READ-MBP+FLAGS~).\n4. Read access when RADDR=00011 is selected (~READ-MBn~).\n5. Read access when WADDR=001xx (~WRITE-AR:MBn~). Note, even though\nwe respond on WADDR, this is a READ operat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"
- note removed: "Main Register File"
- note removed: "Register Address Decoding"
- note removed: "Register Reads"
- note removed: "←"
- moved on the sheet: U?A

Commit message: Add MBU init circuitry, move things around
Parts:
- added C? (x3): 100nF, Capacitor_SMD:C_0805_2012Metric, symbol Device:C_Small
- added R6: 4.7kΩ, Resistor_SMD:R_0805_2012Metric, symbol Device:R_Small
- added RN1, RN2: 4.7kΩ, Resistor_THT:R_Array_SIP5, symbol Device:R_Network04
- added U12, U?: 74LVC1G74, alexios:TSSOP-8_3x3mm_P0.65mm, symbol alexios:74LVC1G74
- added U13, U?: 74AHC1G125, alexios:SOT-23-5_HandSoldering, symbol alexios:74AHC1G125
- added U? (x2): 74LVC1G32, symbol alexios:74LVC1G32
- gave numbers to parts that had none: 33
Connections:
- net LED0 is gone; now on net LED1: U6.12 (1Y3)
- net +5V: now also C?.1, C?.1, C?.1, R6.1, U12.1 (CLK), U12.2 (D), U?.5 (VCC), U?.5 (VCC), U?.8 (VCC)
- net AEXT0: now also RN2.5 (R4)
- net AEXT1: now also RN2.4 (R3)
- net AEXT2: now also RN2.3 (R2)
- net AEXT3: now also RN2.2 (R1)
- net AEXT4: now also RN1.5 (R4)
- net AEXT5: now also RN1.4 (R3)
- net AEXT6: now also RN1.3 (R2)
- net AEXT7: now also U13.4
- net GND: now also C?.2, C?.2, C?.2, RN1.1 (common), RN2.1 (common), U?.3 (GND), U?.3 (GND), U?.4 (GND); no longer U7.27 (A14)
- net LED1: no longer U6.9 (2Y3)
- net LED2: now also U6.9 (2Y3); no longer U5.12 (1Y3)
- net LED3: now also U5.12 (1Y3); no longer U5.9 (2Y3)
- net LED4: now also U5.9 (2Y3)
- net WSTB: now also U?.1
- net ~IOMBR: now also U?.2
- new net: U12.6 (~CLR), U?.4
- new net ~DIS: U12.3 (~Q), U13.1, U7.27 (A14)
- new net ~FPRAM~∕ROM: R6.2, U13.2
- new net ~RESET: U12.7 (~PRE)
- no-connect marks 24 -> 26
Other:
- note added: "45ns EPROM"
- note added: "IR[0:2], IR[8:11]"
- note added: "MBU Enable"
- note added: "Signals IBUS[8..15] are purposefully not driven\nhere! They are handled by the flag unit."
- note added: "The MBU is disabled after reset and enabled\nwhen it's first written to."
- note added: "mbu_rom.bin"
- note removed: "IBUS[8..15] are purposefully not driven here!\nThey are handled by the flag unit."
- note removed: "We only use 7 lines: bits 0–2 and 8–11."
- moved on the sheet: C10, C4, C5, C6, C7, C8, C9, JP1, JP2, JP3, JP4, JP5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
