File: kicad/cft/cft-bus/cft_ws_busen.sch (KiCad schematic (older format))
At the start: 31 parts, among them U22 ICS501, U34 74LVC1G32, U43 74LVC1G04, U44 74LVC1G3208, U45 74LVC1G125, U46 74AHC1G32, U47 74LVC1G74, U48 74HC245, U49 74LVC1G11, U50 74HC245

Commit message: Reworking CTL and BUS boards. Added WAITING# signal to bus.
Changed lines of the file:
@@
 Text Notes 7250 1650 0    50   ~ 0
 Allow for impedance matching resistors\nif needed.
-Text Label 1750 3850 0    50   ~ 0
-CLK3
 Wire Wire Line
 	1650 3850 2000 3850
@@
 Text HLabel 1650 3950 0    50   Input ~ 0
 ~RESET
-Text HLabel 1650 3850 0    50   Input ~ 0
-CLK3
 Wire Wire Line
 	4700 3950 5150 3950
@@
 Wire Wire Line
 	3100 3500 3100 3650
+Text Label 3650 3850 2    50   ~ 0
+CLK3
+Text Notes 2400 3800 0    100  ~ 20
+TODO: REWORK THIS.
 Wire Bus Line
 	8750 3250 8750 5600
 Wire Bus Line
 	6850 3600 6850 6050
-Text Label 3650 3850 2    50   ~ 0
+Text HLabel 1650 3850 0    50   Input ~ 0
 CLK3
-Text Notes 2550 3700 0    100  ~ 20
-TODO: REWORK THIS.
+Text Label 1750 3850 0    50   ~ 0
+CLK3
 $EndSCHEMATC

Commit message: Reworking boards for new bus definitions and control store.
Parts:
- added C54, C55: 100nF, alexios:C_SMD_0805_2012Metric_Pad1.15x1.40mm_HandSolder, symbol Device:C_Small
- added D2: D_ALT, alexios:SOD-323, symbol Device:D_ALT
- added R10: 100Ω, alexios:R_SMD_0805_2012Metric_Pad1.15x1.40mm_HandSolder, symbol Device:R_Small
- added R11: 4.7kΩ, alexios:R_SMD_0805_2012Metric_Pad1.15x1.40mm_HandSolder, symbol Device:R_Small
- added TP6, TP7: TestPoint, TestPoint:TestPoint_Pad_1.0x1.0mm, symbol Connector:TestPoint
- added U51: 74LVC1G3208, alexios:SOT-23-6_Handsoldering, symbol alexios:74LVC1G3208
- added U52: 74LVC1G17, alexios:SOT-23-5_HandSoldering, symbol alexios:74LVC1G17
- U53: renamed from U?; footprint (none) -> alexios:SOT-23-6_Handsoldering
- gave numbers to parts that had none: 1
Connections:
- net +5V: now also C54.1, C55.1, U51.5 (VCC), U52.5 (VCC)
- net GND: now also C54.2, C55.2, R11.1, U51.2 (GND), U52.3 (GND)
- net ~WAITING: now also TP4.1, U51.1, U51.3, U51.6; no longer U44.6
- net at U47.5 (Q): no longer TP4.1
- net ~RESET renamed ~RSTHOLD
- new net: D2.1 (K), R10.1, R11.2
- new net: R10.2, TP7.1, U52.2
- new net: D2.2 (A), U51.4
- new net ~WAITING-DELAYED: TP6.1, U44.6, U52.4
- no-connect marks 2 -> 3
Other:
- note added: "(1)"
- note added: "(1) Held low during Wait State"
- note added: "Delay ~WAITING~ so its positive\nedge comes after ~WSTB~'s. Include\nfootprints for experimenting."
- note added: "Optional impedance\nmatching resistor."
- note added: "Write; No Wait State"
- note added: "Write; One Wait State"
- note added: "~WEN"
- note added: "~WS~"
- note added: "~W\n"
- note added: "~W~"
- note removed: "Allow for impedance matching resistors\nif needed."
- note removed: "TODO: REWORK THIS."
- moved on the sheet: R12, TP4

Commit message: Working on CTL board.
Parts:
- removed U51: 74LVC1G3208, alexios:SOT-23-6_Handsoldering, symbol alexios:74LVC1G3208
- added TP8: TestPoint, TestPoint:TestPoint_Pad_1.0x1.0mm, symbol Connector:TestPoint
- added U42: 74HC08, alexios:SOIC-14, symbol alexios:74HC08
Connections:
- net +5V: now also U42.10, U42.12, U42.13, U42.14 (VCC), U42.9
- net GND: now also U42.7 (GND)
- net ~WAITING: now also U42.1, U42.4, U42.5; no longer TP4.1
- net ~WAITING-DELAYED: now also U42.2; no longer U44.6
- net at D2.2 (A): now also TP4.1, U42.6
- new net: TP8.1, U42.3, U44.6
- no-connect marks 3 -> 5
Other:
- moved on the sheet: C54, C55, TP4, TP6, U52B

Commit message: Fixing serious potential processor bug by readjusting clocks and establishing standard waveforms.
Changed lines of the file:
@@
 ~W\n
 Wire Notes Line width 12 style solid
-	9700 4900 9900 4900
+	9700 4900 9800 4900
 Wire Notes Line width 12 style solid
-	9900 4900 9900 5000
+	9800 4900 9800 5000
 Wire Notes Line width 12 style solid
 	9950 5000 9950 4900
 Wire Notes Line width 12 style solid
-	9900 5000 9950 5000
+	9800 5000 9950 5000
 Wire Notes Line width 12 style solid
-	10700 4900 10700 5000
+	10600 4900 10600 5000
 Wire Notes Line width 12 style solid
 	10750 5000 10750 4900
 Wire Notes Line width 12 style solid
-	10700 5000 10750 5000
+	10600 5000 10750 5000
 Wire Notes Line width 12 style solid
 	10750 4900 10900 4900
@@
 	10770 4750 10900 4750
 Wire Notes Line width 12 style solid
-	9950 4900 10700 4900
+	9950 4900 10600 4900
 Wire Notes Line width 12 style solid
 	9970 4750 10650 4750

Commit message: Fixed timing issues with MBU, improving write waveforms.
Parts:
- removed U48, U50: 74HC245, alexios:SOIC-20W, symbol alexios:74HC245
- added JP4: Jumper_3_Bridged12, Jumper:SolderJumper-3_P1.3mm_Bridged12_RoundedPad1.0x1.5mm, symbol Jumper:Jumper_3_Bridged12
- added U48, U50: 74ACT245, alexios:SOIC-20W, symbol alexios:74ACT245
Connections:
- net +5V: now also U48.20 (VCC), U50.20 (VCC)
- net DB0: now also U48.18 (B0)
- net DB1: now also U48.17 (B1)
- net DB10: now also U50.16 (B2)
- net DB11: now also U50.15 (B3)
- net DB12: now also U50.14 (B4)
- net DB13: now also U50.13 (B5)
- net DB14: now also U50.12 (B6)
- net DB15: now also U50.11 (B7)
- net DB2: now also U48.16 (B2)
- net DB3: now also U48.15 (B3)
- net DB4: now also U48.14 (B4)
- net DB5: now also U48.13 (B5)
- net DB6: now also U48.12 (B6)
- net DB7: now also U48.11 (B7)
- net DB8: now also U50.18 (B0)
- net DB9: now also U50.17 (B1)
- net GND: now also U48.10 (GND), U50.10 (GND)
- net IBUS0: now also U48.2 (A0)
- net IBUS1: now also U48.3 (A1)
- net IBUS10: now also U50.4 (A2)
- net IBUS11: now also U50.5 (A3)
- net IBUS12: now also U50.6 (A4)
- net IBUS13: now also U50.7 (A5)
- net IBUS14: now also U50.8 (A6)
- net IBUS15: now also U50.9 (A7)
- net IBUS2: now also U48.4 (A2)
- net IBUS3: now also U48.5 (A3)
- net IBUS4: now also U48.6 (A4)
- net IBUS5: now also U48.7 (A5)
- net IBUS6: now also U48.8 (A6)
- net IBUS7: now also U48.9 (A7)
- net IBUS8: now also U50.2 (A0)
- net IBUS9: now also U50.3 (A1)
- net ~BUSEN: now also U48.19 (CE), U50.19 (CE)
- net ~R: now also U48.1 (A→B), U50.1 (A→B)
- net ~WAITING: now also JP4.3 (B)
- net at TP8.1, U42.3: now also JP4.1 (A); no longer U44.6
- new net: JP4.2 (C), U44.6
Other:
- note added: "NOTE: HCT or ACT family!"
- moved on the sheet: D2, R10, R11, TP4, TP6, TP7, TP8, U42A, U42B, U52A

Commit message: Worked out simpler Wait State and Write drivers.
Parts:
- removed C55: 100nF, alexios:C_SMD_0805_2012Metric_Pad1.15x1.40mm_HandSolder, symbol Device:C_Small
- removed D2: D_ALT, alexios:SOD-323, symbol Device:D_ALT
- removed JP3, JP4: Jumper_3_Bridged12, Jumper:SolderJumper-3_P1.3mm_Bridged12_RoundedPad1.0x1.5mm, symbol Jumper:Jumper_3_Bridged12
- removed R11: 4.7kΩ, alexios:R_SMD_0805_2012Metric_Pad1.15x1.40mm_HandSolder, symbol Device:R_Small
- removed TP4, TP6, TP7, TP8: TestPoint, TestPoint:TestPoint_Pad_1.0x1.0mm, symbol Connector:TestPoint
- removed U22: ICS501, alexios:SOIC-8, symbol alexios:ICS501
- removed U42: 74HC08, alexios:SOIC-14, symbol alexios:74HC08
- removed U44: 74LVC1G3208, alexios:SOT-23-6_Handsoldering, symbol alexios:74LVC1G3208
- removed U46: 74AHC1G32, alexios:SOT-23-5_HandSoldering, symbol alexios:74AHC1G32
- removed U52: 74LVC1G17, alexios:SOT-23-5_HandSoldering, symbol alexios:74LVC1G17
- removed U53: 74LVC1G373, alexios:SOT-23-6_Handsoldering, symbol alexios:74LVC1G373
- added U22: 74LVC1G17, alexios:SOT-23-5_HandSoldering, symbol alexios:74LVC1G17
- added U42: 74LVC1G74, alexios:TSSOP-8_3x3mm_P0.65mm, symbol alexios:74AUC1G74
- added U44: 74LVC1G0832, alexios:SOT-23-6_Handsoldering, symbol alexios:74LVC1G0832
- added U46: 74LVC1G32, alexios:SOT-23-5_HandSoldering, symbol alexios:74LVC1G32
- R10: value 100Ω -> 0Ω
Connections:
- net +5V: now also U22.5 (VCC), U42.1 (CLK), U42.2 (D), U42.8 (VCC), U44.2 (GND), U46.5 (VCC)
- net CLK4: now also U34.2; no longer U34.1
- net GND: now also U22.3 (GND), U42.4 (GND), U44.5 (VCC), U46.3 (GND)
- net ~HALT: now also TP1.1
- net ~WAITING: now also U44.1
- net ~WEN: now also R10.1, U44.6
- net ~WS: now also U46.1
- net ~WS-in-T34: now also U46.4
- net ~WSTB: now also U42.3 (~Q), U44.3
- net ~W₀: now also U44.4
- net at U43.4, U45.1: no longer TP1.1
- net at R10.2: now also U22.2
- net at U34.4: now also U42.7 (~PRE)
- new net: U22.4, U34.1
- new net CLK2: U42.6 (~CLR)
- new net ~T34: U46.2
- no-connect marks 5 -> 2
Other:
- note added: "CLK1"
- note added: "CLK2"
- note added: "Optional impedance\nmatching resistors."
- note added: "Pull-up may be\noptional, test first!"
- note added: "Wait States must be asserted:\n\n • As early as possible during T3 or T4.\n • At the latest one flip-flop setup time before CLK3 goes high.\n • Remain low at least one hold time after CLK3 goes high.\n\nExecution of the current microinstruction will then be protracted by a whole number of processor cycles, ending on\nthe cycle where ~WS~ was not asserted on the rising edge of CLK3. To generate wa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"
- note added: "Write Strobe"
- note added: "~IO~\n\nX\n0\nX\n1"
- note added: "~WAITING"
- note added: "~WAITING~\n\n X\n X\n 1\n 1\n 1"
- note added: "~WEN~\n\n X\n 1\n 1\n 0\n 0"
- note added: "~WS\n"
- note removed: "(1)"
- note removed: "(1) Held low during Wait State"
- note removed: "8×CLK4"
- note removed: "CLK×4"
- note removed: "Delay ~WAITING~ so its positive\nedge comes after ~WSTB~'s. Include\nfootprints for experimenting."
- note removed: "Optional impedance\nmatching resistor."
- note removed: "Optional, low-jitter\nwrite strobe generator.\nPositive edge 31.25ns\nafter CLK4 goes low."
- note removed: "Pull-up may be optional, test!"
- note removed: "Wait States must be asserted:\n\n • During CLK3.\n • At the latest one flip-flop setup time before CLK3 goes high.\n • Remain low at least one hold time after CLK3 goes high.\n\nExecution of the current microinstruction will then be protracted by a whole number of\nprocessor cycles, ending on the cycle where ~WS~ was not asserted on the rising edge\nof CLK3.\n\nTo generate wait states for slow de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"
- note removed: "~IO~\n\n X\n 0\n X\n 1"
- note removed: "~WAITING~\n\n X\n 0\n 1\n 1\n 1"
- note removed: "~WEN~\n\n X\n X\n 1\n 0\n 0"
- note removed: "~WS~"
- note removed: "~W~"
- note removed: "~W~ strobes come at most approximately 9ns after ~WSTB~."
- moved on the sheet: R12, R13, R14, R8, TP1, TP2, TP3, U43A, U45A, U47A

Commit message: All tests passing again, updating schematics.
Parts:
- removed TP1, TP2: TestPoint, TestPoint:TestPoint_Pad_1.0x1.0mm, symbol Connector:TestPoint
- removed U22: 74LVC1G17, alexios:SOT-23-5_HandSoldering, symbol alexios:74LVC1G17
- added R11, R15, R16, R17, R18, R19, R20, R21, R22: 0Ω, alexios:R_SMD_0805_2012Metric_Pad1.15x1.40mm_HandSolder, symbol Device:R_Small
- added U22: 74LVC1G14, alexios:SOT-23-5_HandSoldering, symbol alexios:74LVC1G14
Connections:
- net +5V: now also U22.5 (VCC)
- net CLK2: now also R17.1; no longer U42.6 (~CLR)
- net CLK3: now also R21.1; no longer U47.1 (CLK)
- net GND: now also U22.3 (GND)
- net ~HALT: now also R11.1; no longer U43.2
- net ~RSTHOLD: now also R22.1; no longer U47.6 (~CLR)
- net ~WEN: now also R15.1, R16.2
- net ~WS: now also R19.1
- net ~WS-in-T34: now also R20.2; no longer TP3.1, U47.7 (~PRE)
- net ~W₀: now also R18.1; no longer U45.2
- net at R10.2: now also U22.2
- net at U34.1: now also R15.2, R16.1
- net CLK4: no longer names the net of U34.2
- net CLK4: now also U22.4
- new net: R21.2, U47.1 (CLK)
- new net: R22.2, U47.6 (~CLR)
- new net: R19.2, R20.1, TP3.1, U47.7 (~PRE)
- new net: R18.2, U45.2
- new net: R11.2, U43.2
- new net: R17.2, U42.6 (~CLR)
Other:
- note added: "0Ω Shunts"
- note added: "Optional"
- note added: "Using 0Ω 0805 shunts as a\ncombination testpoint, jumper\nand pads for impedance-\nmatching resistors."
- moved on the sheet: C36, C54, R10, R14, U34A, U42A, U46A

Commit message: Synced schematics with recent timing changes.
Parts:
- removed R19, R20: 0Ω, alexios:R_SMD_0805_2012Metric_Pad1.15x1.40mm_HandSolder, symbol Device:R_Small
- removed U22: 74LVC1G14, alexios:SOT-23-5_HandSoldering, symbol alexios:74LVC1G14
- added JP3: Jumper_3_Bridged12, Jumper:SolderJumper-3_P1.3mm_Bridged12_RoundedPad1.0x1.5mm, symbol alexios:Jumper_3_Bridged12
- added U22: 74LVC1G04, alexios:SOT-23-5_HandSoldering, symbol alexios:74LVC1G04
Connections:
- net +5V: now also U22.5 (VCC)
- net GND: now also U22.3 (GND)
- net ~WS: now also JP3.1 (A)
- net ~WS-in-T34: now also JP3.3 (B)
- net at TP3.1, U47.7 (~PRE): now also JP3.2 (C)
- net HALT: now reaches U43.4, U45.1
- net ~WEN-DELAYED: now reaches R15.2, R16.1, U34.1
- net at U34.2: now also U22.4
- net at R10.2: now also U22.2
Other:
- note added: "Also used by the AR."
- note added: "Pull-up used to slow\ndown negative edge.\nMay be optional,\ntest first!"
- note removed: "Pull-up may be\noptional, test first!"
- moved on the sheet: R11, R16, TP3, U43A
