File: kicad/cft/cft-ctl/cpu_cs.sch (KiCad schematic (older format))
At the start: 6 parts, among them U24 74HC138, U25 74AC541, U26 74AC541

Commit message: Worked on CTL board.
Parts:
- removed unit 2 of U24
- removed unit 2 of U25
- added U?: 74HC138, alexios:SOIC-14, symbol alexios:74HC138
- added U?: 74AC541, alexios:SOIC-20W, symbol alexios:74AC541
- renumbered C20 to C?, C21 to C?, C22 to C?, U25 to U?, U26 to U?, U24 to U?
Connections:
- net +5V: now also U?.16 (VCC), U?.20 (VCC)
- net GND: now also U?.10 (GND), U?.8 (GND)
Changed lines of the file:
@@
 EESchema Schematic File Version 4
-LIBS:cft-pb0-cache
+LIBS:cft-ctl-cache
 EELAYER 30 0
 EELAYER END
 $Descr A4 11693 8268
 encoding utf-8
-Sheet 5 13
+Sheet 9 12
 Title "Constant Store"
 Date ""
 Rev ""
 Comp ""
-Comment1 "CUB"
+Comment1 "CTL"
 Comment2 ""
 Comment3 ""
@@
 P 1000 7250
 AR Path="/5E4DDD44/5E51C06B" Ref="#PWR?"  Part="1"
-AR Path="/5E507DE3/5E51C06B" Ref="#PWR060"  Part="1"
-F 0 "#PWR060" H 1000 7100 50  0001 C CNN
+AR Path="/5E507DE3/5E51C06B" Ref="#PWR?"  Part="1"
+AR Path="/5DF0FEB9/5E51C06B" Ref="#PWR?"  Part="1"
+F 0 "#PWR?" H 1000 7100 50  0001 C CNN
 F 1 "+5V" H 1015 7423 50  0000 C CNN
 F 2 "" H 1000 7250 50  0001 C CNN
@@
 P 1000 7450
 AR Path="/5E4DDD44/5E51C071" Ref="#PWR?"  Part="1"
-AR Path="/5E507DE3/5E51C071" Ref="#PWR063"  Part="1"
-F 0 "#PWR063" H 1000 7200 50  0001 C CNN
+AR Path="/5E507DE3/5E51C071" Ref="#PWR?"  Part="1"
+AR Path="/5DF0FEB9/5E51C071" Ref="#PWR?"  Part="1"
+F 0 "#PWR?" H 1000 7200 50  0001 C CNN
 F 1 "GND" H 1005 7277 50  0000 C CNN
 F 2 "" H 1000 7450 50  0001 C CNN
@@
 AR Path="/5E51C077" Ref="C?"  Part="1"
 AR Path="/5E4DDD44/5E51C077" Ref="C?"  Part="1"
-AR Path="/5E507DE3/5E51C077" Ref="C20"  Part="1"
-F 0 "C20" H 909 7396 50  0000 R CNN
+AR Path="/5E507DE3/5E51C077" Ref="C?"  Part="1"
+AR Path="/5DF0FEB9/5E51C077" Ref="C?"  Part="1"
+F 0 "C?" H 909 7396 50  0000 R CNN
 F 1 "100nF" H 909 7305 50  0000 R CNN
 F 2 "Capacitor_SMD:C_0805_2012Metric" H 1000 7350 50  0001 C CNN
@@
 AR Path="/5E51C0B5" Ref="C?"  Part="1"
 AR Path="/5E4DDD44/5E51C0B5" Ref="C?"  Part="1"
-AR Path="/5E507DE3/5E51C0B5" Ref="C21"  Part="1"
-F 0 "C21" H 2359 7396 50  0000 R CNN
+AR Path="/5E507DE3/5E51C0B5" Ref="C?"  Part="1"
+AR Path="/5DF0FEB9/5E51C0B5" Ref="C?"  Part="1"
+F 0 "C?" H 2359 7396 50  0000 R CNN
 F 1 "100nF" H 2359 7305 50  0000 R CNN
 F 2 "Capacitor_SMD:C_0805_2012Metric" H 2450 7350 50  0001 C CNN
@@
 P 2450 7450
 AR Path="/5E4DDD44/5E51C0BB" Ref="#PWR?"  Part="1"
-AR Path="/5E507DE3/5E51C0BB" Ref="#PWR064"  Part="1"
-F 0 "#PWR064" H 2450 7200 50  0001 C CNN
+AR Path="/5E507DE3/5E51C0BB" Ref="#PWR?"  Part="1"
+AR Path="/5DF0FEB9/5E51C0BB" Ref="#PWR?"  Part="1"
+F 0 "#PWR?" H 2450 7200 50  0001 C CNN
 F 1 "GND" H 2455 7277 50  0000 C CNN
 F 2 "" H 2450 7450 50  0001 C CNN
@@
 P 2450 7250
 AR Path="/5E4DDD44/5E51C0C1" Ref="#PWR?"  Part="1"
-AR Path="/5E507DE3/5E51C0C1" Ref="#PWR061"  Part="1"
-F 0 "#PWR061" H 2450 7100 50  0001 C CNN
+AR Path="/5E507DE3/5E51C0C1" Ref="#PWR?"  Part="1"
+AR Path="/5DF0FEB9/5E51C0C1" Ref="#PWR?"  Part="1"
+F 0 "#PWR?" H 2450 7100 50  0001 C CNN
 F 1 "+5V" H 2465 7423 50  0000 C CNN
 F 2 "" H 2450 7250 50  0001 C CNN
@@
 P 7100 3050
 AR Path="/5E4DDD44/5E55BF66" Ref="U?"  Part="1"
-AR Path="/5E507DE3/5E55BF66" Ref="U25"  Part="1"
-F 0 "U25" H 7100 3817 50  0000 C CNN
+AR Path="/5E507DE3/5E55BF66" Ref="U?"  Part="1"
+AR Path="/5DF0FEB9/5E55BF66" Ref="U?"  Part="1"
+F 0 "U?" H 7100 3817 50  0000 C CNN
 F 1 "74AC541" H 7100 3726 50  0000 C CNN
 F 2 "alexios:SOIC-20W" H 7100 3050 50  0001 C CNN
@@
 P 7100 4600
 AR Path="/5E4DDD44/5E55BF6C" Ref="U?"  Part="1"
-AR Path="/5E507DE3/5E55BF6C" Ref="U26"  Part="1"
-F 0 "U26" H 7100 5367 50  0000 C CNN
+AR Path="/5E507DE3/5E55BF6C" Ref="U?"  Part="1"
+AR Path="/5DF0FEB9/5E55BF6C" Ref="U?"  Part="1"
+F 0 "U?" H 7100 5367 50  0000 C CNN
 F 1 "74AC541" H 7100 5276 50  0000 C CNN
 F 2 "alexios:SOIC-20W" H 7100 4600 50  0001 C CNN
@@
 	6500 2750 6500 2850
 $Comp
-L power:GND #PWR056
-U 1 1 5E6CB311
+L power:GND #PWR?
+U 1 1 5DEFC7D1
 P 6500 3250
-F 0 "#PWR056" H 6500 3000 50  0001 C CNN
+F 0 "#PWR?" H 6500 3000 50  0001 C CNN
 F 1 "GND" H 6350 3250 50  0000 C CNN
 F 2 "" H 6500 3250 50  0001 C CNN
@@
 	6500 2850 6500 2950
 $Comp
-L power:GND #PWR058
-U 1 1 5E6DE76B
+L power:GND #PWR?
+U 1 1 5DEFC7D2
 P 6500 4800
-F 0 "#PWR058" H 6500 4550 50  0001 C CNN
+F 0 "#PWR?" H 6500 4550 50  0001 C CNN
 F 1 "GND" H 6350 4800 50  0000 C CNN
 F 2 "" H 6500 4800 50  0001 C CNN
@@
 $Comp
 L alexios:74HC138 U?
-U 2 1 5E89BF6D
+U 2 1 5DEFC7D3
 P 1350 7350
-AR Path="/5DC89E19/5E89BF6D" Ref="U?"  Part="1"
-AR Path="/5E507DE3/5E89BF6D" Ref="U24"  Part="2"
-AR Path="/5E89BF6D" Ref="U?"  Part="2"
-F 0 "U24" H 1530 7396 50  0000 L CNN
+AR Path="/5DC89E19/5DEFC7D3" Ref="U?"  Part="1"
+AR Path="/5E507DE3/5DEFC7D3" Ref="U?"  Part="2"
+AR Path="/5DEFC7D3" Ref="U?"  Part="2"
+AR Path="/5DF0FEB9/5DEFC7D3" Ref="U?"  Part="2"
+F 0 "U?" H 1530 7396 50  0000 L CNN
 F 1 "74HC138" H 1530 7305 50  0000 L CNN
 F 2 "alexios:SOIC-14" H 1350 7350 50  0001 C CNN
@@
 $Comp
 L alexios:74AC541 U?
-U 2 1 5E89CE71
+U 2 1 5DEFC7D4
 P 2800 7350
-AR Path="/5E4DDD44/5E89CE71" Ref="U?"  Part="1"
-AR Path="/5E507DE3/5E89CE71" Ref="U25"  Part="2"
-F 0 "U25" H 2980 7396 50  0000 L CNN
+AR Path="/5E4DDD44/5DEFC7D4" Ref="U?"  Part="1"
+AR Path="/5E507DE3/5DEFC7D4" Ref="U?"  Part="2"
+AR Path="/5DF0FEB9/5DEFC7D4" Ref="U?"  Part="2"
+F 0 "U?" H 2980 7396 50  0000 L CNN
 F 1 "74AC541" H 2980 7305 50  0000 L CNN
 F 2 "alexios:SOIC-20W" H 2800 7350 50  0001 C CNN
@@
 AR Path="/5E8B296C" Ref="C?"  Part="1"
 AR Path="/5E4DDD44/5E8B296C" Ref="C?"  Part="1"
-AR Path="/5E507DE3/5E8B296C" Ref="C22"  Part="1"
-F 0 "C22" H 3809 7396 50  0000 R CNN
+AR Path="/5E507DE3/5E8B296C" Ref="C?"  Part="1"
+AR Path="/5DF0FEB9/5E8B296C" Ref="C?"  Part="1"
+F 0 "C?" H 3809 7396 50  0000 R CNN
 F 1 "100nF" H 3809 7305 50  0000 R CNN
 F 2 "Capacitor_SMD:C_0805_2012Metric" H 3900 7350 50  0001 C CNN
@@
 P 3900 7450
 AR Path="/5E4DDD44/5E8B2972" Ref="#PWR?"  Part="1"
-AR Path="/5E507DE3/5E8B2972" Ref="#PWR065"  Part="1"
-F 0 "#PWR065" H 3900 7200 50  0001 C CNN
+AR Path="/5E507DE3/5E8B2972" Ref="#PWR?"  Part="1"
+AR Path="/5DF0FEB9/5E8B2972" Ref="#PWR?"  Part="1"
+F 0 "#PWR?" H 3900 7200 50  0001 C CNN
 F 1 "GND" H 3905 7277 50  0000 C CNN
 F 2 "" H 3900 7450 50  0001 C CNN
@@
 P 3900 7250
 AR Path="/5E4DDD44/5E8B2978" Ref="#PWR?"  Part="1"
-AR Path="/5E507DE3/5E8B2978" Ref="#PWR062"  Part="1"
-F 0 "#PWR062" H 3900 7100 50  0001 C CNN
+AR Path="/5E507DE3/5E8B2978" Ref="#PWR?"  Part="1"
+AR Path="/5DF0FEB9/5E8B2978" Ref="#PWR?"  Part="1"
+F 0 "#PWR?" H 3900 7100 50  0001 C CNN
 F 1 "+5V" H 3915 7423 50  0000 C CNN
 F 2 "" H 3900 7250 50  0001 C CNN
@@
 P 4250 7350
 AR Path="/5E4DDD44/5E8B297E" Ref="U?"  Part="1"
-AR Path="/5E507DE3/5E8B297E" Ref="U26"  Part="2"
-F 0 "U26" H 4430 7396 50  0000 L CNN
+AR Path="/5E507DE3/5E8B297E" Ref="U?"  Part="2"
+AR Path="/5DF0FEB9/5E8B297E" Ref="U?"  Part="2"
+F 0 "U?" H 4430 7396 50  0000 L CNN
 F 1 "74AC541" H 4430 7305 50  0000 L CNN
 F 2 "alexios:SOIC-20W" H 4250 7350 50  0001 C CNN
@@
 	6050 5000 6600 5000
 $Comp
-L power:GND #PWR057
-U 1 1 5DC46A7B
+L power:GND #PWR?
+U 1 1 5DEFC7BA
 P 6500 3550
-F 0 "#PWR057" H 6500 3300 50  0001 C CNN
+F 0 "#PWR?" H 6500 3300 50  0001 C CNN
 F 1 "GND" H 6505 3377 50  0000 C CNN
 F 2 "" H 6500 3550 50  0001 C CNN
@@
 $EndComp
 $Comp
-L power:GND #PWR059
-U 1 1 5DC46AA3
+L power:GND #PWR?
+U 1 1 5DEFC7BB
 P 6500 5100
-F 0 "#PWR059" H 6500 4850 50  0001 C CNN
+F 0 "#PWR?" H 6500 4850 50  0001 C CNN
 F 1 "GND" H 6505 4927 50  0000 C CNN
 F 2 "" H 6500 5100 50  0001 C CNN
@@
 P 4250 2950
 AR Path="/5DC89E19/5E56A57B" Ref="U?"  Part="1"
-AR Path="/5E507DE3/5E56A57B" Ref="U24"  Part="1"
+AR Path="/5E507DE3/5E56A57B" Ref="U?"  Part="1"
 AR Path="/5E56A57B" Ref="U?"  Part="1"
-F 0 "U24" H 4250 3617 50  0000 C CNN
+AR Path="/5DF0FEB9/5E56A57B" Ref="U?"  Part="1"
+F 0 "U?" H 4250 3617 50  0000 C CNN
 F 1 "74HC138" H 4250 3526 50  0000 C CNN
 F 2 "alexios:SOIC-14" H 4250 2950 50  0001 C CNN
@@
 	2850 2650 2950 2750
 $Comp
-L power:+5V #PWR0165
+L power:+5V #PWR?
 U 1 1 5E03D7B4
 P 3750 3150
-F 0 "#PWR0165" H 3750 3000 50  0001 C CNN
+F 0 "#PWR?" H 3750 3000 50  0001 C CNN
 F 1 "+5V" H 3765 3323 50  0000 C CNN
 F 2 "" H 3750 3150 50  0001 C CNN
@@
 $EndComp
 $Comp
-L power:GND #PWR0167
+L power:GND #PWR?
 U 1 1 5E040054
 P 3750 3350
-F 0 "#PWR0167" H 3750 3100 50  0001 C CNN
+F 0 "#PWR?" H 3750 3100 50  0001 C CNN
 F 1 "GND" H 3755 3177 50  0000 C CNN
 F 2 "" H 3750 3350 50  0001 C CNN

Commit message: Investigating board layout
Parts:
- gave numbers to parts that had none: 6
Changed lines of the file:
@@
 EESchema Schematic File Version 4
 LIBS:cft-ctl-cache
-EELAYER 30 0
+EELAYER 26 0
 EELAYER END
 $Descr A4 11693 8268
 encoding utf-8
-Sheet 9 12
+Sheet 9 13
 Title "Constant Store"
 Date ""
@@
 P 1000 7250
 AR Path="/5E4DDD44/5E51C06B" Ref="#PWR?"  Part="1"
-AR Path="/5E507DE3/5E51C06B" Ref="#PWR?"  Part="1"
+AR Path="/5E507DE3/5E51C06B" Ref="#PWR0138"  Part="1"
 AR Path="/5DF0FEB9/5E51C06B" Ref="#PWR?"  Part="1"
-F 0 "#PWR?" H 1000 7100 50  0001 C CNN
+F 0 "#PWR0138" H 1000 7100 50  0001 C CNN
 F 1 "+5V" H 1015 7423 50  0000 C CNN
 F 2 "" H 1000 7250 50  0001 C CNN
@@
 P 1000 7450
 AR Path="/5E4DDD44/5E51C071" Ref="#PWR?"  Part="1"
-AR Path="/5E507DE3/5E51C071" Ref="#PWR?"  Part="1"
+AR Path="/5E507DE3/5E51C071" Ref="#PWR0139"  Part="1"
 AR Path="/5DF0FEB9/5E51C071" Ref="#PWR?"  Part="1"
-F 0 "#PWR?" H 1000 7200 50  0001 C CNN
+F 0 "#PWR0139" H 1000 7200 50  0001 C CNN
 F 1 "GND" H 1005 7277 50  0000 C CNN
 F 2 "" H 1000 7450 50  0001 C CNN
@@
 AR Path="/5E51C077" Ref="C?"  Part="1"
 AR Path="/5E4DDD44/5E51C077" Ref="C?"  Part="1"
-AR Path="/5E507DE3/5E51C077" Ref="C?"  Part="1"
+AR Path="/5E507DE3/5E51C077" Ref="C20"  Part="1"
 AR Path="/5DF0FEB9/5E51C077" Ref="C?"  Part="1"
-F 0 "C?" H 909 7396 50  0000 R CNN
+F 0 "C20" H 909 7396 50  0000 R CNN
 F 1 "100nF" H 909 7305 50  0000 R CNN
 F 2 "Capacitor_SMD:C_0805_2012Metric" H 1000 7350 50  0001 C CNN
@@
 AR Path="/5E51C0B5" Ref="C?"  Part="1"
 AR Path="/5E4DDD44/5E51C0B5" Ref="C?"  Part="1"
-AR Path="/5E507DE3/5E51C0B5" Ref="C?"  Part="1"
+AR Path="/5E507DE3/5E51C0B5" Ref="C21"  Part="1"
 AR Path="/5DF0FEB9/5E51C0B5" Ref="C?"  Part="1"
-F 0 "C?" H 2359 7396 50  0000 R CNN
+F 0 "C21" H 2359 7396 50  0000 R CNN
 F 1 "100nF" H 2359 7305 50  0000 R CNN
 F 2 "Capacitor_SMD:C_0805_2012Metric" H 2450 7350 50  0001 C CNN
@@
 P 2450 7450
 AR Path="/5E4DDD44/5E51C0BB" Ref="#PWR?"  Part="1"
-AR Path="/5E507DE3/5E51C0BB" Ref="#PWR?"  Part="1"
+AR Path="/5E507DE3/5E51C0BB" Ref="#PWR0140"  Part="1"
 AR Path="/5DF0FEB9/5E51C0BB" Ref="#PWR?"  Part="1"
-F 0 "#PWR?" H 2450 7200 50  0001 C CNN
+F 0 "#PWR0140" H 2450 7200 50  0001 C CNN
 F 1 "GND" H 2455 7277 50  0000 C CNN
 F 2 "" H 2450 7450 50  0001 C CNN
@@
 P 2450 7250
 AR Path="/5E4DDD44/5E51C0C1" Ref="#PWR?"  Part="1"
-AR Path="/5E507DE3/5E51C0C1" Ref="#PWR?"  Part="1"
+AR Path="/5E507DE3/5E51C0C1" Ref="#PWR0153"  Part="1"
 AR Path="/5DF0FEB9/5E51C0C1" Ref="#PWR?"  Part="1"
-F 0 "#PWR?" H 2450 7100 50  0001 C CNN
+F 0 "#PWR0153" H 2450 7100 50  0001 C CNN
 F 1 "+5V" H 2465 7423 50  0000 C CNN
 F 2 "" H 2450 7250 50  0001 C CNN
@@
 P 7100 3050
 AR Path="/5E4DDD44/5E55BF66" Ref="U?"  Part="1"
-AR Path="/5E507DE3/5E55BF66" Ref="U?"  Part="1"
+AR Path="/5E507DE3/5E55BF66" Ref="U25"  Part="1"
 AR Path="/5DF0FEB9/5E55BF66" Ref="U?"  Part="1"
-F 0 "U?" H 7100 3817 50  0000 C CNN
+F 0 "U25" H 7100 3817 50  0000 C CNN
 F 1 "74AC541" H 7100 3726 50  0000 C CNN
 F 2 "alexios:SOIC-20W" H 7100 3050 50  0001 C CNN
@@
 P 7100 4600
 AR Path="/5E4DDD44/5E55BF6C" Ref="U?"  Part="1"
-AR Path="/5E507DE3/5E55BF6C" Ref="U?"  Part="1"
+AR Path="/5E507DE3/5E55BF6C" Ref="U26"  Part="1"
 AR Path="/5DF0FEB9/5E55BF6C" Ref="U?"  Part="1"
-F 0 "U?" H 7100 5367 50  0000 C CNN
+F 0 "U26" H 7100 5367 50  0000 C CNN
 F 1 "74AC541" H 7100 5276 50  0000 C CNN
 F 2 "alexios:SOIC-20W" H 7100 4600 50  0001 C CNN
@@
 	6500 2750 6500 2850
 $Comp
-L power:GND #PWR?
+L power:GND #PWR0154
 U 1 1 5DEFC7D1
 P 6500 3250
-F 0 "#PWR?" H 6500 3000 50  0001 C CNN
+F 0 "#PWR0154" H 6500 3000 50  0001 C CNN
 F 1 "GND" H 6350 3250 50  0000 C CNN
 F 2 "" H 6500 3250 50  0001 C CNN
@@
 	6500 2850 6500 2950
 $Comp
-L power:GND #PWR?
+L power:GND #PWR0155
 U 1 1 5DEFC7D2
 P 6500 4800
-F 0 "#PWR?" H 6500 4550 50  0001 C CNN
+F 0 "#PWR0155" H 6500 4550 50  0001 C CNN
 F 1 "GND" H 6350 4800 50  0000 C CNN
 F 2 "" H 6500 4800 50  0001 C CNN
@@
 P 1350 7350
 AR Path="/5DC89E19/5DEFC7D3" Ref="U?"  Part="1"
-AR Path="/5E507DE3/5DEFC7D3" Ref="U?"  Part="2"
+AR Path="/5E507DE3/5DEFC7D3" Ref="U24"  Part="2"
 AR Path="/5DEFC7D3" Ref="U?"  Part="2"
 AR Path="/5DF0FEB9/5DEFC7D3" Ref="U?"  Part="2"
-F 0 "U?" H 1530 7396 50  0000 L CNN
+F 0 "U24" H 1530 7396 50  0000 L CNN
 F 1 "74HC138" H 1530 7305 50  0000 L CNN
 F 2 "alexios:SOIC-14" H 1350 7350 50  0001 C CNN
@@
 P 2800 7350
 AR Path="/5E4DDD44/5DEFC7D4" Ref="U?"  Part="1"
-AR Path="/5E507DE3/5DEFC7D4" Ref="U?"  Part="2"
+AR Path="/5E507DE3/5DEFC7D4" Ref="U25"  Part="2"
 AR Path="/5DF0FEB9/5DEFC7D4" Ref="U?"  Part="2"
-F 0 "U?" H 2980 7396 50  0000 L CNN
+F 0 "U25" H 2980 7396 50  0000 L CNN
 F 1 "74AC541" H 2980 7305 50  0000 L CNN
 F 2 "alexios:SOIC-20W" H 2800 7350 50  0001 C CNN
@@
 AR Path="/5E8B296C" Ref="C?"  Part="1"
 AR Path="/5E4DDD44/5E8B296C" Ref="C?"  Part="1"
-AR Path="/5E507DE3/5E8B296C" Ref="C?"  Part="1"
+AR Path="/5E507DE3/5E8B296C" Ref="C22"  Part="1"
 AR Path="/5DF0FEB9/5E8B296C" Ref="C?"  Part="1"
-F 0 "C?" H 3809 7396 50  0000 R CNN
+F 0 "C22" H 3809 7396 50  0000 R CNN
 F 1 "100nF" H 3809 7305 50  0000 R CNN
 F 2 "Capacitor_SMD:C_0805_2012Metric" H 3900 7350 50  0001 C CNN
@@
 P 3900 7450
 AR Path="/5E4DDD44/5E8B2972" Ref="#PWR?"  Part="1"
-AR Path="/5E507DE3/5E8B2972" Ref="#PWR?"  Part="1"
+AR Path="/5E507DE3/5E8B2972" Ref="#PWR0156"  Part="1"
 AR Path="/5DF0FEB9/5E8B2972" Ref="#PWR?"  Part="1"
-F 0 "#PWR?" H 3900 7200 50  0001 C CNN
+F 0 "#PWR0156" H 3900 7200 50  0001 C CNN
 F 1 "GND" H 3905 7277 50  0000 C CNN
 F 2 "" H 3900 7450 50  0001 C CNN
@@
 P 3900 7250
 AR Path="/5E4DDD44/5E8B2978" Ref="#PWR?"  Part="1"
-AR Path="/5E507DE3/5E8B2978" Ref="#PWR?"  Part="1"
+AR Path="/5E507DE3/5E8B2978" Ref="#PWR0157"  Part="1"
 AR Path="/5DF0FEB9/5E8B2978" Ref="#PWR?"  Part="1"
-F 0 "#PWR?" H 3900 7100 50  0001 C CNN
+F 0 "#PWR0157" H 3900 7100 50  0001 C CNN
 F 1 "+5V" H 3915 7423 50  0000 C CNN
 F 2 "" H 3900 7250 50  0001 C CNN
@@
 P 4250 7350
 AR Path="/5E4DDD44/5E8B297E" Ref="U?"  Part="1"
-AR Path="/5E507DE3/5E8B297E" Ref="U?"  Part="2"
+AR Path="/5E507DE3/5E8B297E" Ref="U26"  Part="2"
 AR Path="/5DF0FEB9/5E8B297E" Ref="U?"  Part="2"
-F 0 "U?" H 4430 7396 50  0000 L CNN
+F 0 "U26" H 4430 7396 50  0000 L CNN
 F 1 "74AC541" H 4430 7305 50  0000 L CNN
 F 2 "alexios:SOIC-20W" H 4250 7350 50  0001 C CNN
@@
 	6050 5000 6600 5000
 $Comp
-L power:GND #PWR?
+L power:GND #PWR0158
 U 1 1 5DEFC7BA
 P 6500 3550
-F 0 "#PWR?" H 6500 3300 50  0001 C CNN
+F 0 "#PWR0158" H 6500 3300 50  0001 C CNN
 F 1 "GND" H 6505 3377 50  0000 C CNN
 F 2 "" H 6500 3550 50  0001 C CNN
@@
 $EndComp
 $Comp
-L power:GND #PWR?
+L power:GND #PWR0159
 U 1 1 5DEFC7BB
 P 6500 5100
-F 0 "#PWR?" H 6500 4850 50  0001 C CNN
+F 0 "#PWR0159" H 6500 4850 50  0001 C CNN
 F 1 "GND" H 6505 4927 50  0000 C CNN
 F 2 "" H 6500 5100 50  0001 C CNN
@@
 P 4250 2950
 AR Path="/5DC89E19/5E56A57B" Ref="U?"  Part="1"
-AR Path="/5E507DE3/5E56A57B" Ref="U?"  Part="1"
+AR Path="/5E507DE3/5E56A57B" Ref="U24"  Part="1"
 AR Path="/5E56A57B" Ref="U?"  Part="1"
 AR Path="/5DF0FEB9/5E56A57B" Ref="U?"  Part="1"
-F 0 "U?" H 4250 3617 50  0000 C CNN
+F 0 "U24" H 4250 3617 50  0000 C CNN
 F 1 "74HC138" H 4250 3526 50  0000 C CNN
 F 2 "alexios:SOIC-14" H 4250 2950 50  0001 C CNN
@@
 	2850 2650 2950 2750
 $Comp
-L power:+5V #PWR?
+L power:+5V #PWR0160
 U 1 1 5E03D7B4
 P 3750 3150
-F 0 "#PWR?" H 3750 3000 50  0001 C CNN
+F 0 "#PWR0160" H 3750 3000 50  0001 C CNN
 F 1 "+5V" H 3765 3323 50  0000 C CNN
 F 2 "" H 3750 3150 50  0001 C CNN
@@
 $EndComp
 $Comp
-L power:GND #PWR?
+L power:GND #PWR0161
 U 1 1 5E040054
 P 3750 3350
-F 0 "#PWR?" H 3750 3100 50  0001 C CNN
+F 0 "#PWR0161" H 3750 3100 50  0001 C CNN
 F 1 "GND" H 3755 3177 50  0000 C CNN
 F 2 "" H 3750 3350 50  0001 C CNN
