File: kicad/cft/cft-ctl/cft_sbu.sch (KiCad schematic (older format))
At the start: 40 parts, among them U1 74HC251, U4 74LVC1G86, U5 74HC251, U56 74LVC1G373, U6 74LVC1G04, U7 74LVC1G11, U8 74LVC1G74, U9 74LVC1G332

Commit message: Reworked the SBU.
Connections:
- net labels added: CEXT10, CEXT8, CEXT9, CEXT[8..10]
- net labels removed: CRSVD10, CRSVD8, CRSVD9, CSRSVD10, CSRSVD8, CSRSVD9, CSRSVD[8..10]
Changed lines of the file:
@@
 Text Label 8300 2350 3    50   ~ 0
 ~COND0
-Text Label 6600 4150 0    50   ~ 0
-CRSVD10
 $Comp
 L alexios:74HC251 U?
@@
 Wire Wire Line
 	6950 3950 6600 3950
-Text Label 6600 3950 0    50   ~ 0
-CRSVD8
 Wire Wire Line
 	6950 4050 6600 4050
-Text Label 6600 4050 0    50   ~ 0
-CRSVD9
 Text Notes 8400 6100 0    50   ~ 0
 Metastability protection latch
@@
 Wire Notes Line width 24 style solid
 	8550 2350 8550 1550
-Text Label 8950 2950 0    50   ~ 0
-CRSVD10
-Text Label 8950 2750 0    50   ~ 0
-CRSVD8
-Text Label 8950 2850 0    50   ~ 0
-CRSVD9
 Entry Wire Line
 	6500 3850 6600 3950
@@
 	10100 3600 10200 3500
 Text Label 6750 3600 0    50   ~ 0
-CSRSVD[8..10]
-Text HLabel 8900 2750 0    50   3State ~ 0
-CSRSVD8
-Text HLabel 8900 2850 0    50   3State ~ 0
-CSRSVD9
-Text HLabel 8900 2950 0    50   3State ~ 0
-CSRSVD10
+CEXT[8..10]
 Text Notes 8450 2600 0    50   ~ 0
 Conditional inputs for future expansion
@@
 Wire Bus Line
 	5750 1800 5750 2500
+Text Label 8950 2750 0    50   ~ 0
+CEXT8
+Text Label 8950 2850 0    50   ~ 0
+CEXT9
+Text Label 8950 2950 0    50   ~ 0
+CEXT10
+Text HLabel 8900 2750 0    50   3State ~ 0
+CEXT8
+Text HLabel 8900 2850 0    50   3State ~ 0
+CEXT9
+Text HLabel 8900 2950 0    50   3State ~ 0
+CEXT10
+Text Label 6950 3950 2    50   ~ 0
+CEXT8
+Text Label 6950 4050 2    50   ~ 0
+CEXT9
+Text Label 6950 4150 2    50   ~ 0
+CEXT10
 $EndSCHEMATC

Commit message: Reworkd Interrupt FSM schematics.
Parts:
- D6: value D_Schottky_ALT -> CUS520; Mouser (none) -> 757-CUS520H3F; £0.043/100
- D7, D8: value D_Schottky_ALT -> CUS520
Changed lines of the file:
@@
 P 8100 1500
 F 0 "D6" H 8100 1600 50  0000 C CNN
-F 1 "D_Schottky_ALT" H 8100 1400 50  0000 C CNN
+F 1 "CUS520" H 8100 1400 50  0000 C CNN
 F 2 "alexios:SOD-323" H 8100 1500 50  0001 C CNN
 F 3 "~" H 8100 1500 50  0001 C CNN
+F 4 "757-CUS520H3F; £0.043/100" H 8100 1500 50  0001 C CNN "Mouser"
 	1    8100 1500
 	1    0    0    -1
@@
 P 8100 4050
 F 0 "D8" H 8100 4150 50  0000 C CNN
-F 1 "D_Schottky_ALT" H 8100 3950 50  0000 C CNN
+F 1 "CUS520" H 8100 3950 50  0000 C CNN
 F 2 "alexios:SOD-323" H 8100 4050 50  0001 C CNN
 F 3 "~" H 8100 4050 50  0001 C CNN
@@
 P 8100 2000
 F 0 "D7" H 8100 2100 50  0000 C CNN
-F 1 "D_Schottky_ALT" H 8100 1900 50  0000 C CNN
+F 1 "CUS520" H 8100 1900 50  0000 C CNN
 F 2 "alexios:SOD-323" H 8100 2000 50  0001 C CNN
 F 3 "~" H 8100 2000 50  0001 C CNN
@@
 Wire Wire Line
 	10000 2950 10100 2950
-Wire Bus Line
-	1050 5750 5650 5750
-Wire Bus Line
-	1050 1700 5650 1700
-Wire Bus Line
-	1650 5250 1650 5650
-Wire Bus Line
-	6500 3700 6500 4050
-Wire Bus Line
-	10200 2850 10200 3500
-Wire Bus Line
-	5750 2900 5750 5650
-Wire Bus Line
-	1400 1800 1400 4350
-Wire Bus Line
-	5750 1800 5750 2500
 Text Label 8950 2750 0    50   ~ 0
 CEXT8
@@
 Text Label 6950 4150 2    50   ~ 0
 CEXT10
+Wire Bus Line
+	1050 5750 5650 5750
+Wire Bus Line
+	1050 1700 5650 1700
+Wire Bus Line
+	1650 5250 1650 5650
+Wire Bus Line
+	6500 3700 6500 4050
+Wire Bus Line
+	10200 2850 10200 3500
+Wire Bus Line
+	5750 2900 5750 5650
+Wire Bus Line
+	1400 1800 1400 4350
+Wire Bus Line
+	5750 1800 5750 2500
 $EndSCHEMATC

Commit message: Bug fixes. Experimental board layout. Changed AGL and IR addresses to save two '138s.
Parts:
- removed C1, C4, C8: 100nF, Capacitor_SMD:C_0805_2012Metric, symbol Device:C_Small
- removed U6: 74LVC1G04, alexios:SOT-23-5_HandSoldering, symbol alexios:74AHC1G04
- removed U7: 74LVC1G11, alexios:SOT-23-6_Handsoldering, symbol alexios:74LVC1G11
- removed U9: 74LVC1G332, alexios:SOT-23-6_Handsoldering, symbol alexios:74LVC1G332
- U10: renamed from U?; footprint (none) -> alexios:SOIC-16
- U2, U3: renamed from U?; footprint (none) -> alexios:SOIC-14
- U4: value 74AHC1G86 -> 74LVC1G86
- gave numbers to parts that had none: 6
Other:
- moved on the sheet: C20, C21, C5, C9, U10C, U3D, U56B, U8B

Commit message: Routing CTL board. Fixing schematic bugs.
Parts:
- C2, C20, C21, C3, C5, C6, C7, C9: footprint Capacitor_SMD:C_0805_2012Metric -> alexios:C_SMD_0805_2012Metric_Pad1.15x1.40mm_HandSolder
Connections:
- net SL: now also U3.5; no longer U3.4
- net SV: now also U3.4; no longer U3.5
Changed lines of the file:
@@
 EESchema Schematic File Version 4
-LIBS:cft-ctl-cache
-EELAYER 26 0
+EELAYER 30 0
 EELAYER END
 $Descr A4 11693 8268
@@
 F 0 "C6" H 859 7446 50  0000 R CNN
 F 1 "100nF" H 859 7355 50  0000 R CNN
-F 2 "Capacitor_SMD:C_0805_2012Metric" H 950 7400 50  0001 C CNN
+F 2 "alexios:C_SMD_0805_2012Metric_Pad1.15x1.40mm_HandSolder" H 950 7400 50  0001 C CNN
 F 3 "~" H 950 7400 50  0001 C CNN
 	1    950  7400
@@
 F 0 "C7" H 2209 7446 50  0000 R CNN
 F 1 "100nF" H 2209 7355 50  0000 R CNN
-F 2 "Capacitor_SMD:C_0805_2012Metric" H 2300 7400 50  0001 C CNN
+F 2 "alexios:C_SMD_0805_2012Metric_Pad1.15x1.40mm_HandSolder" H 2300 7400 50  0001 C CNN
 F 3 "~" H 2300 7400 50  0001 C CNN
 	1    2300 7400
@@
 F 0 "C9" H 4909 7446 50  0000 R CNN
 F 1 "100nF" H 4909 7355 50  0000 R CNN
-F 2 "Capacitor_SMD:C_0805_2012Metric" H 5000 7400 50  0001 C CNN
+F 2 "alexios:C_SMD_0805_2012Metric_Pad1.15x1.40mm_HandSolder" H 5000 7400 50  0001 C CNN
 F 3 "~" H 5000 7400 50  0001 C CNN
 	1    5000 7400
@@
 F 0 "C2" H 859 6746 50  0000 R CNN
 F 1 "100nF" H 859 6655 50  0000 R CNN
-F 2 "Capacitor_SMD:C_0805_2012Metric" H 950 6700 50  0001 C CNN
+F 2 "alexios:C_SMD_0805_2012Metric_Pad1.15x1.40mm_HandSolder" H 950 6700 50  0001 C CNN
 F 3 "~" H 950 6700 50  0001 C CNN
 	1    950  6700
@@
 F 0 "C3" H 2209 6746 50  0000 R CNN
 F 1 "100nF" H 2209 6655 50  0000 R CNN
-F 2 "Capacitor_SMD:C_0805_2012Metric" H 2300 6700 50  0001 C CNN
+F 2 "alexios:C_SMD_0805_2012Metric_Pad1.15x1.40mm_HandSolder" H 2300 6700 50  0001 C CNN
 F 3 "~" H 2300 6700 50  0001 C CNN
 	1    2300 6700
@@
 F 0 "C5" H 3559 6746 50  0000 R CNN
 F 1 "100nF" H 3559 6655 50  0000 R CNN
-F 2 "Capacitor_SMD:C_0805_2012Metric" H 3650 6700 50  0001 C CNN
+F 2 "alexios:C_SMD_0805_2012Metric_Pad1.15x1.40mm_HandSolder" H 3650 6700 50  0001 C CNN
 F 3 "~" H 3650 6700 50  0001 C CNN
 	1    3650 6700
@@
 Text Label 8300 2350 3    50   ~ 0
 ~COND0
-$Comp
-L alexios:74HC251 U?
-U 1 1 5F031563
-P 7450 4550
-AR Path="/5F031563" Ref="U?"  Part="1"
-AR Path="/5EFCF155/5F031563" Ref="U5"  Part="1"
-F 0 "U5" H 7450 5417 50  0000 C CNN
-F 1 "74HC251" H 7450 5326 50  0000 C CNN
-F 2 "alexios:SOIC-16" H 7450 4500 50  0001 C CNN
-F 3 "http://www.ti.com/lit/gpn/sn74LS251" H 7450 4500 50  0001 C CNN
-	1    7450 4550
-	1    0    0    -1
-$EndComp
 $Comp
 L alexios:74AHC1G86 U?
@@
 F 0 "C21" H 4909 6746 50  0000 R CNN
 F 1 "100nF" H 4909 6655 50  0000 R CNN
-F 2 "Capacitor_SMD:C_0805_2012Metric" H 5000 6700 50  0001 C CNN
+F 2 "alexios:C_SMD_0805_2012Metric_Pad1.15x1.40mm_HandSolder" H 5000 6700 50  0001 C CNN
 F 3 "~" H 5000 6700 50  0001 C CNN
 	1    5000 6700
@@
 L alexios:74AC32 U3
 U 2 1 5E7773BA
-P 3150 4050
-F 0 "U3" H 3150 4125 50  0000 C CNN
-F 1 "74AC32" H 3150 4034 50  0000 C CNN
-F 2 "alexios:SOIC-14" H 3150 4050 50  0001 C CNN
-F 3 "http://www.ti.com/lit/gpn/sn74LS32" H 3150 4050 50  0001 C CNN
-	2    3150 4050
-	1    0    0    -1
+P 3150 4450
+F 0 "U3" H 3150 3983 50  0000 C CNN
+F 1 "74AC32" H 3150 4074 50  0000 C CNN
+F 2 "alexios:SOIC-14" H 3150 4450 50  0001 C CNN
+F 3 "http://www.ti.com/lit/gpn/sn74LS32" H 3150 4450 50  0001 C CNN
+	2    3150 4450
+	1    0    0    1
 $EndComp
 $Comp
@@
 F 0 "C20" H 3559 7446 50  0000 R CNN
 F 1 "100nF" H 3559 7355 50  0000 R CNN
-F 2 "Capacitor_SMD:C_0805_2012Metric" H 3650 7400 50  0001 C CNN
+F 2 "alexios:C_SMD_0805_2012Metric_Pad1.15x1.40mm_HandSolder" H 3650 7400 50  0001 C CNN
 F 3 "~" H 3650 7400 50  0001 C CNN
 	1    3650 7400
@@
 Connection ~ 3650 6800
 Connection ~ 3650 6600
+$Comp
+L alexios:74HC251 U?
+U 1 1 5F031563
+P 7450 4550
+AR Path="/5F031563" Ref="U?"  Part="1"
+AR Path="/5EFCF155/5F031563" Ref="U5"  Part="1"
+F 0 "U5" H 7450 5417 50  0000 C CNN
+F 1 "74HC251" H 7450 5326 50  0000 C CNN
+F 2 "alexios:SOIC-16" H 7450 4500 50  0001 C CNN
+F 3 "http://www.ti.com/lit/gpn/sn74LS251" H 7450 4500 50  0001 C CNN
+	1    7450 4550
+	1    0    0    -1
+$EndComp
+Wire Bus Line
+	1050 5750 5650 5750
 Wire Bus Line
 	1650 5250 1650 5650
@@
 	1050 1700 5650 1700
 Wire Bus Line
-	1050 5750 5650 5750
-Wire Bus Line
 	6500 3700 6500 4050

Commit message: Routing CTL board.
Connections:
- net SVL: now also U3.9; no longer U3.10
- net SZN: now also U3.10; no longer U3.9
Changed lines of the file:
@@
 L alexios:74AC32 U3
 U 3 1 5E77741B
-P 3900 3600
-F 0 "U3" H 3900 3675 50  0000 C CNN
-F 1 "74AC32" H 3900 3584 50  0000 C CNN
-F 2 "alexios:SOIC-14" H 3900 3600 50  0001 C CNN
-F 3 "http://www.ti.com/lit/gpn/sn74LS32" H 3900 3600 50  0001 C CNN
-	3    3900 3600
-	1    0    0    -1
+P 3900 4000
+F 0 "U3" H 3900 3533 50  0000 C CNN
+F 1 "74AC32" H 3900 3624 50  0000 C CNN
+F 2 "alexios:SOIC-14" H 3900 4000 50  0001 C CNN
+F 3 "http://www.ti.com/lit/gpn/sn74LS32" H 3900 4000 50  0001 C CNN
+	3    3900 4000
+	1    0    0    1
 $EndComp
 $Comp

Commit message: Routing CTL board
Connections:
- net ~COND0 renamed ~COND₀
- net ~COND1 renamed ~COND₁
Changed lines of the file:
@@
 ~SKIPEXT
 Text Label 8300 4600 3    50   ~ 0
-~COND0
+~COND₀
 $Comp
 L alexios:74LVC1G74 U?
@@
 Text Label 9900 5700 2    50   ~ 0
 CLK4
-Text Label 8650 5600 2    50   ~ 0
-~COND0
 Text HLabel 10700 4050 2    50   Output ~ 0
 ~COND
@@
 Connection ~ 8300 4050
 Text Label 8300 2350 3    50   ~ 0
-~COND0
+~COND₀
 $Comp
 L alexios:74AHC1G86 U?
@@
 ~RESET
 Text Label 9900 5600 2    50   ~ 0
-~COND1
+~COND₁
 Wire Notes Line width 24 style solid
 	8450 3750 10100 3750
@@
 Wire Bus Line
 	5750 1800 5750 2500
+Text Label 8650 5600 2    50   ~ 0
+~COND₀
 $EndSCHEMATC
