File: kicad/cft/cft-ctl/cft_microcode.sch (KiCad schematic (older format))
At the start: 19 parts, among them U43 74LVC1G08, U44 74HC161, U45 74HC85, U46 74LVC1G00, U47 SN74ACT1071

Commit message: Fine-tuning ALU and CTL boards.
Parts:
- JP4, JP5, JP6: footprint Jumper:SolderJumper-2_P1.3mm_Bridged_Pad1.0x1.5mm -> Jumper:SolderJumper-2_P1.3mm_Bridged_RoundedPad1.0x1.5mm
Other:
- note added: "2019 Design Update: both micro-Address Vector and micro-Control Vector have changed significantly\nin this version. Fields are much more vertical now, but the processor is also much more capable."
- note added: "The µPC controls the running of the processor. It counts up to 16, so microprograms can only have\nup to 16 steps. It resets to 0000 when the Control Unit asserts ~END~ or a processor extension\ncard asserts ~ENDEXT~ on the bus. It increments at the end of a processor cycle (rising edge of\nCLK4), and only when ~RSTHOLD~, ~HALT~ and ~WS~ are all deasserted."
- note removed: "2019 Design Update: both micro-Address Vector and\nmicro-Control Vector have changed significantly in this\nversion. Fields are much more vertical now."
- note removed: "The µPC controls the running of the processor. It counts up to 16, so\nmicroprograms can only have up to 16 steps. It resets to 0000 when the\nControl Unit asserts ~END~ or a processor extension card asserts ~ENDEXT~\non the bus. It increments at the end of a processor cycle (rising edge of\nCLK4), and only when ~RSTHOLD~, ~HALT~ and ~WS~ are all deasserted."
- moved on the sheet: C33, C34, JP4, JP5, JP6, R1, R24, R25, R26, R3, R4, U44A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

Commit message: Interim checkin. Redoing µPC and wait states.
Parts:
- removed U43: 74LVC1G08, alexios:SOT-23-5_HandSoldering, symbol alexios:74AHC1G08
- added U29: 74LVC1G0832, alexios:SOT-23-6_Handsoldering, symbol alexios:74LVC1G0832
- added U?: 74LVC1G3208, symbol alexios:74LVC1G3208
Connections:
- net labels added: CLK3
- wire segments 182 -> 181
Other:
- note added: "TODO: Rework This"
- note added: "~ENDEXT~\n\n X\n 0\n X"
- note added: "~END~\n\n X\n X\n 0"
- note added: "~WS~\n\n 0\n 1\n 1"
- note added: "~µPCCLR~\n\n 1\n 1\n 0"
Changed lines of the file:
@@
 Comment4 "sequencer.v"
 $EndDescr
-$Comp
-L alexios:74AHC1G08 U?
-U 1 1 5DEB2D66
-P 2150 1950
-AR Path="/5DEB2D66" Ref="U?"  Part="1"
-AR Path="/5DEAC282/5DEB2D66" Ref="U43"  Part="1"
-F 0 "U43" H 2075 2217 50  0000 C CNN
-F 1 "74LVC1G08" H 2075 2126 50  0000 C CNN
-F 2 "alexios:SOT-23-5_HandSoldering" H 1800 1950 50  0001 C CNN
-F 3 "http://www.ti.com/lit/sg/scyt129e/scyt129e.pdf" H 1800 1950 50  0001 C CNN
-	1    2150 1950
-	1    0    0    -1
-$EndComp
-Text Label 1550 1900 0    50   ~ 0
+Text Label 1550 1850 0    50   ~ 0
 ~ENDEXT
 Wire Wire Line
-	1550 2000 1850 2000
-Text HLabel 1150 1900 0    50   Input ~ 0
+	1550 1950 1850 1950
+Text HLabel 1150 1850 0    50   Input ~ 0
 ~ENDEXT
-Text Label 1550 2000 0    50   ~ 0
+Text Label 1550 1950 0    50   ~ 0
 ~END
 Wire Wire Line
@@
 	1    0    0    -1
 $EndComp
-Text Label 2350 1950 0    50   ~ 0
-~µPCCLR
 Text HLabel 1150 2550 0    50   Input ~ 0
 ~RSTHOLD
@@
 Text Label 1550 2150 0    50   ~ 0
 ~WS
-Wire Wire Line
-	2300 1950 2700 1950
-Wire Wire Line
-	2700 1950 2700 2050
 Text Label 3700 2150 2    50   ~ 0
 ~WS
@@
 Text Label 5000 1850 2    50   ~ 0
 UPC3
-Wire Wire Line
-	1150 1900 1200 1900
 Text Label 3700 2250 2    50   ~ 0
 ~HALT
@@
 Text HLabel 1150 4200 0    50   Input ~ 0
 ~COND
-Wire Wire Line
-	1150 2150 3750 2150
-Wire Wire Line
-	1150 2350 3750 2350
 Text HLabel 6650 6100 2    50   3State ~ 0
 FPD[0..7]
@@
 $EndComp
 Wire Wire Line
-	1200 1700 1200 1900
-Connection ~ 1200 1900
-Wire Wire Line
-	1200 1900 1850 1900
+	1200 1700 1200 1850
+Wire Wire Line
+	1200 1850 1850 1850
 Wire Wire Line
 	1350 1700 1350 2250
@@
 Wire Wire Line
 	1150 5650 2650 5650
-Connection ~ 2250 7300
-Connection ~ 2250 7500
-$Comp
-L alexios:74AHC1G08 U?
-U 2 1 5DEB32A6
-P 2700 7300
-AR Path="/5DEB32A6" Ref="U?"  Part="1"
-AR Path="/5DEAC282/5DEB32A6" Ref="U43"  Part="2"
-F 0 "U43" H 2780 7246 50  0000 L CNN
-F 1 "74LVC1G08" H 2780 7155 50  0000 L CNN
-F 2 "alexios:SOT-23-5_HandSoldering" H 2350 7300 50  0001 C CNN
-F 3 "http://www.ti.com/lit/sg/scyt129e/scyt129e.pdf" H 2350 7300 50  0001 C CNN
-	2    2700 7300
-	1    0    0    -1
-$EndComp
 $Comp
 L alexios:SN74ACT1071 U?
@@
 Wire Wire Line
 	1250 2250 1350 2250
+Connection ~ 1200 1850
+Wire Wire Line
+	1150 1850 1200 1850
+$Comp
+L alexios:74LVC1G0832 U29
+U 2 1 5ED0FCC2
+P 2600 7400
+F 0 "U29" H 2780 7446 50  0000 L CNN
+F 1 "74LVC1G0832" H 2780 7355 50  0000 L CNN
+F 2 "alexios:SOT-23-6_Handsoldering" H 2600 7400 50  0001 C CNN
+F 3 "http://www.ti.com/lit/ds/symlink/sn74lvc1g0832.pdf" H 2600 7400 50  0001 C CNN
+	2    2600 7400
+	1    0    0    -1
+$EndComp
+Connection ~ 2250 7500
+Connection ~ 2250 7300
+Text Notes -1900 2450 0    50   ~ 0
+~WS~\n\n 0\n 1\n 1
+Text Notes -1000 2450 0    50   ~ 0
+~µPCCLR~\n\n  1\n  1\n  0
+Wire Notes Line width 12 style solid
+	-1950 2000 -600 2000
+Wire Notes Line width 12 style solid
+	-600 2000 -600 2500
+Wire Notes Line width 12 style solid
+	-1950 2000 -1950 2500
+Wire Notes Line style solid
+	-1950 2160 -600 2160
+Wire Notes Line
+	-1060 2000 -1060 2500
+Wire Notes Line width 12 style solid
+	-1950 2500 -600 2500
+Text Notes -1350 2450 0    50   ~ 0
+~END~\n\n  X\n  X\n  0
+Text Notes -1700 2450 0    50   ~ 0
+~ENDEXT~\n\n   X\n   0\n   X
+Wire Wire Line
+	1150 2150 3750 2150
+$Comp
+L alexios:74LVC1G3208 U?
+U 1 1 5EDB6618
+P 2200 1950
+F 0 "U?" H 2225 2264 50  0000 C CNN
+F 1 "74LVC1G3208" H 2225 2173 50  0000 C CNN
+F 2 "" H 1875 1750 50  0001 C CNN
+F 3 "http://www.ti.com/lit/sg/scyt129e/scyt129e.pdf" H 1875 1750 50  0001 C CNN
+	1    2200 1950
+	1    0    0    -1
+$EndComp
+Wire Wire Line
+	1150 2350 3750 2350
+Wire Wire Line
+	1150 2050 1850 2050
+Text Label 1550 2050 0    50   ~ 0
+CLK3
+Text HLabel 1150 2050 0    50   Input ~ 0
+CLK3
+Text Notes 1850 2000 0    100  ~ 20
+TODO: Rework This
+Wire Notes Line
+	1350 3050 2000 3050
+Wire Notes Line
+	2000 3050 2000 3950
+Wire Notes Line
+	2000 3950 1350 3950
+Wire Notes Line
+	1350 3950 1350 3050
 Wire Bus Line
 	4550 3050 4550 3800

Commit message: Interim checkin.
Changed lines of the file:
@@
 Wire Wire Line
 	1150 2150 3750 2150
-$Comp
-L alexios:74LVC1G3208 U?
-U 1 1 5EDB6618
-P 2200 1950
-F 0 "U?" H 2225 2264 50  0000 C CNN
-F 1 "74LVC1G3208" H 2225 2173 50  0000 C CNN
-F 2 "" H 1875 1750 50  0001 C CNN
-F 3 "http://www.ti.com/lit/sg/scyt129e/scyt129e.pdf" H 1875 1750 50  0001 C CNN
-	1    2200 1950
-	1    0    0    -1
-$EndComp
 Wire Wire Line
 	1150 2350 3750 2350
@@
 Text HLabel 1150 2050 0    50   Input ~ 0
 CLK3
-Text Notes 1850 2000 0    100  ~ 20
+Text Notes 1900 1950 0    100  ~ 20
 TODO: Rework This
 Wire Notes Line
@@
 Wire Bus Line
 	9800 3000 9800 3450
+$Comp
+L alexios:74LVC1G3208 U?
+U 1 1 5EDB6618
+P -450 1400
+F 0 "U?" H -425 1714 50  0000 C CNN
+F 1 "74LVC1G3208" H -425 1623 50  0000 C CNN
+F 2 "" H -775 1200 50  0001 C CNN
+F 3 "http://www.ti.com/lit/sg/scyt129e/scyt129e.pdf" H -775 1200 50  0001 C CNN
+	1    -450 1400
+	1    0    0    -1
+$EndComp
 $EndSCHEMATC

Commit message: Working on updated µPC
Parts:
- removed U?: 74LVC1G3208, symbol alexios:74LVC1G3208
- added R?: 4.7kΩ, alexios:R_SMD_0805_2012Metric_Pad1.15x1.40mm_HandSolder, symbol Device:R_Small
- added U?: 74LVC1G373, symbol alexios:74LVC1G373
- added U?: 74LVC1G74, symbol alexios:74LVC1G74
- added U?: 74LVC1G0832, symbol alexios:74LVC1G0832
Connections:
- net labels added: ~WAITING
- wire segments 181 -> 205
- no-connect marks 3 -> 4
Other:
- note added: "Remove if BUS board is present!"
Changed lines of the file:
@@
 $Descr A4 11693 8268
 encoding utf-8
-Sheet 4 11
+Sheet 3 11
 Title "Microcode Sequencer"
 Date ""
@@
 Wire Notes Line
 	1350 3950 1350 3050
+$Comp
+L alexios:74LVC1G373 U?
+U 1 1 5ECAD5C4
+P -5750 3400
+F 0 "U?" H -5750 3767 50  0000 C CNN
+F 1 "74LVC1G373" H -5750 3676 50  0000 C CNN
+F 2 "" H -5850 3425 50  0001 C CNN
+F 3 "http://www.ti.com/lit/sg/scyt129e/scyt129e.pdf" H -5850 3425 50  0001 C CNN
+	1    -5750 3400
+	1    0    0    -1
+$EndComp
+$Comp
+L alexios:74LVC1G74 U?
+U 1 1 5ECAE60D
+P -4500 3450
+F 0 "U?" H -4500 3867 50  0000 C CNN
+F 1 "74LVC1G74" H -4500 3776 50  0000 C CNN
+F 2 "" H -4050 3450 50  0001 C CNN
+F 3 "https://assets.nexperia.com/documents/data-sheet/74LVC1G74.pdf" H -4050 3450 50  0001 C CNN
+	1    -4500 3450
+	1    0    0    -1
+$EndComp
+$Comp
+L power:GND #PWR?
+U 1 1 5ECD0CBA
+P -6250 3550
+F 0 "#PWR?" H -6250 3300 50  0001 C CNN
+F 1 "GND" H -6150 3550 50  0000 C CNN
+F 2 "" H -6250 3550 50  0001 C CNN
+F 3 "" H -6250 3550 50  0001 C CNN
+	1    -6250 3550
+	1    0    0    -1
+$EndComp
+Wire Wire Line
+	-6200 3500 -6250 3500
+Wire Wire Line
+	-6250 3500 -6250 3550
+Text Label -6800 3300 0    50   ~ 0
+~WS
+Wire Wire Line
+	-6800 3300 -6450 3300
+Text Label -6800 3700 0    50   ~ 0
+CLK3
+Wire Wire Line
+	-5300 3300 -4950 3300
+Wire Wire Line
+	-4950 3600 -5300 3600
+Text Label -5000 3600 2    50   ~ 0
+~RESET
+Text Label -5000 3500 2    50   ~ 0
+CLK3
+$Comp
+L Device:R_Small R?
+U 1 1 5EE87FE0
+P -6450 3050
+AR Path="/5EE87FE0" Ref="R?"  Part="1"
+AR Path="/5CC0D65F/5EE87FE0" Ref="R?"  Part="1"
+AR Path="/5D54E677/5EE87FE0" Ref="R?"  Part="1"
+AR Path="/5D62E1DC/5EE87FE0" Ref="R?"  Part="1"
+AR Path="/5DEAC282/5EE87FE0" Ref="R?"  Part="1"
+AR Path="/5F67D4B5/5EE87FE0" Ref="R?"  Part="1"
+AR Path="/5D46B22D/5EE87FE0" Ref="R?"  Part="1"
+F 0 "R?" H -6500 2900 50  0000 R CNN
+F 1 "4.7kΩ" H -6500 3000 50  0000 R CNN
+F 2 "alexios:R_SMD_0805_2012Metric_Pad1.15x1.40mm_HandSolder" H -6450 3050 50  0001 C CNN
+F 3 "~" H -6450 3050 50  0001 C CNN
+	1    -6450 3050
+	-1   0    0    1
+$EndComp
+Wire Wire Line
+	-6450 3150 -6450 3300
+Connection ~ -6450 3300
+Wire Wire Line
+	-6450 3300 -6200 3300
+Wire Wire Line
+	-6450 2900 -6450 2950
+$Comp
+L power:+5V #PWR?
+U 1 1 5EEAA993
+P -6450 2900
+F 0 "#PWR?" H -6450 2750 50  0001 C CNN
+F 1 "+5V" H -6435 3073 50  0000 C CNN
+F 2 "" H -6450 2900 50  0001 C CNN
+F 3 "" H -6450 2900 50  0001 C CNN
+	1    -6450 2900
+	1    0    0    -1
+$EndComp
+Wire Notes Line
+	-6600 2650 -6100 2650
+Wire Notes Line
+	-6100 2650 -6100 3200
+Wire Notes Line
+	-6100 3200 -6600 3200
+Wire Notes Line
+	-6600 3200 -6600 2650
+$Comp
+L alexios:74LVC1G0832 U?
+U 1 1 5EF32D3C
+P -3500 4050
+F 0 "U?" H -3475 3769 50  0000 C CNN
+F 1 "74LVC1G0832" H -3475 3860 50  0000 C CNN
+F 2 "" H -3500 4050 50  0001 C CNN
+F 3 "http://www.ti.com/lit/ds/symlink/sn74lvc1g0832.pdf" H -3500 4050 50  0001 C CNN
+	1    -3500 4050
+	1    0    0    1
+$EndComp
+Wire Wire Line
+	-3850 4050 -6800 4050
+Wire Wire Line
+	-6800 4150 -3850 4150
+Wire Wire Line
+	-4950 3400 -5000 3400
+Wire Wire Line
+	-5000 3400 -5000 3250
+$Comp
+L power:+5V #PWR?
+U 1 1 5F0024CB
+P -5000 3250
+F 0 "#PWR?" H -5000 3100 50  0001 C CNN
+F 1 "+5V" H -4985 3423 50  0000 C CNN
+F 2 "" H -5000 3250 50  0001 C CNN
+F 3 "" H -5000 3250 50  0001 C CNN
+	1    -5000 3250
+	1    0    0    -1
+$EndComp
+Wire Wire Line
+	-4050 3300 -3900 3300
+Wire Wire Line
+	-3900 3300 -3900 3950
+Wire Wire Line
+	-3900 3950 -3850 3950
+Text Label -3900 3700 1    50   ~ 0
+~WAITING
+NoConn ~ -4050 3600
+Text Label -3950 4050 2    50   ~ 0
+~ENDEXT
+Text Label -3950 4150 2    50   ~ 0
+~END
+Text Label -2600 4050 2    50   ~ 0
+~µPCCLR
+Wire Wire Line
+	-3100 4050 -2600 4050
+Wire Wire Line
+	-5400 3700 -5400 3500
+Wire Wire Line
+	-6800 3700 -6450 3700
+Wire Wire Line
+	-5400 3500 -4950 3500
+Wire Wire Line
+	-6200 3400 -6450 3400
+Wire Wire Line
+	-6450 3400 -6450 3700
+Connection ~ -6450 3700
+Wire Wire Line
+	-6450 3700 -5400 3700
+Text Label -6800 4050 0    50   ~ 0
+~ENDEXT
+Text Label -6800 4150 0    50   ~ 0
+~END
+Wire Wire Line
+	-5300 3800 -6800 3800
+Wire Wire Line
+	-5300 3600 -5300 3800
+Text Label -6800 3800 0    50   ~ 0
+~RESET
+Text Notes -6050 2900 0    50   ~ 0
+Remove if BUS board is present!
 Wire Bus Line
 	4550 3050 4550 3800
@@
 Wire Bus Line
 	9800 3000 9800 3450
-$Comp
-L alexios:74LVC1G3208 U?
-U 1 1 5EDB6618
-P -450 1400
-F 0 "U?" H -425 1714 50  0000 C CNN
-F 1 "74LVC1G3208" H -425 1623 50  0000 C CNN
-F 2 "" H -775 1200 50  0001 C CNN
-F 3 "http://www.ti.com/lit/sg/scyt129e/scyt129e.pdf" H -775 1200 50  0001 C CNN
-	1    -450 1400
-	1    0    0    -1
-$EndComp
 $EndSCHEMATC

Commit message: Reworking CTL and BUS boards. Added WAITING# signal to bus.
Parts:
- removed C34, C35: 100nF, alexios:C_SMD_0805_2012Metric_Pad1.15x1.40mm_HandSolder, symbol Device:C_Small
- removed R?: 4.7kΩ, alexios:R_SMD_0805_2012Metric_Pad1.15x1.40mm_HandSolder, symbol Device:R_Small
- removed U29: 74LVC1G0832, alexios:SOT-23-6_Handsoldering, symbol alexios:74LVC1G0832
- removed U44: 74HC161, alexios:SOIC-16, symbol alexios:74HC161
- removed U?: 74LVC1G373, symbol alexios:74LVC1G373
- removed U?: 74LVC1G74, symbol alexios:74LVC1G74
- removed U?: 74LVC1G0832, symbol alexios:74LVC1G0832
Connections:
- no-connect marks 4 -> 2
Other:
- note added: "The Microprogram Sequencer"
- note added: "This is the inner sanctum of the control unit, reading, and decoding microprograms\ninto various fields."
- note removed: "Microprogram Counter (µPC)"
- note removed: "Remove if BUS board is present!"
- note removed: "TODO: Rework This"
- note removed: "The µPC controls the running of the processor. It counts up to 16, so microprograms can only have\nup to 16 steps. It resets to 0000 when the Control Unit asserts ~END~ or a processor extension\ncard asserts ~ENDEXT~ on the bus. It increments at the end of a processor cycle (rising edge of\nCLK4), and only when ~RSTHOLD~, ~HALT~ and ~WS~ are all deasserted."
- note removed: "~ENDEXT~\n\n X\n 0\n X"
- note removed: "~END~\n\n X\n X\n 0"
- note removed: "~WS~ is pulled up by the Wait State Handler circuitry."
- note removed: "~WS~\n\n 0\n 1\n 1"
- note removed: "~µPCCLR~\n\n 1\n 1\n 0"
- moved on the sheet: C37, C38, R24, U45B, U46B

Commit message: Reworking boards for new bus definitions and control store.
Parts:
- removed R26: 4.7kΩ, alexios:R_SMD_0805_2012Metric_Pad1.15x1.40mm_HandSolder, symbol Device:R_Small
- removed U46: 74LVC1G00, alexios:SOT-23-5_HandSoldering, symbol alexios:74LVC1G00
- added C34: 100nF, alexios:C_SMD_0805_2012Metric_Pad1.15x1.40mm_HandSolder, symbol Device:C_Small
- added U29: 74LVC1G74, alexios:SOIC-8, symbol alexios:74LVC1G74
- added U46: 74LVC1G373, alexios:SOT-23-6_Handsoldering, symbol alexios:74LVC1G373
Connections:
- net +5V: now also C34.1, U29.7 (~PRE), U29.8 (VCC), U46.5 (VCC)
- net GND: now also C34.2, U29.4 (GND), U46.2 (GND), U46.6 (~OE)
- net ~CSE: now also U29.3 (~Q)
- net ~HALT: now also U46.3 (D)
- net ~RESET: now also U29.6 (~CLR)
- new net: U29.2 (D), U46.4 (Q)
- new net CLK1: U29.1 (CLK), U46.1 (LE)
- no-connect marks 2 -> 3
Other:
- note added: "The Microcode Store is enabled when ~RESET~ and ~HALT~\nare both deasserted. This is synced with CLK1 to ensure\nthe processor doesn't halt mid-microinstruction."
- note removed: "Remove\npull-up if\nIN-RSVD used."
- note removed: "The Microcode Store is enabled\nwhen ~RESET~ and ~HALT~\nare both deasserted."
- moved on the sheet: C33, C37, C38, JP4, JP5, JP6, R1, R24, R25, R3, R4, U45A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
