File: kicad/cft/cft-ctl/cft-ctl.sch (KiCad schematic (older format))
At the start: 5 parts, among them U9 74LVC1G32

Commit message: Reworking CTL and BUS boards. Added WAITING# signal to bus.
Changed lines of the file:
@@
 $Descr A4 11693 8268
 encoding utf-8
-Sheet 1 11
+Sheet 1 12
 Title "Control Unit Board"
 Date ""
@@
 Comment4 ""
 $EndDescr
-Text Label 900  4750 0    50   ~ 0
-IN-RSVD
-Text Label 900  4650 0    50   ~ 0
-~COND
 Text Label 3250 5650 2    50   ~ 0
 FPD[0..7]
@@
 	8350 3300 7800 3300
 Wire Wire Line
+	8350 4200 7800 4200
+Wire Wire Line
+	8350 4300 7800 4300
+Wire Wire Line
 	8350 4100 7800 4100
-Wire Wire Line
-	8350 4200 7800 4200
-Wire Wire Line
-	8350 4000 7800 4000
 Wire Wire Line
 	8350 3900 7800 3900
@@
 Text Label 7800 3900 0    50   ~ 0
 ~WS
-Text Label 7800 4000 0    50   ~ 0
+Text Label 7800 4100 0    50   ~ 0
 ~ENDEXT
-Text Label 7800 4100 0    50   ~ 0
+Text Label 7800 4200 0    50   ~ 0
 ~SKIPEXT
-Text Label 7800 4200 0    50   ~ 0
+Text Label 7800 4300 0    50   ~ 0
 ~HALT
 Text Label 7800 4500 0    50   ~ 0
@@
 Wire Wire Line
 	9500 5500 10100 5500
-Text Label 900  4450 0    50   ~ 0
-IDX0
-Text Label 900  4550 0    50   ~ 0
-IDX1
-$Sheet
-S 1500 3500 1150 2450
-U 5DEAC282
-F0 "Microprogram Sequencer" 50
-F1 "cft_microcode.sch" 50
-F2 "~ENDEXT" I L 1500 4250 50
-F3 "~RSTHOLD" I L 1500 3750 50
-F4 "~WS" I L 1500 4350 50
-F5 "~HALT" I L 1500 4150 50
-F6 "CLK4" I L 1500 4050 50
-F7 "~RESET" I L 1500 3650 50
-F8 "RADDR[0..4]" O R 2650 3650 50
-F9 "WADDR[0..4]" O R 2650 3750 50
-F10 "COND[0..4]" O R 2650 3850 50
-F11 "ACTION[0..3]" O R 2650 3950 50
-F12 "~MEM" O R 2650 4050 50
-F13 "~IO" O R 2650 4150 50
-F14 "~R" O R 2650 4250 50
-F15 "~WEN" O R 2650 4350 50
-F16 "~END" O R 2650 4450 50
-F17 "~IRQSµC" I L 1500 5750 50
-F18 "IN-RSVD" I L 1500 4750 50
-F19 "~COND" I L 1500 4650 50
-F20 "FPD[0..7]" T R 2650 5650 50
-F21 "~FPµA0" I R 2650 5250 50
-F22 "~FPµC0" I R 2650 5350 50
-F23 "~FPµC1" I R 2650 5450 50
-F24 "~FPµC2" I R 2650 5550 50
-F25 "FPFETCH" O R 2650 5150 50
-F26 "IDX0" I L 1500 4450 50
-F27 "IDX1" I L 1500 4550 50
-F28 "IR7" I L 1500 4850 50
-F29 "IR8" I L 1500 4950 50
-F30 "IR9" I L 1500 5050 50
-F31 "IR10" I L 1500 5150 50
-F32 "IR11" I L 1500 5250 50
-F33 "IR12" I L 1500 5350 50
-F34 "IR13" I L 1500 5450 50
-F35 "IR14" I L 1500 5550 50
-F36 "IR15" I L 1500 5650 50
-F37 "CLK2" I L 1500 3850 50
-F38 "CLK3" I L 1500 3950 50
-$EndSheet
 Wire Wire Line
 	900  3850 1500 3850
 Text Label 900  3850 0    50   ~ 0
 CLK2
-Wire Wire Line
-	1500 5750 1000 5750
-Text Label 900  4850 0    50   ~ 0
-IR7
-Text Label 900  4950 0    50   ~ 0
-IR8
-Text Label 900  5050 0    50   ~ 0
-IR9
-Text Label 900  5150 0    50   ~ 0
-IR10
-Text Label 900  5250 0    50   ~ 0
-IR11
-Text Label 900  5350 0    50   ~ 0
-IR12
-Text Label 900  5450 0    50   ~ 0
-IR13
-Text Label 900  5550 0    50   ~ 0
-IR14
-Text Label 900  5650 0    50   ~ 0
-IR15
-Text Label 1000 5750 0    50   ~ 0
-~IRQSµC
 Text Label 10100 5500 2    50   ~ 0
 IN-RSVD
@@
 Text Label 10100 4600 2    50   ~ 0
 POWEROK
-Entry Wire Line
-	800  5650 900  5550
-Entry Wire Line
-	800  5550 900  5450
-Entry Wire Line
-	800  5450 900  5350
-Entry Wire Line
-	800  5350 900  5250
-Entry Wire Line
-	800  5250 900  5150
-Entry Wire Line
-	800  5150 900  5050
-Entry Wire Line
-	800  5050 900  4950
-Entry Wire Line
-	800  4950 900  4850
-Entry Wire Line
-	800  5750 900  5650
 Wire Bus Line
 	2650 3650 3250 3650
@@
 Wire Wire Line
 	900  3650 1500 3650
-Text Label 800  5450 1    50   ~ 0
-IR[0..15]
 Text Notes 800  1000 0    100  ~ 20
 The Control Unit Board
@@
 F20 "~R" U L 8350 3700 50
 F21 "~WS" U L 8350 3900 50
-F22 "~ENDEXT" U L 8350 4000 50
-F23 "~SKIPEXT" U L 8350 4100 50
-F24 "~HALT" U L 8350 4200 50
+F22 "~ENDEXT" U L 8350 4100 50
+F23 "~SKIPEXT" U L 8350 4200 50
+F24 "~HALT" U L 8350 4300 50
 F25 "ACTION[0..3]" U L 8350 4500 50
 F26 "WADDR[0..4]" U L 8350 4600 50
@@
 F67 "C39" U R 9500 5400 50
 F68 "C40" U R 9500 5500 50
+F69 "~WAITING" O L 8350 4000 50
 $EndSheet
-Wire Wire Line
-	1500 4650 900  4650
-Wire Wire Line
-	1500 5650 900  5650
-Wire Wire Line
-	1500 5550 900  5550
-Wire Wire Line
-	1500 5450 900  5450
-Wire Wire Line
-	1500 5350 900  5350
-Wire Wire Line
-	1500 5250 900  5250
-Wire Wire Line
-	1500 5150 900  5150
-Wire Wire Line
-	1500 5050 900  5050
-Wire Wire Line
-	1500 4950 900  4950
-Wire Wire Line
-	1500 4850 900  4850
-Wire Wire Line
-	1500 4550 900  4550
-Wire Wire Line
-	1500 4450 900  4450
-Wire Wire Line
-	900  4750 1500 4750
 Wire Wire Line
 	1500 4150 900  4150
@@
 F14 "CEXT10" T L 4200 5750 50
 $EndSheet
+Wire Wire Line
+	8350 4000 7800 4000
+Text Label 7800 4000 0    50   ~ 0
+~WAITING
+$Sheet
+S 1500 3500 1150 2450
+U 5DEAC282
+F0 "Microprogram Sequencer" 50
+F1 "cft_microcode.sch" 50
+F2 "~ENDEXT" I L 1500 4250 50
+F3 "~RSTHOLD" I L 1500 3750 50
+F4 "~WS" I L 1500 4350 50
+F5 "~HALT" I L 1500 4150 50
+F6 "CLK4" I L 1500 4050 50
+F7 "~RESET" I L 1500 3650 50
+F8 "RADDR[0..4]" O R 2650 3650 50
+F9 "WADDR[0..4]" O R 2650 3750 50
+F10 "COND[0..4]" O R 2650 3850 50
+F11 "ACTION[0..3]" O R 2650 3950 50
+F12 "~MEM" O R 2650 4050 50
+F13 "~IO" O R 2650 4150 50
+F14 "~R" O R 2650 4250 50
+F15 "~WEN" O R 2650 4350 50
+F16 "~END" O R 2650 4450 50
+F17 "~IRQSµC" I L 1500 5750 50
+F18 "IN-RSVD" I L 1500 4750 50
+F19 "~COND" I L 1500 4650 50
+F20 "FPD[0..7]" T R 2650 5650 50
+F21 "~FPµA0" I R 2650 5250 50
+F22 "~FPµC0" I R 2650 5350 50
+F23 "~FPµC1" I R 2650 5450 50
+F24 "~FPµC2" I R 2650 5550 50
+F25 "FPFETCH" O R 2650 5150 50
+F26 "IDX0" I L 1500 4450 50
+F27 "IDX1" I L 1500 4550 50
+F28 "IR7" I L 1500 4850 50
+F29 "IR8" I L 1500 4950 50
+F30 "IR9" I L 1500 5050 50
+F31 "IR10" I L 1500 5150 50
+F32 "IR11" I L 1500 5250 50
+F33 "IR12" I L 1500 5350 50
+F34 "IR13" I L 1500 5450 50
+F35 "IR14" I L 1500 5550 50
+F36 "IR15" I L 1500 5650 50
+F37 "CLK2" I L 1500 3850 50
+F38 "CLK3" I L 1500 3950 50
+F39 "~WAITING" I L 1500 5850 50
+$EndSheet
+Wire Wire Line
+	900  4750 1500 4750
+Wire Wire Line
+	1500 4450 900  4450
+Wire Wire Line
+	1500 4550 900  4550
+Wire Wire Line
+	1500 4850 900  4850
+Wire Wire Line
+	1500 4950 900  4950
+Wire Wire Line
+	1500 5050 900  5050
+Wire Wire Line
+	1500 5150 900  5150
+Wire Wire Line
+	1500 5250 900  5250
+Wire Wire Line
+	1500 5350 900  5350
+Wire Wire Line
+	1500 5450 900  5450
+Wire Wire Line
+	1500 5550 900  5550
+Wire Wire Line
+	1500 5650 900  5650
+Wire Wire Line
+	1500 4650 900  4650
+Text Label 800  5450 1    50   ~ 0
+IR[0..15]
+Entry Wire Line
+	800  5750 900  5650
+Entry Wire Line
+	800  4950 900  4850
+Entry Wire Line
+	800  5050 900  4950
+Entry Wire Line
+	800  5150 900  5050
+Entry Wire Line
+	800  5250 900  5150
+Entry Wire Line
+	800  5350 900  5250
+Entry Wire Line
+	800  5450 900  5350
+Entry Wire Line
+	800  5550 900  5450
+Entry Wire Line
+	800  5650 900  5550
+Text Label 1000 5750 0    50   ~ 0
+~IRQSµC
+Text Label 900  5650 0    50   ~ 0
+IR15
+Text Label 900  5550 0    50   ~ 0
+IR14
+Text Label 900  5450 0    50   ~ 0
+IR13
+Text Label 900  5350 0    50   ~ 0
+IR12
+Text Label 900  5250 0    50   ~ 0
+IR11
+Text Label 900  5150 0    50   ~ 0
+IR10
+Text Label 900  5050 0    50   ~ 0
+IR9
+Text Label 900  4950 0    50   ~ 0
+IR8
+Text Label 900  4850 0    50   ~ 0
+IR7
+Wire Wire Line
+	1500 5750 1000 5750
+Text Label 900  4550 0    50   ~ 0
+IDX1
+Text Label 900  4450 0    50   ~ 0
+IDX0
+Text Label 900  4650 0    50   ~ 0
+~COND
+Text Label 900  4750 0    50   ~ 0
+IN-RSVD
+Wire Wire Line
+	1500 5850 1000 5850
+Text Label 1000 5850 0    50   ~ 0
+~WAITING
 Wire Bus Line
 	9950 1450 9950 2100

Commit message: Working on CTL board.
Changed lines of the file:
@@
 F15 "~WEN" O R 2650 4350 50
 F16 "~END" O R 2650 4450 50
-F17 "~IRQSµC" I L 1500 5750 50
-F18 "IN-RSVD" I L 1500 4750 50
-F19 "~COND" I L 1500 4650 50
-F20 "FPD[0..7]" T R 2650 5650 50
-F21 "~FPµA0" I R 2650 5250 50
-F22 "~FPµC0" I R 2650 5350 50
-F23 "~FPµC1" I R 2650 5450 50
-F24 "~FPµC2" I R 2650 5550 50
-F25 "FPFETCH" O R 2650 5150 50
-F26 "IDX0" I L 1500 4450 50
-F27 "IDX1" I L 1500 4550 50
-F28 "IR7" I L 1500 4850 50
-F29 "IR8" I L 1500 4950 50
-F30 "IR9" I L 1500 5050 50
-F31 "IR10" I L 1500 5150 50
-F32 "IR11" I L 1500 5250 50
-F33 "IR12" I L 1500 5350 50
-F34 "IR13" I L 1500 5450 50
-F35 "IR14" I L 1500 5550 50
-F36 "IR15" I L 1500 5650 50
-F37 "CLK2" I L 1500 3850 50
-F38 "CLK3" I L 1500 3950 50
-F39 "~WAITING" I L 1500 5850 50
+F17 "~IRQSµC" I L 1500 5650 50
+F18 "~COND" I L 1500 4650 50
+F19 "FPD[0..7]" T R 2650 5650 50
+F20 "~FPµA0" I R 2650 5250 50
+F21 "~FPµC0" I R 2650 5350 50
+F22 "~FPµC1" I R 2650 5450 50
+F23 "~FPµC2" I R 2650 5550 50
+F24 "FPFETCH" O R 2650 5150 50
+F25 "IDX0" I L 1500 4450 50
+F26 "IDX1" I L 1500 4550 50
+F27 "IR7" I L 1500 4750 50
+F28 "IR8" I L 1500 4850 50
+F29 "IR9" I L 1500 4950 50
+F30 "IR10" I L 1500 5050 50
+F31 "IR11" I L 1500 5150 50
+F32 "IR12" I L 1500 5250 50
+F33 "IR13" I L 1500 5350 50
+F34 "IR14" I L 1500 5450 50
+F35 "IR15" I L 1500 5550 50
+F36 "CLK2" I L 1500 3850 50
+F37 "CLK3" I L 1500 3950 50
+F38 "~WAITING" I L 1500 5750 50
 $EndSheet
-Wire Wire Line
-	900  4750 1500 4750
 Wire Wire Line
 	1500 4450 900  4450
 Wire Wire Line
 	1500 4550 900  4550
+Wire Wire Line
+	1500 4750 900  4750
 Wire Wire Line
 	1500 4850 900  4850
@@
 	1500 5550 900  5550
 Wire Wire Line
-	1500 5650 900  5650
-Wire Wire Line
 	1500 4650 900  4650
-Text Label 800  5450 1    50   ~ 0
+Text Label 800  5350 1    50   ~ 0
 IR[0..15]
 Entry Wire Line
-	800  5750 900  5650
+	800  5650 900  5550
+Entry Wire Line
+	800  4850 900  4750
 Entry Wire Line
 	800  4950 900  4850
@@
 Entry Wire Line
 	800  5550 900  5450
-Entry Wire Line
-	800  5650 900  5550
-Text Label 1000 5750 0    50   ~ 0
+Text Label 1000 5650 0    50   ~ 0
 ~IRQSµC
-Text Label 900  5650 0    50   ~ 0
+Text Label 900  5550 0    50   ~ 0
 IR15
-Text Label 900  5550 0    50   ~ 0
+Text Label 900  5450 0    50   ~ 0
 IR14
-Text Label 900  5450 0    50   ~ 0
+Text Label 900  5350 0    50   ~ 0
 IR13
-Text Label 900  5350 0    50   ~ 0
+Text Label 900  5250 0    50   ~ 0
 IR12
-Text Label 900  5250 0    50   ~ 0
+Text Label 900  5150 0    50   ~ 0
 IR11
-Text Label 900  5150 0    50   ~ 0
+Text Label 900  5050 0    50   ~ 0
 IR10
-Text Label 900  5050 0    50   ~ 0
+Text Label 900  4950 0    50   ~ 0
 IR9
-Text Label 900  4950 0    50   ~ 0
+Text Label 900  4850 0    50   ~ 0
 IR8
-Text Label 900  4850 0    50   ~ 0
+Text Label 900  4750 0    50   ~ 0
 IR7
 Wire Wire Line
-	1500 5750 1000 5750
+	1500 5650 1000 5650
 Text Label 900  4550 0    50   ~ 0
 IDX1
@@
 Text Label 900  4650 0    50   ~ 0
 ~COND
-Text Label 900  4750 0    50   ~ 0
-IN-RSVD
 Wire Wire Line
-	1500 5850 1000 5850
-Text Label 1000 5850 0    50   ~ 0
+	1500 5750 1000 5750
+Text Label 1000 5750 0    50   ~ 0
 ~WAITING
 Wire Bus Line
 	9950 1450 9950 2100
 Wire Bus Line
-	800  4950 800  5750
+	800  4850 800  5650
 $EndSCHEMATC

Commit message: Synced schematics with recent timing changes.
Parts:
- added JP1: Jumper_3_Bridged12, Jumper:SolderJumper-2_P1.3mm_Bridged_RoundedPad1.0x1.5mm, symbol alexios:Jumper_3_Bridged12
Connections:
- net ~WAITING: now also JP1.1 (A)
- net ~WS: now also JP1.3 (B)
- new net ~µPC-INH: JP1.2 (C)
Changed lines of the file:
@@
 F36 "CLK2" I L 1500 3850 50
 F37 "CLK3" I L 1500 3950 50
-F38 "~WAITING" I L 1500 5750 50
+F38 "~µPC-INH" I L 1500 5750 50
 $EndSheet
 Wire Wire Line
@@
 	1500 5750 1000 5750
 Text Label 1000 5750 0    50   ~ 0
-~WAITING
+~µPC-INH
 $Sheet
 S 8350 1450 1150 4200
@@
 Text Label 7800 3900 0    50   ~ 0
 ~WEN
-Wire Bus Line
-	800  4850 800  5650
-Wire Bus Line
-	9950 1450 9950 2100
 Wire Wire Line
 	6250 3750 6250 5750
@@
 Text Label 5950 4450 2    50   ~ 0
 ~COND
+Wire Wire Line
+	7150 5100 7650 5100
+Text Label 7650 5100 2    50   ~ 0
+~µPC-INH
+$Comp
+L alexios:Jumper_3_Bridged12 JP1
+U 1 1 6091E201
+P 7000 5100
+F 0 "JP1" V 7000 5167 50  0000 L CNN
+F 1 "Jumper_3_Bridged12" H 7000 5210 50  0001 C CNN
+F 2 "Jumper:SolderJumper-2_P1.3mm_Bridged_RoundedPad1.0x1.5mm" H 7000 5100 50  0001 C CNN
+F 3 "~" H 7000 5100 50  0001 C CNN
+	1    7000 5100
+	0    -1   1    0
+$EndComp
+Wire Wire Line
+	7000 4850 7000 4800
+Wire Wire Line
+	7000 4800 6400 4800
+Wire Wire Line
+	7000 5350 7000 5400
+Wire Wire Line
+	7000 5400 6400 5400
+Text Label 6400 4800 0    50   ~ 0
+~WAITING
+Text Label 6400 5400 0    50   ~ 0
+~WS
+Wire Bus Line
+	9950 1450 9950 2100
+Wire Bus Line
+	800  4850 800  5650
 $EndSCHEMATC

Commit message: Reverted pinout to drop WEN. Routing BUS board.
Changed lines of the file:
@@
 F68 "C40" U R 9500 5500 50
 F69 "~WAITING" O L 8350 4100 50
-F70 "~WEN" U L 8350 3900 50
 $EndSheet
 Wire Wire Line
-	8350 3900 7800 3900
-Text Label 7800 3900 0    50   ~ 0
-~WEN
-Wire Wire Line
 	6250 3750 6250 5750

Commit message: Working on CTL board.
Changed lines of the file:
@@
 	900  3850 1500 3850
 Text Label 900  3850 0    50   ~ 0
-CLK2
+CLK1
 Text Label 10100 5500 2    50   ~ 0
 IN-RSVD
@@
 	1500 4050 900  4050
 Text Label 900  3950 0    50   ~ 0
-CLK3
+CLK2
 Wire Wire Line
 	6250 6550 6250 5850
@@
 F34 "IR14" I L 1500 5450 50
 F35 "IR15" I L 1500 5550 50
-F36 "CLK2" I L 1500 3850 50
-F37 "CLK3" I L 1500 3950 50
+F36 "CLK1" I L 1500 3850 50
+F37 "CLK2" I L 1500 3950 50
 F38 "~µPC-INH" I L 1500 5750 50
 $EndSheet

Commit message: Working on CTL and Front Panel boards.
Parts:
- JP1: footprint Jumper:SolderJumper-2_P1.3mm_Bridged_RoundedPad1.0x1.5mm -> Jumper:SolderJumper-3_P1.3mm_Bridged12_RoundedPad1.0x1.5mm
Changed lines of the file:
@@
 F 0 "JP1" V 7000 5167 50  0000 L CNN
 F 1 "Jumper_3_Bridged12" H 7000 5210 50  0001 C CNN
-F 2 "Jumper:SolderJumper-2_P1.3mm_Bridged_RoundedPad1.0x1.5mm" H 7000 5100 50  0001 C CNN
+F 2 "Jumper:SolderJumper-3_P1.3mm_Bridged12_RoundedPad1.0x1.5mm" H 7000 5100 50  0001 C CNN
 F 3 "~" H 7000 5100 50  0001 C CNN
 	1    7000 5100
