File: kicad/cft/cft-ctl/cpu_microcode_fp.sch (KiCad schematic (older format))
At the start: 8 parts, among them U16 74HC541, U17 74HC541, U21 74HC541, U31 74HC541

Commit message: Routing CTL board. Fixing schematic bugs.
Parts:
- C39, C40, C41, C43: footprint Capacitor_SMD:C_0805_2012Metric -> alexios:C_SMD_0805_2012Metric_Pad1.15x1.40mm_HandSolder
Changed lines of the file:
@@
 EESchema Schematic File Version 4
-LIBS:cft-ctl-cache
-EELAYER 26 0
+EELAYER 30 0
 EELAYER END
 $Descr A4 11693 8268
 encoding utf-8
-Sheet 8 11
+Sheet 7 11
 Title "Microcode Front Panel Buffers"
 Date ""
@@
 F 0 "C39" H 3959 5446 50  0000 R CNN
 F 1 "100nF" H 3959 5355 50  0000 R CNN
-F 2 "Capacitor_SMD:C_0805_2012Metric" H 4050 5400 50  0001 C CNN
+F 2 "alexios:C_SMD_0805_2012Metric_Pad1.15x1.40mm_HandSolder" H 4050 5400 50  0001 C CNN
 F 3 "~" H 4050 5400 50  0001 C CNN
 	1    4050 5400
@@
 F 0 "C43" H 5259 5446 50  0000 R CNN
 F 1 "100nF" H 5259 5355 50  0000 R CNN
-F 2 "Capacitor_SMD:C_0805_2012Metric" H 5350 5400 50  0001 C CNN
+F 2 "alexios:C_SMD_0805_2012Metric_Pad1.15x1.40mm_HandSolder" H 5350 5400 50  0001 C CNN
 F 3 "~" H 5350 5400 50  0001 C CNN
 	1    5350 5400
@@
 F 0 "C40" H 3959 6146 50  0000 R CNN
 F 1 "100nF" H 3959 6055 50  0000 R CNN
-F 2 "Capacitor_SMD:C_0805_2012Metric" H 4050 6100 50  0001 C CNN
+F 2 "alexios:C_SMD_0805_2012Metric_Pad1.15x1.40mm_HandSolder" H 4050 6100 50  0001 C CNN
 F 3 "~" H 4050 6100 50  0001 C CNN
 	1    4050 6100
@@
 F 0 "C41" H 5259 6146 50  0000 R CNN
 F 1 "100nF" H 5259 6055 50  0000 R CNN
-F 2 "Capacitor_SMD:C_0805_2012Metric" H 5350 6100 50  0001 C CNN
+F 2 "alexios:C_SMD_0805_2012Metric_Pad1.15x1.40mm_HandSolder" H 5350 6100 50  0001 C CNN
 F 3 "~" H 5350 6100 50  0001 C CNN
 	1    5350 6100
