File: kicad/cft/cft-reg/bus.sch (KiCad schematic (older format))
At the start: 3 parts, among them P1 CFT-2019-Bus

Commit message: Working on ALU.
Parts:
- renumbered C7 to C?, C8 to C?, P1 to P?
Changed lines of the file:
@@
 EESchema Schematic File Version 4
+LIBS:cft-alu-cache
 LIBS:cft-reg-cache
 EELAYER 30 0
@@
 $Descr A4 11693 8268
 encoding utf-8
-Sheet 2 6
+Sheet 8 8
 Title ""
 Date ""
@@
 $EndDescr
 $Comp
-L alexios:CFT-2019-Bus P1
+L alexios:CFT-2019-Bus P?
 U 1 1 5D36087B
 P 3150 1600
-AR Path="/5D34E810/5D36087B" Ref="P1"  Part="1"
+AR Path="/5D34E810/5D36087B" Ref="P?"  Part="1"
 AR Path="/5D36B851/5D36087B" Ref="P?"  Part="1"
 AR Path="/5F1DB2E8/5D36087B" Ref="P?"  Part="1"
 AR Path="/5D36087B" Ref="P?"  Part="1"
-F 0 "P1" H 3150 1767 50  0000 C CNN
+F 0 "P?" H 3150 1767 50  0000 C CNN
 F 1 "CFT-2019-Bus" H 3150 1676 50  0000 C CNN
 F 2 "alexios:CFT-2019-Card-Edge" H 3100 700 50  0001 C CNN
@@
 $EndComp
 $Comp
-L alexios:CFT-2019-Bus P1
+L alexios:CFT-2019-Bus P?
 U 2 1 5D360881
 P 5900 1600
-AR Path="/5D34E810/5D360881" Ref="P1"  Part="2"
+AR Path="/5D34E810/5D360881" Ref="P?"  Part="2"
 AR Path="/5D36B851/5D360881" Ref="P?"  Part="2"
 AR Path="/5F1DB2E8/5D360881" Ref="P?"  Part="2"
 AR Path="/5D360881" Ref="P?"  Part="2"
-F 0 "P1" H 5900 1767 50  0000 C CNN
+F 0 "P?" H 5900 1767 50  0000 C CNN
 F 1 "CFT-2019-Bus" H 5900 1676 50  0000 C CNN
 F 2 "alexios:CFT-2019-Card-Edge" H 5850 700 50  0001 C CNN
@@
 RADDR[0..4]
 $Comp
-L alexios:CFT-2019-Bus P1
+L alexios:CFT-2019-Bus P?
 U 4 1 5D360875
 P 9350 4650
-AR Path="/5D34E810/5D360875" Ref="P1"  Part="4"
+AR Path="/5D34E810/5D360875" Ref="P?"  Part="4"
 AR Path="/5D36B851/5D360875" Ref="P?"  Part="4"
 AR Path="/5F1DB2E8/5D360875" Ref="P?"  Part="4"
 AR Path="/5D360875" Ref="P?"  Part="4"
-F 0 "P1" H 9350 4817 50  0000 C CNN
+F 0 "P?" H 9350 4817 50  0000 C CNN
 F 1 "CFT-2019-Bus" H 9350 4726 50  0000 C CNN
 F 2 "alexios:CFT-2019-Card-Edge" H 9300 3750 50  0001 C CNN
@@
 AR Path="/5F67D4B5/5D360869" Ref="#PWR?"  Part="1"
 AR Path="/5D360869" Ref="#PWR?"  Part="1"
-AR Path="/5D34E810/5D360869" Ref="#PWR016"  Part="1"
+AR Path="/5D34E810/5D360869" Ref="#PWR?"  Part="1"
 AR Path="/5D36B851/5D360869" Ref="#PWR?"  Part="1"
 AR Path="/5F1DB2E8/5D360869" Ref="#PWR?"  Part="1"
-F 0 "#PWR016" H 8800 4650 50  0001 C CNN
+F 0 "#PWR?" H 8800 4650 50  0001 C CNN
 F 1 "+5V" H 8742 4837 50  0000 R CNN
 F 2 "" H 8800 4800 50  0001 C CNN
@@
 AR Path="/5F67D4B5/5D360863" Ref="#PWR?"  Part="1"
 AR Path="/5D360863" Ref="#PWR?"  Part="1"
-AR Path="/5D34E810/5D360863" Ref="#PWR017"  Part="1"
+AR Path="/5D34E810/5D360863" Ref="#PWR?"  Part="1"
 AR Path="/5D36B851/5D360863" Ref="#PWR?"  Part="1"
 AR Path="/5F1DB2E8/5D360863" Ref="#PWR?"  Part="1"
-F 0 "#PWR017" H 8800 4950 50  0001 C CNN
+F 0 "#PWR?" H 8800 4950 50  0001 C CNN
 F 1 "GND" H 8722 5163 50  0000 R CNN
 F 2 "" H 8800 5200 50  0001 C CNN
@@
 AR Path="/5F67D4B5/5D360855" Ref="#PWR?"  Part="1"
 AR Path="/5D360855" Ref="#PWR?"  Part="1"
-AR Path="/5D34E810/5D360855" Ref="#PWR018"  Part="1"
+AR Path="/5D34E810/5D360855" Ref="#PWR?"  Part="1"
 AR Path="/5D36B851/5D360855" Ref="#PWR?"  Part="1"
 AR Path="/5F1DB2E8/5D360855" Ref="#PWR?"  Part="1"
-F 0 "#PWR018" H 9900 4650 50  0001 C CNN
+F 0 "#PWR?" H 9900 4650 50  0001 C CNN
 F 1 "+5V" H 9915 4973 50  0000 C CNN
 F 2 "" H 9900 4800 50  0001 C CNN
@@
 AR Path="/5F67D4B5/5D36084F" Ref="#PWR?"  Part="1"
 AR Path="/5D36084F" Ref="#PWR?"  Part="1"
-AR Path="/5D34E810/5D36084F" Ref="#PWR019"  Part="1"
+AR Path="/5D34E810/5D36084F" Ref="#PWR?"  Part="1"
 AR Path="/5D36B851/5D36084F" Ref="#PWR?"  Part="1"
 AR Path="/5F1DB2E8/5D36084F" Ref="#PWR?"  Part="1"
-F 0 "#PWR019" H 9900 4950 50  0001 C CNN
+F 0 "#PWR?" H 9900 4950 50  0001 C CNN
 F 1 "GND" H 9905 5027 50  0000 C CNN
 F 2 "" H 9900 5200 50  0001 C CNN
@@
 	8350 3700 8800 3700
 $Comp
-L alexios:CFT-2019-Bus P1
+L alexios:CFT-2019-Bus P?
 U 3 1 5D3608F9
 P 9300 1650
-AR Path="/5D34E810/5D3608F9" Ref="P1"  Part="3"
+AR Path="/5D34E810/5D3608F9" Ref="P?"  Part="3"
 AR Path="/5D36B851/5D3608F9" Ref="P?"  Part="3"
 AR Path="/5F1DB2E8/5D3608F9" Ref="P?"  Part="3"
 AR Path="/5D3608F9" Ref="P?"  Part="3"
-F 0 "P1" H 9300 1817 50  0000 C CNN
+F 0 "P?" H 9300 1817 50  0000 C CNN
 F 1 "CFT-2019-Bus" H 9300 1726 50  0000 C CNN
 F 2 "alexios:CFT-2019-Card-Edge" H 9250 750 50  0001 C CNN
@@
 P 8800 5000
 AR Path="/5D8FC46B" Ref="C?"  Part="1"
-AR Path="/5D34E810/5D8FC46B" Ref="C7"  Part="1"
+AR Path="/5D34E810/5D8FC46B" Ref="C?"  Part="1"
 AR Path="/5F1DB2E8/5D8FC46B" Ref="C?"  Part="1"
-F 0 "C7" H 8712 5046 50  0000 R CNN
+F 0 "C?" H 8712 5046 50  0000 R CNN
 F 1 "47µF" H 8712 4955 50  0000 R CNN
 F 2 "Capacitor_THT:CP_Radial_D6.3mm_P2.50mm" H 8800 5000 50  0001 C CNN
@@
 P 9900 5000
 AR Path="/5D908E0A" Ref="C?"  Part="1"
-AR Path="/5D34E810/5D908E0A" Ref="C8"  Part="1"
+AR Path="/5D34E810/5D908E0A" Ref="C?"  Part="1"
 AR Path="/5F1DB2E8/5D908E0A" Ref="C?"  Part="1"
-F 0 "C8" H 9988 5046 50  0000 L CNN
+F 0 "C?" H 9988 5046 50  0000 L CNN
 F 1 "47µF" H 9988 4955 50  0000 L CNN
 F 2 "Capacitor_THT:CP_Radial_D6.3mm_P2.50mm" H 9900 5000 50  0001 C CNN

Commit message: Added RUEN# and WUEN# signals to the expansion bus.
Connections:
- net RSVD7 renamed ~RUEN
- net RSVD8 renamed ~WUEN
Changed lines of the file:
@@
 EESchema Schematic File Version 4
-LIBS:cft-alu-cache
 LIBS:cft-reg-cache
 EELAYER 30 0
@@
 $Descr A4 11693 8268
 encoding utf-8
-Sheet 8 8
+Sheet 2 6
 Title ""
 Date ""
@@
 Wire Wire Line
 	6500 2550 7200 2550
-Wire Wire Line
-	6500 2650 7200 2650
-Wire Wire Line
-	6500 2750 7200 2750
 Text Label 7200 2050 2    50   ~ 0
 RSVD1
@@
 Text Label 7200 2550 2    50   ~ 0
 RSVD6
-Text Label 7200 2650 2    50   ~ 0
-RSVD7
-Text Label 7200 2750 2    50   ~ 0
-RSVD8
 Entry Wire Line
 	7200 2050 7300 2150
@@
 Entry Wire Line
 	7200 2550 7300 2650
-Entry Wire Line
-	7200 2650 7300 2750
-Entry Wire Line
-	7200 2750 7300 2850
 Entry Bus Bus
 	7200 6150 7300 6050
@@
 Wire Wire Line
 	9800 4800 9900 4800
+Wire Wire Line
+	6500 2650 6800 2650
+Wire Wire Line
+	6500 2750 6800 2750
+Text Label 6800 2650 2    50   ~ 0
+~RUEN
+Text Label 6800 2750 2    50   ~ 0
+~WUEN
 Wire Bus Line
 	7000 3950 7000 5750
@@
 Wire Bus Line
 	2050 2850 2050 5250
+Text HLabel 6800 2650 2    50   UnSpc ~ 0
+~RUEN
+Text HLabel 6800 2750 2    50   UnSpc ~ 0
+~WUEN
 $EndSCHEMATC

Commit message: Reassigned A72 & A73 to GND
Connections:
- net RSVD5 is gone; now on net ~ENDEXT: P?.A32 (~ENDEXT)
- net RSVD6 is gone; now on net ~SKIPEXT: P?.A33 (~SKIPEXT)
- net GND: now also P?.B2 (GND), P?.B82 (GND)
Other:
- moved on the sheet: C?
Changed lines of the file:
@@
 	4900 4150 5300 4150
-Wire Wire Line
-	6500 1750 7250 1750
-Wire Wire Line
-	6500 1850 7250 1850
 Wire Wire Line
 	6500 1950 7250 1950
@@
 Text Label 4900 4150 0    50   ~ 0
 FPD7
-Text Label 7200 1750 2    50   ~ 0
-~ENDEXT
-Text Label 7200 1850 2    50   ~ 0
-~SKIPEXT
 Text Label 7200 1950 2    50   ~ 0
 ~HALT
@@
 Text HLabel 4150 2650 2    50   UnSpc ~ 0
 ~WS
-Text HLabel 7250 1750 2    50   UnSpc ~ 0
-~ENDEXT
-Text HLabel 7250 1850 2    50   UnSpc ~ 0
-~SKIPEXT
 Text HLabel 7250 1950 2    50   UnSpc ~ 0
 ~HALT
@@
 L power:+5V #PWR?
 U 1 1 5D360869
-P 8800 4800
+P 8900 4800
 AR Path="/5F67D4B5/5D360869" Ref="#PWR?"  Part="1"
 AR Path="/5D360869" Ref="#PWR?"  Part="1"
@@
 AR Path="/5D36B851/5D360869" Ref="#PWR?"  Part="1"
 AR Path="/5F1DB2E8/5D360869" Ref="#PWR?"  Part="1"
-F 0 "#PWR?" H 8800 4650 50  0001 C CNN
-F 1 "+5V" H 8742 4837 50  0000 R CNN
-F 2 "" H 8800 4800 50  0001 C CNN
-F 3 "" H 8800 4800 50  0001 C CNN
-	1    8800 4800
+F 0 "#PWR?" H 8900 4650 50  0001 C CNN
+F 1 "+5V" H 8842 4837 50  0000 R CNN
+F 2 "" H 8900 4800 50  0001 C CNN
+F 3 "" H 8900 4800 50  0001 C CNN
+	1    8900 4800
 	1    0    0    -1
 $EndComp
@@
 L power:GND #PWR?
 U 1 1 5D360863
-P 8800 5200
+P 8900 5350
 AR Path="/5F67D4B5/5D360863" Ref="#PWR?"  Part="1"
 AR Path="/5D360863" Ref="#PWR?"  Part="1"
@@
 AR Path="/5D36B851/5D360863" Ref="#PWR?"  Part="1"
 AR Path="/5F1DB2E8/5D360863" Ref="#PWR?"  Part="1"
-F 0 "#PWR?" H 8800 4950 50  0001 C CNN
-F 1 "GND" H 8722 5163 50  0000 R CNN
-F 2 "" H 8800 5200 50  0001 C CNN
-F 3 "" H 8800 5200 50  0001 C CNN
-	1    8800 5200
+F 0 "#PWR?" H 8900 5100 50  0001 C CNN
+F 1 "GND" H 8822 5313 50  0000 R CNN
+F 2 "" H 8900 5350 50  0001 C CNN
+F 3 "" H 8900 5350 50  0001 C CNN
+	1    8900 5350
 	1    0    0    -1
 $EndComp
-Wire Wire Line
-	8800 4800 8800 4900
 $Comp
 L power:+5V #PWR?
 U 1 1 5D360855
-P 9900 4800
+P 9800 4800
 AR Path="/5F67D4B5/5D360855" Ref="#PWR?"  Part="1"
 AR Path="/5D360855" Ref="#PWR?"  Part="1"
@@
 AR Path="/5D36B851/5D360855" Ref="#PWR?"  Part="1"
 AR Path="/5F1DB2E8/5D360855" Ref="#PWR?"  Part="1"
-F 0 "#PWR?" H 9900 4650 50  0001 C CNN
-F 1 "+5V" H 9915 4973 50  0000 C CNN
-F 2 "" H 9900 4800 50  0001 C CNN
-F 3 "" H 9900 4800 50  0001 C CNN
-	1    9900 4800
+F 0 "#PWR?" H 9800 4650 50  0001 C CNN
+F 1 "+5V" H 9815 4973 50  0000 C CNN
+F 2 "" H 9800 4800 50  0001 C CNN
+F 3 "" H 9800 4800 50  0001 C CNN
+	1    9800 4800
 	1    0    0    -1
 $EndComp
@@
 L power:GND #PWR?
 U 1 1 5D36084F
-P 9900 5200
+P 9800 5350
 AR Path="/5F67D4B5/5D36084F" Ref="#PWR?"  Part="1"
 AR Path="/5D36084F" Ref="#PWR?"  Part="1"
@@
 AR Path="/5D36B851/5D36084F" Ref="#PWR?"  Part="1"
 AR Path="/5F1DB2E8/5D36084F" Ref="#PWR?"  Part="1"
-F 0 "#PWR?" H 9900 4950 50  0001 C CNN
-F 1 "GND" H 9905 5027 50  0000 C CNN
-F 2 "" H 9900 5200 50  0001 C CNN
-F 3 "" H 9900 5200 50  0001 C CNN
-	1    9900 5200
+F 0 "#PWR?" H 9800 5100 50  0001 C CNN
+F 1 "GND" H 9805 5177 50  0000 C CNN
+F 2 "" H 9800 5350 50  0001 C CNN
+F 3 "" H 9800 5350 50  0001 C CNN
+	1    9800 5350
 	1    0    0    -1
 $EndComp
 Wire Wire Line
-	9900 4800 9900 4900
-Wire Wire Line
-	9900 5100 9900 5200
+	9800 4800 9800 4900
+Wire Wire Line
+	9800 5100 9800 5200
 Wire Wire Line
 	8350 1800 8800 1800
@@
 Wire Wire Line
 	6500 2350 7200 2350
-Wire Wire Line
-	6500 2450 7200 2450
-Wire Wire Line
-	6500 2550 7200 2550
 Text Label 7200 2050 2    50   ~ 0
 RSVD1
@@
 Text Label 7200 2350 2    50   ~ 0
 RSVD4
-Text Label 7200 2450 2    50   ~ 0
-RSVD5
-Text Label 7200 2550 2    50   ~ 0
-RSVD6
 Entry Wire Line
 	7200 2050 7300 2150
@@
 Entry Wire Line
 	7200 2350 7300 2450
-Entry Wire Line
-	7200 2450 7300 2550
-Entry Wire Line
-	7200 2550 7300 2650
 Entry Bus Bus
 	7200 6150 7300 6050
@@
 	7200 6150 1350 6150
 Text HLabel 1350 6150 0    50   UnSpc ~ 0
-RSVD[0..8]
+RSVD[1..4]
 Text Label 1450 6150 0    50   ~ 0
-RSVD[0..8]
-$Comp
-L Device:CP_Small C?
-U 1 1 5D8FC46B
-P 8800 5000
-AR Path="/5D8FC46B" Ref="C?"  Part="1"
-AR Path="/5D34E810/5D8FC46B" Ref="C?"  Part="1"
-AR Path="/5F1DB2E8/5D8FC46B" Ref="C?"  Part="1"
-F 0 "C?" H 8712 5046 50  0000 R CNN
-F 1 "47µF" H 8712 4955 50  0000 R CNN
-F 2 "Capacitor_THT:CP_Radial_D6.3mm_P2.50mm" H 8800 5000 50  0001 C CNN
-F 3 "~" H 8800 5000 50  0001 C CNN
-	1    8800 5000
-	1    0    0    -1
-$EndComp
-$Comp
-L Device:CP_Small C?
-U 1 1 5D908E0A
-P 9900 5000
-AR Path="/5D908E0A" Ref="C?"  Part="1"
-AR Path="/5D34E810/5D908E0A" Ref="C?"  Part="1"
-AR Path="/5F1DB2E8/5D908E0A" Ref="C?"  Part="1"
-F 0 "C?" H 9988 5046 50  0000 L CNN
-F 1 "47µF" H 9988 4955 50  0000 L CNN
-F 2 "Capacitor_THT:CP_Radial_D6.3mm_P2.50mm" H 9900 5000 50  0001 C CNN
-F 3 "~" H 9900 5000 50  0001 C CNN
-	1    9900 5000
-	1    0    0    -1
-$EndComp
+RSVD[1..4]
 Text HLabel 8350 1800 0    50   UnSpc ~ 0
 C1
@@
 C40
 Wire Wire Line
-	8950 4900 8900 4900
-Connection ~ 8800 4800
-Wire Wire Line
-	8800 5100 8800 5200
+	8900 5200 8950 5200
+Connection ~ 9800 4800
+Wire Wire Line
+	6500 2650 6900 2650
+Wire Wire Line
+	6500 2750 6900 2750
+Text Label 6850 2650 2    50   ~ 0
+~RUEN
+Text Label 6850 2750 2    50   ~ 0
+~WUEN
+Text HLabel 6900 2650 2    50   UnSpc ~ 0
+~RUEN
+Text HLabel 6900 2750 2    50   UnSpc ~ 0
+~WUEN
+Wire Wire Line
+	9750 4800 9800 4800
+Connection ~ 9800 4900
+Wire Wire Line
+	9750 4900 9800 4900
+$Comp
+L Device:CP_Small C?
+U 1 1 5D908E0A
+P 9800 5000
+AR Path="/5D908E0A" Ref="C?"  Part="1"
+AR Path="/5D34E810/5D908E0A" Ref="C?"  Part="1"
+AR Path="/5F1DB2E8/5D908E0A" Ref="C?"  Part="1"
+F 0 "C?" H 9888 5046 50  0000 L CNN
+F 1 "47µF" H 9888 4955 50  0000 L CNN
+F 2 "Capacitor_THT:CP_Radial_D6.3mm_P2.50mm" H 9800 5000 50  0001 C CNN
+F 3 "~" H 9800 5000 50  0001 C CNN
+	1    9800 5000
+	1    0    0    -1
+$EndComp
+Wire Wire Line
+	9750 5100 9800 5100
+Connection ~ 9800 5100
+Wire Wire Line
+	9750 5200 9800 5200
+Wire Wire Line
+	9800 5200 9800 5300
+Connection ~ 9800 5200
+Wire Wire Line
+	9750 5300 9800 5300
+Connection ~ 9800 5300
+Wire Wire Line
+	9800 5300 9800 5350
 Wire Wire Line
 	8950 5100 8900 5100
 Wire Wire Line
+	8900 4800 8950 4800
+Wire Wire Line
+	8900 4800 8900 4900
+Connection ~ 8900 4800
+Connection ~ 8900 4900
+Wire Wire Line
+	8900 4900 8950 4900
+$Comp
+L Device:CP_Small C?
+U 1 1 5D8FC46B
+P 8900 5000
+AR Path="/5D8FC46B" Ref="C?"  Part="1"
+AR Path="/5D34E810/5D8FC46B" Ref="C?"  Part="1"
+AR Path="/5F1DB2E8/5D8FC46B" Ref="C?"  Part="1"
+F 0 "C?" H 8812 5046 50  0000 R CNN
+F 1 "47µF" H 8812 4955 50  0000 R CNN
+F 2 "Capacitor_THT:CP_Radial_D6.3mm_P2.50mm" H 8900 5000 50  0001 C CNN
+F 3 "~" H 8900 5000 50  0001 C CNN
+	1    8900 5000
+	1    0    0    -1
+$EndComp
+Wire Wire Line
 	8900 5100 8900 5200
-Wire Wire Line
-	8900 5200 8950 5200
-Wire Wire Line
-	8900 5200 8800 5200
+Connection ~ 8900 5100
 Connection ~ 8900 5200
-Connection ~ 8800 5200
-Wire Wire Line
-	9750 5200 9800 5200
-Connection ~ 9900 5200
-Wire Wire Line
-	9750 5100 9800 5100
-Wire Wire Line
-	9800 5100 9800 5200
-Connection ~ 9800 5200
-Wire Wire Line
-	9800 5200 9900 5200
-Connection ~ 9900 4800
-Wire Wire Line
-	8900 4900 8900 4800
-Connection ~ 8900 4800
-Wire Wire Line
-	8900 4800 8950 4800
-Wire Wire Line
-	8800 4800 8900 4800
-Wire Wire Line
-	9750 4800 9800 4800
-Wire Wire Line
-	9800 4900 9800 4800
-Wire Wire Line
-	9750 4900 9800 4900
-Connection ~ 9800 4800
-Wire Wire Line
-	9800 4800 9900 4800
-Wire Wire Line
-	6500 2650 6800 2650
-Wire Wire Line
-	6500 2750 6800 2750
-Text Label 6800 2650 2    50   ~ 0
-~RUEN
-Text Label 6800 2750 2    50   ~ 0
-~WUEN
+Wire Wire Line
+	8900 5200 8900 5300
+Wire Wire Line
+	8950 5300 8900 5300
+Connection ~ 8900 5300
+Wire Wire Line
+	8900 5300 8900 5350
+Text HLabel 6900 2550 2    50   UnSpc ~ 0
+~SKIPEXT
+Text HLabel 6900 2450 2    50   UnSpc ~ 0
+~ENDEXT
+Text Label 6850 2550 2    50   ~ 0
+~SKIPEXT
+Text Label 6850 2450 2    50   ~ 0
+~ENDEXT
+Wire Wire Line
+	6500 2550 6900 2550
+Wire Wire Line
+	6500 2450 6900 2450
+Wire Bus Line
+	7300 2150 7300 6050
 Wire Bus Line
 	7000 3950 7000 5750
@@
 	7200 2950 7200 5950
 Wire Bus Line
-	7300 2150 7300 6050
-Wire Bus Line
 	4350 2850 4350 5450
 Wire Bus Line
@@
 Wire Bus Line
 	2050 2850 2050 5250
-Text HLabel 6800 2650 2    50   UnSpc ~ 0
-~RUEN
-Text HLabel 6800 2750 2    50   UnSpc ~ 0
-~WUEN
 $EndSCHEMATC

Commit message: Preparing for manufacture.
Parts:
- gave numbers to parts that had none: 3
Connections:
- no-connect marks 0 -> 52
