File: kicad/cft/cft-reg/cft-reg-dr-sp.sch (KiCad schematic (older format))
At the start: 16 parts, among them U24 74HC193, U25 74HC193, U26 74HC193, U27 74HC193, U28 74HCT541, U29 74HCT541, U30 74HCT541, U31 74HCT541

Commit message: Routing REG board.
Parts:
- C35: footprint Jumper:SolderJumper-2_P1.3mm_Open_RoundedPad1.0x1.5mm -> alexios:SMD_0805_2012Metric_Pad1.15x1.40mm_HandSolder
Connections:
- net Q0: no longer U29.2 (A0), U31.2 (A0)
- net Q1: no longer U29.3 (A1), U31.3 (A1)
- net Q10: now also U29.4 (A2), U31.4 (A2)
- net Q11: now also U29.5 (A3), U31.5 (A3)
- net Q12: now also U29.6 (A4), U31.6 (A4)
- net Q13: now also U29.7 (A5), U31.7 (A5)
- net Q14: now also U29.8 (A6), U31.8 (A6)
- net Q15: now also U29.9 (A7), U31.9 (A7)
- net Q2: no longer U29.4 (A2), U31.4 (A2)
- net Q3: no longer U29.5 (A3), U31.5 (A3)
- net Q4: no longer U29.6 (A4), U31.6 (A4)
- net Q5: no longer U29.7 (A5), U31.7 (A5)
- net Q6: no longer U29.8 (A6), U31.8 (A6)
- net Q7: no longer U29.9 (A7), U31.9 (A7)
- net Q8: now also U29.2 (A0), U31.2 (A0)
- net Q9: now also U29.3 (A1), U31.3 (A1)
Changed lines of the file:
@@
-$Comp
-L Device:C_Small C?
-U 1 1 5D9BFF9F
-P 10450 4550
-AR Path="/5CC0D65F/5D9BFF9F" Ref="C?"  Part="1"
-AR Path="/5CE16E65/5D9BFF9F" Ref="C?"  Part="1"
-AR Path="/5D9BFF9F" Ref="C?"  Part="1"
-AR Path="/5D54E677/5D9BFF9F" Ref="C?"  Part="1"
-AR Path="/5D62E1DC/5D9BFF9F" Ref="C?"  Part="1"
-AR Path="/5D79EA4B/5D9BFF9F" Ref="C?"  Part="1"
-AR Path="/5D892D5E/5D9BFF9F" Ref="C?"  Part="1"
-AR Path="/5D9672D4/5D9BFF9F" Ref="C?"  Part="1"
-AR Path="/5D967A8B/5D9BFF9F" Ref="C35"  Part="1"
-AR Path="/5D9746D0/5D9BFF9F" Ref="C?"  Part="1"
-AR Path="/5D9BD2A8/5D9BFF9F" Ref="C43"  Part="1"
-F 0 "C43" H 10359 4596 50  0000 R CNN
-F 1 "100nF" H 10359 4505 50  0000 R CNN
-F 2 "Jumper:SolderJumper-2_P1.3mm_Open_RoundedPad1.0x1.5mm" H 10450 4550 50  0001 C CNN
-F 3 "~" H 10450 4550 50  0001 C CNN
-	1    10450 4550
-	1    0    0    -1
-$EndComp
 $Comp
 L Device:C_Small C?
@@
 Connection ~ 10450 3750
 Connection ~ 10450 3950
-Connection ~ 10450 4450
-Connection ~ 10450 4650
 $Comp
 L alexios:74HCT541 U?
@@
 Wire Wire Line
 	4200 3300 4900 3300
-Text Label 4300 2600 0    50   ~ 0
-Q0
-Text Label 4300 2700 0    50   ~ 0
-Q1
-Text Label 4300 2800 0    50   ~ 0
-Q2
-Text Label 4300 2900 0    50   ~ 0
-Q3
-Text Label 4300 3000 0    50   ~ 0
-Q4
-Text Label 4300 3100 0    50   ~ 0
-Q5
-Text Label 4300 3200 0    50   ~ 0
-Q6
-Text Label 4300 3300 0    50   ~ 0
-Q7
 Wire Wire Line
 	4200 4200 4900 4200
@@
 Q7
 Wire Wire Line
-	4200 5750 4900 5750
-Wire Wire Line
-	4200 5850 4900 5850
-Wire Wire Line
-	4200 5950 4900 5950
-Wire Wire Line
-	4200 6050 4900 6050
-Wire Wire Line
-	4200 6150 4900 6150
-Wire Wire Line
-	4200 6250 4900 6250
-Wire Wire Line
-	4200 6350 4900 6350
-Wire Wire Line
-	4200 6450 4900 6450
-Text Label 4300 5750 0    50   ~ 0
-Q0
-Text Label 4300 5850 0    50   ~ 0
-Q1
-Text Label 4300 5950 0    50   ~ 0
-Q2
-Text Label 4300 6050 0    50   ~ 0
-Q3
-Text Label 4300 6150 0    50   ~ 0
-Q4
-Text Label 4300 6250 0    50   ~ 0
-Q5
-Text Label 4300 6350 0    50   ~ 0
-Q6
-Text Label 4300 6450 0    50   ~ 0
-Q7
-Wire Wire Line
 	5900 5750 6400 5750
 Wire Wire Line
@@
 Text Label 5950 3300 0    50   ~ 0
 IBUS15
+Text Label 4300 2600 0    50   ~ 0
+Q8
+Text Label 4300 2700 0    50   ~ 0
+Q9
+Text Label 4300 2800 0    50   ~ 0
+Q10
+Text Label 4300 2900 0    50   ~ 0
+Q11
+Text Label 4300 3000 0    50   ~ 0
+Q12
+Text Label 4300 3100 0    50   ~ 0
+Q13
+Text Label 4300 3200 0    50   ~ 0
+Q14
+Text Label 4300 3300 0    50   ~ 0
+Q15
+Wire Wire Line
+	4200 5750 4900 5750
+Wire Wire Line
+	4200 5850 4900 5850
+Wire Wire Line
+	4200 5950 4900 5950
+Wire Wire Line
+	4200 6050 4900 6050
+Wire Wire Line
+	4200 6150 4900 6150
+Wire Wire Line
+	4200 6250 4900 6250
+Wire Wire Line
+	4200 6350 4900 6350
+Wire Wire Line
+	4200 6450 4900 6450
+Text Label 4300 5750 0    50   ~ 0
+Q8
+Text Label 4300 5850 0    50   ~ 0
+Q9
+Text Label 4300 5950 0    50   ~ 0
+Q10
+Text Label 4300 6050 0    50   ~ 0
+Q11
+Text Label 4300 6150 0    50   ~ 0
+Q12
+Text Label 4300 6250 0    50   ~ 0
+Q13
+Text Label 4300 6350 0    50   ~ 0
+Q14
+Text Label 4300 6450 0    50   ~ 0
+Q15
 Wire Bus Line
 	1100 650  6250 650
@@
 Wire Bus Line
 	4100 1150 4100 6550
+$Comp
+L Device:C_Small C?
+U 1 1 5E24BF44
+P 10450 4550
+AR Path="/5CC0D65F/5E24BF44" Ref="C?"  Part="1"
+AR Path="/5CE16E65/5E24BF44" Ref="C?"  Part="1"
+AR Path="/5E24BF44" Ref="C?"  Part="1"
+AR Path="/5D54E677/5E24BF44" Ref="C?"  Part="1"
+AR Path="/5D62E1DC/5E24BF44" Ref="C?"  Part="1"
+AR Path="/5D79EA4B/5E24BF44" Ref="C?"  Part="1"
+AR Path="/5D892D5E/5E24BF44" Ref="C?"  Part="1"
+AR Path="/5D9672D4/5E24BF44" Ref="C?"  Part="1"
+AR Path="/5D967A8B/5E24BF44" Ref="C35"  Part="1"
+AR Path="/5D9746D0/5E24BF44" Ref="C?"  Part="1"
+AR Path="/5D9BD2A8/5E24BF44" Ref="C43"  Part="1"
+F 0 "C43" H 10359 4596 50  0000 R CNN
+F 1 "100nF" H 10359 4505 50  0000 R CNN
+F 2 "alexios:SMD_0805_2012Metric_Pad1.15x1.40mm_HandSolder" H 10450 4550 50  0001 C CNN
+F 3 "~" H 10450 4550 50  0001 C CNN
+	1    10450 4550
+	1    0    0    -1
+$EndComp
+Connection ~ 10450 4450
+Connection ~ 10450 4650
 $EndSCHEMATC

Commit message: Preparing for manufacture.
Other:
- note removed: "Data Register (DR)"
Changed lines of the file:
@@
 encoding utf-8
 Sheet 6 6
-Title ""
+Title "Data Register (DR)"
 Date ""
-Rev ""
+Rev "1941"
 Comp ""
-Comment1 ""
+Comment1 "REG"
 Comment2 ""
 Comment3 ""
-Comment4 ""
+Comment4 "reg_sp.v"
 $EndDescr
 Wire Wire Line
@@
 Entry Wire Line
 	6400 5750 6500 5650
-Text Notes 7100 6950 0    197  ~ 39
-Data Register (DR)
 $Comp
 L alexios:74HCT541 U?
