File: kicad/cft/cft-reg/cft-reg-ac.sch (KiCad schematic (older format))
At the start: 22 parts, among them U13 74HC193, U14 74HC193, U15 74HC193, U16 74HC193, U17 74AHC1G08, U18 74HCT541, U19 74HCT541, U20 74HCT541, U21 74HCT541, U22 74HC688, U23 74HC688

Commit message: Preparing for manufacture.
Other:
- note removed: "Accumulator (AC)"
Changed lines of the file:
@@
 encoding utf-8
 Sheet 4 6
-Title ""
+Title "Accumulator (AC)"
 Date ""
-Rev ""
+Rev "1941"
 Comp ""
-Comment1 ""
+Comment1 "REG"
 Comment2 ""
 Comment3 ""
-Comment4 ""
+Comment4 "reg_ac.v"
 $EndDescr
 Wire Wire Line
@@
 	1    0    0    -1
 $EndComp
-Text Notes 7100 6950 0    197  ~ 39
-Accumulator (AC)
 Text Notes 6650 7450 2    50   ~ 0
 ~ACCPL~ toggles the L register whenever the Accumulator wraps around.
