File: kicad/cft/tic/tic.sch (KiCad schematic (older format))
At the start: 27 parts, among them U17 74HC541, U18 74HC541, U19 74LVC1G02, U20 74HC138, U21 74HC541, U22 74HC138, U24 AMS1117-3.3, U26 74HC259, U31 74HC541, U37 74HC590, U38 74AC251, U39 DS12C887+, U40 8254, U42 74HC112, U49 74HC541

Commit message: Fine-tuning BUS board.
Parts:
- removed U37: 74HC590, alexios:SOIC-16, symbol alexios:74HC590
- removed U38: 74AC251, alexios:SOIC-16, symbol alexios:74AC251
- removed U39: DS12C887+, alexios:eDIP-24-DS12x_W15.24mm, symbol alexios:DS12C887+
Connections:
- net labels added: ~IC2CS, ~TMCS
- net labels removed: CEXT8, CEXT9, COND0, COND1, COND2, COND3, COND4, DIV128, DIV16, DIV2, DIV256, DIV32, DIV4, DIV64, DIV8, FL, FN, FPCLK, FPFETCH∕~EXEC, FV, FZ, IDXEN, IN-RSVD, IR0, IR1, IR2, IR3, IR4, IR5, IR6, IR[0..6], PC10, PC11, PC12, PC13, PC14, PC15, POWEROK, ~FLAGWE, ~FPCLK~⁄CLK, ~FPFLAGS, ~FPIRH, ~FPIRL, ~FPRESET, ~FPµA0, ~FPµC0, ~FPµC1, ~FPµC2, ~WEN
- wire segments 299 -> 269
- no-connect marks 10 -> 9
Other:
- note removed: "1 MHz"
- note removed: "1 µs"
- note removed: "125 KHz"
- note removed: "128 µs"
- note removed: "15.625 KHz"
- note removed: "16 µs"
- note removed: "2 µs"
- note removed: "250 KHz"
- note removed: "31.25 KHz"
- note removed: "32 µs"
- note removed: "4 µs"
- note removed: "500 KHz"
- note removed: "62.5 KHz"
- note removed: "64 µs"
- note removed: "7.8125 KHz"
- note removed: "8 µs"
- note removed: "For future expansion"
- note removed: "← ALU"
- note removed: "← BUS"
- note removed: "← DFP"
- note removed: "← PSU (backplane)"
- note removed: "← REG"
- note removed: "→ ALU"
- note removed: "→ BUS.MBU"
- note removed: "→ DFP"
- moved on the sheet: U20A, U40A

Commit message: Working on TIC board
Parts:
- removed U19: 74LVC1G02, alexios:SOT-23-5_HandSoldering, symbol alexios:74LVC1G02
- removed U20, U22: 74HC138, alexios:SOIC-16, symbol alexios:74HC138
- removed U42: 74HC112, symbol alexios:74HC112
- added JP?: SolderJumper_2_Open, symbol Jumper:SolderJumper_2_Open
- added U?: 74LVC1G08, symbol alexios:74LVC1G08
- added U?: 8254, alexios:DIP-24_W15.24mm_socket, symbol alexios:8254
Connections:
- net labels added: AB2, D0, D1, D2, D3, D4, D5, D6, D7, IRQ7, ~IO14, ~IO18, ~IO1C, ~RIO10, ~RIO11, ~WIO10, ~WIO11
- net labels removed: ~IC2CS, ~SEL, ~TMCS
- wire segments 269 -> 293
Other:
- note added: "Address Decoding & Wait States"
- note added: "Adjust resistor\nvalues as required"
- note removed: "IO=&030–037"
- moved on the sheet: U21A, U31A

Commit message: Working on TIC board.
Parts:
- removed R1, R2: 4.7kΩ, Resistor_SMD:R_Array_Convex_4x0603, symbol Device:R_Pack04_Split
- removed U17, U18, U21, U31, U49: 74HC541, alexios:SOIC-20W, symbol alexios:74HC541
- removed U26: 74HC259, alexios:SOIC-16, symbol alexios:74HC259
- removed U?: 74LVC1G08, symbol alexios:74LVC1G08
Connections:
- net labels removed: DB10, DB11, DB12, DB13, DB14, DB15, DB8, DB9, FPD0, FPD1, FPD2, FPD3, FPD4, FPD5, FPD6, FPD7, IEN0, IEN1, IEN2, IEN3, IEN4, IEN5, IEN6, IEN7, IRF0, IRF1, IRF2, IRF3, IRF4, IRF5, IRF6, IRF7, ~FPIRF, ~IRQ0, ~IRQ1, ~IRQ2, ~IRQ3, ~IRQ4, ~IRQ5, ~IRQ6, ~IRQ7, ~RIER, ~RISR, ~WIER
- wire segments 293 -> 132

Commit message: Minor changes.
Connections:
- net labels added: ~FPIEN, ~FPIRF, ~RIER, ~RISR, ~WIER
- wire segments 132 -> 141
Changed lines of the file:
@@
 $EndSheet
 Wire Wire Line
-	1100 2400 750  2400
+	1100 2400 650  2400
 Wire Wire Line
-	1100 2500 750  2500
+	1100 2500 650  2500
 Wire Wire Line
-	1100 2600 750  2600
+	1100 2600 650  2600
 Wire Wire Line
-	1100 2700 750  2700
+	1100 2700 650  2700
 Wire Wire Line
-	1100 2800 750  2800
+	1100 2800 650  2800
 Wire Wire Line
-	750  2950 1100 2950
+	650  2950 1100 2950
 Wire Wire Line
-	750  3050 1100 3050
+	650  3050 1100 3050
 Wire Wire Line
-	750  3150 1100 3150
+	650  3150 1100 3150
 Wire Wire Line
-	750  3250 1100 3250
+	650  3250 1100 3250
 Wire Wire Line
-	750  3350 1100 3350
+	650  3350 1100 3350
 Wire Wire Line
-	750  3450 1100 3450
+	650  3450 1100 3450
 Wire Wire Line
-	750  3550 1100 3550
+	650  3550 1100 3550
 Wire Wire Line
-	2550 2400 2250 2400
+	2700 2400 2250 2400
 Wire Wire Line
-	2550 2500 2250 2500
+	2700 2500 2250 2500
 Wire Wire Line
-	2550 2600 2250 2600
+	2700 2600 2250 2600
 Wire Wire Line
-	2550 2800 2250 2800
+	2700 2800 2250 2800
 Wire Wire Line
-	2250 2900 2550 2900
+	2250 2900 2700 2900
 Wire Wire Line
-	2250 3100 2550 3100
+	2250 3100 2700 3100
 Wire Wire Line
-	2250 3200 2550 3200
+	2250 3200 2700 3200
 Wire Wire Line
-	2250 3550 2550 3550
+	2250 3550 2700 3550
 Text Notes 700  2000 0    100  ~ 20
 Address Decoding & Wait States
-Text Label 750  2400 0    50   ~ 0
+Text Label 650  2400 0    50   ~ 0
 ~RESET
-Text Label 750  2500 0    50   ~ 0
+Text Label 650  2500 0    50   ~ 0
 CLK3
-Text Label 750  2600 0    50   ~ 0
+Text Label 650  2600 0    50   ~ 0
 ~SYSDEV
-Text Label 750  2700 0    50   ~ 0
+Text Label 650  2700 0    50   ~ 0
 ~R
-Text Label 750  2800 0    50   ~ 0
+Text Label 650  2800 0    50   ~ 0
 ~W
-Text Label 750  2950 0    50   ~ 0
+Text Label 650  2950 0    50   ~ 0
 AB1
-Text Label 750  3050 0    50   ~ 0
+Text Label 650  3050 0    50   ~ 0
 AB2
-Text Label 750  3150 0    50   ~ 0
+Text Label 650  3150 0    50   ~ 0
 AB3
-Text Label 750  3250 0    50   ~ 0
+Text Label 650  3250 0    50   ~ 0
 AB4
-Text Label 750  3350 0    50   ~ 0
+Text Label 650  3350 0    50   ~ 0
 AB5
-Text Label 750  3450 0    50   ~ 0
+Text Label 650  3450 0    50   ~ 0
 AB6
-Text Label 750  3550 0    50   ~ 0
+Text Label 650  3550 0    50   ~ 0
 AB7
-Text Label 2550 2400 2    50   ~ 0
+Text Label 2700 2400 2    50   ~ 0
 ~IO14
-Text Label 2550 2500 2    50   ~ 0
+Text Label 2700 2500 2    50   ~ 0
 ~IO18
-Text Label 2550 2600 2    50   ~ 0
+Text Label 2700 2600 2    50   ~ 0
 ~IO1C
-Text Label 2550 2800 2    50   ~ 0
+Text Label 2700 2800 2    50   ~ 0
 ~RIO10
-Text Label 2550 2900 2    50   ~ 0
+Text Label 2700 2900 2    50   ~ 0
 ~RIO11
-Text Label 2550 3100 2    50   ~ 0
+Text Label 2700 3100 2    50   ~ 0
 ~WIO10
-Text Label 2550 3200 2    50   ~ 0
+Text Label 2700 3200 2    50   ~ 0
 ~WIO11
-Text Label 2550 3550 2    50   ~ 0
+Text Label 2700 3550 2    50   ~ 0
 ~WS
 $Sheet
-S 1100 4050 1150 2200
+S 1100 4050 1150 1250
 U 5F160E7C
 F0 "Interrupt Controller" 50
 F1 "irc.sch" 50
-F2 "DB[0..15]" T L 1100 4850 50
-F3 "~RIER" I R 2250 4950 50
-F4 "FPD[0..7]" T L 1100 4700 50
+F2 "DB[0..15]" T L 1100 4600 50
+F3 "~RIER" I L 1100 4750 50
+F4 "FPD[0..7]" T R 2250 5150 50
 F5 "CLK3" I L 1100 4450 50
 F6 "CLK2" I L 1100 4350 50
 F7 "~RESET" I L 1100 4200 50
-F8 "~WIER" I R 2250 4800 50
-F9 "~IRQ[0..7]" I L 1100 5100 50
-F10 "~RISR" I R 2250 4600 50
-F11 "~FPIEN" I R 2250 4500 50
-F12 "~FPIRF" I R 2250 4400 50
+F8 "~WIER" I L 1100 4850 50
+F9 "~IRQ[0..7]" I L 1100 5150 50
+F10 "~RISR" I L 1100 5000 50
+F11 "~FPIEN" I R 2250 4950 50
+F12 "~FPIRF" I R 2250 5050 50
 $EndSheet
+Wire Bus Line
+	1100 5150 650  5150
+Wire Wire Line
+	1100 4200 650  4200
+Wire Wire Line
+	1100 4350 650  4350
+Wire Wire Line
+	1100 4450 650  4450
+Wire Wire Line
+	1100 4600 650  4600
+Wire Wire Line
+	1100 4750 650  4750
+Wire Wire Line
+	1100 4850 650  4850
+Wire Wire Line
+	1100 5000 650  5000
+Wire Wire Line
+	2250 4950 2700 4950
+Wire Wire Line
+	2250 5050 2700 5050
+Wire Bus Line
+	2700 5150 2250 5150
+Text Label 2700 4950 2    50   ~ 0
+~FPIEN
+Text Label 2700 5050 2    50   ~ 0
+~FPIRF
+Text Label 650  5150 0    50   ~ 0
+~IRQ[0..7]
+Text Label 650  4200 0    50   ~ 0
+~RESET
+Text Label 650  4350 0    50   ~ 0
+CLK2
+Text Label 650  4450 0    50   ~ 0
+CLK3
+Text Label 650  4600 0    50   ~ 0
+DB[0..15]
+Text Label 650  4750 0    50   ~ 0
+~RIER
+Text Label 650  4850 0    50   ~ 0
+~WIER
+Text Label 650  5000 0    50   ~ 0
+~RISR
+Text Label 2700 5150 2    50   ~ 0
+FPD[0..7]
 $EndSCHEMATC

Commit message: Working on TIC board schematics.
Parts:
- removed C?: 22µF, symbol Device:CP_Small
- removed C?: 10µF, symbol Device:CP_Small
- removed JP?: SolderJumper_2_Open, symbol Jumper:SolderJumper_2_Open
- removed JP?: SolderJumper_3_Bridged12, symbol alexios:SolderJumper_3_Bridged12
- removed R? (x2): 4.7kΩ, symbol Device:R_Small
- removed U24: AMS1117-3.3, Package_TO_SOT_SMD:SOT-223-3_TabPin2, symbol Regulator_Linear:AMS1117-3.3
- removed U?: PCA9564, symbol alexios:PCA9564
- added C4: 100nF, symbol Device:C_Small
- added U1: 74HC574, symbol alexios:74HC574
- added U2: M48T02-70PC1, alexios:eDIP-24_W15.24mm, symbol alexios:M48T02-70PC1
- U4: renamed from U?; value 8254 -> M48T02-70PC1; footprint alexios:DIP-24_W15.24mm_socket -> alexios:eDIP-24_W15.24mm
- gave numbers to parts that had none: 2
Connections:
- net labels added: RTCA0, RTCA1, RTCA2, RTCA3, RTCA4, RTCA5, RTCA6, RTCA7, ~RTCAW, ~RTCCS, ~RTCR, ~RTCW
- net labels removed: +3.3V-EXT, DB0, DB1, DB2, DB3, DB4, DB5, DB6, DB7, IRQ7, SCL, SDA
- wire segments 141 -> 146
Other:
- note removed: "Adjust resistor\nvalues as required"

Commit message: Working on TIC board.
Parts:
- removed C4: 100nF, symbol Device:C_Small
- removed U1: 74HC574, symbol alexios:74HC574
- removed U2: M48T02-70PC1, alexios:eDIP-24_W15.24mm, symbol alexios:M48T02-70PC1
Connections:
- net labels removed: RTCA0, RTCA1, RTCA2, RTCA3, RTCA4, RTCA5, RTCA6, RTCA7, ~RTCCS
- wire segments 146 -> 107

Commit message: Working on TIC board.
Parts:
- removed C3: 100nF, symbol Device:C_Small
- removed U3: PCA9564, symbol alexios:PCA9564
- added C?: 100nF, symbol Device:C_Small
- added D? (x2): CUS520, alexios:SOD-323, symbol Device:D_Schottky_ALT
- added JP? (x2): Conn_02x03_Odd_Even, symbol Connector_Generic:Conn_02x03_Odd_Even
- added R? (x6): 4.7kΩ, symbol Device:R_Small
- added U? (x2): 74LVC1G11, symbol alexios:74LVC1G11
- added U? (x2): 74LVC1G07, alexios:SOT-23-5_HandSoldering, symbol alexios:74LVC1G07
- added U? (x2): 74HCT245, symbol alexios:74HCT245
- added X?: CXO_DIP8, Oscillator:Oscillator_DIP-8, symbol alexios:CXO_DIP8
Connections:
- net labels added: DB0, DB1, DB2, DB3, DB4, DB5, DB6, DB7, G0-0, G0-1, G0-2, G1-0, G1-1, G1-2, OUT0-0, OUT0-1, OUT0-2, OUT1-0, OUT1-1, OUT1-2, T0D0, T0D1, T0D2, T0D3, T0D4, T0D5, T0D6, T0D7, T1D0, T1D1, T1D2, T1D3, T1D4, T1D5, T1D6, T1D7, T1D[0..7], TCLK, TOD[0..7], ~IRQ0, ~IRQ1, ~IRQ2, ~RTCCS, ~T0CS, ~T1CS
- net labels removed: +3.3V, D0, D1, D2, D3, D4, D5, D6, D7, ~IO14, ~IO18, ~IO1C, ~RIO10, ~RIO11, ~WIO10, ~WIO11
- wire segments 107 -> 216
Other:
- note added: "Interrupt Controller"
- moved on the sheet: U40A, U4A

Commit message: Working on TMR board.
Parts:
- removed C?: 100nF, symbol Device:C_Small
- removed D? (x2): CUS520, alexios:SOD-323, symbol Device:D_Schottky_ALT
- removed JP? (x2): Conn_02x03_Odd_Even, symbol Connector_Generic:Conn_02x03_Odd_Even
- removed R? (x6): 4.7kΩ, symbol Device:R_Small
- removed U4: M48T02-70PC1, alexios:eDIP-24_W15.24mm, symbol alexios:8254
- removed U40: 8254, alexios:DIP-24_W15.24mm_socket, symbol alexios:8254
- removed U? (x2): 74LVC1G11, symbol alexios:74LVC1G11
- removed U? (x2): 74LVC1G07, alexios:SOT-23-5_HandSoldering, symbol alexios:74LVC1G07
- removed U? (x2): 74HCT245, symbol alexios:74HCT245
- removed X?: CXO_DIP8, Oscillator:Oscillator_DIP-8, symbol alexios:CXO_DIP8
- renumbered C59 to C3, C60 to C4
