File: kicad/cft/tic/tty.sch (KiCad schematic (older format))
At the start: 62 parts, among them J601 DB9_Female, J602 DB25_Female, U601 MAX232, U602 MAX232, U603 16C2550, U604 MAX232, U605 MAX232, U606 MAX232, U607 MAX232, U608 16C2550, U609 MAX232, U610 MAX232

Commit message: Work on new TIC board
Parts:
- removed D601, D602, D603, D604: PESD15VS2UT, Package_TO_SOT_SMD:SOT-23, symbol alexios:PESD15VS2UT
- removed J601: DB9_Female, Connector_Dsub:DSUB-9_Female_Horizontal_P2.77x2.84mm_EdgePinOffset4.94mm_Housed_MountingHolesOffset7.48mm, symbol Connector:DB9_Female
- added C?: C_Small, symbol Device:C_Small
- added C?: 1nF 3kV, symbol Device:C_Small
- added J?: DE9-Female-with-Shield, symbol alexios:DE9-Female-with-Shield
- added U? (x2): STC16C554, Package_LCC:PLCC-68, symbol alexios:STC16C554
- added X?: 7.3728 MHz, Oscillator:Oscillator_DIP-8, symbol alexios:CXO_DIP8
- C601, C602: value 10μF -> 1μF
Connections:
- net labels added: AB0, AB1, AB2, AB3, AB4, DB0, DB1, DB2, DB3, DB4, DB5, DB6, DB7, Earth, RS-CTSA, RS-DCDA, RS-DSRA, RS-DTRA, RS-RIA, RS-RTSA, RS-RXA, RS-TXA, ~R, ~RSTHOLD, ~UART-IRQ, ~UARTCS, ~W
- wire segments 343 -> 392
- no-connect marks 16 -> 23
Other:
- note added: "Look at this for ESD protection: https://www.acmesystems.it/pcb_serial"
- note added: "Or 14.7456 MHz."
- note added: "Tantalum or ceramic capacitors."
- moved on the sheet: C601, C602, C603, C604, C605, C606, C607, C608, C609, C622, U601, U602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

Commit message: Work on TIC schematics
Parts:
- removed C603, C611, C620, C621, C627, C628, C629, C630: 10μF, Capacitor_THT:CP_Radial_D6.3mm_P2.50mm, symbol Device:CP_Small
- removed C623, C625, C626, C631, C632, C633, C634: 1μF, Capacitor_THT:CP_Radial_D6.3mm_P2.50mm, symbol Device:CP_Small
- removed D605, D606, D607, D608, D609, D610, D611, D612, D613, D614, D615, D616: PESD15VS2UT, Package_TO_SOT_SMD:SOT-23, symbol alexios:PESD15VS2UT
- removed J602: DB25_Female, Connector_Dsub:DSUB-25_Female_Horizontal_P2.77x2.84mm_EdgePinOffset4.94mm_Housed_MountingHolesOffset7.48mm, symbol Connector:DB25_Female
- removed U602, U606, U607, U609, U610: MAX232, Package_DIP:DIP-16_W7.62mm_Socket, symbol alexios:MAX232
- removed U603, U608: 16C2550, Package_LCC:PLCC-44_THT-Socket, symbol alexios:16C2550
- added C620, C621: 100nF, alexios:C_SMD_0805_2012Metric_Pad1.15x1.40mm_HandSolder, symbol Device:C_Small
- added C623: 47pF, alexios:C_SMD_0805_2012Metric_Pad1.15x1.40mm_HandSolder, symbol Device:C_Small
- added D601, D602: LED_ALT, alexios:LED_0805_2012Metric_Pad1.15x1.40mm_HandSolder, symbol Device:LED_ALT
- added J602: DE9-Female-with-Shield, Connector_Dsub:DSUB-9_Female_Horizontal_P2.77x2.84mm_EdgePinOffset4.94mm_Housed_MountingHolesOffset7.48mm, symbol alexios:DE9-Female-with-Shield
- added J603: USB_OTG, Connector_USB:USB_B_Lumberg_2411_02_Horizontal, symbol Connector:USB_OTG
- added R601, R602: 27Ω, alexios:R_SMD_0805_2012Metric_Pad1.15x1.40mm_HandSolder, symbol Device:R_Small
- added R603, R604: 560Ω, alexios:R_SMD_0805_2012Metric_Pad1.15x1.40mm_HandSolder, symbol Device:R_Small
- added unit 3 of U602
- added unit 4 of U602
- added U603: MAX232, Package_DIP:DIP-16_W7.62mm_Socket, symbol alexios:MAX232
- added U606: FT231XS, Housings_SSOP:SSOP-20_4.4x6.5mm_Pitch0.65mm, symbol alexios:FT231XS
- C603: renamed from C?; footprint (none) -> Capacitor_SMD:C_1206_3216Metric
- C604, C610, C612, C613, C618, C619: value 10μF -> 1μF
- C605: value C_Small -> 100nF
- C611: renamed from C?; value C_Small -> 100nF; footprint (none) -> alexios:C_SMD_0805_2012Metric_Pad1.15x1.40mm_HandSolder
- C622: value C_Small -> 47pF
- C624: value 1μF -> 4.7µF
- J601: renamed from J?; footprint (none) -> Connector_Dsub:DSUB-9_Female_Horizontal_P2.77x2.84mm_EdgePinOffset4.94mm_Housed_MountingHolesOffset7.48mm
- U604: footprint Package_DIP:DIP-16_W7.62mm_Socket -> Package_LCC:PLCC-68_THT-Socket
- gave numbers to parts that had none: 2
Connections:
- net labels added: CTSC, D+, D-, DSRC, DTRC, RS-CTSB, RS-DCDB, RS-DSRB, RS-DTRB, RS-RIB, RS-RTSB, RS-RXB, RS-TXB, RSTHOLD, RTSC, RXC, RXD, TTYD-RX, TTYD-TX, TXC, TXD, USBD+, USBD-, ~RI0, ~RI1, ~RXLED, ~TXLED
- net labels removed: A0, A1, A2, D0, D1, D2, D3, D4, D5, D6, D7, INT0, INT1, INT2, INT3, RESET, RX2, RX3, TX2, TX3, ~CD2, ~CD3, ~CSTTY0, ~CSTTY1, ~CSTTY2, ~CSTTY3, ~CTS2, ~CTS3, ~DSR2, ~DSR3, ~DTR2, ~DTR3, ~IOR, ~IOW, ~OUT0, ~OUT1, ~OUT2, ~OUT3, ~RI2, ~RI3, ~RTS2, ~RTS3, ~RXRDY0, ~RXRDY1, ~RXRDY2, ~RXRDY3, ~TXRDY0, ~TXRDY1, ~TXRDY2, ~TXRDY3
- wire segments 392 -> 261
- no-connect marks 23 -> 17
Other:
- note added: "TTYA"
- note added: "TTYB"
- note added: "TTYC"
- note added: "TTYC: USB serial (FTDI chip)"
- note added: "TTYD/WIFI"
- note added: "USB-Powered FTDI IC"
- moved on the sheet: C601, C602, C603, C605, C606, C607, C611, J601, U601, U602A, U602B, X601

Commit message: Work on TIC board
Parts:
- removed J603: USB_OTG, Connector_USB:USB_B_Lumberg_2411_02_Horizontal, symbol Connector:USB_OTG
- added J1: USB_B_Micro, Connector_USB:USB_Micro-B_Molex_47346-0001, symbol Connector:USB_B_Micro
- added U9: USB6B1, alexios:SOIC-8, symbol alexios:USB6B1
- U601, U603, U605: footprint Package_DIP:DIP-16_W7.62mm_Socket -> alexios:DIP-16_W7.62mm_Socket
- U602: footprint Package_LCC:PLCC-68 -> alexios:PLCC68
- U604: footprint Package_LCC:PLCC-68_THT-Socket -> alexios:DIP-16_W7.62mm_Socket
- U606: footprint Housings_SSOP:SSOP-20_4.4x6.5mm_Pitch0.65mm -> Package_SO:SSOP-20_3.9x8.7mm_P0.635mm
Connections:
- net D+: now also J1.3 (D+), U9.7 (I/O1B); no longer C623.1, R601.1
- net D-: now also J1.2 (D-), U9.6 (I/O2B); no longer C622.1, R602.1
- net Earth: now also J1.6 (Shield)
- net GND: now also J1.5 (GND), U9.4 (GNDA), U9.5 (GNDB)
- net at C621.1, C624.1, D601.1 (K)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: now also U9.1 (VBUSA)
- new net: J1.1 (VBUS), U9.8 (VBUSB)
- new net D'+: C623.1, R601.1, U9.2 (I/O1A)
- new net D'-: C622.1, R602.1, U9.3 (I/O2A)
Other:
- moved on the sheet: C620, C621, C622, C623, C624, D601, D602, R601, R602, R603, R604, U602C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
