File: kicad/cft/cft-ctl-reg/bus.sch (KiCad schematic (older format))
At the start: 3 parts, among them P1201 CFT-2019-Bus

Commit message: Removing
Parts:
- removed C1202: 47µF, Capacitor_THT:CP_Radial_D6.3mm_P2.50mm, symbol Device:CP_Small
- removed unit 4 of P1201
- added C1302: 47µF, Capacitor_THT:CP_Radial_D6.3mm_P2.50mm, symbol Device:CP_Small
- added unit 4 of P1301
- renumbered C1201 to C1301, P1201 to P1301
Connections:
- net +5V: now also C1302.1, P1301.A1 (+5V), P1301.A2 (+5V), P1301.A81 (+5V), P1301.A82 (+5V)
- net GND: now also C1302.2, P1301.A72 (GND), P1301.A73 (GND), P1301.B1 (GND), P1301.B2 (GND), P1301.B81 (GND), P1301.B82 (GND)
Changed lines of the file:
@@
 $Descr A4 11693 8268
 encoding utf-8
-Sheet 12 12
+Sheet 12 17
 Title "CFT Bus Connector"
 Date ""
@@
 $EndDescr
 $Comp
-L alexios:CFT-2019-Bus P?
+L alexios:CFT-2019-Bus P1301
 U 2 1 5D360881
 P 5900 1600
-AR Path="/5D34E810/5D360881" Ref="P?"  Part="2"
+AR Path="/5D34E810/5D360881" Ref="P1301"  Part="2"
 AR Path="/5D36B851/5D360881" Ref="P?"  Part="2"
 AR Path="/5F1DB2E8/5D360881" Ref="P?"  Part="2"
 AR Path="/5D360881" Ref="P?"  Part="2"
-AR Path="/5DD5525C/5D360881" Ref="P1201"  Part="2"
-F 0 "P1201" H 5900 1767 50  0000 C CNN
+AR Path="/5DD5525C/5D360881" Ref="P?"  Part="2"
+F 0 "P1301" H 5900 1767 50  0000 C CNN
 F 1 "CFT-2019-Bus" H 5900 1676 50  0000 C CNN
 F 2 "alexios:CFT-2019-Card-Edge" H 5850 700 50  0001 C CNN
@@
 RADDR[0..4]
 $Comp
-L alexios:CFT-2019-Bus P?
-U 4 1 5D360875
+L alexios:CFT-2019-Bus P1301
+U 4 1 6027EB19
 P 9350 4650
-AR Path="/5D34E810/5D360875" Ref="P?"  Part="4"
-AR Path="/5D36B851/5D360875" Ref="P?"  Part="4"
-AR Path="/5F1DB2E8/5D360875" Ref="P?"  Part="4"
-AR Path="/5D360875" Ref="P?"  Part="4"
-AR Path="/5DD5525C/5D360875" Ref="P1201"  Part="4"
-F 0 "P1201" H 9350 4817 50  0000 C CNN
+AR Path="/5D34E810/6027EB19" Ref="P1301"  Part="4"
+AR Path="/5D36B851/6027EB19" Ref="P?"  Part="4"
+AR Path="/5F1DB2E8/6027EB19" Ref="P?"  Part="4"
+AR Path="/6027EB19" Ref="P?"  Part="4"
+AR Path="/5DD5525C/6027EB19" Ref="P?"  Part="4"
+F 0 "P1301" H 9350 4817 50  0000 C CNN
 F 1 "CFT-2019-Bus" H 9350 4726 50  0000 C CNN
 F 2 "alexios:CFT-2019-Card-Edge" H 9300 3750 50  0001 C CNN
@@
 AR Path="/5F67D4B5/5D360869" Ref="#PWR?"  Part="1"
 AR Path="/5D360869" Ref="#PWR?"  Part="1"
-AR Path="/5D34E810/5D360869" Ref="#PWR?"  Part="1"
+AR Path="/5D34E810/5D360869" Ref="#PWR01301"  Part="1"
 AR Path="/5D36B851/5D360869" Ref="#PWR?"  Part="1"
 AR Path="/5F1DB2E8/5D360869" Ref="#PWR?"  Part="1"
-AR Path="/5DD5525C/5D360869" Ref="#PWR01201"  Part="1"
-F 0 "#PWR01201" H 8900 4650 50  0001 C CNN
+AR Path="/5DD5525C/5D360869" Ref="#PWR?"  Part="1"
+F 0 "#PWR01301" H 8900 4650 50  0001 C CNN
 F 1 "+5V" H 8842 4837 50  0000 R CNN
 F 2 "" H 8900 4800 50  0001 C CNN
@@
 AR Path="/5F67D4B5/5D360863" Ref="#PWR?"  Part="1"
 AR Path="/5D360863" Ref="#PWR?"  Part="1"
-AR Path="/5D34E810/5D360863" Ref="#PWR?"  Part="1"
+AR Path="/5D34E810/5D360863" Ref="#PWR01303"  Part="1"
 AR Path="/5D36B851/5D360863" Ref="#PWR?"  Part="1"
 AR Path="/5F1DB2E8/5D360863" Ref="#PWR?"  Part="1"
-AR Path="/5DD5525C/5D360863" Ref="#PWR01203"  Part="1"
-F 0 "#PWR01203" H 8900 5100 50  0001 C CNN
+AR Path="/5DD5525C/5D360863" Ref="#PWR?"  Part="1"
+F 0 "#PWR01303" H 8900 5100 50  0001 C CNN
 F 1 "GND" H 8822 5313 50  0000 R CNN
 F 2 "" H 8900 5350 50  0001 C CNN
@@
 AR Path="/5F67D4B5/5D360855" Ref="#PWR?"  Part="1"
 AR Path="/5D360855" Ref="#PWR?"  Part="1"
-AR Path="/5D34E810/5D360855" Ref="#PWR?"  Part="1"
+AR Path="/5D34E810/5D360855" Ref="#PWR01302"  Part="1"
 AR Path="/5D36B851/5D360855" Ref="#PWR?"  Part="1"
 AR Path="/5F1DB2E8/5D360855" Ref="#PWR?"  Part="1"
-AR Path="/5DD5525C/5D360855" Ref="#PWR01202"  Part="1"
-F 0 "#PWR01202" H 9800 4650 50  0001 C CNN
+AR Path="/5DD5525C/5D360855" Ref="#PWR?"  Part="1"
+F 0 "#PWR01302" H 9800 4650 50  0001 C CNN
 F 1 "+5V" H 9815 4973 50  0000 C CNN
 F 2 "" H 9800 4800 50  0001 C CNN
@@
 $Comp
 L power:GND #PWR?
-U 1 1 5D36084F
+U 1 1 6027EB15
 P 9800 5350
-AR Path="/5F67D4B5/5D36084F" Ref="#PWR?"  Part="1"
-AR Path="/5D36084F" Ref="#PWR?"  Part="1"
-AR Path="/5D34E810/5D36084F" Ref="#PWR?"  Part="1"
-AR Path="/5D36B851/5D36084F" Ref="#PWR?"  Part="1"
-AR Path="/5F1DB2E8/5D36084F" Ref="#PWR?"  Part="1"
-AR Path="/5DD5525C/5D36084F" Ref="#PWR01204"  Part="1"
-F 0 "#PWR01204" H 9800 5100 50  0001 C CNN
+AR Path="/5F67D4B5/6027EB15" Ref="#PWR?"  Part="1"
+AR Path="/6027EB15" Ref="#PWR?"  Part="1"
+AR Path="/5D34E810/6027EB15" Ref="#PWR01304"  Part="1"
+AR Path="/5D36B851/6027EB15" Ref="#PWR?"  Part="1"
+AR Path="/5F1DB2E8/6027EB15" Ref="#PWR?"  Part="1"
+AR Path="/5DD5525C/6027EB15" Ref="#PWR?"  Part="1"
+F 0 "#PWR01304" H 9800 5100 50  0001 C CNN
 F 1 "GND" H 9805 5177 50  0000 C CNN
 F 2 "" H 9800 5350 50  0001 C CNN
@@
 	8350 3700 8800 3700
 $Comp
-L alexios:CFT-2019-Bus P?
+L alexios:CFT-2019-Bus P1301
 U 3 1 5D3608F9
 P 9300 1650
-AR Path="/5D34E810/5D3608F9" Ref="P?"  Part="3"
+AR Path="/5D34E810/5D3608F9" Ref="P1301"  Part="3"
 AR Path="/5D36B851/5D3608F9" Ref="P?"  Part="3"
 AR Path="/5F1DB2E8/5D3608F9" Ref="P?"  Part="3"
 AR Path="/5D3608F9" Ref="P?"  Part="3"
-AR Path="/5DD5525C/5D3608F9" Ref="P1201"  Part="3"
-F 0 "P1201" H 9300 1817 50  0000 C CNN
+AR Path="/5DD5525C/5D3608F9" Ref="P?"  Part="3"
+F 0 "P1301" H 9300 1817 50  0000 C CNN
 F 1 "CFT-2019-Bus" H 9300 1726 50  0000 C CNN
 F 2 "alexios:CFT-2019-Card-Edge" H 9250 750 50  0001 C CNN
@@
 $Comp
 L Device:CP_Small C?
-U 1 1 5D908E0A
+U 1 1 6027EB1E
 P 9800 5000
-AR Path="/5D908E0A" Ref="C?"  Part="1"
-AR Path="/5D34E810/5D908E0A" Ref="C?"  Part="1"
-AR Path="/5F1DB2E8/5D908E0A" Ref="C?"  Part="1"
-AR Path="/5DD5525C/5D908E0A" Ref="C1202"  Part="1"
-F 0 "C1202" H 9888 5046 50  0000 L CNN
+AR Path="/6027EB1E" Ref="C?"  Part="1"
+AR Path="/5D34E810/6027EB1E" Ref="C1302"  Part="1"
+AR Path="/5F1DB2E8/6027EB1E" Ref="C?"  Part="1"
+AR Path="/5DD5525C/6027EB1E" Ref="C?"  Part="1"
+F 0 "C1302" H 9888 5046 50  0000 L CNN
 F 1 "47µF" H 9888 4955 50  0000 L CNN
 F 2 "Capacitor_THT:CP_Radial_D6.3mm_P2.50mm" H 9800 5000 50  0001 C CNN
@@
 P 8900 5000
 AR Path="/5D8FC46B" Ref="C?"  Part="1"
-AR Path="/5D34E810/5D8FC46B" Ref="C?"  Part="1"
+AR Path="/5D34E810/5D8FC46B" Ref="C1301"  Part="1"
 AR Path="/5F1DB2E8/5D8FC46B" Ref="C?"  Part="1"
-AR Path="/5DD5525C/5D8FC46B" Ref="C1201"  Part="1"
-F 0 "C1201" H 8812 5046 50  0000 R CNN
+AR Path="/5DD5525C/5D8FC46B" Ref="C?"  Part="1"
+F 0 "C1301" H 8812 5046 50  0000 R CNN
 F 1 "47µF" H 8812 4955 50  0000 R CNN
 F 2 "Capacitor_THT:CP_Radial_D6.3mm_P2.50mm" H 8900 5000 50  0001 C CNN
@@
 	6500 2450 6900 2450
 $Comp
-L alexios:CFT-2019-Bus P?
+L alexios:CFT-2019-Bus P1301
 U 1 1 5D36087B
 P 3150 1600
-AR Path="/5D34E810/5D36087B" Ref="P?"  Part="1"
+AR Path="/5D34E810/5D36087B" Ref="P1301"  Part="1"
 AR Path="/5D36B851/5D36087B" Ref="P?"  Part="1"
 AR Path="/5F1DB2E8/5D36087B" Ref="P?"  Part="1"
 AR Path="/5D36087B" Ref="P?"  Part="1"
-AR Path="/5DD5525C/5D36087B" Ref="P1201"  Part="1"
-F 0 "P1201" H 3150 1767 50  0000 C CNN
+AR Path="/5DD5525C/5D36087B" Ref="P?"  Part="1"
+F 0 "P1301" H 3150 1767 50  0000 C CNN
 F 1 "CFT-2019-Bus" H 3150 1676 50  0000 C CNN
 F 2 "alexios:CFT-2019-Card-Edge" H 3100 700 50  0001 C CNN
@@
 NoConn ~ 7200 2350
 $Comp
-L power:PWR_FLAG #FLG01201
-U 1 1 5EB1EF8C
+L power:PWR_FLAG #FLG01301
+U 1 1 6027EB1F
 P 8700 4850
-F 0 "#FLG01201" H 8700 4925 50  0001 C CNN
+F 0 "#FLG01301" H 8700 4925 50  0001 C CNN
 F 1 "PWR_FLAG" V 8700 5150 50  0000 C CNN
 F 2 "" H 8700 4850 50  0001 C CNN
@@
 	8900 4850 8900 4900
 $Comp
-L power:PWR_FLAG #FLG01202
-U 1 1 5EB3E4B0
+L power:PWR_FLAG #FLG01302
+U 1 1 6027EB20
 P 9850 5300
-F 0 "#FLG01202" H 9850 5375 50  0001 C CNN
+F 0 "#FLG01302" H 9850 5375 50  0001 C CNN
 F 1 "PWR_FLAG" V 9850 5428 50  0000 L CNN
 F 2 "" H 9850 5300 50  0001 C CNN
