File: kicad/cft/cft-ctl-reg/cft-ctl.kicad_pcb (KiCad board)
At the start: 4 copper layers, 976.5 x 771.8 mm, 544 parts, among them J1 Conn_01x02, J1 VG64_VME_3Rows_3x32_J1_P1, J2 VG64_VME_3Rows_3x32_J2_P2, SW1 tactile_switch, U1 74LVC1G04, U10 74LVC2G157, U11 74HC574, U12 74HC541, U13 74LVC1G32, U14 74HC574, U15 74HC541, U16 74HC541, U17 74HC138, U18 74LVC1G0832, U19 74HC138, U2 74HC138, U20 74HC541, U21 74HC541, U22 74HC574, U23 74HC541, U24 74LVC1G11, U25 74LVC1G11, U26 74LVC1G00, U27 74HC138, U28 74LVC1G74, U29 74LVC1G08, U3 74HC138, U30 74LVC1G08, U31 74LVC1G74, U32 74LVC1G74, U33 74LVC1G373, U34 74LVC1G04, U35 74LVC1G32, U36 74HC251, U37 74AC08, U38 74AC32, U39 74LVC1G86, U4 74LVC1G32, U40 74HC251, U41 74HC139, U42 74LVC1G74, U43 74LVC1G373, U44 74HC85, U45 SN74ACT1071, U46 74LVC1G74, U47 74LVC1G373, U48 AT27C020, U49 AT27C020, U5 74HC138, U50 AT27C020, U51 74AC157, U52 74HC574, U53 74HC574, U54 74HC574, U55 74HC541, U56 74HC541, U57 74HC541, U58 74HC541, U59 74HC251, U6 74HC590, U60 74AC161, U61 74HC193, U62 74HCT541, U63 74HC193, U64 74HCT541, U65 74HCT541, U66 74HC193, U67 74HCT541, U68 74HC193, U69 74HC193, U7 74LVC1G17, U70 74HCT541, U71 74HC688, U72 74HC193, U73 74HCT541, U74 74HCT541, U75 74HC193, U76 74HCT541, U77 74HC193, U78 74HC688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

Commit message: Removing
Parts:
- removed C1, C10, C12, C14, C15, C16, C17, C18, C19, C20, C21, C22, C23, C24, C25, C26, C27, C28, C29, C30, C31, C32, C33, C34, C35, C36, C37, C38, C39, C40, C41, C42, C43, C44, C45, C46, C47, C48, C49, C50, C51, C52, C53, C54, C55, C57, C59, C61, C62, C63, C64, C65, C66, C67, C68, C69, C70: 100nF, alexios:C_SMD_0805_2012Metric_Pad1.15x1.40mm_HandSolder
- removed C100, C101, C102, C103, C104, C105, C106, C107, C108, C109, C6, C7, C75, C76, C77, C78, C79, C8, C80, C81, C82, C83, C84, C85, C86, C87, C88, C89, C9, C90, C91, C92, C93, C94, C95, C96, C97, C98, C99: 100nF, alexios:SMD_0805_2012Metric_Pad1.15x1.40mm_HandSolder
- removed C11, C56, C58, C60: 10µF, alexios:C_SMD_0805_2012Metric_Pad1.15x1.40mm_HandSolder
- removed C13: 47µF, alexios:C_SMD_0805_2012Metric_Pad1.15x1.40mm_HandSolder
- removed C2, C3, C4, C5, C71, C72, C73, C74: 47µF, Capacitor_THT:CP_Radial_D6.3mm_P2.50mm
- removed D1, D2, D3, D4, D5, D6, D7: CUS520, alexios:SOD-323
- removed J1: Conn_01x02, Connector_PinHeader_2.54mm:PinHeader_1x02_P2.54mm_Horizontal
- removed J1: VG64_VME_3Rows_3x32_J1_P1, alexios:DIN41612_B_3x32_Horizontal
- removed J2: VG64_VME_3Rows_3x32_J2_P2, alexios:DIN41612_B_3x32_Horizontal
- removed JP1, JP4: Jumper_NC_Small, Jumper:SolderJumper-2_P1.3mm_Bridged_RoundedPad1.0x1.5mm
- removed JP2: SolderJumper_3_Open, Jumper:SolderJumper-3_P1.3mm_Open_RoundedPad1.0x1.5mm
- removed JP3: Jumper_3_Bridged12, Jumper:SolderJumper-3_P1.3mm_Bridged12_RoundedPad1.0x1.5mm
- removed JP5, JP7: SolderJumper_3_Bridged23, Jumper:SolderJumper-3_P1.3mm_Open_RoundedPad1.0x1.5mm
- removed JP6: SolderJumper_3_Bridged12, Jumper:SolderJumper-3_P1.3mm_Open_RoundedPad1.0x1.5mm
- removed R1, R10, R11, R12, R14, R15, R16, R2, R22, R23, R24, R25, R26, R27, R29, R3, R31, R32, R33, R34, R35, R36, R4, R5, R6, R61, R62, R7, R8, R9: 4.7kΩ, alexios:R_SMD_0805_2012Metric_Pad1.15x1.40mm_HandSolder
- removed R13, R17, R18, R19, R20, R21, R28, R30: 30Ω, alexios:R_SMD_0805_2012Metric_Pad1.15x1.40mm_HandSolder
- removed R37, R38, R39, R40, R41, R42, R43, R44, R45, R46, R47, R48, R49, R50, R51, R52, R53, R54, R55, R56, R57, R58, R59, R60: 0Ω/30Ω, alexios:R_SMD_0805_2012Metric_Pad1.15x1.40mm_HandSolder
- removed R63: 0Ω, alexios:R_SMD_0805_2012Metric_Pad1.15x1.40mm_HandSolder
- removed the REF** at (63.7, -281.8)
- removed the REF** at (2.73, -281.8)
- removed the REF** at (5.27, -281.8)
- removed the REF** at (7.81, -281.8)
- removed the REF** at (10.3, -281.8)
- removed the REF** at (12.9, -281.8)
- removed the REF** at (15.4, -281.8)
- removed the REF** at (18.0, -281.8)
- removed the REF** at (20.5, -281.8)
- removed the REF** at (23.0, -281.8)
- removed the REF** at (25.6, -281.8)
- removed the REF** at (170.4, -276.7)
- removed the REF** at (28.1, -281.8)
- removed the REF** at (30.7, -281.8)
- removed the REF** at (33.2, -281.8)
- removed the REF** at (86.5, -281.8)
- removed the REF** at (89.1, -281.8)
- removed the REF** at (91.6, -281.8)
- removed the REF** at (94.2, -281.8)
- removed the REF** at (96.7, -281.8)
- removed the REF** at (99.2, -281.8)
- removed the REF** at (101.8, -281.8)
- removed the REF** at (170.4, -279.3)
- removed the REF** at (104.3, -281.8)
- removed the REF** at (106.9, -281.8)
- removed the REF** at (109.4, -281.8)
- removed the REF** at (111.9, -281.8)
- removed the REF** at (114.5, -281.8)
- removed the REF** at (117.0, -281.8)
- removed the REF** at (119.6, -281.8)
- removed the REF** at (122.1, -281.8)
- removed the REF** at (124.6, -281.8)
- removed the REF** at (127.2, -281.8)
- removed the REF** at (170.4, -281.8)
- removed the REF** at (129.7, -281.8)
- removed the REF** at (132.3, -281.8)
- removed the REF** at (134.8, -281.8)
- removed the REF** at (137.3, -281.8)
- removed the REF** at (139.9, -281.8)
- removed the REF** at (142.4, -281.8)
- removed the REF** at (145.0, -281.8)
- removed the REF** at (147.5, -281.8)
- removed the REF** at (150.0, -281.8)
- removed the REF** at (152.6, -281.8)
- removed the REF** at (-50.6, -276.7)
- removed the REF** at (155.1, -281.8)
- removed the REF** at (157.7, -281.8)
- removed the REF** at (160.2, -281.8)
- removed the REF** at (162.7, -281.8)
- removed the REF** at (165.3, -281.8)
- removed the REF** at (-50.6, -284.3)
- removed the REF** at (-45.5, -284.3)
- removed the REF** at (-43.0, -284.3)
- removed the REF** at (-40.5, -284.3)
- removed the REF** at (-37.9, -284.3)
- removed the REF** at (-50.6, -279.3)
- removed the REF** at (-35.4, -284.3)
- removed the REF** at (-32.8, -284.3)
- removed the REF** at (-30.3, -284.3)
- removed the REF** at (-27.8, -284.3)
- removed the REF** at (-25.2, -284.3)
- removed the REF** at (-22.7, -284.3)
- removed the REF** at (-20.1, -284.3)
- removed the REF** at (-17.6, -284.3)
- removed the REF** at (-15.1, -284.3)
- removed the REF** at (-12.5, -284.3)
- removed the REF** at (-50.6, -281.8)
- removed the REF** at (-9.97, -284.3)
- removed the REF** at (-7.43, -284.3)
- removed the REF** at (-4.89, -284.3)
- removed the REF** at (-2.35, -284.3)
- removed the REF** at (0.19, -284.3)
- removed the REF** at (2.73, -284.3)
- removed the REF** at (5.27, -284.3)
- removed the REF** at (7.81, -284.3)
- removed the REF** at (10.3, -284.3)
- removed the REF** at (12.9, -284.3)
- removed the REF** at (-45.5, -279.3)
- removed the REF** at (15.4, -284.3)
- removed the REF** at (18.0, -284.3)
- removed the REF** at (20.5, -284.3)
- removed the REF** at (23.0, -284.3)
- removed the REF** at (25.6, -284.3)
- removed the REF** at (28.1, -284.3)
- removed the REF** at (30.7, -284.3)
- removed the REF** at (33.2, -284.3)
- removed the REF** at (53.5, -284.3)
- removed the REF** at (58.6, -284.3)
- removed the REF** at (-43.0, -279.3)
- removed the REF** at (63.7, -284.3)
- removed the REF** at (86.5, -284.3)
- removed the REF** at (89.1, -284.3)
- removed the REF** at (91.6, -284.3)
- removed the REF** at (94.2, -284.3)
- removed the REF** at (96.7, -284.3)
- removed the REF** at (99.2, -284.3)
- removed the REF** at (101.8, -284.3)
- removed the REF** at (104.3, -284.3)
- removed the REF** at (106.9, -284.3)
- removed the REF** at (-40.5, -279.3)
- removed the REF** at (109.4, -284.3)
- removed the REF** at (111.9, -284.3)
- removed the REF** at (114.5, -284.3)
- removed the REF** at (117.0, -284.3)
- removed the REF** at (119.6, -284.3)
- removed the REF** at (122.1, -284.3)
- removed the REF** at (124.6, -284.3)
- removed the REF** at (127.2, -284.3)
- removed the REF** at (129.7, -284.3)
- removed the REF** at (132.3, -284.3)
- removed the REF** at (53.5, -276.7)
- removed the REF** at (-37.9, -279.3)
- removed the REF** at (134.8, -284.3)
- removed the REF** at (137.3, -284.3)
- removed the REF** at (139.9, -284.3)
- removed the REF** at (142.4, -284.3)
- removed the REF** at (145.0, -284.3)
- removed the REF** at (147.5, -284.3)
- removed the REF** at (150.0, -284.3)
- removed the REF** at (152.6, -284.3)
- removed the REF** at (155.1, -284.3)
- removed the REF** at (157.7, -284.3)
- removed the REF** at (-35.4, -279.3)
- removed the REF** at (160.2, -284.3)
- removed the REF** at (162.7, -284.3)
- removed the REF** at (165.3, -284.3)
- removed the REF** at (170.4, -284.3)
- removed the REF** at (45.9, -296.1)
- removed the REF** at (73.8, -296.1)
- removed the REF** at (48.4, -296.1)
- removed the REF** at (51.0, -296.1)
- removed the REF** at (53.5, -296.1)
- removed the REF** at (56.1, -296.1)
- removed the REF** at (-32.8, -279.3)
- removed the REF** at (58.6, -296.1)
- removed the REF** at (61.1, -296.1)
- removed the REF** at (63.7, -296.1)
- removed the REF** at (66.2, -296.1)
- removed the REF** at (68.8, -296.1)
- removed the REF** at (71.3, -296.1)
- removed the REF** at (45.9, -291.1)
- removed the REF** at (48.4, -291.1)
- removed the REF** at (51.0, -291.1)
- removed the REF** at (53.5, -291.1)
- removed the REF** at (-30.3, -279.3)
- removed the REF** at (56.1, -291.1)
- removed the REF** at (58.6, -291.1)
- removed the REF** at (61.1, -291.1)
- removed the REF** at (63.7, -291.1)
- removed the REF** at (66.2, -291.1)
- removed the REF** at (68.8, -291.1)
- removed the REF** at (71.3, -291.1)
- removed the REF** at (73.8, -291.1)
- removed the REF** at (45.9, -293.6)
- removed the REF** at (48.4, -293.6)
- removed the REF** at (-27.8, -279.3)
- removed the REF** at (51.0, -293.6)
- removed the REF** at (53.5, -293.6)
- removed the REF** at (56.1, -293.6)
- removed the REF** at (58.6, -293.6)
- removed the REF** at (61.1, -293.6)
- removed the REF** at (63.7, -293.6)
- removed the REF** at (66.2, -293.6)
- removed the REF** at (68.8, -293.6)
- removed the REF** at (71.3, -293.6)
- removed the REF** at (73.8, -293.6)
- removed the REF** at (-25.2, -279.3)
- removed the REF** at (37.7, -23.9)
- removed the REF** at (81.9, -23.9)
- removed the REF** at (-51.2, -23.9)
- removed the REF** at (171.0, -23.9)
- removed the REF** at (-22.7, -279.3)
- removed the REF** at (-20.1, -279.3)
- removed the REF** at (-17.6, -279.3)
- removed the REF** at (-15.1, -279.3)
- removed the REF** at (53.5, -279.3)
- removed the REF** at (-12.5, -279.3)
- removed the REF** at (-9.97, -279.3)
- removed the REF** at (-7.43, -279.3)
- removed the REF** at (-4.89, -279.3)
- removed the REF** at (-2.35, -279.3)
- removed the REF** at (0.19, -279.3)
- removed the REF** at (2.73, -279.3)
- removed the REF** at (5.27, -279.3)
- removed the REF** at (7.81, -279.3)
- removed the REF** at (10.3, -279.3)
- removed the REF** at (53.5, -281.8)
- removed the REF** at (12.9, -279.3)
- removed the REF** at (15.4, -279.3)
- removed the REF** at (18.0, -279.3)
- removed the REF** at (20.5, -279.3)
- removed the REF** at (23.0, -279.3)
- removed the REF** at (25.6, -279.3)
- removed the REF** at (28.1, -279.3)
- removed the REF** at (30.7, -279.3)
- removed the REF** at (33.2, -279.3)
- removed the REF** at (86.5, -279.3)
- removed the REF** at (58.6, -276.7)
- removed the REF** at (89.1, -279.3)
- removed the REF** at (91.6, -279.3)
- removed the REF** at (94.2, -279.3)
- removed the REF** at (96.7, -279.3)
- removed the REF** at (99.2, -279.3)
- removed the REF** at (101.8, -279.3)
- removed the REF** at (104.3, -279.3)
- removed the REF** at (106.9, -279.3)
- removed the REF** at (109.4, -279.3)
- removed the REF** at (111.9, -279.3)
- removed the REF** at (58.6, -279.3)
- removed the REF** at (114.5, -279.3)
- removed the REF** at (117.0, -279.3)
- removed the REF** at (119.6, -279.3)
- removed the REF** at (122.1, -279.3)
- removed the REF** at (124.6, -279.3)
- removed the REF** at (127.2, -279.3)
- removed the REF** at (129.7, -279.3)
- removed the REF** at (132.3, -279.3)
- removed the REF** at (134.8, -279.3)
- removed the REF** at (137.3, -279.3)
- removed the REF** at (58.6, -281.8)
- removed the REF** at (139.9, -279.3)
- removed the REF** at (142.4, -279.3)
- removed the REF** at (145.0, -279.3)
- removed the REF** at (147.5, -279.3)
- removed the REF** at (150.0, -279.3)
- removed the REF** at (152.6, -279.3)
- removed the REF** at (155.1, -279.3)
- removed the REF** at (157.7, -279.3)
- removed the REF** at (160.2, -279.3)
- removed the REF** at (162.7, -279.3)
- removed the REF** at (63.7, -276.7)
- removed the REF** at (165.3, -279.3)
- removed the REF** at (-45.5, -281.8)
- removed the REF** at (-43.0, -281.8)
- removed the REF** at (-40.5, -281.8)
- removed the REF** at (-37.9, -281.8)
- removed the REF** at (-35.4, -281.8)
- removed the REF** at (-32.8, -281.8)
- removed the REF** at (-30.3, -281.8)
- removed the REF** at (-27.8, -281.8)
- removed the REF** at (-25.2, -281.8)
- removed the REF** at (63.7, -279.3)
- removed the REF** at (-22.7, -281.8)
- removed the REF** at (-20.1, -281.8)
- removed the REF** at (-17.6, -281.8)
- removed the REF** at (-15.1, -281.8)
- removed the REF** at (-12.5, -281.8)
- removed the REF** at (-9.97, -281.8)
- removed the REF** at (-7.43, -281.8)
- removed the REF** at (-4.89, -281.8)
- removed the REF** at (-2.35, -281.8)
- removed the REF** at (0.19, -281.8)
- removed SW1: tactile_switch, Button_Switch_THT:SW_Tactile_SPST_Angled_PTS645Vx39-2LFS
- removed TP1, TP2, TP3, TP4, TP5: TestPoint, TestPoint:TestPoint_Pad_1.0x1.0mm
- removed U1, U34: 74LVC1G04, alexios:SOT-23-5_HandSoldering
- removed U10: 74LVC2G157, alexios:TSSOP-8_3x3mm_P0.65mm
- removed U11, U14, U22, U52, U53, U54: 74HC574, alexios:DIP-20_W7.62mm_Socket
- removed U12, U15, U16, U20, U21, U23, U55, U56, U57, U58: 74HC541, alexios:DIP-20_W7.62mm_Socket
- removed U13, U35, U4: 74LVC1G32, alexios:SOT-23-5_HandSoldering
- removed U17, U19, U2, U27, U3, U5: 74HC138, Package_DIP:DIP-16_W7.62mm_Socket
- removed U18: 74LVC1G0832, alexios:SOT-23-6_Handsoldering
- removed U24, U25: 74LVC1G11, alexios:SOT-23-6_Handsoldering
- removed U26: 74LVC1G00, alexios:SOT-23-5_HandSoldering
- removed U28, U31, U32, U42, U46: 74LVC1G74, alexios:TSSOP-8_3x3mm_P0.65mm
- removed U29, U30: 74LVC1G08, alexios:SOT-23-5_HandSoldering
- removed U33, U43, U47: 74LVC1G373, alexios:SOT-23-6_Handsoldering
- removed U36, U40, U59: 74HC251, Package_DIP:DIP-16_W7.62mm_Socket
- removed U37: 74AC08, Package_DIP:DIP-14_W7.62mm_Socket
- removed U38: 74AC32, Package_DIP:DIP-14_W7.62mm_Socket
- removed U39: 74LVC1G86, alexios:SOT-23-5_HandSoldering
- removed U41, U8: 74HC139, Package_DIP:DIP-16_W7.62mm_Socket
- removed U44: 74HC85, Package_DIP:DIP-16_W7.62mm_Socket
- removed U45: SN74ACT1071, Package_DIP:DIP-14_W7.62mm_Socket
- removed U48, U49, U50: AT27C020, alexios:PLCC32
- removed U51: 74AC157, Package_DIP:DIP-16_W7.62mm_Socket
- removed U6: 74HC590, Package_DIP:DIP-16_W7.62mm_Socket
- removed U60: 74AC161, Package_DIP:DIP-16_W7.62mm_Socket
- removed U61, U63, U66, U68, U69, U72, U75, U77, U80, U82, U85, U87, U88, U90, U93, U95: 74HC193, Package_DIP:DIP-16_W7.62mm_Socket
- removed U62, U64, U65, U67, U70, U73, U74, U76, U81, U83, U84, U86, U89, U91, U92, U94: 74HCT541, alexios:DIP-20_W7.62mm_Socket
- removed U7: 74LVC1G17, alexios:SOT-23-5_HandSoldering
- removed U71, U78: 74HC688, alexios:DIP-20_W7.62mm_Socket
- removed U79: 74AHC1G08, alexios:SOT-23-5_HandSoldering
- removed U9: 74AC191, Package_DIP:DIP-16_W7.62mm_Socket
- removed X1: 16 MHz, alexios:Crystal_SMD_7050-4Pin_7.0x5.0mm
- added G***: LOGO, alexios:CFT, F.Cu at (254.6, 295.5)
- added P1: VG64_VME_3Rows_3x32_J1_P1, alexios:DIN41612_B_3x32_Horizontal, F.Cu at (40.0, 80.9)
- added P2: VG64_VME_3Rows_3x32_J2_P2, alexios:DIN41612_B_3x32_Horizontal, F.Cu at (173.4, 80.9)
- added REF**: KiCad-Logo2_5mm_SilkScreen, Symbol:KiCad-Logo2_5mm_SilkScreen, F.Cu at (255.9, 329.8)
- added REF**: MountingHole_2.7mm_M2.5, MountingHole:MountingHole_2.7mm_M2.5, F.Cu at (168.3, 352.0)
- added REF**: MountingHole_2.7mm_M2.5, MountingHole:MountingHole_2.7mm_M2.5, F.Cu at (35.1, 352.0)
- added REF**: MountingHole_2.7mm_M2.5, MountingHole:MountingHole_2.7mm_M2.5, F.Cu at (257.4, 352.0)
- added REF**: vero-card-handle-type-C, alexios:vero-card-handle-type-C, F.Cu at (244.8, 349.5)
- added REF**: OSHW-Logo2_7.3x6mm_SilkScreen, Symbol:OSHW-Logo2_7.3x6mm_SilkScreen, F.Cu at (255.9, 310.8)
- added REF**: ESD-Logo_6.6x6mm_SilkScreen, Symbol:ESD-Logo_6.6x6mm_SilkScreen, F.Cu at (255.9, 318.4)
- added REF**: QRCODE-CFT, alexios:QRCODE-CFT, F.Cu at (136.5, 107.5)
- added REF**: MountingHole_2.7mm_M2.5, MountingHole:MountingHole_2.7mm_M2.5, F.Cu at (35.1, 102.0)
- added REF**: MountingHole_2.7mm_M2.5, MountingHole:MountingHole_2.7mm_M2.5, F.Cu at (168.3, 102.0)
- added REF**: MountingHole_2.7mm_M2.5, MountingHole:MountingHole_2.7mm_M2.5, F.Cu at (124.0, 102.0)
- added REF**: MountingHole_2.7mm_M2.5, MountingHole:MountingHole_2.7mm_M2.5, F.Cu at (257.4, 102.0)
- added REF**: MountingHole_2.7mm_M2.5, MountingHole:MountingHole_2.7mm_M2.5, F.Cu at (124.0, 352.0)
- moved REF** 226.3 mm to (47.6, 349.5)
Routing:
- net (no net): track 1648.3 -> 0.00 mm
- net GND: track 32.6 -> 0.00 mm
- net /COND1: track 18.8 -> 0.00 mm
- net /COND2: track 18.8 -> 0.00 mm
- net /COND0: track 18.8 -> 0.00 mm
- net Net-(J2-Pada1): track 12.5 -> 0.00 mm
- net Net-(J1-Padb6): track 12.0 -> 0.00 mm
- net Net-(J1-Padb5): track 12.0 -> 0.00 mm
- net Net-(J1-Padb4): track 12.0 -> 0.00 mm
- net Net-(J1-Padb31): track 12.0 -> 0.00 mm
- net Net-(J1-Padb27): track 12.0 -> 0.00 mm
- net Net-(J1-Padb26): track 12.0 -> 0.00 mm
- net Net-(J1-Padb11): track 12.0 -> 0.00 mm
- net Net-(J1-Padb10): track 12.0 -> 0.00 mm
- net Net-(J1-Padb7): track 12.0 -> 0.00 mm
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Other:
- board size 976.5 x 771.8 mm -> 233.4 x 280 mm
- copper layers 4 -> 2
- rule trace_min: 0.2 -> 0.127
- board text added: "Peripheral Bus"
- board text added: "Processor Bus"
- board text added: "© 2001–2021 Alexios Chouchoulas"
- board text removed: "+5V"
- board text removed: "1 5 10 15 20 25 32"
- board text removed: "10"
- board text removed: "2"
- board text removed: "3"
- board text removed: "32 25 20 15 10 5 1"
- board text removed: "4"
- board text removed: "5"
- board text removed: "6"
- board text removed: "7"
- board text removed: "8"
- board text removed: "9"
- board text removed: "GND"
- board text removed: "JLCJLCJLCJLC"
- board text removed: "a b c"
- board text removed: "keepout areas on both sides for board guides 88 x 55 holes"
- board text removed: "© 2020 Alexios Chouchoulas"
