File: kicad/cft/cft-ctl-reg/cft-reg-ac.sch (KiCad schematic (older format))
At the start: 22 parts, among them U13 74HC193, U14 74HC193, U15 74HC193, U16 74HC193, U17 74AHC1G08, U18 74HCT541, U19 74HCT541, U20 74HCT541, U21 74HCT541, U22 74HC688, U23 74HC688

Commit message: Removing
Parts:
- renumbered C17 to C1501, C23 to C1502, C18 to C1503, C24 to C1504, C19 to C1505, C25 to C1506, C20 to C1507, C26 to C1508, C21 to C1509, C27 to C1510, C22 to C1511, U13 to U1501, U18 to U1502, U22 to U1503, U14 to U1504, U19 to U1505, U20 to U1506, U15 to U1507, U21 to U1508, U16 to U1509, U23 to U1510, U17 to U1511
