File: kicad/cft/cft-board0/cft-board0.sch (KiCad schematic (older format))
At the start: 34 parts, among them P1 CFT-2021-Processor-Bus, P2 CFT-2021-Peripheral-Bus, U101 74LVC1G04, U102 74HC138, U103 74HC138, U104 74HC138, U105 74LVC1G32

Commit message: Route MBU experimentally
Connections:
- net labels added: IR[0..2]
- wire segments 431 -> 426
Changed lines of the file:
@@
 $Descr A4 11693 8268
 encoding utf-8
-Sheet 1 19
+Sheet 1 17
 Title "Control Unit Board"
 Date ""
@@
 ~FPAEXT
 Wire Wire Line
-	12150 -6450 13000 -6450
-Wire Wire Line
-	12150 -6150 13000 -6150
-Text Label 13000 -6450 2    50   ~ 0
-~SYSDEV
-Wire Bus Line
-	12150 -6350 13000 -6350
-Text Label 13000 -6350 2    50   ~ 0
-AB[0..23]
-Text Label 13000 -6150 2    50   ~ 0
-~W
-Wire Bus Line
-	12150 -6050 13000 -6050
-Text Label 13000 -6050 2    50   ~ 0
-DB[0..15]
-Wire Wire Line
 	11000 -5450 10150 -5450
 Text Label 10150 -5450 0    50   ~ 0
@@
 Wire Bus Line
 	11000 -6150 10150 -6150
-Text Label 10150 -6700 0    50   ~ 0
-~RESET
-Wire Wire Line
-	11000 -6700 10150 -6700
 Wire Wire Line
 	15350 -6200 16200 -6200
@@
 Address Register
 Wire Wire Line
-	11000 -5850 10150 -5850
-Wire Wire Line
-	11000 -5750 10150 -5750
-Text Label 10150 -5850 0    50   ~ 0
-IR0
-Text Label 10150 -5750 0    50   ~ 0
-IR1
-Wire Wire Line
-	12150 -6250 13000 -6250
-Text Label 13000 -6250 2    50   ~ 0
-~R
-Wire Wire Line
-	11000 -5650 10150 -5650
-Text Label 10150 -5650 0    50   ~ 0
-IR2
-Wire Wire Line
 	15300 -3650 16150 -3650
 Text Label 16150 -3650 2    50   ~ 0
@@
 Text Label 13350 -6100 0    50   ~ 0
 ~HALT
-Wire Wire Line
-	11000 -6600 10150 -6600
-Text Label 10150 -6600 0    50   ~ 0
-CLK2
-Wire Wire Line
-	11000 -6500 10150 -6500
-Text Label 10150 -6500 0    50   ~ 0
-CLK4
 $Sheet
 S 10950 -4650 1150 450
@@
 F0 "Memory Bank Unit (MBU)" 50
 F1 "mbu.sch" 50
-F2 "~RESET" I L 11000 -6700 50
-F3 "AEXT[0..7]" O R 12150 -6700 50
-F4 "WADDR[0..4]" I L 11000 -6150 50
-F5 "~FPRAM~∕ROM" I L 11000 -5450 50
-F6 "IBUS[0..7]" T L 11000 -6050 50
-F7 "RADDR[0..4]" I L 11000 -6250 50
-F8 "AB[0..7]" I R 12150 -6350 50
-F9 "~W" I R 12150 -6150 50
-F10 "~SYSDEV" I R 12150 -6450 50
-F11 "DB[0..7]" B R 12150 -6050 50
-F12 "~IR-IDX" I L 11000 -5950 50
-F13 "~WAR" O R 12150 -5450 50
-F14 "IR0" I L 11000 -5850 50
-F15 "IR1" I L 11000 -5750 50
-F16 "~R" I R 12150 -6250 50
-F17 "IR2" I L 11000 -5650 50
-F18 "CLK4" I L 11000 -6500 50
-F19 "CLK2" I L 11000 -6600 50
+F2 "AEXT[0..7]" O R 12150 -6700 50
+F3 "WADDR[0..4]" I L 11000 -6150 50
+F4 "~FPRAM~∕ROM" I L 11000 -5450 50
+F5 "IBUS[0..7]" T L 11000 -6050 50
+F6 "RADDR[0..4]" I L 11000 -6250 50
+F7 "~IR-IDX" I L 11000 -5950 50
+F8 "~WAR" O R 12150 -5450 50
+F9 "CLK4" I L 11000 -6500 50
+F10 "CLK2" I L 11000 -6600 50
+F11 "~RSTHOLD" I L 11000 -6700 50
+F12 "IR[0..2]" I L 11000 -5850 50
+F13 "~T34" I L 11000 -6400 50
 $EndSheet
 Wire Wire Line
@@
 $EndComp
 Wire Bus Line
+	11000 -5850 10150 -5850
+Text Label 10150 -5850 0    50   ~ 0
+IR[0..2]
+Wire Wire Line
+	11000 -6700 10150 -6700
+Wire Wire Line
+	11000 -6600 10150 -6600
+Wire Wire Line
+	11000 -6500 10150 -6500
+Wire Wire Line
+	11000 -6400 10150 -6400
+Wire Bus Line
 	2450 -4900 2450 -4100
 Wire Bus Line
@@
 Wire Bus Line
 	-10350 -3450 -10350 -2650
+Text Label 10150 -6700 0    50   ~ 0
+~RSTHOLD
+Text Label 10150 -6600 0    50   ~ 0
+CLK2
+Text Label 10150 -6500 0    50   ~ 0
+CLK3
+Text Label 10150 -6400 0    50   ~ 0
+~T34
 $EndSCHEMATC

Commit message: Work on Board 0.
Connections:
- net labels added: ~FPCTX
- wire segments 426 -> 427
Changed lines of the file:
@@
 F12 "IR[0..2]" I L 11000 -5850 50
 F13 "~T34" I L 11000 -6400 50
+F14 "~FPCTX" I L 11000 -5550 50
+F15 "FPD[0..7]" T R 12150 -5550 50
 $EndSheet
 Wire Wire Line
@@
 Wire Wire Line
 	11000 -6400 10150 -6400
-Wire Bus Line
-	2450 -4900 2450 -4100
-Wire Bus Line
-	2450 -6350 2450 -5550
-Wire Bus Line
-	2450 -3250 2450 -2550
-Wire Bus Line
-	-1200 -6850 -1200 -6200
-Wire Bus Line
-	-10350 -3450 -10350 -2650
 Text Label 10150 -6700 0    50   ~ 0
 ~RSTHOLD
@@
 Text Label 10150 -6400 0    50   ~ 0
 ~T34
+Wire Wire Line
+	10150 -5550 11000 -5550
+Text Label 10150 -5550 0    50   ~ 0
+~FPCTX
+Wire Bus Line
+	12150 -5550 13000 -5550
+Text Label 13000 -5550 2    50   ~ 0
+FPD[0..7]
+Wire Bus Line
+	2450 -4900 2450 -4100
+Wire Bus Line
+	2450 -6350 2450 -5550
+Wire Bus Line
+	2450 -3250 2450 -2550
+Wire Bus Line
+	-1200 -6850 -1200 -6200
+Wire Bus Line
+	-10350 -3450 -10350 -2650
 $EndSCHEMATC

Commit message: Route Board 0
Parts:
- removed U102, U103: 74HC138, alexios:DIP-16_W7.62mm_Socket, symbol alexios:74HC138
- added C1, C2: 100nF, alexios:SMD_0805_2012Metric_Pad1.15x1.40mm_HandSolder, symbol Device:C_Small
- added U1, U2: 16V8, alexios:DIP-20_W7.62mm_Socket, symbol alexios:16V8
Connections:
- net labels added: RADDR[0..1], ~READ_AGL, ~READ_CS, ~READ_DR, ~READ_FL, ~READ_PC, ~WRITE_DR, ~WRITE_FL, ~WRITE_IR, ~WRITE_PC
- wire segments 427 -> 441
- no-connect marks 15 -> 31
Other:
- note removed: "RADDR=010xx"

Commit message: Place and route more of Board 0
Parts:
- renumbered C112 to C104, C104 to C20, C105 to C21, C106 to C22
Connections:
- net labels added: ~READ-CS, ~READ-FL
- net labels removed: ~READ_AGL, ~READ_CS, ~READ_DR, ~READ_FL, ~READ_PC
- wire segments 441 -> 442
Changed lines of the file:
@@
 AR Path="/5CC0D65F/5DD51032" Ref="C?"  Part="1"
 AR Path="/5CE16E65/5DD51032" Ref="C?"  Part="1"
-AR Path="/5DD51032" Ref="C112"  Part="1"
+AR Path="/5DD51032" Ref="C104"  Part="1"
 AR Path="/5D54E677/5DD51032" Ref="C?"  Part="1"
 AR Path="/5D62E1DC/5DD51032" Ref="C?"  Part="1"
@@
 AR Path="/5D892D5E/5DD51032" Ref="C?"  Part="1"
 AR Path="/5D9672D4/5DD51032" Ref="C?"  Part="1"
-F 0 "C112" H 6059 -904 50  0000 R CNN
+F 0 "C104" H 6059 -904 50  0000 R CNN
 F 1 "100nF" H 6059 -995 50  0000 R CNN
 F 2 "alexios:SMD_0805_2012Metric_Pad1.15x1.40mm_HandSolder" H 6150 -950 50  0001 C CNN
@@
 Wire Wire Line
 	19750 -2050 19750 -1950
-$Comp
-L Device:CP_Small C105
-U 1 1 5DF0FF8F
-P 19750 -1850
-AR Path="/5DF0FF8F" Ref="C105"  Part="1"
-AR Path="/5D34E810/5DF0FF8F" Ref="C?"  Part="1"
-AR Path="/5F1DB2E8/5DF0FF8F" Ref="C?"  Part="1"
-AR Path="/5DD3D79F/5DF0FF8F" Ref="C?"  Part="1"
-F 0 "C105" H 19662 -1804 50  0000 R CNN
-F 1 "47µF" H 19662 -1895 50  0000 R CNN
-F 2 "Capacitor_THT:CP_Radial_D6.3mm_P2.50mm" H 19750 -1850 50  0001 C CNN
-F 3 "~" H 19750 -1850 50  0001 C CNN
-	1    19750 -1850
-	1    0    0    -1
-$EndComp
 Wire Wire Line
 	19750 -1750 19750 -1650
@@
 Wire Wire Line
 	19300 -2050 19300 -1950
-$Comp
-L Device:CP_Small C104
-U 1 1 5DF0FFA3
-P 19300 -1850
-AR Path="/5DF0FFA3" Ref="C104"  Part="1"
-AR Path="/5D34E810/5DF0FFA3" Ref="C?"  Part="1"
-AR Path="/5F1DB2E8/5DF0FFA3" Ref="C?"  Part="1"
-AR Path="/5DD3D79F/5DF0FFA3" Ref="C?"  Part="1"
-F 0 "C104" H 19212 -1804 50  0000 R CNN
-F 1 "47µF" H 19212 -1895 50  0000 R CNN
-F 2 "Capacitor_THT:CP_Radial_D6.3mm_P2.50mm" H 19300 -1850 50  0001 C CNN
-F 3 "~" H 19300 -1850 50  0001 C CNN
-	1    19300 -1850
-	1    0    0    -1
-$EndComp
 Wire Wire Line
 	19300 -1750 19300 -1650
@@
 F2 "RADDR[0..1]" I L 10950 -4500 50
 F3 "IBUS[0..15]" B R 12100 -4500 50
-F4 "~READ_CS" I L 10950 -4350 50
+F4 "~READ-CS" I L 10950 -4350 50
 $EndSheet
 Wire Wire Line
 	10950 -4350 10100 -4350
 Text Label 10100 -4350 0    50   ~ 0
-~READ_CS
+~READ-CS
 $Sheet
 S 11000 -6850 1150 1550
@@
 Wire Wire Line
 	20200 -2050 20200 -1950
-$Comp
-L Device:CP_Small C106
-U 1 1 5EFD0822
-P 20200 -1850
-AR Path="/5EFD0822" Ref="C106"  Part="1"
-AR Path="/5D34E810/5EFD0822" Ref="C?"  Part="1"
-AR Path="/5F1DB2E8/5EFD0822" Ref="C?"  Part="1"
-AR Path="/5DD3D79F/5EFD0822" Ref="C?"  Part="1"
-F 0 "C106" H 20112 -1804 50  0000 R CNN
-F 1 "47µF" H 20112 -1895 50  0000 R CNN
-F 2 "Capacitor_THT:CP_Radial_D6.3mm_P2.50mm" H 20200 -1850 50  0001 C CNN
-F 3 "~" H 20200 -1850 50  0001 C CNN
-	1    20200 -1850
-	1    0    0    -1
-$EndComp
 Wire Wire Line
 	20200 -1750 20200 -1650
@@
 F13 "~READ-AGL" O R -8500 -1450 50
 F14 "~WRITE-IR" O R -8500 -1350 50
+F15 "~READ-FL" I R -8500 -1950 50
 $EndSheet
 Wire Bus Line
@@
 NoConn ~ 16700 3250
 Text Label 17200 2550 2    50   ~ 0
-~READ_DR
+~READ-DR
 Text Label 17200 2650 2    50   ~ 0
-~READ_PC
+~READ-PC
 Text Label 17200 2750 2    50   ~ 0
-~READ_FL
+~READ-FL
 Text Label 17200 2850 2    50   ~ 0
-~READ_AGL
+~READ-AGL
 Wire Wire Line
 	15800 4250 15350 4250
@@
 	16700 2950 17200 2950
 Text Label 17200 2950 2    50   ~ 0
-~READ_CS
+~READ-CS
 NoConn ~ 15800 2650
 NoConn ~ 15800 2750
@@
 NoConn ~ 15800 3450
 NoConn ~ 15800 3550
+$Comp
+L Device:CP_Small C22
+U 1 1 5EFD0822
+P 20200 -1850
+AR Path="/5EFD0822" Ref="C22"  Part="1"
+AR Path="/5D34E810/5EFD0822" Ref="C?"  Part="1"
+AR Path="/5F1DB2E8/5EFD0822" Ref="C?"  Part="1"
+AR Path="/5DD3D79F/5EFD0822" Ref="C?"  Part="1"
+F 0 "C22" H 20112 -1804 50  0000 R CNN
+F 1 "47µF" H 20112 -1895 50  0000 R CNN
+F 2 "Capacitor_THT:CP_Radial_D6.3mm_P2.50mm" H 20200 -1850 50  0001 C CNN
+F 3 "~" H 20200 -1850 50  0001 C CNN
+	1    20200 -1850
+	1    0    0    -1
+$EndComp
+$Comp
+L Device:CP_Small C21
+U 1 1 5DF0FF8F
+P 19750 -1850
+AR Path="/5DF0FF8F" Ref="C21"  Part="1"
+AR Path="/5D34E810/5DF0FF8F" Ref="C?"  Part="1"
+AR Path="/5F1DB2E8/5DF0FF8F" Ref="C?"  Part="1"
+AR Path="/5DD3D79F/5DF0FF8F" Ref="C?"  Part="1"
+F 0 "C21" H 19662 -1804 50  0000 R CNN
+F 1 "47µF" H 19662 -1895 50  0000 R CNN
+F 2 "Capacitor_THT:CP_Radial_D6.3mm_P2.50mm" H 19750 -1850 50  0001 C CNN
+F 3 "~" H 19750 -1850 50  0001 C CNN
+	1    19750 -1850
+	1    0    0    -1
+$EndComp
+$Comp
+L Device:CP_Small C20
+U 1 1 5DF0FFA3
+P 19300 -1850
+AR Path="/5DF0FFA3" Ref="C20"  Part="1"
+AR Path="/5D34E810/5DF0FFA3" Ref="C?"  Part="1"
+AR Path="/5F1DB2E8/5DF0FFA3" Ref="C?"  Part="1"
+AR Path="/5DD3D79F/5DF0FFA3" Ref="C?"  Part="1"
+F 0 "C20" H 19212 -1804 50  0000 R CNN
+F 1 "47µF" H 19212 -1895 50  0000 R CNN
+F 2 "Capacitor_THT:CP_Radial_D6.3mm_P2.50mm" H 19300 -1850 50  0001 C CNN
+F 3 "~" H 19300 -1850 50  0001 C CNN
+	1    19300 -1850
+	1    0    0    -1
+$EndComp
+Wire Wire Line
+	-8500 -1950 -7900 -1950
 Wire Bus Line
 	2450 -4900 2450 -4100
@@
 Wire Bus Line
 	-10350 -3450 -10350 -2650
+Text Label -7900 -1950 2    50   ~ 0
+~READ-FL
 $EndSCHEMATC

Commit message: Work on Board 0 schematics
Connections:
- net labels added: ~WRITE-FL
- net labels removed: ~FLAGWE
Changed lines of the file:
@@
 FN
 Text Label -7150 13000 0    50   ~ 0
-~FLAGWE
+~WRITE-FL
 Text Label -7150 13200 0    50   ~ 0
 IR0
@@
 IR[0..6]
 Text Label -1050 -5700 2    50   ~ 0
-~FLAGWE
+~WRITE-FL
 Text Label -1050 -5900 2    50   ~ 0
 FL
@@
 F8 "~IRQSµC" O R -5800 -1100 50
 F9 "IBUS15" I L -6950 -1450 50
-F10 "~FLAGWE" I L -6950 -1350 50
+F10 "~WRITE-FL" I L -6950 -1350 50
 F11 "ACTION[0..3]" I L -6950 -1650 50
 F12 "~ACTION-IDX" O R -5800 -1750 50
@@
 ~END
 Text Label -7550 -1350 0    50   ~ 0
-~FLAGWE
+~WRITE-FL
 Text Label -7550 -1450 0    50   ~ 0
 IBUS15

Commit message: Routing Board 0
Parts:
- removed C101: 100nF, alexios:C_SMD_0805_2012Metric_Pad1.15x1.40mm_HandSolder, symbol Device:C_Small
- removed C104: 100nF, alexios:SMD_0805_2012Metric_Pad1.15x1.40mm_HandSolder, symbol Device:C_Small
- removed JP104: Jumper_NC_Small, Jumper:SolderJumper-2_P1.3mm_Bridged_RoundedPad1.0x1.5mm, symbol Device:Jumper_NC_Small
- removed U104: 74HC138, alexios:DIP-16_W7.62mm_Socket, symbol alexios:74HC138
- removed U105: 74LVC1G32, alexios:SOT-23-5_HandSoldering, symbol alexios:74LVC1G32
Connections:
- net labels added: ~DECDR, ~INCDR, ~INCPC
- net labels removed: ACTION[3..0], ~ACTION-DECDR, ~ACTION-IDX, ~ACTION-INCDR, ~ACTION-INCPC
- wire segments 442 -> 431
- no-connect marks 31 -> 30
Other:
- note removed: "The PC doesn't decrement"

Commit message: Route Board 0
Connections:
- net labels removed: ~WRITE_DR, ~WRITE_FL, ~WRITE_IR, ~WRITE_PC
Changed lines of the file:
@@
 	17200 4350 16700 4350
 Text Label 17200 4050 2    50   ~ 0
-~WRITE_DR
+~WRITE-DR
 Text Label 17200 4150 2    50   ~ 0
-~WRITE_PC
+~WRITE-PC
 Text Label 17200 4250 2    50   ~ 0
-~WRITE_FL
+~WRITE-FL
 Text Label 17200 4350 2    50   ~ 0
-~WRITE_IR
+~WRITE-IR
 NoConn ~ 15800 4550
 NoConn ~ 15800 4650
