File: kicad/cft/cft-board0/cft_ws_busen.sch (KiCad schematic (older format))
At the start: 39 parts, among them U901 74HC14, U903 74LVC1G0832, U904 74LVC1G04, U905 74LVC1G74, U906 74LVC1G125, U907 74LVC1G32, U908 74LVC1G74, U909 74ACT245, U910 74LVC1G11, U911 74ACT245

Commit message: Work on schematic and route board 0
Parts:
- removed C903, C905, C908, C910: 100nF, alexios:C_SMD_0805_2012Metric_Pad1.15x1.40mm_HandSolder, symbol Device:C_Small
- removed JP901: Jumper_3_Bridged12, Jumper:SolderJumper-3_P1.3mm_Bridged12_RoundedPad1.0x1.5mm, symbol alexios:Jumper_3_Bridged12
- removed R903: 4.7kΩ, alexios:R_SMD_0805_2012Metric_Pad1.15x1.40mm_HandSolder, symbol Device:R_Small
- removed R905, R906, R907, R909, R911, R912: 0Ω, alexios:R_SMD_0805_2012Metric_Pad1.15x1.40mm_HandSolder, symbol Device:R_Small
- removed R910: 680Ω, alexios:R_SMD_0805_2012Metric_Pad1.15x1.40mm_HandSolder, symbol Device:R_Small
- removed TP901, TP902: TestPoint, TestPoint:TestPoint_Pad_1.0x1.0mm, symbol Connector:TestPoint
- removed U903: 74LVC1G0832, alexios:SOT-23-6_Handsoldering, symbol alexios:74LVC1G0832
- removed U904: 74LVC1G04, alexios:SOT-23-5_HandSoldering, symbol alexios:74LVC1G04
- removed U905, U908: 74LVC1G74, alexios:TSSOP-8_3x3mm_P0.65mm, symbol alexios:74AUC1G74
- removed U907: 74LVC1G32, alexios:SOT-23-5_HandSoldering, symbol alexios:74LVC1G32
- removed U910: 74LVC1G11, alexios:SOT-23-6_Handsoldering, symbol alexios:74LVC1G11
- added C901: 100nF, alexios:C_SMD_0805_2012Metric_Pad1.15x1.40mm_HandSolder, symbol Device:C_Small
- added C921, C923: 120pF, alexios:C_SMD_0805_2012Metric_Pad1.15x1.40mm_HandSolder, symbol Device:C_Small
- added C922: 22pF, alexios:C_SMD_0805_2012Metric_Pad1.15x1.40mm_HandSolder, symbol Device:C_Small
- added D902, D903: LED_ALT, alexios:LED_0805_2012Metric_Pad1.15x1.40mm_HandSolder, symbol Device:LED_ALT
- added R921, R923: 100Ω, alexios:R_SMD_0805_2012Metric_Pad1.15x1.40mm_HandSolder, symbol Device:R_Small
- added R922, R924: 4.7kΩ, alexios:R_SMD_0805_2012Metric_Pad1.15x1.40mm_HandSolder, symbol Device:R_Small
- added RV902: 1kΩ, alexios:Potentiometer_Bourns_67W, symbol Device:R_POT
- added U901: 16V8, alexios:DIP-20_W7.62mm_Socket, symbol alexios:16V8
- added U902, U904: 74HC74, alexios:DIP-14_W7.62mm_Socket, symbol alexios:74HC74
- added U907: 74LVC1G125, alexios:SOT-23-5_HandSoldering, symbol alexios:74AHC1G125
- R901, R902, R904: value 0Ω -> 680Ω
- renumbered C901 to C903, C911 to C910, U901 to U903, U911 to U910
Connections:
- net labels added: CLK1, DBDIR, T34, ~ABEN, ~CLRRW, ~CLRWS, ~DBEN, ~REN, ~SETR, ~SETW
- net labels removed: CLK2, CLK2', HALT, ~BUSEN, ~T34, ~WAITING0, ~WEN-DELAYED, ~WEN1, ~WS-in-T34, ~WSTB, ~W₀
- wire segments 128 -> 122
Other:
- note added: "Control Logic"
- note added: "Delay"
- note added: "Read/Write Transactions"
- note added: "Termination"
- note added: "Tri-Stating"
- note added: "~DBDIR~\n\n \n \n\n 0\n 0\n\n 1\n 1"
- note added: "~DBEN~\n\n 1\n 1\n\n 0\n 0\n\n 1\n 1"
- note added: "~IO~\n\nX\n1\n\nX\n0\n\nX\n0"
- note added: "~MEM~\n\n X\n 1\n\n 0\n X\n\n 0\n X\n"
- note added: "~REN~\n\n X\n X\n\n 0\n 0\n\n 1\n 1"
- note added: "~RSTHOLD~\n\n 0\n 1\n\n 1\n 1\n\n 1\n 1"
- note added: "~WAITING~\n\n X\n 1\n\n X\n X\n\n X\n X"
- note added: "~WEN~\n\n X\n X\n\n X\n X\n\n X\n X"
- note removed: "Also used by the AR."
- note removed: "Keep the data bus enabled\nwhile waiting."
- note removed: "Keep ~W~ low during a wait state."
- note removed: "Optional"
- note removed: "Optional impedance\nmatching resistors."
- note removed: "Pull-up used to slow\ndown negative edge.\nMay be optional,\ntest first!"
- note removed: "Tristate ~W~ on ~HALT~."
- note removed: "Write Strobe"
- note removed: "~BUSEN~\n\n 0\n 0\n 0\n 1"
- note removed: "~IO~\n\nX\n0\nX\n1"
- note removed: "~MEM~\n\n 0\n X\n X\n 1"
- note removed: "~WAITING~\n\n X\n X\n 0\n 1"
- moved on the sheet: C903, C909, C910, C920, R908, RV901, U903A, U903B, U903C, U903D, U903E, U903F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

Commit message: Route board0
Connections:
- net ~WS: now also R908.2
Changed lines of the file:
@@
 Connection ~ 6900 5750
 Wire Wire Line
-	3700 2150 4450 2150
+	3700 2150 3950 2150
 Wire Wire Line
 	4100 1650 4450 1650
@@
 Text Label 4100 1550 0    50   ~ 0
 ~HALT
+Wire Wire Line
+	3950 1100 3950 2150
 Wire Bus Line
 	9650 3550 9650 5900
 Wire Bus Line
 	7750 3900 7750 6350
+Connection ~ 3950 2150
+Wire Wire Line
+	3950 2150 4450 2150
 $EndSCHEMATC
