File: kicad/cft/cft-board0/cft_ar.sch (KiCad schematic (older format))
At the start: 22 parts, among them U401 74HC138, U402 74HC574, U403 74HC541, U404 74LVC1G08, U405 74LVC1G32, U406 74HC574, U407 74HC541, U408 74HC574, U409 74HC541, U410 74HC541

Commit message: Work on Board 0
Connections:
- net ~ABEN2: no longer U409.19 (~G2)
Changed lines of the file:
@@
 Wire Wire Line
 	4700 6000 4700 5600
-Wire Wire Line
-	4700 5600 5250 5600
 Connection ~ 2650 4300
 Text Label 2650 3350 1    50   ~ 0

Commit message: Place and route more of Board 0
Parts:
- renumbered C404 to C402, C407 to C403, C402 to C404, C403 to C405, C405 to C406, C408 to C407, C406 to C408
Connections:
- net ~ABEN2: now also U409.19 (~G2)
Changed lines of the file:
@@
 $EndComp
-Wire Wire Line
-	4650 1250 4850 1250
-Wire Wire Line
-	4650 1350 4850 1350
-Wire Wire Line
-	4650 1450 4850 1450
-Wire Wire Line
-	4650 1550 4850 1550
-Wire Wire Line
-	4650 1650 4850 1650
-Wire Wire Line
-	4650 1750 4850 1750
-Wire Wire Line
-	4650 1850 4850 1850
-Wire Wire Line
-	4650 1950 4850 1950
 Wire Wire Line
 	4650 2900 4850 2900
@@
 Wire Wire Line
 	4650 3600 4850 3600
-Text Label 4650 1250 0    50   ~ 0
-AR0
-Text Label 4650 1350 0    50   ~ 0
-AR1
-Text Label 4650 1450 0    50   ~ 0
-AR2
-Text Label 4650 1550 0    50   ~ 0
-AR3
-Text Label 4650 1650 0    50   ~ 0
-AR4
-Text Label 4650 1750 0    50   ~ 0
-AR5
-Text Label 4650 1850 0    50   ~ 0
-AR6
-Text Label 4650 1950 0    50   ~ 0
-AR7
 Text Label 4650 2900 0    50   ~ 0
 AR8
@@
 AR15
 Wire Wire Line
-	5050 1250 5250 1250
-Wire Wire Line
-	5050 1350 5250 1350
-Wire Wire Line
-	5050 1450 5250 1450
-Wire Wire Line
-	5050 1550 5250 1550
-Wire Wire Line
-	5050 1650 5250 1650
-Wire Wire Line
-	5050 1750 5250 1750
-Wire Wire Line
-	5050 1850 5250 1850
-Wire Wire Line
-	5050 1950 5250 1950
-Wire Wire Line
 	5050 2900 5250 2900
 Wire Wire Line
@@
 	1    0    0    -1
 $EndComp
-Text Label 5250 1250 2    50   ~ 0
-AR0
-Text Label 5250 1350 2    50   ~ 0
-AR1
-Text Label 5250 1450 2    50   ~ 0
-AR2
-Text Label 5250 1550 2    50   ~ 0
-AR3
-Text Label 5250 1650 2    50   ~ 0
-AR4
-Text Label 5250 1750 2    50   ~ 0
-AR5
-Text Label 5250 1850 2    50   ~ 0
-AR6
-Text Label 5250 1950 2    50   ~ 0
-AR7
 Text Label 5250 2900 2    50   ~ 0
 AR8
@@
 AR15
 Wire Wire Line
-	6250 1250 6500 1250
-Wire Wire Line
-	6250 1350 6500 1350
-Wire Wire Line
-	6250 1450 6500 1450
-Wire Wire Line
-	6250 1550 6500 1550
-Wire Wire Line
-	6250 1650 6500 1650
-Wire Wire Line
-	6250 1750 6500 1750
-Wire Wire Line
-	6250 1850 6500 1850
-Wire Wire Line
-	6250 1950 6500 1950
-Wire Wire Line
 	6250 2900 6500 2900
 Wire Wire Line
@@
 Wire Wire Line
 	3300 3600 3650 3600
-Wire Wire Line
-	3300 1250 3650 1250
-Wire Wire Line
-	3300 1350 3650 1350
-Wire Wire Line
-	3300 1450 3650 1450
-Wire Wire Line
-	3300 1550 3650 1550
-Wire Wire Line
-	3300 1650 3650 1650
-Wire Wire Line
-	3300 1750 3650 1750
-Wire Wire Line
-	3300 1850 3650 1850
-Wire Wire Line
-	3300 1950 3650 1950
-Text Label 3650 1250 2    50   ~ 0
-IBUS0
-Text Label 3650 1350 2    50   ~ 0
-IBUS1
-Text Label 3650 1450 2    50   ~ 0
-IBUS2
-Text Label 3650 1550 2    50   ~ 0
-IBUS3
-Text Label 3650 1650 2    50   ~ 0
-IBUS4
-Text Label 3650 1750 2    50   ~ 0
-IBUS5
-Text Label 3650 1850 2    50   ~ 0
-IBUS6
-Text Label 3650 1950 2    50   ~ 0
-IBUS7
 Text Label 3650 2900 2    50   ~ 0
 IBUS8
@@
 Entry Wire Line
 	6500 3600 6600 3700
-Text Label 6250 1250 0    50   ~ 0
-AB0
-Text Label 6250 1350 0    50   ~ 0
-AB1
-Text Label 6250 1450 0    50   ~ 0
-AB2
-Text Label 6250 1550 0    50   ~ 0
-AB3
-Text Label 6250 1650 0    50   ~ 0
-AB4
-Text Label 6250 1750 0    50   ~ 0
-AB5
-Text Label 6250 1850 0    50   ~ 0
-AB6
-Text Label 6250 1950 0    50   ~ 0
-AB7
 Text Label 6250 2900 0    50   ~ 0
 AB8
@@
 Text HLabel 1000 1500 0    50   Input ~ 0
 AEXT[0..7]
-Wire Wire Line
-	4650 4600 4850 4600
-Wire Wire Line
-	4650 4700 4850 4700
-Wire Wire Line
-	4650 4800 4850 4800
-Wire Wire Line
-	4650 4900 4850 4900
-Wire Wire Line
-	4650 5000 4850 5000
-Wire Wire Line
-	4650 5100 4850 5100
-Wire Wire Line
-	4650 5200 4850 5200
-Wire Wire Line
-	4650 5300 4850 5300
-Text Label 4650 4600 0    50   ~ 0
-AR16
-Text Label 4650 4700 0    50   ~ 0
-AR17
-Text Label 4650 4800 0    50   ~ 0
-AR18
-Text Label 4650 4900 0    50   ~ 0
-AR19
-Text Label 4650 5000 0    50   ~ 0
-AR20
-Text Label 4650 5100 0    50   ~ 0
-AR21
-Text Label 4650 5200 0    50   ~ 0
-AR22
-Text Label 4650 5300 0    50   ~ 0
-AR23
 Wire Wire Line
 	5250 4600 5050 4600
@@
 AR Path="/5CC0D65F/5D344142" Ref="C?"  Part="1"
 AR Path="/5D344142" Ref="C?"  Part="1"
-AR Path="/5CC06F10/5D344142" Ref="C404"  Part="1"
-F 0 "C404" H 809 6796 50  0000 R CNN
+AR Path="/5CC06F10/5D344142" Ref="C402"  Part="1"
+F 0 "C402" H 809 6796 50  0000 R CNN
 F 1 "100nF" H 809 6705 50  0000 R CNN
 F 2 "alexios:C_SMD_0805_2012Metric_Pad1.15x1.40mm_HandSolder" H 900 6750 50  0001 C CNN
@@
 AR Path="/5CC0D65F/5D34414E" Ref="C?"  Part="1"
 AR Path="/5D34414E" Ref="C?"  Part="1"
-AR Path="/5CC06F10/5D34414E" Ref="C405"  Part="1"
-F 0 "C405" H 2209 6796 50  0000 R CNN
+AR Path="/5CC06F10/5D34414E" Ref="C406"  Part="1"
+F 0 "C406" H 2209 6796 50  0000 R CNN
 F 1 "100nF" H 2209 6705 50  0000 R CNN
 F 2 "alexios:C_SMD_0805_2012Metric_Pad1.15x1.40mm_HandSolder" H 2300 6750 50  0001 C CNN
@@
 AR Path="/5CC0D65F/5D34415A" Ref="C?"  Part="1"
 AR Path="/5D34415A" Ref="C?"  Part="1"
-AR Path="/5CC06F10/5D34415A" Ref="C407"  Part="1"
-F 0 "C407" H 809 7446 50  0000 R CNN
+AR Path="/5CC06F10/5D34415A" Ref="C403"  Part="1"
+F 0 "C403" H 809 7446 50  0000 R CNN
 F 1 "100nF" H 809 7355 50  0000 R CNN
 F 2 "alexios:C_SMD_0805_2012Metric_Pad1.15x1.40mm_HandSolder" H 900 7400 50  0001 C CNN
@@
 AR Path="/5CC0D65F/5D344166" Ref="C?"  Part="1"
 AR Path="/5D344166" Ref="C?"  Part="1"
-AR Path="/5CC06F10/5D344166" Ref="C408"  Part="1"
-F 0 "C408" H 2209 7446 50  0000 R CNN
+AR Path="/5CC06F10/5D344166" Ref="C407"  Part="1"
+F 0 "C407" H 2209 7446 50  0000 R CNN
 F 1 "100nF" H 2209 7355 50  0000 R CNN
 F 2 "alexios:C_SMD_0805_2012Metric_Pad1.15x1.40mm_HandSolder" H 2300 7400 50  0001 C CNN
@@
 AR Path="/5CC0D65F/5D34419E" Ref="C?"  Part="1"
 AR Path="/5D34419E" Ref="C?"  Part="1"
-AR Path="/5CC06F10/5D34419E" Ref="C406"  Part="1"
-F 0 "C406" H 3609 6796 50  0000 R CNN
+AR Path="/5CC06F10/5D34419E" Ref="C408"  Part="1"
+F 0 "C408" H 3609 6796 50  0000 R CNN
 F 1 "100nF" H 3609 6705 50  0000 R CNN
 F 2 "alexios:C_SMD_0805_2012Metric_Pad1.15x1.40mm_HandSolder" H 3700 6750 50  0001 C CNN
@@
 AR Path="/5CC0D65F/5E3EB5F8" Ref="C?"  Part="1"
 AR Path="/5E3EB5F8" Ref="C?"  Part="1"
-AR Path="/5CC06F10/5E3EB5F8" Ref="C402"  Part="1"
-F 0 "C402" H 809 5496 50  0000 R CNN
+AR Path="/5CC06F10/5E3EB5F8" Ref="C404"  Part="1"
+F 0 "C404" H 809 5496 50  0000 R CNN
 F 1 "100nF" H 809 5405 50  0000 R CNN
 F 2 "alexios:C_SMD_0805_2012Metric_Pad1.15x1.40mm_HandSolder" H 900 5450 50  0001 C CNN
@@
 AR Path="/5CC0D65F/604EA909" Ref="C?"  Part="1"
 AR Path="/604EA909" Ref="C?"  Part="1"
-AR Path="/5CC06F10/604EA909" Ref="C403"  Part="1"
-F 0 "C403" H 809 6146 50  0000 R CNN
+AR Path="/5CC06F10/604EA909" Ref="C405"  Part="1"
+F 0 "C405" H 809 6146 50  0000 R CNN
 F 1 "100nF" H 809 6055 50  0000 R CNN
 F 2 "alexios:C_SMD_0805_2012Metric_Pad1.15x1.40mm_HandSolder" H 900 6100 50  0001 C CNN
@@
 Text Notes 1450 2450 0    50   ~ 0
 Optional
+Wire Wire Line
+	4700 5600 5250 5600
+Wire Wire Line
+	3300 1250 3650 1250
+Wire Wire Line
+	3300 1350 3650 1350
+Wire Wire Line
+	3300 1450 3650 1450
+Wire Wire Line
+	3300 1550 3650 1550
+Wire Wire Line
+	3300 1650 3650 1650
+Wire Wire Line
+	3300 1750 3650 1750
+Wire Wire Line
+	3300 1850 3650 1850
+Wire Wire Line
+	3300 1950 3650 1950
+Text Label 3650 1250 2    50   ~ 0
+IBUS0
+Text Label 3650 1350 2    50   ~ 0
+IBUS1
+Text Label 3650 1450 2    50   ~ 0
+IBUS2
+Text Label 3650 1550 2    50   ~ 0
+IBUS3
+Text Label 3650 1650 2    50   ~ 0
+IBUS4
+Text Label 3650 1750 2    50   ~ 0
+IBUS5
+Text Label 3650 1850 2    50   ~ 0
+IBUS6
+Text Label 3650 1950 2    50   ~ 0
+IBUS7
+Wire Wire Line
+	4650 1250 4850 1250
+Wire Wire Line
+	4650 1350 4850 1350
+Wire Wire Line
+	4650 1450 4850 1450
+Wire Wire Line
+	4650 1550 4850 1550
+Wire Wire Line
+	4650 1650 4850 1650
+Wire Wire Line
+	4650 1750 4850 1750
+Wire Wire Line
+	4650 1850 4850 1850
+Wire Wire Line
+	4650 1950 4850 1950
+Text Label 4650 1250 0    50   ~ 0
+AR0
+Text Label 4650 1350 0    50   ~ 0
+AR1
+Text Label 4650 1450 0    50   ~ 0
+AR2
+Text Label 4650 1550 0    50   ~ 0
+AR3
+Text Label 4650 1650 0    50   ~ 0
+AR4
+Text Label 4650 1750 0    50   ~ 0
+AR5
+Text Label 4650 1850 0    50   ~ 0
+AR6
+Text Label 4650 1950 0    50   ~ 0
+AR7
+Wire Wire Line
+	5050 1250 5250 1250
+Wire Wire Line
+	5050 1350 5250 1350
+Wire Wire Line
+	5050 1450 5250 1450
+Wire Wire Line
+	5050 1550 5250 1550
+Wire Wire Line
+	5050 1650 5250 1650
+Wire Wire Line
+	5050 1750 5250 1750
+Wire Wire Line
+	5050 1850 5250 1850
+Wire Wire Line
+	5050 1950 5250 1950
+Text Label 5250 1250 2    50   ~ 0
+AR0
+Text Label 5250 1350 2    50   ~ 0
+AR1
+Text Label 5250 1450 2    50   ~ 0
+AR2
+Text Label 5250 1550 2    50   ~ 0
+AR3
+Text Label 5250 1650 2    50   ~ 0
+AR4
+Text Label 5250 1750 2    50   ~ 0
+AR5
+Text Label 5250 1850 2    50   ~ 0
+AR6
+Text Label 5250 1950 2    50   ~ 0
+AR7
+Wire Wire Line
+	6250 1250 6500 1250
+Wire Wire Line
+	6250 1350 6500 1350
+Wire Wire Line
+	6250 1450 6500 1450
+Wire Wire Line
+	6250 1550 6500 1550
+Wire Wire Line
+	6250 1650 6500 1650
+Wire Wire Line
+	6250 1750 6500 1750
+Wire Wire Line
+	6250 1850 6500 1850
+Wire Wire Line
+	6250 1950 6500 1950
+Text Label 6250 1250 0    50   ~ 0
+AB0
+Text Label 6250 1350 0    50   ~ 0
+AB1
+Text Label 6250 1450 0    50   ~ 0
+AB2
+Text Label 6250 1550 0    50   ~ 0
+AB3
+Text Label 6250 1650 0    50   ~ 0
+AB4
+Text Label 6250 1750 0    50   ~ 0
+AB5
+Text Label 6250 1850 0    50   ~ 0
+AB6
+Text Label 6250 1950 0    50   ~ 0
+AB7
 Wire Bus Line
 	6900 950  6900 1200
@@
 Wire Bus Line
 	4950 950  4950 5200
+Text Label 4650 5300 0    50   ~ 0
+AR23
+Text Label 4650 5200 0    50   ~ 0
+AR22
+Text Label 4650 5100 0    50   ~ 0
+AR21
+Text Label 4650 5000 0    50   ~ 0
+AR20
+Text Label 4650 4900 0    50   ~ 0
+AR19
+Text Label 4650 4800 0    50   ~ 0
+AR18
+Text Label 4650 4700 0    50   ~ 0
+AR17
+Text Label 4650 4600 0    50   ~ 0
+AR16
+Wire Wire Line
+	4650 5300 4850 5300
+Wire Wire Line
+	4650 5200 4850 5200
+Wire Wire Line
+	4650 5100 4850 5100
+Wire Wire Line
+	4650 5000 4850 5000
+Wire Wire Line
+	4650 4900 4850 4900
+Wire Wire Line
+	4650 4800 4850 4800
+Wire Wire Line
+	4650 4700 4850 4700
+Wire Wire Line
+	4650 4600 4850 4600
 $EndSCHEMATC

Commit message: Work on schematic and route board 0
Parts:
- removed C404, C405: 100nF, alexios:C_SMD_0805_2012Metric_Pad1.15x1.40mm_HandSolder, symbol Device:C_Small
- removed JP401, JP402: Jumper_3_Bridged12, Jumper:SolderJumper-3_P1.3mm_Bridged12_RoundedPad1.0x1.5mm, symbol alexios:Jumper_3_Bridged12
- removed U404: 74LVC1G08, alexios:SOT-23-5_HandSoldering, symbol alexios:74AHC1G08
- removed U405: 74LVC1G32, alexios:SOT-23-5_HandSoldering, symbol alexios:74LVC1G32
Connections:
- net ~ABEN2 is gone; now on net GND: U403.19 (~G2), U407.19 (~G2), U409.19 (~G2)
- net ~ABEN1 renamed ~ABEN
Other:
- note removed: "Optional"

Commit message: Cleaning up board
Parts:
- added R410: 4.7kΩ, alexios:R_SMD_0805_2012Metric_Pad1.15x1.40mm_HandSolder, symbol Device:R_Small
Connections:
- net +5V: now also R410.1
- net ~FPAEXT: now also R410.2
Changed lines of the file:
@@
 	1    0    0    -1
 $EndComp
-Text HLabel 7650 5550 0    50   Input ~ 0
+Text HLabel 7350 5550 0    50   Input ~ 0
 ~FPAEXT
 Text HLabel 10150 5600 2    50   3State ~ 0
 FPD[0..7]
 Wire Wire Line
-	7650 5550 8100 5550
+	7350 5550 7600 5550
 Text Label 7800 5550 0    50   ~ 0
 ~FPAEXT
@@
 Text HLabel 7450 1800 0    50   Input ~ 0
 ~IO
+$Comp
+L Device:R_Small R?
+U 1 1 60AF5E1B
+P 7600 5400
+AR Path="/61F95ACC/60AF5E1B" Ref="R?"  Part="1"
+AR Path="/5F63066B/60AF5E1B" Ref="R?"  Part="1"
+AR Path="/5D69F3FD/60AF5E1B" Ref="R?"  Part="1"
+AR Path="/5CC06F10/60AF5E1B" Ref="R410"  Part="1"
+F 0 "R410" H 7658 5446 50  0000 L CNN
+F 1 "4.7kΩ" H 7658 5355 50  0000 L CNN
+F 2 "alexios:R_SMD_0805_2012Metric_Pad1.15x1.40mm_HandSolder" H 7600 5400 50  0001 C CNN
+F 3 "~" H 7600 5400 50  0001 C CNN
+	1    7600 5400
+	-1   0    0    -1
+$EndComp
+$Comp
+L power:+5V #PWR?
+U 1 1 60AF5E21
+P 7600 5300
+AR Path="/61F95ACC/60AF5E21" Ref="#PWR?"  Part="1"
+AR Path="/5F63066B/60AF5E21" Ref="#PWR?"  Part="1"
+AR Path="/5D69F3FD/60AF5E21" Ref="#PWR?"  Part="1"
+F 0 "#PWR?" H 7600 5150 50  0001 C CNN
+F 1 "+5V" H 7615 5473 50  0000 C CNN
+F 2 "" H 7600 5300 50  0001 C CNN
+F 3 "" H 7600 5300 50  0001 C CNN
+	1    7600 5300
+	1    0    0    -1
+$EndComp
+Wire Wire Line
+	7600 5500 7600 5550
 Wire Bus Line
 	6900 950  6900 1200
@@
 Wire Bus Line
 	4950 950  4950 5200
+Connection ~ 7600 5550
+Wire Wire Line
+	7600 5550 8100 5550
 $EndSCHEMATC
