File: kicad/cft/cft-board0/flag_unit.sch (KiCad schematic (older format))
At the start: 10 parts, among them U1201 74HC541, U1202 74HC138, U1203 74LVC1G0832, U1204 74HC138, U1205 74HC541

Commit message: Route Board 0
Parts:
- removed C1203, C1204, C1205: 100nF, alexios:C_SMD_0805_2012Metric_Pad1.15x1.40mm_HandSolder, symbol Device:C_Small
- removed U1202, U1204: 74HC138, alexios:DIP-16_W7.62mm_Socket, symbol alexios:74HC138
- removed U1203: 74LVC1G0832, alexios:SOT-23-6_Handsoldering, symbol alexios:74LVC1G0832
Connections:
- net ~FLAGOE renamed ~READ_FLAGS
- no-connect marks 11 -> 0
Other:
- note removed: "RADDR or WADDR = 01101 → Read/Write MBP & Flags\nRADDR or WADDR = 01110 → Read/Write Flags"
- note removed: "RADDR=01xxx"
- note removed: "WADDR=011xx"

Commit message: Place and route more of Board 0
Parts:
- renumbered U1205 to U1202
Connections:
- net ~READ_FLAGS renamed ~READ-FL
Changed lines of the file:
@@
 	7600 1750 7050 1750
 Text Label 7250 2350 0    50   ~ 0
-~FLAGOE
+~READ-FL
 Text Label 9700 6250 2    50   ~ 0
 FPD[0..7]
@@
 AR Path="/5D676F64" Ref="U?"  Part="1"
 AR Path="/5D65F6EF/5D676F64" Ref="U?"  Part="1"
-AR Path="/5D69F3FD/5D676F64" Ref="U1205"  Part="1"
-F 0 "U1205" H 8100 6067 50  0000 C CNN
+AR Path="/5D69F3FD/5D676F64" Ref="U1202"  Part="1"
+F 0 "U1202" H 8100 6067 50  0000 C CNN
 F 1 "74HC541" H 8100 5976 50  0000 C CNN
 F 2 "alexios:DIP-20_W7.62mm_Socket" H 8100 5300 50  0001 C CNN
@@
 AR Path="/5F4B0011/5DDC83B3" Ref="U?"  Part="2"
 AR Path="/5F63066B/5DDC83B3" Ref="U?"  Part="2"
-AR Path="/5D69F3FD/5DDC83B3" Ref="U1205"  Part="2"
-F 0 "U1205" H 10080 5296 50  0000 L CNN
+AR Path="/5D69F3FD/5DDC83B3" Ref="U1202"  Part="2"
+F 0 "U1202" H 10080 5296 50  0000 L CNN
 F 1 "74HC541" H 10080 5205 50  0000 L CNN
 F 2 "alexios:DIP-20_W7.62mm_Socket" H 9900 5250 50  0001 C CNN
@@
 These traces are named, but connected to ground directly.\nThe traces on the board are long so they can be cut and the\nsignals repurposed (e.g. tied to Vcc).
 Text Label 2000 2350 0    50   ~ 0
-~FLAGOE
+~READ-FL
 Text HLabel 1950 2350 0    50   Input ~ 0
-~READ_FLAGS
+~READ-FL
 Wire Wire Line
 	1950 2350 7600 2350

Commit message: Cleaning up board
Parts:
- added R1201: 4.7kΩ, alexios:R_SMD_0805_2012Metric_Pad1.15x1.40mm_HandSolder, symbol Device:R_Small
- added RN1201: 10kΩ, Resistor_THT:R_Array_SIP5, symbol Device:R_Network04
Connections:
- net +5V: now also R1201.1
- net FL: now also RN1201.3 (R2)
- net FN: now also RN1201.5 (R4)
- net FV: now also RN1201.2 (R1)
- net FZ: now also RN1201.4 (R3)
- net GND: now also RN1201.1 (common)
- net ~FPFLAGS: now also R1201.2
Changed lines of the file:
@@
 ~FPFLAGS
 Wire Wire Line
-	7600 5700 1900 5700
+	7600 5700 2500 5700
 $Comp
 L power:GND #PWR?
@@
 Wire Wire Line
 	6750 5500 1900 5500
-Wire Wire Line
-	6850 5300 1900 5300
-Wire Wire Line
-	6950 5200 1900 5200
-Wire Wire Line
-	7050 5100 1900 5100
-Wire Wire Line
-	7150 5000 1900 5000
 Text HLabel 1900 5500 0    50   Input ~ 0
 FI
@@
 Wire Wire Line
 	1950 2350 7600 2350
+$Comp
+L Device:R_Small R?
+U 1 1 609A7128
+P 2500 4750
+AR Path="/61F95ACC/609A7128" Ref="R?"  Part="1"
+AR Path="/5F63066B/609A7128" Ref="R?"  Part="1"
+AR Path="/5D69F3FD/609A7128" Ref="R1201"  Part="1"
+F 0 "R1201" H 2559 4796 50  0000 L CNN
+F 1 "4.7kΩ" H 2559 4705 50  0000 L CNN
+F 2 "alexios:R_SMD_0805_2012Metric_Pad1.15x1.40mm_HandSolder" H 2500 4750 50  0001 C CNN
+F 3 "~" H 2500 4750 50  0001 C CNN
+	1    2500 4750
+	-1   0    0    -1
+$EndComp
+$Comp
+L power:+5V #PWR?
+U 1 1 609A712E
+P 2500 4650
+AR Path="/61F95ACC/609A712E" Ref="#PWR?"  Part="1"
+AR Path="/5F63066B/609A712E" Ref="#PWR?"  Part="1"
+AR Path="/5D69F3FD/609A712E" Ref="#PWR0123"  Part="1"
+F 0 "#PWR0123" H 2500 4500 50  0001 C CNN
+F 1 "+5V" H 2515 4823 50  0000 C CNN
+F 2 "" H 2500 4650 50  0001 C CNN
+F 3 "" H 2500 4650 50  0001 C CNN
+	1    2500 4650
+	1    0    0    -1
+$EndComp
+Wire Wire Line
+	2500 4850 2500 5700
+Connection ~ 2500 5700
+Wire Wire Line
+	2500 5700 1900 5700
+$Comp
+L power:GND #PWR?
+U 1 1 609C9CF9
+P 3250 6200
+AR Path="/61F95ACC/609C9CF9" Ref="#PWR?"  Part="1"
+AR Path="/61F95ACC/6888FBA2/609C9CF9" Ref="#PWR?"  Part="1"
+AR Path="/5D69F3FD/609C9CF9" Ref="#PWR0124"  Part="1"
+F 0 "#PWR0124" H 3250 5950 50  0001 C CNN
+F 1 "GND" H 3255 6027 50  0000 C CNN
+F 2 "" H 3250 6200 50  0001 C CNN
+F 3 "" H 3250 6200 50  0001 C CNN
+	1    3250 6200
+	-1   0    0    -1
+$EndComp
+Wire Wire Line
+	1900 5100 3050 5100
+Wire Wire Line
+	1900 5000 2950 5000
+Wire Wire Line
+	1900 5200 3150 5200
+Wire Wire Line
+	1900 5300 3250 5300
+Wire Wire Line
+	2950 5800 2950 5000
+Connection ~ 2950 5000
+Wire Wire Line
+	2950 5000 7150 5000
+Wire Wire Line
+	3050 5800 3050 5100
+Connection ~ 3050 5100
+Wire Wire Line
+	3050 5100 7050 5100
+Wire Wire Line
+	3150 5800 3150 5200
+Connection ~ 3150 5200
+Wire Wire Line
+	3150 5200 6950 5200
+Wire Wire Line
+	3250 5800 3250 5300
+Connection ~ 3250 5300
+Wire Wire Line
+	3250 5300 6850 5300
+$Comp
+L Device:R_Network04 RN?
+U 1 1 609C9CFF
+P 3050 6000
+AR Path="/61F95ACC/6888FBA2/609C9CFF" Ref="RN?"  Part="1"
+AR Path="/61F95ACC/609C9CFF" Ref="RN?"  Part="1"
+AR Path="/5D69F3FD/609C9CFF" Ref="RN1201"  Part="1"
+F 0 "RN1201" H 2770 5954 50  0000 R CNN
+F 1 "10kΩ" H 2770 6045 50  0000 R CNN
+F 2 "Resistor_THT:R_Array_SIP5" V 3525 6000 50  0001 C CNN
+F 3 "http://www.vishay.com/docs/31509/csc.pdf" H 3050 6000 50  0001 C CNN
+	1    3050 6000
+	-1   0    0    1
+$EndComp
 Wire Bus Line
 	9050 4900 9050 6150

Commit message: ERC/DRC board 0, route, fine-tune
Changed lines of the file:
@@
 $Descr A4 11693 8268
 encoding utf-8
-Sheet 9 17
+Sheet 17 17
 Title "Flag Unit"
 Date ""
@@
 Text Label 7250 5700 0    50   ~ 0
 ~FPFLAGS
-Wire Wire Line
-	7600 5700 2500 5700
 $Comp
 L power:GND #PWR?
@@
 	1    0    0    -1
 $EndComp
-Wire Wire Line
-	2500 4850 2500 5700
-Connection ~ 2500 5700
-Wire Wire Line
-	2500 5700 1900 5700
 $Comp
 L power:GND #PWR?
@@
 	-1   0    0    1
 $EndComp
+Wire Wire Line
+	1900 5700 2500 5700
+Wire Wire Line
+	2500 4850 2500 5700
 Wire Bus Line
 	9050 4900 9050 6150
 Wire Bus Line
 	9050 1550 9050 2850
+Connection ~ 2500 5700
+Wire Wire Line
+	2500 5700 7600 5700
 $EndSCHEMATC
