File: kicad/cft/cft-board0/cpu_cs.sch (KiCad schematic (older format))
At the start: 7 parts, among them U501 74AC541, U502 74HC138, U503 74AC541

Commit message: Route Board 0
Parts:
- removed C501: 100nF, alexios:C_SMD_0805_2012Metric_Pad1.15x1.40mm_HandSolder, symbol Device:C_Small
- removed JP501: SolderJumper_2_Bridged, Jumper:SolderJumper-2_P1.3mm_Bridged_RoundedPad1.0x1.5mm, symbol Jumper:SolderJumper_2_Bridged
- removed U502: 74HC138, alexios:DIP-16_W7.62mm_Socket, symbol alexios:74HC138
Connections:
- net labels added: RADDR[0..1], ~READ_CS
- net labels removed: RADDR2, RADDR3, RADDR4, RADDR[0..4], T34, ~CSEN
- wire segments 60 -> 50
- no-connect marks 7 -> 0
Other:
- note removed: "For testing, T34 may be\nconnected to ~CSEN~, or JP1\ncan be bridged to ground."
- note removed: "RADDR=001xx"
- moved on the sheet: U501A, U503A

Commit message: Place and route more of Board 0
Parts:
- renumbered C502 to C501
Connections:
- net ~READ_CS renamed ~READ-CS
Changed lines of the file:
@@
 AR Path="/5E507DE3/5E51C0B5" Ref="C?"  Part="1"
 AR Path="/5DF0FEB9/5E51C0B5" Ref="C?"  Part="1"
-AR Path="/5E25A7FA/5E51C0B5" Ref="C502"  Part="1"
-F 0 "C502" H 2359 7396 50  0000 R CNN
+AR Path="/5E25A7FA/5E51C0B5" Ref="C501"  Part="1"
+F 0 "C501" H 2359 7396 50  0000 R CNN
 F 1 "100nF" H 2359 7305 50  0000 R CNN
 F 2 "alexios:C_SMD_0805_2012Metric_Pad1.15x1.40mm_HandSolder" H 2450 7350 50  0001 C CNN
@@
 	4000 2750 3400 2750
 Text Label 3500 3950 0    50   ~ 0
-~CSOE
+~READ-CS
 Text Notes 4050 4050 2    50   ~ 0
 RADDR=001XX
 Text Label 5450 3950 2    50   ~ 0
-~CSOE
+~READ-CS
 Wire Wire Line
 	5500 4050 5600 4050
 Text Label 5450 5500 2    50   ~ 0
-~CSOE
+~READ-CS
 Wire Wire Line
 	5500 5600 5600 5600
@@
 The Constant Store
 Text HLabel 3400 3950 0    50   Input ~ 0
-~READ_CS
+~READ-CS
 Connection ~ 5050 3950
 Wire Wire Line
