File: kicad/cft/cft-board1/bus_interface.sch (KiCad schematic (older format))
At the start: 11 parts, among them U2004 74HC139, U2005 74LVC1G11, U2006 74HC74, U2010 74HC139, U37 74HC138, U38 74HC138

Commit message: Route board 1
Parts:
- renumbered U2010 to U2004
Changed lines of the file:
@@
 $Descr A4 11693 8268
 encoding utf-8
-Sheet 20 20
+Sheet 19 20
 Title ""
 Date ""
@@
 ~R
 $Comp
-L alexios:74HC139 U2010
+L alexios:74HC139 U2004
 U 1 1 60AF2A38
 P 7200 1550
-F 0 "U2010" H 7200 1917 50  0000 C CNN
+F 0 "U2004" H 7200 1917 50  0000 C CNN
 F 1 "74HC139" H 7200 1826 50  0000 C CNN
 F 2 "alexios:SOIC-16" H 7200 1550 50  0001 C CNN
@@
 NoConn ~ 7700 2150
 $Comp
-L alexios:74HC139 U2010
+L alexios:74HC139 U2004
 U 2 1 60AF2A3E
 P 7200 2150
-F 0 "U2010" H 7850 2000 50  0000 L CNN
+F 0 "U2004" H 7850 2000 50  0000 L CNN
 F 1 "74HC139" H 7850 1900 50  0000 L CNN
 F 2 "alexios:SOIC-16" H 7200 2150 50  0001 C CNN

Commit message: Move to GAL for IRC decoding
Parts:
- removed unit 1 of U38
Changed lines of the file:
@@
 $Descr A4 11693 8268
 encoding utf-8
-Sheet 17 20
+Sheet 20 20
 Title ""
 Date ""
@@
 Wire Wire Line
 	4000 2750 4050 2750
-$Comp
-L alexios:74HC138 U?
-U 1 1 60AF2A23
-P 4550 2550
-AR Path="/5F3EA987/60AF2A23" Ref="U?"  Part="1"
-AR Path="/60AF2A23" Ref="U?"  Part="1"
-AR Path="/61F95ACC/60AF2A23" Ref="U?"  Part="1"
-AR Path="/5D65F6EF/60AF2A23" Ref="U?"  Part="1"
-AR Path="/5D69F3FD/60AF2A23" Ref="U?"  Part="1"
-AR Path="/5F67D4B5/60AF2A23" Ref="U?"  Part="1"
-AR Path="/60AA2B43/60AF2A23" Ref="U38"  Part="1"
-AR Path="/61C2F29F/60AF2A23" Ref="U2003"  Part="1"
-F 0 "U2003" H 4550 3217 50  0000 C CNN
-F 1 "74HC138" H 4550 3126 50  0000 C CNN
-F 2 "alexios:SOIC-16" H 4550 2550 50  0001 C CNN
-F 3 "http://www.ti.com/lit/gpn/sn74LS138" H 4550 2550 50  0001 C CNN
-	1    4550 2550
-	1    0    0    -1
-$EndComp
 Text Label 3750 2150 0    50   ~ 0
 AB2
