File: kicad/cft/cft-board1/clock_quadruppler.sch (KiCad schematic (older format))
At the start: 18 parts, among them U11 74HC04, U12 74AC86, U21 74LVC1G04, U46 ICS501

Commit message: Rearrange sheet numbers, prepare for layout
Parts:
- renumbered C17 to C301, C13 to C302, C48 to C303, C53 to C304, JP6 to JP301, JP7 to JP302, JP2 to JP303, R3 to R301, R5 to R302, R4 to R303, R7 to R304, TP5 to TP301, TP6 to TP302, TP7 to TP303, U11 to U301, U12 to U302, U21 to U303, U46 to U304, U11 to U305

Commit message: Renumber schematics, start of board layout
Parts:
- U701: renamed from U301; footprint alexios:SOIC-14 -> alexios:DIP-14_W7.62mm_Socket
- U702: renamed from U302; footprint alexios:SOIC-14 -> alexios:DIP-14_W7.62mm_Socket
- U705: renamed from U305; footprint alexios:SOIC-14 -> alexios:DIP-14_W7.62mm_Socket
- renumbered C301 to C701, C302 to C702, C303 to C703, C304 to C704, JP301 to JP701, JP302 to JP702, JP303 to JP703, R301 to R701, R302 to R702, R303 to R703, R304 to R704, TP301 to TP701, TP302 to TP702, TP303 to TP703, U303 to U703, U304 to U704

Commit message: Work on Board1 schematics and PCB
Parts:
- added C?: 100nF, alexios:C_SMD_0805_2012Metric_Pad1.15x1.40mm_HandSolder, symbol Device:C_Small
- added U?: 74AC74, symbol alexios:74AC74
- added X?: CXO_DIP8, Oscillator:Oscillator_DIP-8, symbol alexios:CXO_DIP8
Connections:
- net +5V: now also C?.1, X?.8 (Vcc)
- net GND: now also C?.2, X?.2 (GND), X?.3 (GND), X?.4 (GND), X?.6 (GND), X?.7 (GND)
- new net: U?.2 (D), U?.6 (~Q)
Changed lines of the file:
@@
 Wire Notes Line
 	8000 5700 8000 2450
+$Comp
+L alexios:CXO_DIP8 X?
+U 1 1 60A9A739
+P 8800 5500
+F 0 "X?" H 8900 5867 50  0000 C CNN
+F 1 "CXO_DIP8" H 8900 5776 50  0000 C CNN
+F 2 "Oscillator:Oscillator_DIP-8" H 8950 5100 50  0001 C CNN
+F 3 "http://cdn-reichelt.de/documents/datenblatt/B400/OSZI.pdf" H 8900 5450 50  0001 C CNN
+	1    8800 5500
+	1    0    0    -1
+$EndComp
+$Comp
+L alexios:74AC74 U?
+U 1 1 60A9D4D3
+P 10400 5500
+F 0 "U?" H 10400 5917 50  0000 C CNN
+F 1 "74AC74" H 10400 5826 50  0000 C CNN
+F 2 "" H 10350 5650 50  0001 C CNN
+F 3 "74xx/74hc_hct74.pdf" H 10350 5650 50  0001 C CNN
+	1    10400 5500
+	1    0    0    -1
+$EndComp
+Wire Wire Line
+	9950 5450 9850 5450
+Wire Wire Line
+	9850 5450 9850 5000
+Wire Wire Line
+	9850 5000 11000 5000
+Wire Wire Line
+	11000 5000 11000 5650
+Wire Wire Line
+	11000 5650 10850 5650
+$Comp
+L power:+5V #PWR?
+U 1 1 60AB727D
+P 8450 5300
+F 0 "#PWR?" H 8450 5150 50  0001 C CNN
+F 1 "+5V" H 8465 5473 50  0000 C CNN
+F 2 "" H 8450 5300 50  0001 C CNN
+F 3 "" H 8450 5300 50  0001 C CNN
+	1    8450 5300
+	1    0    0    -1
+$EndComp
+Wire Wire Line
+	8450 5300 8450 5400
+Wire Wire Line
+	8450 5400 8500 5400
+$Comp
+L power:GND #PWR?
+U 1 1 60AC2902
+P 8450 5750
+F 0 "#PWR?" H 8450 5500 50  0001 C CNN
+F 1 "GND" H 8455 5577 50  0000 C CNN
+F 2 "" H 8450 5750 50  0001 C CNN
+F 3 "" H 8450 5750 50  0001 C CNN
+	1    8450 5750
+	1    0    0    -1
+$EndComp
+Wire Wire Line
+	8500 5700 8450 5700
+Wire Wire Line
+	8450 5700 8450 5750
+$Comp
+L Device:C_Small C?
+U 1 1 60ACF0CA
+P 8450 5550
+AR Path="/5CC0D65F/60ACF0CA" Ref="C?"  Part="1"
+AR Path="/60ACF0CA" Ref="C?"  Part="1"
+AR Path="/5EF76914/60ACF0CA" Ref="C?"  Part="1"
+AR Path="/6A313729/60ACF0CA" Ref="C?"  Part="1"
+AR Path="/5DC89E19/5D0A147D/60ACF0CA" Ref="C?"  Part="1"
+AR Path="/5DC89E19/5D396E91/60ACF0CA" Ref="C?"  Part="1"
+AR Path="/5DF75CDE/60ACF0CA" Ref="C?"  Part="1"
+AR Path="/5DF75CDE/5EF12B5A/60ACF0CA" Ref="C?"  Part="1"
+F 0 "C?" H 8359 5596 50  0000 R CNN
+F 1 "100nF" H 8359 5505 50  0000 R CNN
+F 2 "alexios:C_SMD_0805_2012Metric_Pad1.15x1.40mm_HandSolder" H 8450 5550 50  0001 C CNN
+F 3 "~" H 8450 5550 50  0001 C CNN
+	1    8450 5550
+	1    0    0    -1
+$EndComp
+Wire Wire Line
+	8450 5400 8450 5450
+Connection ~ 8450 5400
+Wire Wire Line
+	8450 5650 8450 5700
+Connection ~ 8450 5700
 $EndSCHEMATC

Commit message: Work on board1
Parts:
- removed U?: 74AC74, symbol alexios:74AC74
- X701: renamed from X?; footprint Oscillator:Oscillator_DIP-8 -> alexios:Oscillator_DIP-8-socket
- gave numbers to parts that had none: 1
Changed lines of the file:
@@
 	8000 5700 8000 2450
 $Comp
-L alexios:CXO_DIP8 X?
+L alexios:CXO_DIP8 X701
 U 1 1 60A9A739
 P 8800 5500
-F 0 "X?" H 8900 5867 50  0000 C CNN
+F 0 "X701" H 8900 5867 50  0000 C CNN
 F 1 "CXO_DIP8" H 8900 5776 50  0000 C CNN
-F 2 "Oscillator:Oscillator_DIP-8" H 8950 5100 50  0001 C CNN
+F 2 "alexios:Oscillator_DIP-8-socket" H 8950 5100 50  0001 C CNN
 F 3 "http://cdn-reichelt.de/documents/datenblatt/B400/OSZI.pdf" H 8900 5450 50  0001 C CNN
 	1    8800 5500
-	1    0    0    -1
-$EndComp
-$Comp
-L alexios:74AC74 U?
-U 1 1 60A9D4D3
-P 10400 5500
-F 0 "U?" H 10400 5917 50  0000 C CNN
-F 1 "74AC74" H 10400 5826 50  0000 C CNN
-F 2 "" H 10350 5650 50  0001 C CNN
-F 3 "74xx/74hc_hct74.pdf" H 10350 5650 50  0001 C CNN
-	1    10400 5500
 	1    0    0    -1
 $EndComp
@@
 	11000 5650 10850 5650
 $Comp
-L power:+5V #PWR?
+L power:+5V #PWR0150
 U 1 1 60AB727D
 P 8450 5300
-F 0 "#PWR?" H 8450 5150 50  0001 C CNN
+F 0 "#PWR0150" H 8450 5150 50  0001 C CNN
 F 1 "+5V" H 8465 5473 50  0000 C CNN
 F 2 "" H 8450 5300 50  0001 C CNN
@@
 	8450 5400 8500 5400
 $Comp
-L power:GND #PWR?
+L power:GND #PWR0151
 U 1 1 60AC2902
 P 8450 5750
-F 0 "#PWR?" H 8450 5500 50  0001 C CNN
+F 0 "#PWR0151" H 8450 5500 50  0001 C CNN
 F 1 "GND" H 8455 5577 50  0000 C CNN
 F 2 "" H 8450 5750 50  0001 C CNN
@@
 AR Path="/5DC89E19/5D396E91/60ACF0CA" Ref="C?"  Part="1"
 AR Path="/5DF75CDE/60ACF0CA" Ref="C?"  Part="1"
-AR Path="/5DF75CDE/5EF12B5A/60ACF0CA" Ref="C?"  Part="1"
-F 0 "C?" H 8359 5596 50  0000 R CNN
+AR Path="/5DF75CDE/5EF12B5A/60ACF0CA" Ref="C705"  Part="1"
+F 0 "C705" H 8359 5596 50  0000 R CNN
 F 1 "100nF" H 8359 5505 50  0000 R CNN
 F 2 "alexios:C_SMD_0805_2012Metric_Pad1.15x1.40mm_HandSolder" H 8450 5550 50  0001 C CNN

Commit message: Add SRU GAL, layout and route Board 1
Parts:
- removed JP701, JP702: SolderJumper_2_Bridged, alexios:SolderJumper-2_P1.3mm_Bridged_RoundedPad1.0x1.5mm, symbol Jumper:SolderJumper_2_Bridged
- removed TP701, TP702, TP703: TestPoint, TestPoint:TestPoint_Pad_1.0x1.0mm, symbol Connector:TestPoint
- removed U703: 74LVC1G04, alexios:SOT-23-5_HandSoldering, symbol alexios:74LVC1G04
- removed U704: ICS501, alexios:SOIC-8, symbol alexios:ICS501
- added JP701, JP702: SolderJumper_2_Open, alexios:SolderJumper-2_P1.3mm_Open_RoundedPad1.0x1.5mm, symbol Jumper:SolderJumper_2_Open
- added R705: 100Ω, alexios:R_SMD_0805_2012Metric_Pad1.15x1.40mm_HandSolder, symbol Device:R_Small
- added R706: 30Ω, alexios:R_SMD_0805_2012Metric_Pad1.15x1.40mm_HandSolder, symbol Device:R_Small
- added R707: 0Ω, alexios:R_SMD_0805_2012Metric_Pad1.15x1.40mm_HandSolder, symbol Device:R_Small
- added U703: 74AC14, alexios:DIP-14_W7.62mm_Socket, symbol alexios:74AC14
- C704: value 100nF -> 120pF
- JP703: footprint Jumper:SolderJumper-2_P1.3mm_Open_RoundedPad1.0x1.5mm -> alexios:SolderJumper-2_P1.3mm_Open_RoundedPad1.0x1.5mm
- renumbered U705 to U701
Connections:
- net labels added: 16MHz
- wire segments 63 -> 60
- no-connect marks 4 -> 6
Other:
- note added: "0Ω, 30Ω or 100Ω as required\nfor signal integrity."
- note added: "Termination is optional."
- note removed: "16 MHZ PLL-synced"
- note removed: "An ICS501 cheap PLL-based clock multiplier IC can be used\ninstead of the delay line/XOR tree. It has the advantage of\nbeing much more reliable at clock generation, with less\njitter and less calibration needed.\n\nU21 is an optional inverter. Testing shows this may be\nneeded to shift the clock output phase by 180° (plus\npropagation delay, of course). If not installed, pins\n2 and 4 need to be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"
- note removed: "Bridge JP2 to disable\nclock output."
- note removed: "Bridge JP6 if U21\nis not needed."
- note removed: "JP7 is bridged by\ndefault (×4 clock).\nBreak for ×2."
- note removed: "PLL Option"
- note removed: "U46"
- moved on the sheet: C701, C702, C705, X701
