File: kicad/cft/cft-board1/alu_decoder.sch (KiCad schematic (older format))
At the start: 12 parts, among them U39 74AC138, U40 74HC138, U41 74HC138, U42 74HC138, U48 74LVC1G04

Commit message: Rearrange sheet numbers, prepare for layout
Parts:
- renumbered C50 to C201, C41 to C202, C42 to C203, C43 to C204, C44 to C205, JP3 to JP201, JP4 to JP202, U39 to U201, U40 to U202, U48 to U203, U41 to U204, U42 to U205

Commit message: Renumber schematics, start of board layout
Parts:
- removed C204, C205: 100nF, alexios:C_SMD_0805_2012Metric_Pad1.15x1.40mm_HandSolder, symbol Device:C_Small
- removed JP201, JP202: Jumper_NC_Small, Jumper:SolderJumper-2_P1.3mm_Bridged_RoundedPad1.0x1.5mm, symbol Device:Jumper_NC_Small
- removed U201: 74AC138, alexios:SOIC-16, symbol alexios:74HC138
- removed U202, U204, U205: 74HC138, alexios:SOIC-16, symbol alexios:74HC138
- removed U203: 74LVC1G04, alexios:SOT-23-5_HandSoldering, symbol alexios:74LVC1G04
- added U201, U202, U203: ATF16V8B, alexios:DIP-20_W7.62mm_Socket, symbol alexios:ATF16V8B
Connections:
- net +5V: now also U201.20 (VCC), U202.20 (VCC), U203.20 (VCC)
- net ACP: now also U201.13 (IO7)
- net ACTION0: now also U203.2 (I1)
- net ACTION1: now also U203.3 (I2)
- net ACTION2: now also U203.4 (I3)
- net ACTION3: now also U203.5 (I4)
- net CLK4: now also U202.1 (I/CLK), U203.1 (I/CLK)
- net GND: now also U201.10 (GND), U202.10 (GND), U203.10 (GND)
- net RADDR0: now also U201.2 (I1)
- net RADDR1: now also U201.3 (I2)
- net RADDR2: now also U201.4 (I3)
- net RADDR3: now also U201.5 (I4)
- net RADDR4: now also U201.6 (I5)
- net T34: now also U201.1 (I/CLK)
- net WADDR0: now also U202.2 (I1)
- net WADDR1: now also U202.3 (I2)
- net WADDR2: now also U202.4 (I3)
- net WADDR3: now also U202.5 (I4)
- net WADDR4: now also U202.6 (I5)
- net ~ACTION-CLL: now also U203.13 (IO7)
- net ~ACTION-CPL: now also U203.12 (IO8)
- net ~ACTION-SRU: now also U203.14 (IO6)
- net ~ALU-OP: now also U201.12 (IO8)
- net ~READ-ALU-B: now also U201.15 (IO5)
- net ~READ-ALU-Y: now also U201.14 (IO6)
- net ~WRITE-ALU-B: now also U202.12 (IO8)
- new net ~DECAC: U203.16 (IO4)
- new net ~DECSP: U203.18 (IO2)
- new net ~INCAC: U203.15 (IO5)
- new net ~INCSP: U203.17 (I03)
- new net ~READ-AC: U201.16 (IO4)
- new net ~READ-SP: U201.17 (I03)
- new net ~WRITE-AC: U202.13 (IO7)
- new net ~WRITE-SP: U202.14 (IO6)
- no-connect marks 24 -> 21
Other:
- note removed: "0000"
- note removed: "0001"
- note removed: "0010"
- note removed: "0011"
- note removed: "0100"
- note removed: "0101"
- note removed: "0110"
- note removed: "0111"
- note removed: "1X0XX\nX1X00\n----\n11000"
- note removed: "ACTION=0xxx"
- note removed: "Base\n~Y4~\n\nFinal"
- note removed: "NOTE: Use 74AC!"
- note removed: "RADDR = 10xxx\n(8 addresses)"
- note removed: "RADDR=10xxx"
- note removed: "RADDR=1x0xx"
- note removed: "WADDR=1x0xx"

Commit message: Work on Board1 schematics and PCB
Connections:
- net ~ALUOE: now reaches U201.18 (IO2)
- no-connect marks 21 -> 20
Changed lines of the file:
@@
 ~READ-SP
 NoConn ~ 4850 1200
-NoConn ~ 4850 1300
 Text Label 3650 1300 0    50   ~ 0
 RADDR0
@@
 Text HLabel 5500 4200 2    50   Output ~ 0
 ~WRITE-ALU-B
+Wire Wire Line
+	4850 1300 5500 1300
+Text Label 5400 1300 2    50   ~ 0
+~ALUOE
+Text HLabel 5500 1300 2    50   Output ~ 0
+~ALUOE
 $EndSCHEMATC

Commit message: Add SRU GAL, layout and route Board 1
Connections:
- net ~WRITE-AC: now also U202.18 (IO2); no longer U202.13 (IO7)
- net ~WRITE-ALU-B: now also U202.13 (IO7); no longer U202.12 (IO8)
- net ~WRITE-SP: now also U202.12 (IO8); no longer U202.14 (IO6)
Changed lines of the file:
@@
 NoConn ~ 3950 4400
 NoConn ~ 4850 3500
-NoConn ~ 4850 3600
 $Comp
 L alexios:ATF16V8B U201
@@
 Text Label 3650 1700 0    50   ~ 0
 RADDR4
+Text Label 5400 4100 2    50   ~ 0
+~WRITE-B
+Text Label 5400 3600 2    50   ~ 0
+~WRITE-AC
 Text Label 5400 4200 2    50   ~ 0
-~WRITE-B
-Text Label 5400 4100 2    50   ~ 0
-~WRITE-AC
-Text Label 5400 4000 2    50   ~ 0
 ~WRITE-SP
 NoConn ~ 4850 3700
 NoConn ~ 4850 3800
-$Comp
-L alexios:ATF16V8B U203
-U 1 1 63A656B3
-P 4400 6350
-F 0 "U203" H 4400 7100 50  0000 C CNN
-F 1 "ATF16V8B" H 4400 7000 50  0000 C CNN
-F 2 "alexios:DIP-20_W7.62mm_Socket" H 4400 6350 50  0001 C CNN
-F 3 "https://ww1.microchip.com/downloads/en/DeviceDoc/Atmel-0364-PLD-ATF16V8B-8BQ-8BQL-Datasheet.pdf" H 4400 6350 50  0001 C CNN
-F 4 "ALADEC00" V 4400 6350 50  0000 C CNB "Signature"
-F 5 "alu-action-decode.jed" H 4400 5700 50  0000 C CNN "Image Filename"
-	1    4400 6350
-	1    0    0    -1
-$EndComp
 $Comp
 L alexios:ATF16V8B U203
@@
 ACTION[0..3]
 Wire Wire Line
-	4850 4000 5500 4000
+	4850 4200 5500 4200
+Wire Wire Line
+	4850 3600 5500 3600
 Wire Wire Line
 	4850 4100 5500 4100
-Wire Wire Line
-	4850 4200 5500 4200
-Text HLabel 5500 4000 2    50   Output ~ 0
+Text HLabel 5500 4200 2    50   Output ~ 0
 ~WRITE-SP
+Text HLabel 5500 3600 2    50   Output ~ 0
+~WRITE-AC
 Text HLabel 5500 4100 2    50   Output ~ 0
-~WRITE-AC
-Text HLabel 5500 4200 2    50   Output ~ 0
 ~WRITE-ALU-B
 Wire Wire Line
@@
 $EndComp
 NoConn ~ 4850 3900
+NoConn ~ 4850 4000
+$Comp
+L alexios:ATF16V8B U203
+U 1 1 63A656B3
+P 4400 6350
+F 0 "U203" H 4400 7100 50  0000 C CNN
+F 1 "ATF16V8B" H 4400 7000 50  0000 C CNN
+F 2 "alexios:DIP-20_W7.62mm_Socket" H 4400 6350 50  0001 C CNN
+F 3 "https://ww1.microchip.com/downloads/en/DeviceDoc/Atmel-0364-PLD-ATF16V8B-8BQ-8BQL-Datasheet.pdf" H 4400 6350 50  0001 C CNN
+F 4 "ALADEC00" V 4400 6350 50  0000 C CNB "Signature"
+F 5 "alu-action-decode.jed" H 4400 5700 50  0000 C CNN "Image Filename"
+	1    4400 6350
+	1    0    0    -1
+$EndComp
 $EndSCHEMATC
