File: kicad/cft/cft-board1/alu_port_b.sch (KiCad schematic (older format))
At the start: 10 parts, among them U26 74HC574, U27 74HC541, U28 74HC574, U29 74HC541, U4 74LVC1G08

Commit message: Rearrange sheet numbers, prepare for layout
Parts:
- renumbered C27 to C501, C28 to C502, C33 to C503, C29 to C504, C30 to C505, U26 to U501, U27 to U502, U4 to U503, U28 to U504, U29 to U505

Commit message: Renumber schematics, start of board layout
Parts:
- U401: renamed from U501; footprint alexios:SOIC-20W -> alexios:DIP-20_W7.62mm_Socket
- U402: renamed from U502; footprint alexios:SOIC-20W -> alexios:DIP-20_W7.62mm_Socket
- U404: renamed from U504; footprint alexios:SOIC-20W -> alexios:DIP-20_W7.62mm_Socket
- U405: renamed from U505; footprint alexios:SOIC-20W -> alexios:DIP-20_W7.62mm_Socket
- renumbered C501 to C401, C502 to C402, C503 to C403, C504 to C404, C505 to C405, U503 to U403

Commit message: Route Board 1
Parts:
- removed C403: 100nF, alexios:C_SMD_0805_2012Metric_Pad1.15x1.40mm_HandSolder, symbol Device:C_Small
- removed U403: 74LVC1G08, alexios:SOT-23-5_HandSoldering, symbol alexios:74LVC1G08
Connections:
- net CP is gone; now on net BCP: U401.11 (CP), U404.11 (CP)
Other:
- note added: "The SRU GAL asserts BCP when:\n\n1. The CU asserts ~WRITE-ALU-B~\n2. When the SRU needs to write temporary values\n to the B port."
- moved on the sheet: C401, C402, C404, C405, U401B, U402B, U404B, U405B
