File: kicad/cft/cft-dfp-pod/cft-dfp-pod.kicad_pcb (KiCad board)
At the start: 2 copper layers, 280 x 164.6 mm, 196 parts, among them J101 AVR-ISP-6, J102 Conn_01x06, P1 CFT-2019-Bus, P2 CFT-2019-Bus, SW1 SW_DIP_x08, U1001 74HC574, U1002 74HC574, U1003 74HC574, U101 ATmega64-16AU, U102 74LVC1G04, U103 74HC139, U104 74LVC1G07, U105 74LVC1G07, U106 74LVC1G07, U107 74AC573, U108 74HC590, U109 74LVC1G04, U110 74HC540, U1101 SN74ACT1073, U1102 SN74ACT1071, U1103 SN74ACT1071, U1104 SN74ACT1071, U1105 SN74ACT1071, U1106 SN74ACT1071, U1107 SN74ACT1071, U1108 SN74ACT1073, U1109 SN74ACT1071, U111 74HC138, U112 74HC138, U113 74HC138, U115 74LVC1G07, U1201 74HC138, U1202 74HC138, U1203 74HC138, U1204 74HC138, U1205 74HC138, U1206 74HC138, U1301 74LVC1G17, U1302 74LVC1G17, U401 74HC74, U402 74HC74, U403 74LVC1G11, U404 74HC253, U501 74HC138, U502 74HC112, U503 74HC251, U504 74LVC1G07, U601 74HC574, U602 74HC574, U603 74HC574, U604 74HC574, U605 74HC574, U606 74HC574, U701 74HC574, U702 74HC574, U703 74HC574, U704 74HC574, U801 74HC574, U802 74HC574, U803 74HC574, U804 74HC574, U901 74HC574, U902 74HC574, U903 74HC541, X101 CXO, X102 33 MHz?

Commit message: Route first version of DFP pod module
Parts:
- removed C1001, C1002, C1003, C104, C105, C107, C108, C109, C110, C1101, C1102, C1103, C1104, C1105, C1106, C1107, C1108, C1109, C111, C112, C113, C114, C115, C116, C118, C119, C120, C1201, C1202, C1203, C1204, C1205, C1206, C121, C122, C123, C1301, C1302, C1303, C1304, C401, C402, C403, C404, C501, C502, C503, C504, C601, C602, C603, C604, C605, C606, C701, C702, C703, C704, C801, C802, C803, C804, C901, C902, C903: 100nF, alexios:SMD_0805_2012Metric_Pad1.15x1.40mm_HandSolder
- removed C101, C102, C103, C106, C117: 1µF, alexios:SMD_0805_2012Metric_Pad1.15x1.40mm_HandSolder
- removed C124, C125, C126, C127, C128, C129, C201, C202, C301, C302: 47µF, Capacitor_THT:CP_Radial_D6.3mm_P2.50mm
- removed D1301, D1302: D_ALT, Diode_SMD:D_0805_2012Metric_Pad1.15x1.40mm_HandSolder
- removed D1303, D1304: LED_ALT, alexios:LED_0805_2012Metric_Pad1.15x1.40mm_HandSolder
- removed G*** (x2): LOGO, alexios:CFT
- removed J101: AVR-ISP-6, Connector_IDC:IDC-Header_2x03_P2.54mm_Horizontal
- removed J102: Conn_01x06, Connector_PinHeader_2.54mm:PinHeader_1x06_P2.54mm_Horizontal
- removed JP101: Conn_02x03_Odd_Even, Connector_PinHeader_2.54mm:PinHeader_2x03_P2.54mm_Vertical
- removed P1: CFT-2019-Bus, alexios:CFT-2019-Card-Edge-Double-Width
- removed P2: CFT-2019-Bus, alexios:CFT-2019-Card-Edge-P2-Connector
- removed R101, R102, R103: 4.7kΩ, alexios:SMD_0805_2012Metric_Pad1.15x1.40mm_HandSolder
- removed R104, R105, R106, R107, R108, R401, R402, R501: 30Ω, alexios:SMD_0805_2012Metric_Pad1.15x1.40mm_HandSolder
- removed R1301, R1302: 220kΩ, alexios:SMD_0805_2012Metric_Pad1.15x1.40mm_HandSolder
- removed R1303, R1304: 1.2kΩ, alexios:SMD_0805_2012Metric_Pad1.15x1.40mm_HandSolder
- removed REF** (x2): vero-card-handle-type-C, alexios:vero-card-handle-type-C
- removed REF** (x2): OSHW-Logo_19x20mm_SilkScreen, Symbol:OSHW-Logo_19x20mm_SilkScreen
- removed REF**: ESD-Logo_13.2x12mm_SilkScreen, Symbol:ESD-Logo_13.2x12mm_SilkScreen
- removed REF** (x2): QRCODE-CFT, alexios:QRCODE-CFT
- removed REF**: SIGNATURESILK, alexios:SIGNATURE
- removed REF** (x4): MountingHole_2.5mm, MountingHole:MountingHole_2.5mm
- removed REF**: WEEE-Logo_5.6x8mm_SilkScreen, Symbol:WEEE-Logo_5.6x8mm_SilkScreen
- removed REF**: KiCad-Logo2_8mm_SilkScreen, Symbol:KiCad-Logo2_8mm_SilkScreen
- removed RN901: 4.7kΩ, Resistor_THT:R_Array_SIP9
- removed SW1: SW_DIP_x08, Button_Switch_THT:SW_DIP_SPSTx08_Piano_10.8x21.88mm_W7.62mm_P2.54mm
- removed TP101, TP102, TP104, TP105, TP106, TP107, TP108, TP109, TP110, TP111, TP112, TP113, TP114: TestPoint, TestPoint:TestPoint_THTPad_D1.0mm_Drill0.5mm
- removed U1001, U1002, U1003, U601, U602, U603, U604, U605, U606, U701, U702, U703, U704, U801, U802, U803, U804, U901, U902: 74HC574, alexios:SOIC-20W
- removed U101: ATmega64-16AU, alexios:TQFP-64
- removed U102, U109: 74LVC1G04, alexios:SOT-23-5_HandSoldering
- removed U103: 74HC139, alexios:SOIC-16
- removed U104, U105, U106, U115, U504: 74LVC1G07, alexios:SOT-23-5_HandSoldering
- removed U107: 74AC573, alexios:SOIC-20W
- removed U108: 74HC590, alexios:SOIC-16
- removed U110: 74HC540, alexios:SOIC-20W
- removed U1101, U1108: SN74ACT1073, alexios:SOIC-20W
- removed U1102, U1103, U1104, U1105, U1106, U1107, U1109: SN74ACT1071, alexios:SOIC-14
- removed U111, U112, U113, U1201, U1202, U1203, U1204, U1205, U1206, U501: 74HC138, alexios:SOIC-16
- removed U1301, U1302: 74LVC1G17, alexios:SOT-23-5_HandSoldering
- removed U401, U402: 74HC74, alexios:SOIC-14
- removed U403: 74LVC1G11, alexios:SOT-23-6_Handsoldering
- removed U404: 74HC253, alexios:SOIC-16
- removed U502: 74HC112, alexios:SOIC-16
- removed U503: 74HC251, alexios:SOIC-16
- removed U903: 74HC541, alexios:SOIC-20W
- removed X101: CXO, alexios:Crystal_SMD_7050-4Pin_7.0x5.0mm
- removed X102: 33 MHz?, alexios:Oscillator_DIP-8-socket
- added C1: 100nF, alexios:SMD_0805_2012Metric_Pad1.15x1.40mm_HandSolder, F.Cu at (104.5, 128.9)
- added C2: 100nF, alexios:SMD_0805_2012Metric_Pad1.15x1.40mm_HandSolder, F.Cu at (120.3, 128.9)
- added C3: 100nF, alexios:SMD_0805_2012Metric_Pad1.15x1.40mm_HandSolder, F.Cu at (102.3, 144.2)
- added C4: 100nF, alexios:SMD_0805_2012Metric_Pad1.15x1.40mm_HandSolder, F.Cu at (118.9, 144.2)
- added C5: 100nF, alexios:SMD_0805_2012Metric_Pad1.15x1.40mm_HandSolder, B.Cu at (105.4, 136.4)
- added D1: LED_ALT, alexios:LED_0805_2012Metric_Pad1.15x1.40mm_HandSolder, F.Cu at (84.9, 163.2)
- added D2: LED_ALT, alexios:LED_0805_2012Metric_Pad1.15x1.40mm_HandSolder, F.Cu at (89.0, 163.2)
- added J1: Conn_01x24_Male, Connector_PinHeader_2.54mm:PinHeader_2x12_P2.54mm_Vertical, F.Cu at (85.5, 129.6)
- added J2: Conn_01x24_Male, Connector_PinHeader_2.54mm:PinHeader_2x12_P2.54mm_Vertical, F.Cu at (126.2, 129.6)
- added J3: Conn_01x16_Male, Connector_PinHeader_2.54mm:PinHeader_2x08_P2.54mm_Vertical, F.Cu at (98.6, 165.8)
- added R1: 330Ω, alexios:R_SMD_0805_2012Metric_Pad1.15x1.40mm_HandSolder, F.Cu at (86.9, 163.2)
- added R2: 330Ω, alexios:R_SMD_0805_2012Metric_Pad1.15x1.40mm_HandSolder, F.Cu at (91.0, 163.2)
- added RN1: 30Ω, Resistor_SMD:R_Array_Convex_4x0402, B.Cu at (116.4, 134.0)
- added RN2: 30Ω, Resistor_SMD:R_Array_Convex_4x0402, B.Cu at (116.4, 139.1)
- added RN3: 30Ω, Resistor_SMD:R_Array_Convex_4x0402, B.Cu at (116.4, 149.3)
- added RN4: 30Ω, Resistor_SMD:R_Array_Convex_4x0402, B.Cu at (116.4, 154.3)
- added U1: 74HC574, alexios:SOIC-20W, F.Cu at (93.2, 130.8)
- added U2: 74HC574, alexios:SOIC-20W, F.Cu at (93.2, 146.1)
- added U3: 74HC574, alexios:SOIC-20W, F.Cu at (109.7, 130.8)
- added U4: 74HC574, alexios:SOIC-20W, F.Cu at (109.7, 146.1)
- added U5: SN74ACT1073, alexios:SOIC-20W, B.Cu at (110.1, 149.3)
Routing:
- net +5V: track 2209.4 -> 136.9 mm, vias 50 -> 5
- net /FPD1: track 736.4 -> 70.1 mm, vias 9 -> 4
- net /FPD4: track 733.9 -> 73.2 mm, vias 9 -> 4
- net /FPD3: track 731.5 -> 71.3 mm, vias 9 -> 3
- net /FPD5: track 725.2 -> 67.8 mm, vias 9 -> 4
- net /FPD2: track 724.2 -> 72.3 mm, vias 9 -> 4
- net /FPD0: track 724.0 -> 74.6 mm, vias 9 -> 4
- net /FPD6: track 710.2 -> 71.4 mm, vias 9 -> 4
- net /FPD7: track 707.5 -> 71.3 mm, vias 9 -> 3
- net /FPA2: track 567.4 -> 0.00 mm, vias 14 -> 0
- net /~FPRESET: track 469.5 -> 0.00 mm, vias 11 -> 0
- net /Address Bus Pod/AB6: track 467.9 -> 0.00 mm, vias 11 -> 0
- net /Address Bus Pod/AB7: track 465.6 -> 0.00 mm, vias 11 -> 0
- net /FPA4: track 461.2 -> 0.00 mm, vias 10 -> 0
- net /~R: track 460.4 -> 0.00 mm, vias 12 -> 0
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- removed copper zone on F.Cu, net +5V
Other:
- board size 280 x 164.6 mm -> 50.8 x 43.2 mm
- board text removed: "1945"
- board text removed: "AB H In"
- board text removed: "AB H Out"
- board text removed: "AB L In"
- board text removed: "AB L Out"
- board text removed: "AB M In"
- board text removed: "AB M Out"
- board text removed: "ACT"
- board text removed: "ACTION Out"
- board text removed: "ADD 13.2mm to the gap!"
- board text removed: "Bus Hold"
- board text removed: "CFT Address Decoders & Wait State Generator"
- board text removed: "DB H In"
- board text removed: "DB H Out"
- board text removed: "DB L In"
- board text removed: "DB L Out"
- board text removed: "DSR In"
- board text removed: "FPA Read dcdr."
- board text removed: "FPA Write decoders"
- board text removed: "Front Panel Row dcdr."
- board text removed: "Front Panel scan counter"
- board text removed: "GND"
- board text removed: "IBus H In"
- board text removed: "IBus H Out"
- board text removed: "IBus L In"
- board text removed: "IBus L Out"
- board text removed: "IRQ"
- board text removed: "IRQ6"
- board text removed: "IRQ7"
- board text removed: "ISP"
- board text removed: "Interrupt"
- board text removed: "Multi-Function Display"
- board text removed: "OR H Out"
- board text removed: "OR L Out"
- board text removed: "PG3"
- board text removed: "PG4"
- board text removed: "Panel Module dcdr."
- board text removed: "RADDR Out"
- board text removed: "RX"
- board text removed: "RXD"
- board text removed: "Remote Debugging & Virtual Panel (µCU)"
- board text removed: "Run/Stop/Step State Machine"
- board text removed: "Serial (TTYD)"
- board text removed: "State Lights (A5)"
- board text removed: "TXD"
- board text removed: "U11xx: Bus Hold"
- board text removed: "WADDR Out"
- board text removed: "WARNING: THIS IS NOT PCI EXPRESS. Do not plug into PCI Express receptacles, not even extension cables. Damage may occur."
- board text removed: "www.bedroomlan.org/cft"
- board text removed: "~FPHALT"
- board text removed: "~FPIRQ"
- board text removed: "~FPOE31~"
- board text removed: "~FPOE~ Decoders"
- board text removed: "~FPRESET~"
- board text removed: "~RESET"
- board text removed: "~RSTHOLD"
- board text removed: "~SCANCLR~"
- board text removed: "© 2019 Alexios Chouchoulas"
- board text removed: "µCU Address Latch"
- board text removed: "→0x84"
- board text removed: "→0x85"
- board text removed: "→0x86"
- board text removed: "→0x87"
- board text removed: "⎐"

Commit message: Add board-wide bypass capacitors
Parts:
- added C6: 1uF, alexios:SMD_0805_2012Metric_Pad1.15x1.40mm_HandSolder, B.Cu at (93.8, 131.2)
- added C7: 1uF, alexios:SMD_0805_2012Metric_Pad1.15x1.40mm_HandSolder, B.Cu at (122.9, 135.9)
Connections:
- J2 pad 21: Net-(J2-Pad21) -> GND
- J2 pad 22: Net-(J2-Pad22) -> GND
- J2 pad 23: Net-(J2-Pad23) -> GND
- J2 pad 24: Net-(J2-Pad24) -> GND
Routing:
- net GND: vias 9 -> 10

Commit message: Fine-tune pod board
Parts:
- removed J3: Conn_01x16_Male, Connector_PinHeader_2.54mm:PinHeader_2x08_P2.54mm_Vertical
- added G***: LOGO, alexios:CFT, B.Cu at (105.2, 156.2)
- added P3: Conn_01x18_Male, Connector_PinHeader_2.54mm:PinHeader_2x09_P2.54mm_Vertical, F.Cu at (97.6, 165.8)
- added REF**: SIGNATURESILK, alexios:SIGNATURE, F.Cu at (120.6, 168.4)
- moved C7 3.37 mm to (121.7, 132.8), turned to 270 degrees
- renumbered J1 to P1, J2 to P2
Routing:
- net +5V: track 136.9 -> 120.9 mm
- net /D5: track 79.2 -> 77.4 mm
- net GND: track 69.4 -> 71.2 mm
- net /D9: track 65.8 -> 64.0 mm
- net /D10: track 63.2 -> 61.7 mm
- net /D11: track 55.5 -> 56.9 mm
- net /D8: track 43.9 -> 44.6 mm
- net /D14: track 42.2 -> 42.9 mm
- net /D13: track 55.7 -> 56.3 mm
- net /D12: track 42.2 -> 42.8 mm
- net /D6: track 96.8 -> 97.4 mm
- net /D15: track 44.5 -> 45.0 mm
- added copper zone on B.Cu, net +5V
- added copper zone on F.Cu, net +5V
Other:
- board text added: "2129"
- board text added: "Bus Hold"
- board text added: "DFP 16-bit Pod"
- board text added: "High"
- board text added: "Input"
- board text added: "Low"
- board text added: "OE"
- board text added: "Output"
- board text added: "R"
